File: hardware/liger.sch (KiCad schematic (older format))
At the start: 54 parts, among them U1? SPX3819

Commit message: all current data sheets are done
Parts:
- removed D? (x4): LED, symbol LED
- added D? (x4): LED, LEDs:LED_0603, symbol LED
- D?: footprint (none) -> LEDs:LED_0603; Part Number (none) -> LS Q976-NR-1
- P?: footprint (none) -> Connect:USB_Micro-B; Part Number (none) -> 10118194-0001LF
- P? (x2): footprint (none) -> Pin_Headers:Pin_Header_Angled_1x10
- Relay?: Part Number (none) -> V23105A5001A201
- SW?: footprint (none) -> Buttons_Switches_SMD:SW_SPST_KMR2; Part Number (none) -> KMR211NG LFS
- U?: footprint (none) -> libraries:Electret; Part Number (none) -> CMC-5044PF-A
Connections:
- net +3V3: now also D?.2 (A), D?.2 (A)
- net at C?.1, D?.2 (A), U?.10 (3V3OUT)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: now also D?.2 (A), D?.2 (A)
- net at R?.1: now also D?.1 (K) (x3)
- net at Q?.2 (S), R?.1: now also D?.1 (K)
Changed lines of the file:
@@
 F 1 "V23105" H 8850 1400 50  0000 L CNN
 F 2 "garage-opener:V23105" H 8400 1550 50  0001 C CNN
-F 3 "file:///home/chris/Downloads/ENG_SS_108-98007_L.pdf" H 8400 1550 50  0001 C CNN
+F 3 "http://www.te.com/commerce/DocumentDelivery/DDEController?Action=srchrtrv&DocNm=1393792-2&DocType=Customer+Drawing&DocLang=English" H 8400 1550 50  0001 C CNN
+F 4 "V23105A5001A201" H 8400 1550 60  0001 C CNN "Part Number"
 	1    8400 1550
 	1    0    0    -1
@@
 F 0 "P?" H 10325 1375 50  0000 C CNN
 F 1 "USB_OTG" H 10000 1700 50  0000 C CNN
-F 2 "" V 9950 1400 50  0000 C CNN
+F 2 "Connect:USB_Micro-B" V 9950 1400 50  0001 C CNN
 F 3 "" V 9950 1400 50  0000 C CNN
+F 4 "10118194-0001LF" H 10000 1500 60  0001 C CNN "Part Number"
 	1    10000 1500
 	1    0    0    -1
@@
 F 0 "U?" H 900 1600 60  0000 C CNN
 F 1 "electret_microphone" H 750 2350 60  0000 C CNN
-F 2 "" H 650 2000 60  0000 C CNN
+F 2 "libraries:Electret" H 650 2000 60  0001 C CNN
 F 3 "http://www.mouser.com/ds/2/670/cmc-5044pf-a-515902.pdf" H 650 2000 60  0001 C CNN
+F 4 "CMC-5044PF-A" H 750 1850 60  0001 C CNN "Part Number"
 	1    750  1850
 	1    0    0    -1
@@
 F 0 "P?" H 5600 6200 50  0000 C CNN
 F 1 "CONN_01X10" V 5700 5650 50  0000 C CNN
-F 2 "" H 5600 5650 50  0000 C CNN
+F 2 "Pin_Headers:Pin_Header_Angled_1x10" H 5600 5650 50  0001 C CNN
 F 3 "" H 5600 5650 50  0000 C CNN
 	1    5600 5650
@@
 F 0 "P?" H 6400 6150 50  0000 C CNN
 F 1 "CONN_01X10" V 6500 5600 50  0000 C CNN
-F 2 "" H 6400 5600 50  0000 C CNN
+F 2 "Pin_Headers:Pin_Header_Angled_1x10" H 6400 5600 50  0001 C CNN
 F 3 "" H 6400 5600 50  0000 C CNN
 	1    6400 5600
@@
 $EndComp
 $Comp
-L LED D?
-U 1 1 576895D1
-P 1500 4400
-F 0 "D?" H 1500 4500 50  0000 C CNN
-F 1 "LED" H 1500 4300 50  0000 C CNN
-F 2 "" H 1500 4400 50  0000 C CNN
-F 3 "" H 1500 4400 50  0000 C CNN
-	1    1500 4400
-	0    -1   -1   0
-$EndComp
-$Comp
 L +3.3V #PWR?
 U 1 1 57689636
@@
 Text GLabel 650  5100 3    60   Input ~ 0
 IO2
-$Comp
-L LED D?
-U 1 1 5768A3FF
-P 2700 3500
-F 0 "D?" H 2700 3600 50  0000 C CNN
-F 1 "LED" H 2700 3400 50  0000 C CNN
-F 2 "" H 2700 3500 50  0000 C CNN
-F 3 "" H 2700 3500 50  0000 C CNN
-	1    2700 3500
-	0    -1   -1   0
-$EndComp
 Wire Wire Line
 	2700 3700 2700 3800
@@
 F 0 "SW?" H 2850 4710 50  0000 C CNN
 F 1 "SW_PUSH" H 2700 4520 50  0000 C CNN
-F 2 "" H 2700 4600 50  0000 C CNN
-F 3 "" H 2700 4600 50  0000 C CNN
+F 2 "Buttons_Switches_SMD:SW_SPST_KMR2" H 2700 4600 50  0001 C CNN
+F 3 "http://www.mouser.com/ds/2/60/KMR2_9aug12-25127.pdf" H 2700 4600 50  0001 C CNN
+F 4 "KMR211NG LFS" H 2700 4600 60  0001 C CNN "Part Number"
 	1    2700 4600
 	0    1    1    0
@@
 $Comp
 L LED D?
-U 1 1 576C6652
-P 13950 2250
-F 0 "D?" H 13950 2350 50  0000 C CNN
-F 1 "LED" H 13950 2150 50  0000 C CNN
-F 2 "" H 13950 2250 50  0000 C CNN
-F 3 "" H 13950 2250 50  0000 C CNN
-	1    13950 2250
-	1    0    0    -1
-$EndComp
-$Comp
-L LED D?
-U 1 1 576C66E1
-P 13950 1800
-F 0 "D?" H 13950 1900 50  0000 C CNN
-F 1 "LED" H 14100 1750 50  0000 C CNN
-F 2 "" H 13950 1800 50  0000 C CNN
-F 3 "" H 13950 1800 50  0000 C CNN
-	1    13950 1800
-	1    0    0    -1
-$EndComp
-$Comp
-L LED D?
 U 1 1 576C671E
 P 13950 1600
 F 0 "D?" H 13950 1700 50  0000 C CNN
 F 1 "LED" H 14100 1550 50  0000 C CNN
-F 2 "" H 13950 1600 50  0000 C CNN
-F 3 "" H 13950 1600 50  0000 C CNN
+F 2 "LEDs:LED_0603" H 13950 1600 50  0001 C CNN
+F 3 "http://www.osram-os.com/Graphics/XPic9/00128792_0.pdf" H 13950 1600 50  0001 C CNN
+F 4 "LS Q976-NR-1" H 13950 1600 60  0001 C CNN "Part Number"
 	1    13950 1600
 	1    0    0    -1
@@
 	-1   0    0    1
 $EndComp
+$Comp
+L LED D?
+U 1 1 57710784
+P 1500 4400
+F 0 "D?" H 1500 4500 50  0000 C CNN
+F 1 "LED" H 1650 4350 50  0000 C CNN
+F 2 "LEDs:LED_0603" H 1500 4400 50  0001 C CNN
+F 3 "http://www.osram-os.com/Graphics/XPic9/00128792_0.pdf" H 1500 4400 50  0001 C CNN
+F 4 "LS Q976-NR-1" H 1500 4400 60  0001 C CNN "Part Number"
+	1    1500 4400
+	0    -1   -1   0
+$EndComp
+$Comp
+L LED D?
+U 1 1 577107D2
+P 2700 3500
+F 0 "D?" H 2700 3600 50  0000 C CNN
+F 1 "LED" H 2850 3450 50  0000 C CNN
+F 2 "LEDs:LED_0603" H 2700 3500 50  0001 C CNN
+F 3 "http://www.osram-os.com/Graphics/XPic9/00128792_0.pdf" H 2700 3500 50  0001 C CNN
+F 4 "LS Q976-NR-1" H 2700 3500 60  0001 C CNN "Part Number"
+	1    2700 3500
+	0    -1   -1   0
+$EndComp
+$Comp
+L LED D?
+U 1 1 577108E3
+P 13950 1800
+F 0 "D?" H 13950 1900 50  0000 C CNN
+F 1 "LED" H 14100 1750 50  0000 C CNN
+F 2 "LEDs:LED_0603" H 13950 1800 50  0001 C CNN
+F 3 "http://www.osram-os.com/Graphics/XPic9/00128792_0.pdf" H 13950 1800 50  0001 C CNN
+F 4 "LS Q976-NR-1" H 13950 1800 60  0001 C CNN "Part Number"
+	1    13950 1800
+	1    0    0    -1
+$EndComp
+$Comp
+L LED D?
+U 1 1 577108EA
+P 13950 2250
+F 0 "D?" H 13950 2350 50  0000 C CNN
+F 1 "LED" H 14100 2200 50  0000 C CNN
+F 2 "LEDs:LED_0603" H 13950 2250 50  0001 C CNN
+F 3 "http://www.osram-os.com/Graphics/XPic9/00128792_0.pdf" H 13950 2250 50  0001 C CNN
+F 4 "LS Q976-NR-1" H 13950 2250 60  0001 C CNN "Part Number"
+	1    13950 2250
+	1    0    0    -1
+$EndComp
 $EndSCHEMATC

Commit message: update
Parts:
- P?: footprint (none) -> Pin_Headers:Pin_Header_Angled_1x02
Connections:
- net EN renamed TOUT
Changed lines of the file:
@@
 EESchema Schematic File Version 2
-LIBS:glass-break-cache
-LIBS:liger
-LIBS:liger-cache
-LIBS:garage-opener-cache
-LIBS:glass-break
-LIBS:SR086-SOIC
 LIBS:power
 LIBS:device
@@
 LIBS:contrib
 LIBS:valves
+LIBS:liger-cache
 EELAYER 25 0
 EELAYER END
@@
 $EndComp
 Text GLabel 3600 1750 2    60   Input ~ 0
-EN
+TOUT
 $Comp
 L SPX3819 U1?
@@
 F 0 "P?" H 9250 1850 50  0000 C CNN
 F 1 "CONN_01X02" V 9350 1700 50  0000 C CNN
-F 2 "" H 9250 1700 50  0000 C CNN
+F 2 "Pin_Headers:Pin_Header_Angled_1x02" H 9250 1700 50  0001 C CNN
 F 3 "" H 9250 1700 50  0000 C CNN
 	1    9250 1700
@@
 	1    0    0    -1
 $EndComp
+Text Label 3650 1700 0    60   ~ 0
+ADC
 $EndSCHEMATC
