File: hardware/_saved_liger.sch (KiCad schematic (older format))
At the start: 60 parts, among them P1 CONN_01X10, P2 CONN_01X10, P3 USB_OTG, P4 CONN_01X02, P5 CONN_01X04, Q1 Q_NMOS_GSD, Q2 Q_PMOS_GSD, Q3 Q_NPN_BEC, Q4 Q_NPN_BEC, SW1 SW_PUSH, U1 electret_microphone, U11 SPX3819, U2 ADA4075, U3 ESP-WROOM-02, U4 FT230XS, U5 PT5529B/L2/H2-F

Commit message: update
Parts:
- Relay1: footprint garage-opener:V23105 -> libraries:V23105
Changed lines of the file:
@@
 F 0 "Relay1" H 7750 1750 50  0000 L CNN
 F 1 "V23105" H 8850 1400 50  0000 L CNN
-F 2 "garage-opener:V23105" H 8400 1550 50  0001 C CNN
+F 2 "libraries:V23105" H 8400 1550 50  0001 C CNN
 F 3 "file:///home/chris/Downloads/ENG_SS_108-98007_L%20(3).pdf" H 8400 1550 50  0001 C CNN
 F 4 "V23105A5001A201" H 8400 1550 60  0001 C CNN "Part Number"
@@
 F 1 "USB_OTG" H 8300 4350 50  0000 C CNN
 F 2 "Connect:USB_Micro-B" V 8250 4050 50  0001 C CNN
-F 3 "http://portal.fciconnect.com/Comergent//fci/drawing/10118194.pdf" V 8250 4050 50  0000 C CNN
+F 3 "http://portal.fciconnect.com/Comergent//fci/drawing/10118194.pdf" V 8250 4050 50  0001 C CNN
 F 4 "10118194-0001LF" H 8300 4150 60  0001 C CNN "Part Number"
 	1    8300 4150
