File: hardware/_autosave-liger.kicad_pcb (KiCad board)
At the start: 2 copper layers, 50 x 92.1 mm, 76 parts, among them P1 CONN_01X10, P2 CONN_01X10, P4 CONN_01X02, P5 CONN_01X04, Q1 Q_NMOS_GSD, Q2 Q_PMOS_GSD, Q3 Q_NPN_BEC, Q4 Q_NPN_BEC, Q5 Q_NPN_BEC, SW1 SW_PUSH, SW2 LED-switch, U1 MEMS-SPM0408LE5H, U11 SPX3819, U2 OPA344, U3 ESP-WROOM-02, U4 LNK4023D, U5 PT5529B/L2/H2-F, U6 EPC1716D

Commit message: update
Parts:
- moved Q3 139.3 mm to (32.9, 138.8)
- moved R14 123.8 mm to (33.6, 144.5)
- moved P4 123.7 mm to (-53.8, 121.4)
- moved D4 103.5 mm to (22.0, 141.9), turned to 90 degrees
Changed lines of the file:
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@@
     (tags "capacitor 0603")
     (attr smd)
-    (fp_text reference C10 (at 0 -1.9 180) (layer F.SilkS)
+    (fp_text reference C10 (at -1.204 1.778 180) (layer F.SilkS)
       (effects (font (size 1 1) (thickness 0.15)))
     )
@@
   )
   (module Diodes_SMD:SMA_Standard (layer F.Cu)
-    (at 56.458735 44.306508)
+    (at 21.971 141.859 90)
     (descr "Diode SMA")
     (tags "Diode SMA")
     (attr smd)
-    (fp_text reference D4 (at 0 -3.81) (layer F.SilkS)
-      (effects (font (size 1 1) (thickness 0.15)))
-    )
-    (fp_text value D (at 0 4.3) (layer F.Fab)
+    (fp_text reference D4 (at 4.572 -0.127 180) (layer F.SilkS)
+      (effects (font (size 1 1) (thickness 0.15)))
+    )
+    (fp_text value D (at 0 4.3 90) (layer F.Fab)
       (effects (font (size 1 1) (thickness 0.15)))
     )
@@
     (fp_line (start 3.5 2) (end -3.5 2) (layer F.CrtYd) (width 0.05))
     (fp_line (start -3.5 2) (end -3.5 -2) (layer F.CrtYd) (width 0.05))
-    (fp_text user K (at -2.9 2.95) (layer F.SilkS)
-      (effects (font (size 1 1) (thickness 0.15)))
-    )
-    (fp_text user A (at 2.9 2.9) (layer F.SilkS)
+    (fp_text user K (at -2.9 2.95 90) (layer F.SilkS)
+      (effects (font (size 1 1) (thickness 0.15)))
+    )
+    (fp_text user A (at 2.9 2.9 90) (layer F.SilkS)
       (effects (font (size 1 1) (thickness 0.15)))
     )
@@
     (fp_line (start -2.25044 1.75006) (end 2.25044 1.75006) (layer F.SilkS) (width 0.15))
     (fp_line (start -2.25044 -1.75006) (end 2.25044 -1.75006) (layer F.SilkS) (width 0.15))
-    (pad 1 smd rect (at -1.99898 0) (size 2.49936 1.80086) (layers F.Cu F.Paste F.Mask)
+    (pad 1 smd rect (at -1.99898 0 90) (size 2.49936 1.80086) (layers F.Cu F.Paste F.Mask)
       (net 8 +5V))
-    (pad 2 smd rect (at 1.99898 0) (size 2.49936 1.80086) (layers F.Cu F.Paste F.Mask)
+    (pad 2 smd rect (at 1.99898 0 90) (size 2.49936 1.80086) (layers F.Cu F.Paste F.Mask)
       (net 21 "Net-(D4-Pad2)"))
     (model Diodes_SMD.3dshapes/SMA_Standard.wrl
@@
   )
   (module Terminal_Blocks:TerminalBlock_Pheonix_MKDS1.5-2pol (layer F.Cu)
-    (at 44.808735 46.846508)
+    (at -53.848 121.412)
     (descr "2-way 5mm pitch terminal block, Phoenix MKDS series")
     (fp_text reference P4 (at 2.5 5.9) (layer F.SilkS)
@@
   )
   (module TO_SOT_Packages_SMD:SOT-23 (layer F.Cu)
-    (at 97.534448 15.446508)
+    (at 32.893 138.811)
     (descr "SOT-23, Standard")
     (tags SOT-23)
@@
   )
   (module Resistors_SMD:R_0603_HandSoldering (layer F.Cu)
-    (at 93.278735 35.996508)
+    (at 33.612 144.526)
     (descr "Resistor SMD 0603, hand soldering")
     (tags "resistor 0603")
@@
     (tags "resistor 0603")
     (attr smd)
-    (fp_text reference R29 (at 0 -1.9 180) (layer F.SilkS)
+    (fp_text reference R29 (at 0.678 1.651 180) (layer F.SilkS)
       (effects (font (size 1 1) (thickness 0.15)))
     )
@@
       (net 8 +5V))
   )
-  (gr_line (start 135.382 21.59) (end 135.382 141.605) (layer Dwgs.User) (width 0.2))
-  (gr_line (start 210.439 21.59) (end 135.382 21.59) (layer Dwgs.User) (width 0.2))
-  (gr_line (start 210.439 141.605) (end 210.439 21.59) (layer Dwgs.User) (width 0.2))
+  (gr_line (start 136.906 21.59) (end 136.906 141.605) (layer Dwgs.User) (width 0.2))
+  (gr_line (start 211.963 21.59) (end 136.906 21.59) (layer Dwgs.User) (width 0.2))
+  (gr_line (start 211.963 141.605) (end 211.963 21.59) (layer Dwgs.User) (width 0.2))
   (gr_line (start 135.382 141.605) (end 210.439 141.605) (layer Dwgs.User) (width 0.2))
   (gr_circle (center 173.609 33.909) (end 173.736 31.496) (layer Dwgs.User) (width 0.2))
