File: hardware/_autosave-liger.kicad_pcb (KiCad board)
At the start: 2 copper layers, 43.2 x 92.2 mm, 54 parts, among them P1 CONN_01X20, P2 CONN_01X20, P3 CONN_01X03, P4 CONN_01X03, P5 CONN_01X04, P6 CONN_01X04, Q1 Q_NPN_BEC, Q2 Q_NMOS_GSD, Q3 Q_PMOS_GSD, U1 ESP-WROOM-32, U12 soft-button-4x, U2 PT5529B/L2/H2-F, U3 MEMS-SPM0408LE5H, U4 OPA344, U5 SPX3819, U6 OPA344, U7 RGB-LED, U8 Amplifier-D-TS4962IQT

Commit message: updatge
Parts:
- U3: moved to B.Cu
- moved R6 58.0 mm to (162.2, 54.5), turned to 0 degrees
- moved U6 43.5 mm to (159.1, 86.8)
- moved R7 41.3 mm to (143.1, 58.2)
- moved U3 28.2 mm to (147.1, 58.6)
Changed lines of the file:
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@@
   )
   (module Resistors_SMD:R_0603_HandSoldering (layer F.Cu)
-    (at 115.638027 89.114302 270)
-    (descr "Resistor SMD 0603, hand soldering")
-    (tags "resistor 0603")
-    (attr smd)
-    (fp_text reference R6 (at 0 -1.45 270) (layer F.SilkS)
-      (effects (font (size 1 1) (thickness 0.15)))
-    )
-    (fp_text value 100K (at 0 1.55 270) (layer F.Fab)
-      (effects (font (size 1 1) (thickness 0.15)))
-    )
-    (fp_text user %R (at 0 0 270) (layer F.Fab)
-      (effects (font (size 0.4 0.4) (thickness 0.075)))
-    )
-    (fp_line (start -0.8 0.4) (end -0.8 -0.4) (layer F.Fab) (width 0.1))
-    (fp_line (start 0.8 0.4) (end -0.8 0.4) (layer F.Fab) (width 0.1))
-    (fp_line (start 0.8 -0.4) (end 0.8 0.4) (layer F.Fab) (width 0.1))
-    (fp_line (start -0.8 -0.4) (end 0.8 -0.4) (layer F.Fab) (width 0.1))
-    (fp_line (start 0.5 0.68) (end -0.5 0.68) (layer F.SilkS) (width 0.12))
-    (fp_line (start -0.5 -0.68) (end 0.5 -0.68) (layer F.SilkS) (width 0.12))
-    (fp_line (start -1.96 -0.7) (end 1.95 -0.7) (layer F.CrtYd) (width 0.05))
-    (fp_line (start -1.96 -0.7) (end -1.96 0.7) (layer F.CrtYd) (width 0.05))
-    (fp_line (start 1.95 0.7) (end 1.95 -0.7) (layer F.CrtYd) (width 0.05))
-    (fp_line (start 1.95 0.7) (end -1.96 0.7) (layer F.CrtYd) (width 0.05))
-    (pad 1 smd rect (at -1.1 0 270) (size 1.2 0.9) (layers F.Cu F.Paste F.Mask)
+    (at 162.15 54.5)
+    (descr "Resistor SMD 0603, hand soldering")
+    (tags "resistor 0603")
+    (attr smd)
+    (fp_text reference R6 (at 0 -1.45) (layer F.SilkS)
+      (effects (font (size 1 1) (thickness 0.15)))
+    )
+    (fp_text value 100K (at 0 1.55) (layer F.Fab)
+      (effects (font (size 1 1) (thickness 0.15)))
+    )
+    (fp_text user %R (at 0 0) (layer F.Fab)
+      (effects (font (size 0.4 0.4) (thickness 0.075)))
+    )
+    (fp_line (start -0.8 0.4) (end -0.8 -0.4) (layer F.Fab) (width 0.1))
+    (fp_line (start 0.8 0.4) (end -0.8 0.4) (layer F.Fab) (width 0.1))
+    (fp_line (start 0.8 -0.4) (end 0.8 0.4) (layer F.Fab) (width 0.1))
+    (fp_line (start -0.8 -0.4) (end 0.8 -0.4) (layer F.Fab) (width 0.1))
+    (fp_line (start 0.5 0.68) (end -0.5 0.68) (layer F.SilkS) (width 0.12))
+    (fp_line (start -0.5 -0.68) (end 0.5 -0.68) (layer F.SilkS) (width 0.12))
+    (fp_line (start -1.96 -0.7) (end 1.95 -0.7) (layer F.CrtYd) (width 0.05))
+    (fp_line (start -1.96 -0.7) (end -1.96 0.7) (layer F.CrtYd) (width 0.05))
+    (fp_line (start 1.95 0.7) (end 1.95 -0.7) (layer F.CrtYd) (width 0.05))
+    (fp_line (start 1.95 0.7) (end -1.96 0.7) (layer F.CrtYd) (width 0.05))
+    (pad 1 smd rect (at -1.1 0) (size 1.2 0.9) (layers F.Cu F.Paste F.Mask)
       (net 52 3V3))
-    (pad 2 smd rect (at 1.1 0 270) (size 1.2 0.9) (layers F.Cu F.Paste F.Mask)
+    (pad 2 smd rect (at 1.1 0) (size 1.2 0.9) (layers F.Cu F.Paste F.Mask)
       (net 3 "Net-(C2-Pad2)"))
     (model ${KISYS3DMOD}/Resistors_SMD.3dshapes/R_0603.wrl
@@
   )
   (module Resistors_SMD:R_0603_HandSoldering (layer F.Cu)
-    (at 115.638027 89.114302 270)
-    (descr "Resistor SMD 0603, hand soldering")
-    (tags "resistor 0603")
-    (attr smd)
-    (fp_text reference R7 (at 0 -1.45 270) (layer F.SilkS)
+    (at 143.09 58.21 270)
+    (descr "Resistor SMD 0603, hand soldering")
+    (tags "resistor 0603")
+    (attr smd)
+    (fp_text reference R7 (at -0.95 1.58 360) (layer F.SilkS)
       (effects (font (size 1 1) (thickness 0.15)))
     )
@@
       (net 15 5V))
   )
-  (module footprints:mems-mic (layer F.Cu)
-    (at 146.07064 86.79872)
-    (fp_text reference U3 (at 0.2032 3.48488) (layer F.SilkS)
-      (effects (font (size 1 1) (thickness 0.15)))
-    )
-    (fp_text value MEMS-SPM0408LE5H (at -0.06604 -3.2004) (layer F.Fab)
-      (effects (font (size 1 1) (thickness 0.15)))
-    )
-    (fp_line (start -1.90064 -2.30272) (end -1.90064 2.49728) (layer F.SilkS) (width 0.15))
-    (fp_line (start 1.89936 -2.30272) (end -1.90064 -2.30272) (layer F.SilkS) (width 0.15))
-    (fp_line (start 1.89936 2.49728) (end 1.89936 -2.30272) (layer F.SilkS) (width 0.15))
-    (fp_line (start 1.49936 2.49728) (end 1.89936 2.49728) (layer F.SilkS) (width 0.15))
-    (fp_line (start 1.49936 2.49728) (end -1.90064 2.49728) (layer F.SilkS) (width 0.15))
-    (pad 3 smd circle (at -1.25064 1.84728) (size 0.5 0.5) (layers *.Mask F.Cu F.Paste)
-      (net 1 GND))
-    (pad 3 smd circle (at 1.24936 1.84728) (size 0.5 0.5) (layers *.Mask F.Cu F.Paste)
-      (net 1 GND))
-    (pad 3 smd circle (at 1.22436 -0.35272) (size 0.6 0.6) (layers F.Cu F.Paste B.SilkS F.Mask)
+  (module footprints:mems-mic (layer B.Cu)
+    (at 147.05064 58.59728)
+    (fp_text reference U3 (at 0.2032 -3.48488) (layer B.SilkS)
+      (effects (font (size 1 1) (thickness 0.15)) (justify mirror))
+    )
+    (fp_text value MEMS-SPM0408LE5H (at -0.06604 3.2004) (layer B.Fab)
+      (effects (font (size 1 1) (thickness 0.15)) (justify mirror))
+    )
+    (fp_line (start -1.90064 2.30272) (end -1.90064 -2.49728) (layer B.SilkS) (width 0.15))
+    (fp_line (start 1.89936 2.30272) (end -1.90064 2.30272) (layer B.SilkS) (width 0.15))
+    (fp_line (start 1.89936 -2.49728) (end 1.89936 2.30272) (layer B.SilkS) (width 0.15))
+    (fp_line (start 1.49936 -2.49728) (end 1.89936 -2.49728) (layer B.SilkS) (width 0.15))
+    (fp_line (start 1.49936 -2.49728) (end -1.90064 -2.49728) (layer B.SilkS) (width 0.15))
+    (pad 3 smd circle (at -1.25064 -1.84728) (size 0.5 0.5) (layers *.Mask B.Cu B.Paste)
+      (net 1 GND))
+    (pad 3 smd circle (at 1.24936 -1.84728) (size 0.5 0.5) (layers *.Mask B.Cu B.Paste)
+      (net 1 GND))
+    (pad 3 smd circle (at 1.22436 0.35272) (size 0.6 0.6) (layers B.Cu B.Paste F.SilkS B.Mask)
       (net 1 GND) (solder_mask_margin 0.1))
-    (pad 6 smd circle (at 1.24936 -1.55272) (size 0.6 0.6) (layers *.Mask F.Cu F.Paste)
+    (pad 6 smd circle (at 1.24936 1.55272) (size 0.6 0.6) (layers *.Mask B.Cu B.Paste)
       (net 52 3V3))
-    (pad 3 smd circle (at -0.00064 -1.55272) (size 0.6 0.6) (layers *.Mask F.Cu F.Paste)
-      (net 1 GND))
-    (pad 1 smd circle (at -1.25064 -1.55272) (size 0.6 0.6) (layers *.Mask F.Cu F.Paste)
+    (pad 3 smd circle (at -0.00064 1.55272) (size 0.6 0.6) (layers *.Mask B.Cu B.Paste)
+      (net 1 GND))
+    (pad 1 smd circle (at -1.25064 1.55272) (size 0.6 0.6) (layers *.Mask B.Cu B.Paste)
       (net 13 "Net-(C2-Pad1)"))
-    (pad 2 smd circle (at -1.20064 -0.35272) (size 0.6 0.6) (layers *.Mask F.Cu F.Paste)
+    (pad 2 smd circle (at -1.20064 0.35272) (size 0.6 0.6) (layers *.Mask B.Cu B.Paste)
       (net 2 "Net-(C1-Pad2)"))
-    (pad 3 thru_hole circle (at 0.0254 1.03632) (size 1.676 1.676) (drill 1.016) (layers *.Cu *.Mask)
+    (pad 3 thru_hole circle (at 0.0254 -1.03632) (size 1.676 1.676) (drill 1.016) (layers *.Cu *.Mask)
       (net 1 GND))
   )
@@
   )
   (module TO_SOT_Packages_SMD:SOT-23-5 (layer F.Cu)
-    (at 115.638027 89.114302 270)
+    (at 159.05 86.76 270)
     (descr "5-pin SOT23 package")
     (tags SOT-23-5)
@@
     )
   )
-  (gr_line (start 217.75 114.65) (end 217.75 47.65) (layer Dwgs.User) (width 0.2))
-  (gr_line (start 250.75 114.65) (end 217.75 114.65) (layer Dwgs.User) (width 0.2))
-  (gr_line (start 250.75 47.65) (end 250.75 114.65) (layer Dwgs.User) (width 0.2))
-  (gr_line (start 217.75 47.65) (end 250.75 47.65) (layer Dwgs.User) (width 0.2))
+  (gr_line (start 325 109.49) (end 325 42.49) (layer Dwgs.User) (width 0.2))
+  (gr_line (start 358 109.49) (end 325 109.49) (layer Dwgs.User) (width 0.2))
+  (gr_line (start 358 42.49) (end 358 109.49) (layer Dwgs.User) (width 0.2))
+  (gr_line (start 325 42.49) (end 358 42.49) (layer Dwgs.User) (width 0.2))
   (gr_circle (center 147.664463 130.513302) (end 147.918463 133.561302) (layer Edge.Cuts) (width 0.15))
   (dimension 67.183 (width 0.3) (layer Cmts.User)
@@
   (gr_line (start 125.713028 127.595302) (end 142.350028 127.595302) (layer Edge.Cuts) (width 0.15))
   (gr_line (start 125.713028 49.236302) (end 142.604028 49.236302) (layer Edge.Cuts) (width 0.15))
-  (gr_line (start 381.35 133.85) (end 381.337028 18.849302) (layer Dwgs.User) (width 0.2))
-  (gr_line (start 306.280028 133.85) (end 381.337028 133.85) (layer Dwgs.User) (width 0.2))
-  (gr_line (start 306.280028 18.849302) (end 306.25 133.85) (layer Dwgs.User) (width 0.2))
-  (gr_line (start 381.337028 18.849302) (end 306.280028 18.849302) (layer Dwgs.User) (width 0.2))
+  (gr_line (start 376.5 133) (end 376.5 18.95) (layer Dwgs.User) (width 0.2))
+  (gr_line (start 306.5 133) (end 376.5 133) (layer Dwgs.User) (width 0.2))
+  (gr_line (start 306.480028 18.999302) (end 306.5 133) (layer Dwgs.User) (width 0.2))
+  (gr_line (start 376.5 18.95) (end 306.480028 18.949302) (layer Dwgs.User) (width 0.2))
   (gr_circle (center 147.684028 40.095641) (end 147.811028 42.508641) (layer Dwgs.User) (width 0.2))
   (gr_circle (center 147.684028 47.458302) (end 147.938028 50.506302) (layer Edge.Cuts) (width 0.15))
