File: hardware/_autosave-liger.kicad_pcb (KiCad board)
At the start: 2 copper layers, 33.1 x 92.2 mm, 56 parts, among them J1 Conn_02x08_Odd_Even, Q1 Q_NPN_BEC, Q4 PMOS-DMG3413L, U1 ESP-WROOM-32, U10 EKMC1601112, U12 soft-button-4x, U2 IR-RX-TSOP34438, U3 SPH0645LM4H-B, U4 MCP73831T, U5 MAX98357AETE+T, U6 SI7020-A20, U8 TSL45315CL, U9 AP2112

Commit message: update
Parts:
- J1: moved to F.Cu
- moved U1 161.7 mm to (185.1, -79.8)
- moved U4 139.0 mm to (126.9, 68.2), turned to 90 degrees
- moved LS1 135.5 mm to (151.3, -24.1), turned to 0 degrees
- moved U10 115.9 mm to (189.6, -51.1)
- moved J1 63.8 mm to (140.0, 62.8)
