File: hardware/liger.kicad_pcb (KiCad board)
At the start: 2 copper layers, 0 parts

Commit message: update
Parts:
- added BR1: DF08S, footprints:surfacemount-diodebridge, F.Cu at (36.7, 144.6)
- added C1: 4.7uf, Capacitors_SMD:C_0603_HandSoldering, F.Cu at (119.2, 40.9)
- added C10: 1000pF, Capacitors_SMD:C_0603_HandSoldering, F.Cu at (63.9, 26.9)
- added C11: 220nF, Capacitors_SMD:C_0603_HandSoldering, F.Cu at (99.4, 54.3)
- added C12: 330pF, Capacitors_SMD:C_0805_HandSoldering, F.Cu at (35.3, 62.1)
- added C13: 2.2uF, Capacitors_SMD:C_0603_HandSoldering, F.Cu at (99.1, 60.2)
- added C14: 2.2pF, Capacitors_SMD:C_0603_HandSoldering, F.Cu at (105.3, 54.1)
- added C15: 560uF, Capacitors_ThroughHole:C_Radial_D8_L11.5_P3.5, F.Cu at (52.6, 59.6)
- added C2: 4.7uF, Capacitors_SMD:C_0603, F.Cu at (116.6, 35.0)
- added C3: 12uF, Capacitors_ThroughHole:C_Radial_D10_L13_P5, F.Cu at (52.8, 31.3)
- added C4: 1uf, Capacitors_SMD:C_0603, F.Cu at (120.4, 26.3)
- added C5: 1uf, Capacitors_SMD:C_0603, F.Cu at (68.7, 26.9)
- added C6: 0.1uF, Capacitors_SMD:C_0603, F.Cu at (116.8, 46.7)
- added C7: 100pF, Capacitors_SMD:C_0603_HandSoldering, F.Cu at (104.1, 60.2)
- added C8: 12uF, Capacitors_ThroughHole:C_Radial_D10_L13_P5, F.Cu at (83.1, 32.7)
- added C9: 560uF, Capacitors_ThroughHole:C_Radial_D8_L11.5_P3.5, F.Cu at (98.9, 22.7)
- added D1: LED, LEDs:LED_0603, F.Cu at (76.7, 68.5)
- added D2: LED, LEDs:LED_0603, F.Cu at (120.6, 31.7)
- added D3: D, Diodes_SMD:SMB_Handsoldering, F.Cu at (71.2, 58.1)
- added D4: D, Diodes_SMD:SMA_Standard, F.Cu at (62.6, 58.8)
- added D5: D, Diodes_SMD:SMB_Handsoldering, F.Cu at (96.1, 33.1)
- added D6: D, Diodes_SMD:SMB_Handsoldering, F.Cu at (110.1, 20.5)
- added D7: D, Diodes_SMD:SMB_Handsoldering, F.Cu at (89.1, 44.1)
- added D8: LED, LEDs:LED-3MM, F.Cu at (34.2, 48.6)
- added L1: BEAD, Resistors_SMD:R_0805_HandSoldering, F.Cu at (35.4, 55.8)
- added L2: 470uH, Capacitors_ThroughHole:C_Radial_D10_L13_P5, F.Cu at (52.8, 46.0)
- added P1: CONN_01X10, Pin_Headers:Pin_Header_Straight_1x10, F.Cu at (228.4, 85.5)
- added P2: CONN_01X10, Pin_Headers:Pin_Header_Straight_1x10, F.Cu at (274.7, 62.3)
- added P4: CONN_01X02, Terminal_Blocks:TerminalBlock_Pheonix_MKDS1.5-2pol, F.Cu at (63.8, 37.7)
- added P5: CONN_01X04, Pin_Headers:Pin_Header_Angled_1x04, F.Cu at (85.2, 15.8)
- added Q1: Q_NMOS_GSD, TO_SOT_Packages_SMD:SOT-23, F.Cu at (116.8, 13.0)
- added Q2: Q_PMOS_GSD, TO_SOT_Packages_SMD:SOT-23, F.Cu at (79.1, 43.3)
- added Q3: Q_NPN_BEC, TO_SOT_Packages_SMD:SOT-23, F.Cu at (109.7, 29.5)
- added Q4: Q_NPN_BEC, TO_SOT_Packages_SMD:SOT-23, F.Cu at (78.5, 49.9)
- added Q5: Q_NPN_BEC, TO_SOT_Packages_SMD:SOT-23, F.Cu at (63.4, 67.4)
- added R1: 1K, Resistors_SMD:R_0603_HandSoldering, F.Cu at (78.4, 63.1)
- added R10: 1K, Resistors_SMD:R_0603_HandSoldering, F.Cu at (107.8, 42.4)
- added R11: 10K, Resistors_SMD:R_0603_HandSoldering, F.Cu at (90.1, 59.8)
- added R12: 10K, Resistors_SMD:R_0603_HandSoldering, F.Cu at (114.8, 40.9)
- added R13: 10K, Resistors_SMD:R_0603_HandSoldering, F.Cu at (82.8, 65.6)
- added R14: 1K, Resistors_SMD:R_0603_HandSoldering, F.Cu at (100.7, 48.5)
- added R15: 0.82, Resistors_SMD:R_0805_HandSoldering, F.Cu at (25.2, 68.5)
- added R16: 0.91, Resistors_SMD:R_0805_HandSoldering, F.Cu at (19.9, 68.5)
- added R17: 1K, Resistors_SMD:R_0603_HandSoldering, F.Cu at (94.6, 54.3)
- added R18: 270, Resistors_SMD:R_0805_HandSoldering, F.Cu at (14.7, 68.5)
- added R19: 27M, Resistors_SMD:R_1206_HandSoldering, F.Cu at (97.6, 42.2)
- added R2: 1K, Resistors_SMD:R_0603_HandSoldering, F.Cu at (56.5, 68.9)
- added R20: 27M, Resistors_SMD:R_1206_HandSoldering, F.Cu at (104.6, 36.2)
- added R21: 270, Resistors_SMD:R_0805_HandSoldering, F.Cu at (35.4, 68.3)
- added R22: 27M, Resistors_SMD:R_1206_HandSoldering, F.Cu at (71.5, 67.2)
- added R23: 300, Resistors_SMD:R_0603_HandSoldering, F.Cu at (94.6, 60.2)
- added R24: 1K, Resistors_SMD:R_0603_HandSoldering, F.Cu at (100.6, 66.0)
- added R25: 36, Resistors_SMD:R_0603_HandSoldering, F.Cu at (105.2, 48.3)
- added R26: 9.1K, Resistors_SMD:R_0603_HandSoldering, F.Cu at (87.3, 65.6)
- added R27: 620, Resistors_SMD:R_0603_HandSoldering, F.Cu at (112.2, 46.7)
- added R28: 3K, Resistors_SMD:R_0603_HandSoldering, F.Cu at (91.7, 66.0)
- added R29: 4.7, Resistors_SMD:R_0603_HandSoldering, F.Cu at (109.8, 52.6)
- added R3: 6.65K, Resistors_SMD:R_0603_HandSoldering, F.Cu at (110.1, 58.4)
- added R30: 1, Resistors_SMD:R_0603_HandSoldering, F.Cu at (96.2, 66.0)
- added R31: 5.1K, Resistors_SMD:R_0603_HandSoldering, F.Cu at (52.0, 68.9)
- added R4: 1K, Resistors_SMD:R_0603_HandSoldering, F.Cu at (116.5, 29.2)
- added R5: 1K, Resistors_SMD:R_0603_HandSoldering, F.Cu at (96.3, 48.5)
- added R6: 1K, Resistors_SMD:R_0603_HandSoldering, F.Cu at (85.7, 59.8)
- added R7: 1K, Resistors_SMD:R_0603_HandSoldering, F.Cu at (103.3, 42.4)
- added R8: 1K, Resistors_SMD:R_0603_HandSoldering, F.Cu at (110.4, 35.8)
- added R9: 1K, Resistors_SMD:R_0603_HandSoldering, F.Cu at (30.0, 68.3)
- added RT1: 5, Resistors_ThroughHole:Resistor_Horizontal_RM10mm, F.Cu at (62.3, 49.2)
- added Relay1: V23105, libraries:V23105, F.Cu at (51.1, 21.0)
- added SW1: SW_PUSH, Buttons_Switches_SMD:SW_SPST_KMR2, F.Cu at (118.7, 19.8)
- added U11: SPX3819, TO_SOT_Packages_SMD:SOT-23-5, F.Cu at (79.9, 56.8)
- added U2: ADA4075, TO_SOT_Packages_SMD:SOT-23-5, F.Cu at (87.0, 53.5)
- added U3: ESP-WROOM-02, libraries:ESP-WROOM-02, F.Cu at (240.6, 66.6)
- added U4: LNK4023D, Power_Integrations:SO-8, F.Cu at (75.8, 33.9)
- added U5: PT5529B/L2/H2-F, libraries:PT5529B, F.Cu at (107.1, 13.5)
- added U6: EPC1716D, Transformers_CHK:Trafo_CHK-EI30-2VA_1xSec, F.Cu at (25.8, 28.5)

Commit message: update
Parts:
- added U1: MEMS-SPM0408LE5H, footprints:memes-mic, F.Cu at (153.4, 119.8)
- moved R8 82.7 mm to (149.7, 108.5), turned to 270 degrees
- moved C1 82.0 mm to (146.1, 118.3)
- moved R5 80.7 mm to (145.2, 112.7), turned to 270 degrees
- moved U2 77.5 mm to (145.9, 103.9), turned to 270 degrees
- moved C11 77.4 mm to (149.7, 113.1), turned to 270 degrees
- moved R7 76.6 mm to (143.2, 107.8), turned to 270 degrees
- moved R11 74.2 mm to (149.7, 104.1), turned to 90 degrees
- moved R3 62.5 mm to (141.2, 112.7), turned to 270 degrees

Commit message: update
Parts:
- Relay1: footprint libraries:V23105 -> Relays_ThroughHole:Relay_SANYOU_SRD_Series_Form_C
- moved Relay1 107.5 mm to (116.5, 106.3)
- moved R3 7.53 mm to (148.7, 113.3)
- moved R5 5.78 mm to (150.9, 113.2)
- moved R7 5.62 mm to (148.7, 109.0)
- moved U2 3.80 mm to (149.7, 104.0)
- moved C11 3.50 mm to (153.2, 113.1)
- moved R11 3.50 mm to (153.2, 104.1)
- moved R8 3.50 mm to (153.2, 108.5)
- moved C1 0.35 mm to (146.5, 118.3)

Commit message: update
Parts:
- D3: footprint Diodes_SMD:SMB_Handsoldering -> Diodes_SMD:DO-214BA
- D5: footprint Diodes_SMD:SMB_Handsoldering -> Diodes_SMD:SMA_Standard
- RT1: footprint Resistors_ThroughHole:Resistor_Horizontal_RM10mm -> Resistors_ThroughHole:Resistor_Vertical_RM5mm
- moved C8 134.5 mm to (43.7, 161.3)
- moved C3 130.8 mm to (35.9, 161.1), turned to 180 degrees
- moved R20 130.2 mm to (80.2, 164.1), turned to 90 degrees
- moved BR1 128.0 mm to (43.9, 16.8)
- moved U4 124.7 mm to (72.7, 158.6)
- moved L1 113.6 mm to (39.9, 169.3)
- moved R21 105.8 mm to (73.3, 167.1), turned to 180 degrees
- moved R18 104.9 mm to (63.6, 161.3)
- moved L2 103.5 mm to (37.2, 148.3)
- moved R16 99.4 mm to (58.4, 160.2), turned to 270 degrees
- moved R15 95.9 mm to (53.7, 160.1), turned to 270 degrees
- moved Q1 83.0 mm to (46.5, 57.0)
- moved C12 77.1 mm to (101.9, 23.3)
- moved D8 76.6 mm to (103.5, 16.1)
- moved P5 75.7 mm to (19.4, 53.3)
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
Commit message: update
Parts:
- moved BR1 177.4 mm to (10.9, 191.2), turned to 180 degrees
- moved U6 157.9 mm to (99.9, 171.6)
- moved C15 155.0 mm to (156.4, 154.7), turned to 270 degrees
- moved Q5 154.2 mm to (75.9, 182.3)
- moved C14 154.1 mm to (137.7, 192.8), turned to 270 degrees
- moved C9 152.7 mm to (145.2, 154.9), turned to 270 degrees
- moved D5 151.4 mm to (129.6, 170.9), turned to 180 degrees
- moved D3 150.8 mm to (76.2, 172.3), turned to 270 degrees
- moved P5 148.9 mm to (158.7, 105.9), turned to 90 degrees
- moved RT1 148.5 mm to (6.44, 197.8), turned to 180 degrees
- moved R28 148.1 mm to (124.7, 192.7), turned to 270 degrees
- moved C12 144.3 mm to (71.4, 164.3), turned to 90 degrees
- moved C13 142.6 mm to (134.4, 192.8), turned to 270 degrees
- moved R30 135.3 mm to (134.2, 181.0), turned to 270 degrees
- moved D6 133.7 mm to (129.5, 152.7), turned to 180 degrees
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Connections:
- U4 pad 3: Net-(Q5-Pad1) -> Net-(R21-Pad1)
- U4 pad 4: (no net) -> Net-(Q5-Pad1)
Other:
- board outline added: 44.5 x 94.5 mm

Commit message: update
Parts:
- removed D6: D, Diodes_SMD:SMB_Handsoldering
- added SW2: LED-switch, footprints:SMT-led-switch, F.Cu at (155.1, -67.0)
- C14: value 2.2pF -> 2.2uF
- D7: footprint Diodes_SMD:SMB_Handsoldering -> footprints:PMEG45A10EPDAZ-Schottky
- R22: value 27M -> 470K
- R4: value 1K -> 36
- Relay1: value V23105 -> ORWH-SH-105D1F
- U2: value ADA4075 -> OPA344
- U6: footprint Transformers_CHK:Trafo_CHK-EI30-2VA_1xSec -> footprints:PNK-40230
- moved R2 173.1 mm to (52.1, 17.7)
- moved R30 153.7 mm to (-18.9, 168.1)
- moved C14 153.4 mm to (-15.1, 178.8)
- moved C13 147.9 mm to (-12.8, 178.8)
- moved R1 144.4 mm to (150.6, -51.3)
- moved D5 141.7 mm to (-12.1, 167.1), turned to 0 degrees
- moved R26 139.8 mm to (-15.0, 172.6)
- moved R28 136.7 mm to (-10.3, 171.1), turned to 0 degrees
- moved R27 135.4 mm to (-10.3, 173.6), turned to 0 degrees
- moved C1 133.0 mm to (141.0, -14.6)
- moved C11 133.0 mm to (147.7, -19.9)
- moved P5 133.0 mm to (153.2, -27.0)
- moved R11 133.0 mm to (147.7, -28.9)
- moved R3 133.0 mm to (143.2, -19.6)
- moved R5 133.0 mm to (145.4, -19.7)
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Connections:
- P5 pad 1: Net-(P5-Pad1) -> +5V
- P5 pad 2: Net-(P5-Pad2) -> IO12
- P5 pad 3: Net-(P5-Pad3) -> IO14
- P5 pad 4: Net-(P5-Pad4) -> GND
- R1 pad 2: IO2 -> Net-(R1-Pad2)
- R25 pad 1: +5V -> Net-(R25-Pad1)
- R4 pad 1: Net-(D1-Pad1) -> +3V3
- R4 pad 2: IO5 -> Net-(R4-Pad2)
- Relay1 pad 1: Net-(D4-Pad2) -> Net-(P4-Pad2)
- Relay1 pad 2: (no net) -> Net-(D4-Pad2)
- Relay1 pad 3: (no net) -> Net-(P4-Pad1)
- Relay1 pad 5: (no net) -> +5V
- U2 pad 2: Net-(R11-Pad1) -> GND
- U2 pad 4: GND -> Net-(R11-Pad1)
- U2 pad 5: (no net) -> +3V3
Other:
- board size 44.5 x 94.5 mm -> 50 x 92.1 mm

Commit message: update
Parts:
- moved P4 123.7 mm to (-53.8, 121.4)
- moved D4 105.8 mm to (18.2, 142.9), turned to 90 degrees
- moved U6 2.68 mm to (-2.69, 173.8)
Changed lines of the file:
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@@
     (links 156)
     (no_connects 156)
-    (area 148.514999 36.881999 198.703001 129.107001)
+    (area -76.046523 -73.48466 210.539001 183.9135)
     (thickness 1.6)
     (drawings 16)
@@
     (descr "Single phase bridge rectifier case 15.7x15.7")
     (tags "Diode Bridge")
-    (fp_text reference BR1 (at -1.016 4.958 360) (layer F.SilkS)
+    (fp_text reference BR1 (at -1.016 4.958) (layer F.SilkS)
       (effects (font (size 1 1) (thickness 0.15)))
     )
@@
     (descr "Radial Electrolytic Capacitor Diameter 8mm x Length 11.5mm, Pitch 3.5mm")
     (tags "Electrolytic Capacitor")
-    (fp_text reference C9 (at -2.667 -2.921 540) (layer F.SilkS)
+    (fp_text reference C9 (at -2.667 -2.921 180) (layer F.SilkS)
       (effects (font (size 1 1) (thickness 0.15)))
     )
@@
     (tags "capacitor 0603")
     (attr smd)
-    (fp_text reference C13 (at -2.606 -0.762 360) (layer F.SilkS)
+    (fp_text reference C13 (at -2.606 -0.762) (layer F.SilkS)
       (effects (font (size 1 1) (thickness 0.15)))
     )
@@
     (tags "capacitor 0603")
     (attr smd)
-    (fp_text reference C14 (at -2.667 0.381 360) (layer F.SilkS)
+    (fp_text reference C14 (at -2.667 0.381) (layer F.SilkS)
       (effects (font (size 1 1) (thickness 0.15)))
     )
@@
   )
   (module Diodes_SMD:SMA_Standard (layer F.Cu)
-    (at 56.458735 44.306508)
+    (at 18.161 142.90802 90)
     (descr "Diode SMA")
     (tags "Diode SMA")
     (attr smd)
-    (fp_text reference D4 (at 0 -3.81) (layer F.SilkS)
-      (effects (font (size 1 1) (thickness 0.15)))
-    )
-    (fp_text value D (at 0 4.3) (layer F.Fab)
+    (fp_text reference D4 (at 0 -3.81 90) (layer F.SilkS)
+      (effects (font (size 1 1) (thickness 0.15)))
+    )
+    (fp_text value D (at 0 4.3 90) (layer F.Fab)
       (effects (font (size 1 1) (thickness 0.15)))
     )
@@
     (fp_line (start 3.5 2) (end -3.5 2) (layer F.CrtYd) (width 0.05))
     (fp_line (start -3.5 2) (end -3.5 -2) (layer F.CrtYd) (width 0.05))
-    (fp_text user K (at -2.9 2.95) (layer F.SilkS)
-      (effects (font (size 1 1) (thickness 0.15)))
-    )
-    (fp_text user A (at 2.9 2.9) (layer F.SilkS)
+    (fp_text user K (at -2.9 2.95 90) (layer F.SilkS)
+      (effects (font (size 1 1) (thickness 0.15)))
+    )
+    (fp_text user A (at 2.9 2.9 90) (layer F.SilkS)
       (effects (font (size 1 1) (thickness 0.15)))
     )
@@
     (fp_line (start -2.25044 1.75006) (end 2.25044 1.75006) (layer F.SilkS) (width 0.15))
     (fp_line (start -2.25044 -1.75006) (end 2.25044 -1.75006) (layer F.SilkS) (width 0.15))
-    (pad 1 smd rect (at -1.99898 0) (size 2.49936 1.80086) (layers F.Cu F.Paste F.Mask)
+    (pad 1 smd rect (at -1.99898 0 90) (size 2.49936 1.80086) (layers F.Cu F.Paste F.Mask)
       (net 8 +5V))
-    (pad 2 smd rect (at 1.99898 0) (size 2.49936 1.80086) (layers F.Cu F.Paste F.Mask)
+    (pad 2 smd rect (at 1.99898 0 90) (size 2.49936 1.80086) (layers F.Cu F.Paste F.Mask)
       (net 21 "Net-(D4-Pad2)"))
     (model Diodes_SMD.3dshapes/SMA_Standard.wrl
@@
     (tags "resistor 0805")
     (attr smd)
-    (fp_text reference L1 (at -3.556 0 360) (layer F.SilkS)
+    (fp_text reference L1 (at -3.556 0) (layer F.SilkS)
       (effects (font (size 1 1) (thickness 0.15)))
     )
@@
   )
   (module Terminal_Blocks:TerminalBlock_Pheonix_MKDS1.5-2pol (layer F.Cu)
-    (at 44.808735 46.846508)
+    (at -53.848 121.412)
     (descr "2-way 5mm pitch terminal block, Phoenix MKDS series")
     (fp_text reference P4 (at 2.5 5.9) (layer F.SilkS)
@@
     (tags "resistor 0805")
     (attr smd)
-    (fp_text reference R15 (at -3.603 0.254 360) (layer F.SilkS)
+    (fp_text reference R15 (at -3.603 0.254) (layer F.SilkS)
       (effects (font (size 1 1) (thickness 0.15)))
     )
@@
     (tags "resistor 0805")
     (attr smd)
-    (fp_text reference R16 (at -4.017 0 360) (layer F.SilkS)
+    (fp_text reference R16 (at -4.017 0) (layer F.SilkS)
       (effects (font (size 1 1) (thickness 0.15)))
     )
@@
   )
   (module footprints:PNK-40230 (layer F.Cu)
-    (at -5.3594 173.4566)
+    (at -2.6924 173.7614)
     (fp_text reference U6 (at 20.701 -20.955 180) (layer F.SilkS)
       (effects (font (size 1 1) (thickness 0.15)))
@@
       (net 8 +5V))
   )
-  (gr_line (start 135.382 21.59) (end 135.382 141.605) (layer Dwgs.User) (width 0.2))
-  (gr_line (start 210.439 21.59) (end 135.382 21.59) (layer Dwgs.User) (width 0.2))
-  (gr_line (start 210.439 141.605) (end 210.439 21.59) (layer Dwgs.User) (width 0.2))
+  (gr_line (start 136.906 21.59) (end 136.906 141.605) (layer Dwgs.User) (width 0.2))
+  (gr_line (start 211.963 21.59) (end 136.906 21.59) (layer Dwgs.User) (width 0.2))
+  (gr_line (start 211.963 141.605) (end 211.963 21.59) (layer Dwgs.User) (width 0.2))
   (gr_line (start 135.382 141.605) (end 210.439 141.605) (layer Dwgs.User) (width 0.2))
   (gr_circle (center 173.609 33.909) (end 173.736 31.496) (layer Dwgs.User) (width 0.2))

Commit message: update
Parts:
- added P3: CONN_01X02, footprints:pheonix-connector-01x02-5mm, F.Cu at (100.4, 89.3)
- added P6: CONN_01X03, Connectors_Hirose:Hirose_DF13-03P-1.25DSA_03x1.25mm_Straight, F.Cu at (173.0, 100.1)
- added P7: CONN_01X03, Connectors_Hirose:Hirose_DF13-03P-1.25DS_03x1.25mm_Angled, F.Cu at (146.6, 113.0)
- BR1: footprint footprints:surfacemount-diodebridge -> footprints:DF005S; moved to B.Cu
- C10, C12, C13, C14, C7, D3, D4, D7, L1, Q3, Q5, R14, R15, R16, R18, R19, R20, R21, R22, R23, R26, R27, R28, R29, R30, R31, U4: moved to B.Cu
- D5: footprint Diodes_SMD:SMA_Standard -> Diodes_SMD:SOD-323; moved to B.Cu
- P4: footprint Terminal_Blocks:TerminalBlock_Pheonix_MKDS1.5-2pol -> footprints:pheonix-connector-01x02-5mm
- U5: footprint libraries:PT5529B -> footprints:PT5529; moved to B.Cu
- moved R16 199.8 mm to (147.4, 99.9), turned to 0 degrees
- moved C8 191.4 mm to (124.2, 92.8), turned to 180 degrees
- moved L2 190.7 mm to (114.0, 103.5)
- moved RT1 184.1 mm to (102.7, 103.7)
- moved L1 183.5 mm to (119.2, 89.9), turned to 0 degrees
- moved BR1 182.7 mm to (115.6, 89.9)
- moved R20 180.9 mm to (137.0, 104.7), turned to 180 degrees
- moved C3 180.2 mm to (110.3, 95.0), turned to 90 degrees
- moved R15 178.0 mm to (126.0, 114.8), turned to 180 degrees
- moved C12 177.3 mm to (136.2, 90.7)
- moved R19 176.3 mm to (136.8, 98.5)
- moved SW2 173.6 mm to (200.5, 100.6)
- moved R18 171.5 mm to (125.9, 112.3)
- moved D3 170.4 mm to (144.5, 95.8), turned to 0 degrees
- moved R22 169.3 mm to (136.6, 93.7), turned to 0 degrees
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Connections:
- BR1 pad 4: VDD -> HV+
- P4 pad 1: Net-(P4-Pad1) -> HV-
- P4 pad 2: Net-(P4-Pad2) -> RELAY
- RT1 pad 2: VDDA -> HV-
- Relay1 pad 1: Net-(P4-Pad2) -> HV-
- Relay1 pad 3: Net-(P4-Pad1) -> RELAY
Other:
- board size 50 x 92.1 mm -> 115.9 x 92.1 mm
