File: hardware/liger.kicad_pcb (KiCad board)
At the start: 2 copper layers, 43.2 x 92.2 mm, 54 parts, among them P1 CONN_01X20, P2 CONN_01X20, P3 CONN_01X03, P4 CONN_01X03, P5 CONN_01X04, P6 CONN_01X04, Q1 Q_NPN_BEC, Q2 Q_NMOS_GSD, Q3 Q_PMOS_GSD, U1 ESP-WROOM-32, U12 soft-button-4x, U2 PT5529B/L2/H2-F, U3 MEMS-SPM0408LE5H, U4 OPA344, U5 SPX3819, U6 OPA344, U7 RGB-LED, U8 Amplifier-D-TS4962IQT

Commit message: update
Parts:
- moved U6 133.3 mm to (248.9, 84.4)
- moved R7 41.3 mm to (143.1, 58.2)
Changed lines of the file:
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@@
   )
   (module Resistors_SMD:R_0603_HandSoldering (layer F.Cu)
-    (at 115.638027 89.114302 270)
-    (descr "Resistor SMD 0603, hand soldering")
-    (tags "resistor 0603")
-    (attr smd)
-    (fp_text reference R7 (at 0 -1.45 270) (layer F.SilkS)
+    (at 143.09 58.21 270)
+    (descr "Resistor SMD 0603, hand soldering")
+    (tags "resistor 0603")
+    (attr smd)
+    (fp_text reference R7 (at -0.95 1.58 360) (layer F.SilkS)
       (effects (font (size 1 1) (thickness 0.15)))
     )
@@
   )
   (module TO_SOT_Packages_SMD:SOT-23-5 (layer F.Cu)
-    (at 115.638027 89.114302 270)
+    (at 248.88 84.38 270)
     (descr "5-pin SOT23 package")
     (tags SOT-23-5)

Commit message: update
Parts:
- removed P5: CONN_01X04, Pin_Headers:Pin_Header_Straight_1x04_Pitch2.54mm
- D1, D3, LS1, U2: moved to B.Cu
- P3: footprint Pin_Headers:Pin_Header_Straight_1x03_Pitch2.54mm -> open-automation:PIR; moved to B.Cu
- moved P2 137.1 mm to (165.9, 119.4), turned to 180 degrees
- moved D1 110.7 mm to (159.9, 58.3)
- moved U6 90.6 mm to (159.8, 68.2)
- moved P1 85.9 mm to (128.9, 76.0), turned to 0 degrees
- moved U1 83.6 mm to (138.8, 101.8), turned to 0 degrees
- moved R1 75.9 mm to (123.3, 131.6)
- moved R2 75.9 mm to (123.0, 136.0)
- moved Q1 67.8 mm to (121.1, 67.1)
- moved P6 60.0 mm to (151.4, 52.9)
- moved R11 50.4 mm to (160.3, 112.3), turned to 0 degrees
- moved Q2 46.9 mm to (122.3, 89.1), turned to 0 degrees
- moved R9 45.2 mm to (155.6, 67.9)
- moved C4 45.0 mm to (120.1, 121.2)
- moved C5 45.0 mm to (121.6, 122.3)
- moved C6 45.0 mm to (120.9, 117.2)
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
Commit message: update
Parts:
- removed R2: 10K, Resistors_SMD:R_0603_HandSoldering
- moved C5 61.7 mm to (161.2, 74.9), turned to 180 degrees
- moved R18 58.9 mm to (159.7, 50.0), turned to 180 degrees
- moved R19 55.5 mm to (159.7, 55.5), turned to 0 degrees
- moved R17 54.8 mm to (155.8, 51.8), turned to 180 degrees
- moved R25 54.6 mm to (157.2, 124.5)
- moved R14 45.9 mm to (160.1, 77.8), turned to 90 degrees
- moved Q1 44.3 mm to (164.5, 58.4), turned to 180 degrees
- moved R16 42.9 mm to (155.1, 72.2), turned to 0 degrees
- moved C6 42.9 mm to (154.7, 90.8), turned to 180 degrees
- moved R5 41.3 mm to (159.8, 64.2), turned to 90 degrees
- moved R15 41.2 mm to (156.2, 82.2), turned to 90 degrees
- moved Q2 40.6 mm to (159.2, 72.2), turned to 180 degrees
- moved Q3 38.6 mm to (159.2, 82.3)
- moved D2 38.4 mm to (154.5, 82.5), turned to 90 degrees
- moved R12 37.6 mm to (152.4, 96.8)
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Connections:
- P1 pad 3: 3V3 -> 3v3
- P1 pad 4: 3V3 -> 3v3
- U1 pad 2: 3V3 -> 3v3

Commit message: update
Parts:
- moved R8 1.53 mm to (155.5, 96.7)
- moved U5 1.26 mm to (138.8, 122.7)
- moved C3 1.13 mm to (133.5, 123.7)
- moved R11 1.12 mm to (136.8, 126.5)
- moved R18 1.08 mm to (160.7, 50.3)
- moved C4 1.00 mm to (133.4, 121.5)
- moved R12 1.00 mm to (153.4, 96.7)
- moved R19 0.97 mm to (160.6, 55.9)
- moved U6 0.91 mm to (160.6, 53.0)
- moved R5 0.84 mm to (159.9, 65.0)
- moved R7 0.58 mm to (138.7, 56.3)
- moved R9 0.57 mm to (134.3, 56.5)
- moved U4 0.47 mm to (135.4, 61.4)
- moved R6 0.42 mm to (138.8, 62.9)
- moved R13 0.36 mm to (151.2, 96.7)
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Changed lines of the file:
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@@
   )
   (module Capacitors_SMD:C_0603_HandSoldering (layer F.Cu)
-    (at 140.8 56.6 270)
+    (at 140.825 56.45 270)
     (descr "Capacitor SMD 0603, hand soldering")
     (tags "capacitor 0603")
@@
   )
   (module Capacitors_SMD:C_0603_HandSoldering (layer F.Cu)
-    (at 133.444852 124.800468 180)
+    (at 133.475 123.675 180)
     (descr "Capacitor SMD 0603, hand soldering")
     (tags "capacitor 0603")
@@
   )
   (module Capacitors_SMD:C_0603_HandSoldering (layer F.Cu)
-    (at 133.394852 122.500468 180)
+    (at 133.375 121.5 180)
     (descr "Capacitor SMD 0603, hand soldering")
     (tags "capacitor 0603")
@@
   )
   (module Resistors_SMD:R_0603_HandSoldering (layer F.Cu)
-    (at 159.75 64.15 90)
+    (at 159.9 64.975 90)
     (descr "Resistor SMD 0603, hand soldering")
     (tags "resistor 0603")
@@
   )
   (module Resistors_SMD:R_0603_HandSoldering (layer F.Cu)
-    (at 138.8 62.5 270)
+    (at 138.8 62.925 270)
     (descr "Resistor SMD 0603, hand soldering")
     (tags "resistor 0603")
@@
   )
   (module Resistors_SMD:R_0603_HandSoldering (layer F.Cu)
-    (at 138.7 56.85 270)
+    (at 138.725 56.275 270)
     (descr "Resistor SMD 0603, hand soldering")
     (tags "resistor 0603")
@@
   )
   (module Resistors_SMD:R_0603_HandSoldering (layer F.Cu)
-    (at 154 96.75 270)
+    (at 155.525 96.675 270)
     (descr "Resistor SMD 0603, hand soldering")
     (tags "resistor 0603")
@@
   )
   (module Resistors_SMD:R_0603_HandSoldering (layer F.Cu)
-    (at 134.65 56.9 90)
+    (at 134.3 56.45 90)
     (descr "Resistor SMD 0603, hand soldering")
     (tags "resistor 0603")
@@
   )
   (module Resistors_SMD:R_0603_HandSoldering (layer F.Cu)
-    (at 132.1 61.15 270)
+    (at 131.75 61.2 270)
     (descr "Resistor SMD 0603, hand soldering")
     (tags "resistor 0603")
@@
   )
   (module Resistors_SMD:R_0603_HandSoldering (layer F.Cu)
-    (at 135.694852 126.600468)
+    (at 136.8 126.45)
     (descr "Resistor SMD 0603, hand soldering")
     (tags "resistor 0603")
@@
   )
   (module Resistors_SMD:R_0603_HandSoldering (layer F.Cu)
-    (at 152.45 96.75 270)
+    (at 153.45 96.725 270)
     (descr "Resistor SMD 0603, hand soldering")
     (tags "resistor 0603")
@@
   )
   (module Resistors_SMD:R_0603_HandSoldering (layer F.Cu)
-    (at 150.9 96.75 270)
+    (at 151.25 96.675 270)
     (descr "Resistor SMD 0603, hand soldering")
     (tags "resistor 0603")
@@
   )
   (module Resistors_SMD:R_0603_HandSoldering (layer F.Cu)
-    (at 155.75 51.825 180)
+    (at 155.675 51.85 180)
     (descr "Resistor SMD 0603, hand soldering")
     (tags "resistor 0603")
@@
   )
   (module Resistors_SMD:R_0603_HandSoldering (layer F.Cu)
-    (at 159.670631 49.951839 180)
+    (at 160.7 50.275 180)
     (descr "Resistor SMD 0603, hand soldering")
     (tags "resistor 0603")
@@
   )
   (module Resistors_SMD:R_0603_HandSoldering (layer F.Cu)
-    (at 159.745631 55.476839)
+    (at 160.625 55.875)
     (descr "Resistor SMD 0603, hand soldering")
     (tags "resistor 0603")
@@
   )
   (module TO_SOT_Packages_SMD:SOT-23-5 (layer F.Cu)
-    (at 135.7 61.05 180)
+    (at 135.425 61.425 180)
     (descr "5-pin SOT23 package")
     (tags SOT-23-5)
@@
   )
   (module TO_SOT_Packages_SMD:SOT-23-5 (layer F.Cu)
-    (at 137.869852 123.525468 90)
+    (at 138.825 122.7 90)
     (descr "5-pin SOT23 package")
     (tags SOT-23-5)
@@
   )
   (module TO_SOT_Packages_SMD:SOT-23-5 (layer F.Cu)
-    (at 159.745631 52.801839 180)
+    (at 160.625 53.05 180)
     (descr "5-pin SOT23 package")
     (tags SOT-23-5)

Commit message: update
Routing:
- added copper zone on B.Cu, net GND
Changed lines of the file:
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@@
   (gr_circle (center 147.684028 40.095641) (end 147.811028 42.508641) (layer Dwgs.User) (width 0.2))
   (gr_circle (center 147.684028 47.458302) (end 147.938028 50.506302) (layer Edge.Cuts) (width 0.15))
+  (zone (net 1) (net_name GND) (layer B.Cu) (hatch edge 0.508)
+    (connect_pads (clearance 0.508))
+    (min_thickness 0.254)
+    (fill yes (arc_segments 16) (thermal_gap 0.508) (thermal_bridge_width 0.508))
+    (polygon
+      (pts
+        (xy 152.925 43.1) (xy 152.925 49.325) (xy 168.8 49.325) (xy 168.8 127.5) (xy 152.925 127.5)
+        (xy 152.925 135.125) (xy 142.45 135.125) (xy 142.45 127.5) (xy 125.8 127.5) (xy 125.8 49.325)
+        (xy 142.7 49.325) (xy 142.7 43.1)
+      )
+    )
+  )
 )

Commit message: update
Parts:
- moved C5 21.6 mm to (139.6, 75.3)
- moved D2 21.6 mm to (132.9, 82.9)
- moved PROG1 21.6 mm to (135.8, 77.5)
- moved Q2 21.6 mm to (137.6, 72.7)
- moved Q3 21.6 mm to (137.6, 82.8)
- moved R14 21.6 mm to (138.5, 78.3)
- moved R15 21.6 mm to (134.7, 82.6)
- moved R16 21.6 mm to (133.5, 72.7)
- moved R1 10.4 mm to (152.2, 115.0), turned to 90 degrees
- moved R19 6.12 mm to (156.5, 60.4), turned to 270 degrees
- moved R18 5.12 mm to (155.6, 50.8)
- moved U6 5.06 mm to (155.7, 54.0), turned to 90 degrees
- moved R17 4.94 mm to (160.5, 52.9), turned to 0 degrees
- turned R6 to 90 degrees
Routing:
- net 5V: track 0.00 -> 89.3 mm
- net 3V3: track 0.00 -> 74.5 mm, vias 0 -> 4
- net IO35: track 0.00 -> 74.0 mm
- net IO0: track 0.00 -> 71.3 mm, vias 0 -> 4
- net GND: track 0.00 -> 37.6 mm, vias 0 -> 10
- net IO25: track 0.00 -> 31.4 mm, vias 0 -> 1
- net IO17: track 0.00 -> 29.9 mm, vias 0 -> 2
- net TXD: track 0.00 -> 27.5 mm
- net RXD: track 0.00 -> 26.3 mm
- net IO34: track 0.00 -> 25.8 mm
- net Net-(R8-Pad2): track 0.00 -> 25.7 mm, vias 0 -> 1
- net 3v3: track 0.00 -> 25.5 mm
- net SENSOR_VP: track 0.00 -> 23.0 mm
- net IO27: track 0.00 -> 22.5 mm, vias 0 -> 1
- net SENSOR_VN: track 0.00 -> 21.8 mm
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
Commit message: update
Routing:
- net IO17: track 29.9 -> 93.5 mm, vias 2 -> 3
- net GND: track 37.6 -> 39.3 mm, vias 10 -> 11
Other:
- board text added: "GND"
Changed lines of the file:
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@@
   (general
     (links 146)
-    (no_connects 94)
+    (no_connects 39)
     (area 125.638027 42.938301 168.968029 135.290303)
     (thickness 1.6)
-    (drawings 35)
-    (tracks 360)
+    (drawings 37)
+    (tracks 376)
     (zones 0)
     (modules 52)
@@
   )
   (setup
-    (last_trace_width 0.4)
+    (last_trace_width 0.25)
     (user_trace_width 0.25)
     (user_trace_width 0.4)
@@
     )
   )
+  (gr_text GND (at 162.776076 71.33189) (layer F.SilkS)
+    (effects (font (size 1 1) (thickness 0.2)))
+  )
+  (gr_text GND (at 162.9 73.7) (layer F.SilkS)
+    (effects (font (size 1 1) (thickness 0.2)))
+  )
   (gr_line (start 112.080028 30.909302) (end 112.1 144.91) (layer Dwgs.User) (width 0.2))
   (gr_line (start 130.6 121.4) (end 130.6 54.4) (layer Dwgs.User) (width 0.2))
@@
   (gr_circle (center 147.684028 40.095641) (end 147.811028 42.508641) (layer Dwgs.User) (width 0.2))
   (gr_circle (center 147.684028 47.458302) (end 147.938028 50.506302) (layer Edge.Cuts) (width 0.15))
+  (segment (start 161.6 52.9) (end 162.75 52.9) (width 0.25) (layer F.Cu) (net 1))
+  (segment (start 162.75 52.9) (end 163.15 52.5) (width 0.25) (layer F.Cu) (net 1))
+  (via (at 163.15 52.5) (size 0.9) (drill 0.6) (layers F.Cu B.Cu) (net 1))
   (segment (start 152.25 114.1) (end 153.450002 115.300002) (width 0.25) (layer F.Cu) (net 1))
   (segment (start 153.450002 115.300002) (end 153.450002 116.35) (width 0.25) (layer F.Cu) (net 1))
@@
   (segment (start 138.55 82.75) (end 138.55 79.45) (width 0.25) (layer F.Cu) (net 18))
   (segment (start 138.55 79.45) (end 138.5 79.4) (width 0.25) (layer F.Cu) (net 18))
+  (segment (start 164.45 63.3) (end 163.425001 62.275001) (width 0.25) (layer B.Cu) (net 19))
+  (segment (start 148.87 54.052081) (end 148.87 52.85) (width 0.25) (layer B.Cu) (net 19))
+  (segment (start 163.425001 62.275001) (end 152.653999 62.275001) (width 0.25) (layer B.Cu) (net 19))
+  (segment (start 152.653999 62.275001) (end 148.87 58.491002) (width 0.25) (layer B.Cu) (net 19))
+  (segment (start 148.87 58.491002) (end 148.87 54.052081) (width 0.25) (layer B.Cu) (net 19))
+  (segment (start 165.45 63.75) (end 164.9 63.75) (width 0.25) (layer F.Cu) (net 19))
+  (segment (start 164.9 63.75) (end 164.45 63.3) (width 0.25) (layer F.Cu) (net 19))
+  (via (at 164.45 63.3) (size 0.6) (drill 0.4) (layers F.Cu B.Cu) (net 19))
+  (segment (start 165.45 63.75) (end 165.45 63.9) (width 0.25) (layer F.Cu) (net 19))
+  (segment (start 165.45 63.9) (end 167.165001 65.615001) (width 0.25) (layer F.Cu) (net 19))
+  (segment (start 166.739999 100.800001) (end 165.89 101.65) (width 0.25) (layer F.Cu) (net 19))
+  (segment (start 167.165001 65.615001) (end 167.165001 100.374999) (width 0.25) (layer F.Cu) (net 19))
+  (segment (start 167.165001 100.374999) (end 166.739999 100.800001) (width 0.25) (layer F.Cu) (net 19))
   (segment (start 154.55 115.6) (end 154.55 114.27908) (width 0.25) (layer F.Cu) (net 19))
   (segment (start 154.55 114.27908) (end 155.55788 113.2712) (width 0.25) (layer F.Cu) (net 19))

Commit message: update
Parts:
- moved R1 6.79 mm to (151.2, 121.8), turned to 180 degrees
Routing:
- net 5V: track 89.3 -> 201.7 mm, vias 0 -> 6
- net GND: track 39.3 -> 129.6 mm, vias 11 -> 23
- net SPEAKER+: track 0.00 -> 70.3 mm, vias 0 -> 1
- net SPEAKER-: track 0.00 -> 62.8 mm, vias 0 -> 2
- net Net-(R3-Pad1): track 0.00 -> 47.7 mm, vias 0 -> 1
- net 3V3: track 74.5 -> 114.3 mm, vias 4 -> 6
- net IO16: track 14.8 -> 54.6 mm, vias 0 -> 3
- net IO18: track 18.7 -> 55.3 mm, vias 0 -> 3
- net IO34: track 25.8 -> 57.4 mm, vias 0 -> 1
- net IO19: track 19.9 -> 50.5 mm, vias 0 -> 3
- net EN: track 8.20 -> 33.0 mm, vias 0 -> 2
- net IO15: track 19.7 -> 41.1 mm
- net IO4: track 13.3 -> 30.4 mm, vias 0 -> 1
- net IO33: track 16.7 -> 33.8 mm, vias 0 -> 1
- net IO35: track 74.0 -> 88.3 mm, vias 0 -> 2
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Other:
- board text added: "5V 5V TXD RXD I023 I022 I021 I019 I018 I05 I017 I016 I04 I00 I02 I015 SD1 SD0"
- board text added: "GND GND 3V3 3V3 VP VN I034 I035 I032 I033 I025 I026 I027 I014 I012 I013 SD2 SD3 SP+ SP-"
