File: hardware/thermometer.sch (KiCad schematic (older format))
At the start: 2 parts

Commit message: update
Parts:
- R24: Part Number RC0603JR-0710KL -> RC0603JR-07100KL
Changed lines of the file:
@@
 F 1 "100K" V 4750 3450 50  0000 C CNN
 F 2 "Resistors_SMD:R_0603_HandSoldering" V 4680 3450 50  0001 C CNN
-F 3 "http://www.digikey.com/en/resources/datasheets/yageo/rc-series-l-suffix-datasheet" H 4750 3450 50  0001 C CNN
-F 4 "RC0603JR-0710KL" V 4750 3450 60  0001 C CNN "Part Number"
+F 3 "http://www.yageo.com/documents/recent/PYu-RC_Group_51_RoHS_L_7.pdf" H 4750 3450 50  0001 C CNN
+F 4 "RC0603JR-07100KL" V 4750 3450 60  0001 C CNN "Part Number"
 	1    4750 3450
 	1    0    0    -1
