File: hardware/ultrasonic.sch (KiCad schematic (older format))
At the start: 1 part, among them P5 CONN_01X04

Commit message: update
Parts:
- removed P5: CONN_01X04, Pin_Headers:Pin_Header_Straight_1x04_Pitch2.54mm, symbol CONN_01X04
Changed lines of the file:
@@
 Comment4 ""
 $EndDescr
-$Comp
-L CONN_01X04 P5
-U 1 1 5909282F
-P 5700 4150
-F 0 "P5" H 5700 4400 50  0000 C CNN
-F 1 "CONN_01X04" V 5800 4150 50  0000 C CNN
-F 2 "Pin_Headers:Pin_Header_Straight_1x04_Pitch2.54mm" H 5700 4150 50  0001 C CNN
-F 3 "http://sullinscorp.com/catalogs/101_PAGE114-115_.100_FEMALE_HDR.pdf" H 5700 4150 50  0001 C CNN
-F 4 "PPTC041LGBN-RC" H 5700 4150 60  0001 C CNN "Part Number"
-	1    5700 4150
-	0    1    1    0
-$EndComp
 Text Label 5250 3000 0    60   ~ 0
 Ultra-Sonic_Sensor
-Text GLabel 5750 3750 1    60   Input ~ 0
-IO12
-Text GLabel 5650 3750 1    60   Input ~ 0
-IO13
-$Comp
-L GND #PWR019
-U 1 1 59092834
-P 5500 3900
-F 0 "#PWR019" H 5500 3650 50  0001 C CNN
-F 1 "GND" H 5500 3750 50  0000 C CNN
-F 2 "" H 5500 3900 50  0000 C CNN
-F 3 "" H 5500 3900 50  0000 C CNN
-	1    5500 3900
-	0    1    1    0
-$EndComp
-Wire Wire Line
-	5750 3750 5750 3950
-Wire Wire Line
-	5650 3750 5650 3950
-Wire Wire Line
-	5850 3900 5850 3950
-Wire Wire Line
-	5900 3900 5850 3900
-Wire Wire Line
-	5550 3900 5550 3950
-Wire Wire Line
-	5500 3900 5550 3900
-Text GLabel 5900 3900 2    60   Input ~ 0
-5V
 $EndSCHEMATC
