File: hardware/InfraRed.sch (KiCad schematic (older format))
At the start: 12 parts, among them P3 CONN_01X03, Q1 Q_NPN_BEC, U2 PT5529B/L2/H2-F, U6 OPA344

Commit message: update
Parts:
- D3: Part Number QED123 -> 365-1086-ND
- Q1: Part Number MMBT3904LT1G -> MMBT3904LT1GOSCT-ND
- R17: Part Number RC0603JR-071KL -> RC0603JR-0722KL
- R18: Part Number RC0603JR-071KL -> RC0603FR-071ML
- R19: Part Number RC0603JR-071KL -> RC0603JR-07180KL
- U2: Part Number PT5529B/L2/H2-F -> 1080-1161-ND
- U6: Part Number (none) -> 296-41475-1-ND
Changed lines of the file:
@@
 F 2 "footprints:PT5529" H 7300 2600 60  0001 C CNN
 F 3 "http://www.everlight.com/file/ProductFile/PT5529B-L2-H2-F.pdf" H 7300 2600 60  0001 C CNN
-F 4 "PT5529B/L2/H2-F" H 7300 2600 60  0001 C CNN "Part Number"
+F 4 "1080-1161-ND" H 7300 2600 60  0001 C CNN "Part Number"
 	1    7300 2600
 	1    0    0    -1
@@
 F 1 "Q_NPN_BEC" H 8200 5050 50  0000 R CNN
 F 2 "TO_SOT_Packages_SMD:SOT-23" H 7800 5200 50  0001 C CNN
-F 3 "http://www.mouser.com/ds/2/308/MMBT3904LT1-D-113169.pdf" H 7600 5100 50  0001 C CNN
-F 4 "MMBT3904LT1G" H 7600 5100 60  0001 C CNN "Part Number"
+F 3 "http://www.onsemi.com/pub/Collateral/MMBT3904LT1-D.PDF" H 7600 5100 50  0001 C CNN
+F 4 "MMBT3904LT1GOSCT-ND" H 7600 5100 60  0001 C CNN "Part Number"
 	1    7600 5100
 	1    0    0    -1
@@
 F 2 "TO_SOT_Packages_SMD:SOT-23-5" H 4450 2850 50  0001 C CNN
 F 3 "http://www.digikey.com/product-detail/en/texas-instruments/OPA344NA-3K/296-41475-1-ND/5222851" H 4550 2950 50  0001 C CNN
+F 4 "296-41475-1-ND" H 4550 2800 60  0001 C CNN "Part Number"
 	1    4550 2800
 	1    0    0    -1
@@
 F 1 "LED" H 4000 2600 50  0000 C CNN
 F 2 "LEDs:LED_D3.0mm" H 4000 2700 50  0001 C CNN
-F 3 "http://www.mouser.com/ds/2/149/QED123-890063.pdf" H 4000 2700 50  0001 C CNN
-F 4 "QED123" H 4000 2700 60  0001 C CNN "Part Number"
+F 3 "http://www.ttelectronics.com/sites/default/files/download-files/OP993-999_0.pdf" H 4000 2700 50  0001 C CNN
+F 4 "365-1086-ND" H 4000 2700 60  0001 C CNN "Part Number"
 	1    4000 2700
 	-1   0    0    1
@@
 F 1 "180K" V 4450 3550 50  0000 C CNN
 F 2 "Resistors_SMD:R_0603_HandSoldering" V 4380 3550 50  0001 C CNN
-F 3 "http://www.digikey.com/en/resources/datasheets/yageo/rc-series-l-suffix-datasheet" H 4450 3550 50  0001 C CNN
-F 4 "RC0603JR-071KL" V 4450 3550 60  0001 C CNN "Part Number"
+F 3 "http://www.yageo.com/documents/recent/PYu-RC_Group_51_RoHS_L_7.pdf" H 4450 3550 50  0001 C CNN
+F 4 "RC0603JR-07180KL" V 4450 3550 60  0001 C CNN "Part Number"
 	1    4450 3550
 	0    -1   -1   0
@@
 F 1 "22K" V 4000 2900 50  0000 C CNN
 F 2 "Resistors_SMD:R_0603_HandSoldering" V 3930 2900 50  0001 C CNN
-F 3 "http://www.digikey.com/en/resources/datasheets/yageo/rc-series-l-suffix-datasheet" H 4000 2900 50  0001 C CNN
-F 4 "RC0603JR-071KL" V 4000 2900 60  0001 C CNN "Part Number"
+F 3 "http://www.yageo.com/documents/recent/PYu-RC_Group_51_RoHS_L_7.pdf" H 4000 2900 50  0001 C CNN
+F 4 "RC0603JR-0722KL" V 4000 2900 60  0001 C CNN "Part Number"
 	1    4000 2900
 	0    1    1    0
@@
 F 1 "1M" V 4200 2400 50  0000 C CNN
 F 2 "Resistors_SMD:R_0603_HandSoldering" V 4130 2400 50  0001 C CNN
-F 3 "http://www.digikey.com/en/resources/datasheets/yageo/rc-series-l-suffix-datasheet" H 4200 2400 50  0001 C CNN
-F 4 "RC0603JR-071KL" V 4200 2400 60  0001 C CNN "Part Number"
+F 3 "http://www.yageo.com/documents/recent/PYu-RC_Group_51_RoHS_L_7.pdf" H 4200 2400 50  0001 C CNN
+F 4 "RC0603FR-071ML" V 4200 2400 60  0001 C CNN "Part Number"
 	1    4200 2400
 	-1   0    0    1

Commit message: updatE
Connections:
- net 5V: now also P3.1 (P1); no longer P3.3 (P3)
- net GND: now also P3.3 (P3); no longer P3.1 (P1)
Changed lines of the file:
@@
 IR-Receive
 $Comp
-L GND #PWR05
+L GND #PWR8
 U 1 1 59098AF2
 P 7300 3050
-F 0 "#PWR05" H 7300 2800 50  0001 C CNN
+F 0 "#PWR8" H 7300 2800 50  0001 C CNN
 F 1 "GND" H 7300 2900 50  0000 C CNN
 F 2 "" H 7300 3050 50  0000 C CNN
@@
 $EndComp
 $Comp
-L GND #PWR06
+L GND #PWR9
 U 1 1 59098AF9
 P 7700 5500
-F 0 "#PWR06" H 7700 5250 50  0001 C CNN
+F 0 "#PWR9" H 7700 5250 50  0001 C CNN
 F 1 "GND" H 7700 5350 50  0000 C CNN
 F 2 "" H 7700 5500 50  0000 C CNN
@@
 $EndComp
 $Comp
-L GND #PWR07
+L GND #PWR6
 U 1 1 59098B15
-P 4150 4850
-F 0 "#PWR07" H 4150 4600 50  0001 C CNN
-F 1 "GND" H 4150 4700 50  0000 C CNN
-F 2 "" H 4150 4850 50  0000 C CNN
-F 3 "" H 4150 4850 50  0000 C CNN
-	1    4150 4850
-	-1   0    0    1
+P 4150 5150
+F 0 "#PWR6" H 4150 4900 50  0001 C CNN
+F 1 "GND" H 4150 5000 50  0000 C CNN
+F 2 "" H 4150 5150 50  0000 C CNN
+F 3 "" H 4150 5150 50  0000 C CNN
+	1    4150 5150
+	1    0    0    -1
 $EndComp
 Text GLabel 4100 5000 0    60   Input ~ 0
@@
 PIR
 $Comp
-L GND #PWR08
+L GND #PWR7
 U 1 1 590BA36E
 P 4450 3150
-F 0 "#PWR08" H 4450 2900 50  0001 C CNN
+F 0 "#PWR7" H 4450 2900 50  0001 C CNN
 F 1 "GND" H 4450 3000 50  0000 C CNN
 F 2 "" H 4450 3150 50  0000 C CNN
@@
 $EndComp
 $Comp
-L GND #PWR09
+L GND #PWR5
 U 1 1 590BAE9F
 P 3750 2900
-F 0 "#PWR09" H 3750 2650 50  0001 C CNN
+F 0 "#PWR5" H 3750 2650 50  0001 C CNN
 F 1 "GND" H 3750 2750 50  0000 C CNN
 F 2 "" H 3750 2900 50  0000 C CNN
@@
 Text GLabel 4450 2100 1    60   Input ~ 0
 5V
-Text GLabel 4150 5150 3    60   Input ~ 0
+Text GLabel 4150 4850 1    60   Input ~ 0
 5V
 $EndSCHEMATC

Commit message: updatge
Connections:
- net IO18 renamed IO35
Changed lines of the file:
@@
 IR-Receive
 $Comp
-L GND #PWR8
+L GND #PWR05
 U 1 1 59098AF2
 P 7300 3050
-F 0 "#PWR8" H 7300 2800 50  0001 C CNN
+F 0 "#PWR05" H 7300 2800 50  0001 C CNN
 F 1 "GND" H 7300 2900 50  0000 C CNN
 F 2 "" H 7300 3050 50  0000 C CNN
@@
 $EndComp
 $Comp
-L GND #PWR9
+L GND #PWR06
 U 1 1 59098AF9
 P 7700 5500
-F 0 "#PWR9" H 7700 5250 50  0001 C CNN
+F 0 "#PWR06" H 7700 5250 50  0001 C CNN
 F 1 "GND" H 7700 5350 50  0000 C CNN
 F 2 "" H 7700 5500 50  0000 C CNN
@@
 $EndComp
 $Comp
-L GND #PWR6
+L GND #PWR07
 U 1 1 59098B15
 P 4150 5150
-F 0 "#PWR6" H 4150 4900 50  0001 C CNN
+F 0 "#PWR07" H 4150 4900 50  0001 C CNN
 F 1 "GND" H 4150 5000 50  0000 C CNN
 F 2 "" H 4150 5150 50  0000 C CNN
@@
 $EndComp
 Text GLabel 5050 2800 2    60   Input ~ 0
-IO18
+IO35
 Text Label 4250 1750 0    60   ~ 0
 Light-Level
@@
 PIR
 $Comp
-L GND #PWR7
+L GND #PWR08
 U 1 1 590BA36E
 P 4450 3150
-F 0 "#PWR7" H 4450 2900 50  0001 C CNN
+F 0 "#PWR08" H 4450 2900 50  0001 C CNN
 F 1 "GND" H 4450 3000 50  0000 C CNN
 F 2 "" H 4450 3150 50  0000 C CNN
@@
 $EndComp
 $Comp
-L GND #PWR5
+L GND #PWR09
 U 1 1 590BAE9F
 P 3750 2900
-F 0 "#PWR5" H 3750 2650 50  0001 C CNN
+F 0 "#PWR09" H 3750 2650 50  0001 C CNN
 F 1 "GND" H 3750 2750 50  0000 C CNN
 F 2 "" H 3750 2900 50  0000 C CNN

Commit message: update
Parts:
- P3: footprint Pin_Headers:Pin_Header_Straight_1x03_Pitch2.54mm -> open-automation:PIR
Changed lines of the file:
@@
 $Descr A4 11693 8268
 encoding utf-8
-Sheet 3 9
+Sheet 3 8
 Title ""
 Date ""
@@
 F 0 "P3" H 4350 5200 50  0000 L CNN
 F 1 "CONN_01X03" H 4350 4800 50  0001 L CNN
-F 2 "Pin_Headers:Pin_Header_Straight_1x03_Pitch2.54mm" H 4477 4904 50  0001 L CNN
+F 2 "open-automation:PIR" H 4477 4904 50  0001 L CNN
 F 3 "http://sullinscorp.com/catalogs/101_PAGE114-115_.100_FEMALE_HDR.pdf" H 4400 5000 50  0001 C CNN
 	1    4400 5000
