File: hardware/InfraRed.sch (KiCad schematic (older format))
At the start: 12 parts, among them P3 CONN_01X03, Q1 Q_NPN_BEC, U2 PT5529B/L2/H2-F, U6 OPA344

Commit message: update
Parts:
- removed D3: LED, LEDs:LED_D3.0mm, symbol LED
- removed P3: CONN_01X03, open-automation:PIR, symbol CONN_01X03
- removed R17: 22K, Resistors_SMD:R_0603_HandSoldering, symbol R
- removed R18: 1M, Resistors_SMD:R_0603_HandSoldering, symbol R
- removed R19: 180K, Resistors_SMD:R_0603_HandSoldering, symbol R
- removed R3, R4: 1K, Resistors_SMD:R_0603_HandSoldering, symbol R
- removed U6: OPA344, TO_SOT_Packages_SMD:SOT-23-5, symbol OPA344
- added R3, R4: R_1k, Resistors_SMD:R_0603, symbol R_1k
Connections:
- net labels added: IR_RX, IR_TX, V_USB
- net labels removed: 5V, IO16, IO17, IO35, IO4, Light-Level, PIR
- wire segments 33 -> 13
Other:
- moved on the sheet: D1, Q1, R5, U2

Commit message: update
Other:
- moved on the sheet: D1, Q1, R3, R4, R5, U2
Changed lines of the file:
@@
 L PT5529B/L2/H2-F U2
 U 1 1 59098AF0
-P 5250 2550
-F 0 "U2" H 4950 2450 60  0000 C CNN
-F 1 "PT5529B/L2/H2-F" H 5300 2750 60  0000 C CNN
-F 2 "footprints:PT5529" H 5250 2550 60  0001 C CNN
-F 3 "http://www.everlight.com/file/ProductFile/PT5529B-L2-H2-F.pdf" H 5250 2550 60  0001 C CNN
-F 4 "1080-1161-ND" H 5250 2550 60  0001 C CNN "Part Number"
-	1    5250 2550
+P 4900 3000
+F 0 "U2" H 4600 2900 60  0000 C CNN
+F 1 "PT5529B/L2/H2-F" H 4950 3200 60  0000 C CNN
+F 2 "footprints:PT5529" H 4900 3000 60  0001 C CNN
+F 3 "http://www.everlight.com/file/ProductFile/PT5529B-L2-H2-F.pdf" H 4900 3000 60  0001 C CNN
+F 4 "1080-1161-ND" H 4900 3000 60  0001 C CNN "Part Number"
+	1    4900 3000
 	1    0    0    -1
 $EndComp
-Text Label 5000 2150 0    60   ~ 0
+Text Label 4650 2600 0    60   ~ 0
 IR-Receive
 $Comp
-L GND #PWR02
+L GND #PWR2
 U 1 1 59098AF2
-P 5250 3000
-F 0 "#PWR02" H 5250 2750 50  0001 C CNN
-F 1 "GND" H 5250 2850 50  0000 C CNN
-F 2 "" H 5250 3000 50  0000 C CNN
-F 3 "" H 5250 3000 50  0000 C CNN
-	1    5250 3000
+P 4900 3450
+F 0 "#PWR2" H 4900 3200 50  0001 C CNN
+F 1 "GND" H 4900 3300 50  0000 C CNN
+F 2 "" H 4900 3450 50  0000 C CNN
+F 3 "" H 4900 3450 50  0000 C CNN
+	1    4900 3450
 	1    0    0    -1
 $EndComp
-Text GLabel 4550 2950 0    60   Input ~ 0
+Text GLabel 4200 3400 0    60   Input ~ 0
 IR_RX
 $Comp
 L LED D1
 U 1 1 59098AF4
-P 5650 4550
-F 0 "D1" H 5650 4650 50  0000 C CNN
-F 1 "LED" H 5650 4450 50  0000 C CNN
-F 2 "LEDs:LED_D3.0mm" H 5650 4550 50  0001 C CNN
-F 3 "http://www.mouser.com/ds/2/149/QED123-890063.pdf" H 5650 4550 50  0001 C CNN
-F 4 "QED123" H 5650 4550 60  0001 C CNN "Part Number"
-	1    5650 4550
+P 7500 3050
+F 0 "D1" H 7500 3150 50  0000 C CNN
+F 1 "LED" H 7500 2950 50  0000 C CNN
+F 2 "LEDs:LED_D3.0mm" H 7500 3050 50  0001 C CNN
+F 3 "http://www.mouser.com/ds/2/149/QED123-890063.pdf" H 7500 3050 50  0001 C CNN
+F 4 "QED123" H 7500 3050 60  0001 C CNN "Part Number"
+	1    7500 3050
 	0    -1   -1   0
 $EndComp
@@
 L R R5
 U 1 1 59098AF5
-P 5650 4100
-F 0 "R5" V 5730 4100 50  0000 C CNN
-F 1 "36" V 5650 4100 50  0000 C CNN
-F 2 "Resistors_SMD:R_0603_HandSoldering" V 5580 4100 50  0001 C CNN
-F 3 "http://www.yageo.com.tw/exep/pages/download/literatures/PYu-R_INT-thick_7.pdf" H 5650 4100 50  0001 C CNN
-F 4 "RC0603JR-0736RL" V 5650 4100 60  0001 C CNN "Part Number"
-	1    5650 4100
+P 7500 2600
+F 0 "R5" V 7580 2600 50  0000 C CNN
+F 1 "36" V 7500 2600 50  0000 C CNN
+F 2 "Resistors_SMD:R_0603_HandSoldering" V 7430 2600 50  0001 C CNN
+F 3 "http://www.yageo.com.tw/exep/pages/download/literatures/PYu-R_INT-thick_7.pdf" H 7500 2600 50  0001 C CNN
+F 4 "RC0603JR-0736RL" V 7500 2600 60  0001 C CNN "Part Number"
+	1    7500 2600
 	1    0    0    -1
 $EndComp
@@
 L Q_NPN_BEC Q1
 U 1 1 59098AF8
-P 5550 5050
-F 0 "Q1" H 5850 5100 50  0000 R CNN
-F 1 "Q_NPN_BEC" H 6150 5000 50  0000 R CNN
-F 2 "TO_SOT_Packages_SMD:SOT-23" H 5750 5150 50  0001 C CNN
-F 3 "http://www.onsemi.com/pub/Collateral/MMBT3904LT1-D.PDF" H 5550 5050 50  0001 C CNN
-F 4 "MMBT3904LT1GOSCT-ND" H 5550 5050 60  0001 C CNN "Part Number"
-	1    5550 5050
+P 7400 3550
+F 0 "Q1" H 7700 3600 50  0000 R CNN
+F 1 "Q_NPN_BEC" H 8000 3500 50  0000 R CNN
+F 2 "TO_SOT_Packages_SMD:SOT-23" H 7600 3650 50  0001 C CNN
+F 3 "http://www.onsemi.com/pub/Collateral/MMBT3904LT1-D.PDF" H 7400 3550 50  0001 C CNN
+F 4 "MMBT3904LT1GOSCT-ND" H 7400 3550 60  0001 C CNN "Part Number"
+	1    7400 3550
 	1    0    0    -1
 $EndComp
 $Comp
-L GND #PWR03
+L GND #PWR3
 U 1 1 59098AF9
-P 5650 5450
-F 0 "#PWR03" H 5650 5200 50  0001 C CNN
-F 1 "GND" H 5650 5300 50  0000 C CNN
-F 2 "" H 5650 5450 50  0000 C CNN
-F 3 "" H 5650 5450 50  0000 C CNN
-	1    5650 5450
+P 7500 3950
+F 0 "#PWR3" H 7500 3700 50  0001 C CNN
+F 1 "GND" H 7500 3800 50  0000 C CNN
+F 2 "" H 7500 3950 50  0000 C CNN
+F 3 "" H 7500 3950 50  0000 C CNN
+	1    7500 3950
 	1    0    0    -1
 $EndComp
-Text GLabel 4500 5050 0    60   Input ~ 0
+Text GLabel 6350 3550 0    60   Input ~ 0
 IR_TX
-Text Label 4750 4500 0    60   ~ 0
+Text Label 6600 3000 0    60   ~ 0
 IR-Transmit
 Wire Wire Line
-	4800 5050 4500 5050
+	6650 3550 6350 3550
 Wire Wire Line
-	5650 5250 5650 5450
+	7500 3750 7500 3950
 Wire Wire Line
-	5100 5050 5350 5050
+	6950 3550 7200 3550
 Wire Wire Line
-	5650 3800 5650 3950
+	7500 2300 7500 2450
 Wire Wire Line
-	4650 2950 4550 2950
+	4300 3400 4200 3400
 Wire Wire Line
-	5550 2950 5550 2850
+	5200 3400 5200 3300
 Wire Wire Line
-	5350 2950 5550 2950
+	5000 3400 5200 3400
 Wire Wire Line
-	5350 2850 5350 2950
+	5000 3300 5000 3400
 Wire Wire Line
-	5250 2850 5250 3000
+	4900 3300 4900 3450
 Wire Wire Line
-	5150 2950 4950 2950
+	4800 3400 4600 3400
 Wire Wire Line
-	5150 2850 5150 2950
+	4800 3300 4800 3400
 Wire Wire Line
-	5650 4250 5650 4400
+	7500 2750 7500 2900
 Wire Wire Line
-	5650 4700 5650 4850
-Text GLabel 5650 3800 1    60   Input ~ 0
+	7500 3200 7500 3350
+Text GLabel 7500 2300 1    60   Input ~ 0
 3V3
-Text GLabel 5550 2850 1    60   Input ~ 0
+Text GLabel 5200 3300 1    60   Input ~ 0
 V_USB
 $Comp
 L R_1k R3
 U 1 1 59BA28B3
-P 4800 2950
-F 0 "R3" V 4800 2950 50  0000 C CNN
-F 1 "R_1k" V 4725 2950 50  0000 C CNN
-F 2 "Resistors_SMD:R_0603" V 4730 2950 50  0001 C CNN
-F 3 "https://www.digikey.com/product-detail/en/yageo/RC0603JR-071KL/311-1.0KGRCT-ND/729624" V 4880 2950 50  0001 C CNN
-F 4 "RC0603JR-071KL" V 4980 3050 60  0001 C CNN "Part Number"
-	1    4800 2950
+P 4450 3400
+F 0 "R3" V 4450 3400 50  0000 C CNN
+F 1 "R_1k" V 4375 3400 50  0000 C CNN
+F 2 "Resistors_SMD:R_0603" V 4380 3400 50  0001 C CNN
+F 3 "https://www.digikey.com/product-detail/en/yageo/RC0603JR-071KL/311-1.0KGRCT-ND/729624" V 4530 3400 50  0001 C CNN
+F 4 "RC0603JR-071KL" V 4630 3500 60  0001 C CNN "Part Number"
+	1    4450 3400
 	0    1    1    0
 $EndComp
@@
 L R_1k R4
 U 1 1 59BA28E7
-P 4950 5050
-F 0 "R4" V 4950 5050 50  0000 C CNN
-F 1 "R_1k" V 4875 5050 50  0000 C CNN
-F 2 "Resistors_SMD:R_0603" V 4880 5050 50  0001 C CNN
-F 3 "https://www.digikey.com/product-detail/en/yageo/RC0603JR-071KL/311-1.0KGRCT-ND/729624" V 5030 5050 50  0001 C CNN
-F 4 "RC0603JR-071KL" V 5130 5150 60  0001 C CNN "Part Number"
-	1    4950 5050
+P 6800 3550
+F 0 "R4" V 6800 3550 50  0000 C CNN
+F 1 "R_1k" V 6725 3550 50  0000 C CNN
+F 2 "Resistors_SMD:R_0603" V 6730 3550 50  0001 C CNN
+F 3 "https://www.digikey.com/product-detail/en/yageo/RC0603JR-071KL/311-1.0KGRCT-ND/729624" V 6880 3550 50  0001 C CNN
+F 4 "RC0603JR-071KL" V 6980 3650 60  0001 C CNN "Part Number"
+	1    6800 3550
 	0    1    1    0
 $EndComp

Commit message: update
Parts:
- R5: footprint Resistors_SMD:R_0603_HandSoldering -> Resistors_SMD:R_0603
- U2: footprint footprints:PT5529 -> open-automation:PT5529
Changed lines of the file:
@@
 F 0 "U2" H 4600 2900 60  0000 C CNN
 F 1 "PT5529B/L2/H2-F" H 4950 3200 60  0000 C CNN
-F 2 "footprints:PT5529" H 4900 3000 60  0001 C CNN
+F 2 "open-automation:PT5529" H 4900 3000 60  0001 C CNN
 F 3 "http://www.everlight.com/file/ProductFile/PT5529B-L2-H2-F.pdf" H 4900 3000 60  0001 C CNN
 F 4 "1080-1161-ND" H 4900 3000 60  0001 C CNN "Part Number"
@@
 F 0 "R5" V 7580 2600 50  0000 C CNN
 F 1 "36" V 7500 2600 50  0000 C CNN
-F 2 "Resistors_SMD:R_0603_HandSoldering" V 7430 2600 50  0001 C CNN
+F 2 "Resistors_SMD:R_0603" V 7430 2600 50  0001 C CNN
 F 3 "http://www.yageo.com.tw/exep/pages/download/literatures/PYu-R_INT-thick_7.pdf" H 7500 2600 50  0001 C CNN
 F 4 "RC0603JR-0736RL" V 7500 2600 60  0001 C CNN "Part Number"

Commit message: update
Parts:
- U2: value PT5529B/L2/H2-F -> TSOP32538; Part Number 1080-1161-ND -> TSOP32538
Changed lines of the file:
@@
 P 4900 3000
 F 0 "U2" H 4600 2900 60  0000 C CNN
-F 1 "PT5529B/L2/H2-F" H 4950 3200 60  0000 C CNN
+F 1 "TSOP32538" H 4950 3200 60  0000 C CNN
 F 2 "open-automation:PT5529" H 4900 3000 60  0001 C CNN
-F 3 "http://www.everlight.com/file/ProductFile/PT5529B-L2-H2-F.pdf" H 4900 3000 60  0001 C CNN
-F 4 "1080-1161-ND" H 4900 3000 60  0001 C CNN "Part Number"
+F 3 "https://www.digikey.com/product-detail/en/vishay-semiconductor-opto-division/TSOP32538/TSOP32538-ND/4695608" H 4900 3000 60  0001 C CNN
+F 4 "TSOP32538" H 4900 3000 60  0001 C CNN "Part Number"
 	1    4900 3000
 	1    0    0    -1
@@
 IR-Receive
 $Comp
-L GND #PWR02
+L GND #PWR06
 U 1 1 59098AF2
 P 4900 3450
-F 0 "#PWR02" H 4900 3200 50  0001 C CNN
+F 0 "#PWR06" H 4900 3200 50  0001 C CNN
 F 1 "GND" H 4900 3300 50  0000 C CNN
 F 2 "" H 4900 3450 50  0000 C CNN
@@
 $EndComp
 $Comp
-L GND #PWR03
+L GND #PWR07
 U 1 1 59098AF9
 P 7500 3950
-F 0 "#PWR03" H 7500 3700 50  0001 C CNN
+F 0 "#PWR07" H 7500 3700 50  0001 C CNN
 F 1 "GND" H 7500 3800 50  0000 C CNN
 F 2 "" H 7500 3950 50  0000 C CNN

Commit message: update
Parts:
- R3, R4, R5: footprint Resistors_SMD:R_0603 -> Resistors_SMD:R_0603_HandSoldering
Connections:
- net V_USB is gone; now on net 3V3: U2.3 (E_B)
Changed lines of the file:
@@
 IR-Receive
 $Comp
-L GND #PWR06
+L GND #PWR05
 U 1 1 59098AF2
 P 4900 3450
-F 0 "#PWR06" H 4900 3200 50  0001 C CNN
+F 0 "#PWR05" H 4900 3200 50  0001 C CNN
 F 1 "GND" H 4900 3300 50  0000 C CNN
 F 2 "" H 4900 3450 50  0000 C CNN
@@
 F 0 "R5" V 7580 2600 50  0000 C CNN
 F 1 "36" V 7500 2600 50  0000 C CNN
-F 2 "Resistors_SMD:R_0603" V 7430 2600 50  0001 C CNN
+F 2 "Resistors_SMD:R_0603_HandSoldering" V 7430 2600 50  0001 C CNN
 F 3 "http://www.yageo.com.tw/exep/pages/download/literatures/PYu-R_INT-thick_7.pdf" H 7500 2600 50  0001 C CNN
 F 4 "RC0603JR-0736RL" V 7500 2600 60  0001 C CNN "Part Number"
@@
 $EndComp
 $Comp
-L GND #PWR07
+L GND #PWR06
 U 1 1 59098AF9
 P 7500 3950
-F 0 "#PWR07" H 7500 3700 50  0001 C CNN
+F 0 "#PWR06" H 7500 3700 50  0001 C CNN
 F 1 "GND" H 7500 3800 50  0000 C CNN
 F 2 "" H 7500 3950 50  0000 C CNN
@@
 3V3
 Text GLabel 5200 3300 1    60   Input ~ 0
-V_USB
+3V3
 $Comp
 L R_1k R3
@@
 F 0 "R3" V 4450 3400 50  0000 C CNN
 F 1 "R_1k" V 4375 3400 50  0000 C CNN
-F 2 "Resistors_SMD:R_0603" V 4380 3400 50  0001 C CNN
+F 2 "Resistors_SMD:R_0603_HandSoldering" V 4380 3400 50  0001 C CNN
 F 3 "https://www.digikey.com/product-detail/en/yageo/RC0603JR-071KL/311-1.0KGRCT-ND/729624" V 4530 3400 50  0001 C CNN
 F 4 "RC0603JR-071KL" V 4630 3500 60  0001 C CNN "Part Number"
@@
 F 0 "R4" V 6800 3550 50  0000 C CNN
 F 1 "R_1k" V 6725 3550 50  0000 C CNN
-F 2 "Resistors_SMD:R_0603" V 6730 3550 50  0001 C CNN
+F 2 "Resistors_SMD:R_0603_HandSoldering" V 6730 3550 50  0001 C CNN
 F 3 "https://www.digikey.com/product-detail/en/yageo/RC0603JR-071KL/311-1.0KGRCT-ND/729624" V 6880 3550 50  0001 C CNN
 F 4 "RC0603JR-071KL" V 6980 3650 60  0001 C CNN "Part Number"
