File: hardware/InfraRed.sch (KiCad schematic (older format))
At the start: 6 parts, among them Q1 Q_NPN_BEC, U2 TSOP32538

Commit message: update
Parts:
- removed U2: TSOP32538, open-automation:PT5529, symbol PT5529B/L2/H2-F
- added U2: IR-RX-TSOP34438, open-automation:TSOP75338TR, symbol IR-RX-TSOP34438
Connections:
- wire segments 13 -> 11
Other:
- moved on the sheet: D1, Q1, R3, R4, R5
Changed lines of the file:
@@
 $Descr A4 11693 8268
 encoding utf-8
-Sheet 3 10
+Sheet 3 9
 Title ""
 Date ""
@@
 Comment4 ""
 $EndDescr
+Text Label 3725 4300 0    60   ~ 0
+IR-Receive
 $Comp
-L PT5529B/L2/H2-F U2
-U 1 1 59098AF0
-P 4900 3000
-F 0 "U2" H 4600 2900 60  0000 C CNN
-F 1 "TSOP32538" H 4950 3200 60  0000 C CNN
-F 2 "open-automation:PT5529" H 4900 3000 60  0001 C CNN
-F 3 "https://www.digikey.com/product-detail/en/vishay-semiconductor-opto-division/TSOP32538/TSOP32538-ND/4695608" H 4900 3000 60  0001 C CNN
-F 4 "TSOP32538" H 4900 3000 60  0001 C CNN "Part Number"
-	1    4900 3000
+L GND #PWR04
+U 1 1 59098AF2
+P 3525 3650
+F 0 "#PWR04" H 3525 3400 50  0001 C CNN
+F 1 "GND" H 3525 3500 50  0000 C CNN
+F 2 "" H 3525 3650 50  0000 C CNN
+F 3 "" H 3525 3650 50  0000 C CNN
+	1    3525 3650
 	1    0    0    -1
 $EndComp
-Text Label 4650 2600 0    60   ~ 0
-IR-Receive
-$Comp
-L GND #PWR05
-U 1 1 59098AF2
-P 4900 3450
-F 0 "#PWR05" H 4900 3200 50  0001 C CNN
-F 1 "GND" H 4900 3300 50  0000 C CNN
-F 2 "" H 4900 3450 50  0000 C CNN
-F 3 "" H 4900 3450 50  0000 C CNN
-	1    4900 3450
-	1    0    0    -1
-$EndComp
-Text GLabel 4200 3400 0    60   Input ~ 0
+Text GLabel 4875 3550 2    60   Input ~ 0
 IR_RX
 $Comp
 L LED D1
 U 1 1 59098AF4
-P 7500 3050
-F 0 "D1" H 7500 3150 50  0000 C CNN
-F 1 "LED" H 7500 2950 50  0000 C CNN
-F 2 "LEDs:LED_D3.0mm" H 7500 3050 50  0001 C CNN
-F 3 "http://www.mouser.com/ds/2/149/QED123-890063.pdf" H 7500 3050 50  0001 C CNN
-F 4 "QED123" H 7500 3050 60  0001 C CNN "Part Number"
-	1    7500 3050
+P 7625 3100
+F 0 "D1" H 7625 3200 50  0000 C CNN
+F 1 "LED" H 7625 3000 50  0000 C CNN
+F 2 "LEDs:LED_D3.0mm" H 7625 3100 50  0001 C CNN
+F 3 "http://www.mouser.com/ds/2/149/QED123-890063.pdf" H 7625 3100 50  0001 C CNN
+F 4 "QED123" H 7625 3100 60  0001 C CNN "Part Number"
+	1    7625 3100
 	0    -1   -1   0
 $EndComp
@@
 L R R5
 U 1 1 59098AF5
-P 7500 2600
-F 0 "R5" V 7580 2600 50  0000 C CNN
-F 1 "36" V 7500 2600 50  0000 C CNN
-F 2 "Resistors_SMD:R_0603_HandSoldering" V 7430 2600 50  0001 C CNN
-F 3 "http://www.yageo.com.tw/exep/pages/download/literatures/PYu-R_INT-thick_7.pdf" H 7500 2600 50  0001 C CNN
-F 4 "RC0603JR-0736RL" V 7500 2600 60  0001 C CNN "Part Number"
-	1    7500 2600
+P 7625 2650
+F 0 "R5" V 7705 2650 50  0000 C CNN
+F 1 "36" V 7625 2650 50  0000 C CNN
+F 2 "Resistors_SMD:R_0603_HandSoldering" V 7555 2650 50  0001 C CNN
+F 3 "http://www.yageo.com.tw/exep/pages/download/literatures/PYu-R_INT-thick_7.pdf" H 7625 2650 50  0001 C CNN
+F 4 "RC0603JR-0736RL" V 7625 2650 60  0001 C CNN "Part Number"
+	1    7625 2650
 	1    0    0    -1
 $EndComp
@@
 L Q_NPN_BEC Q1
 U 1 1 59098AF8
-P 7400 3550
-F 0 "Q1" H 7700 3600 50  0000 R CNN
-F 1 "Q_NPN_BEC" H 8000 3500 50  0000 R CNN
-F 2 "TO_SOT_Packages_SMD:SOT-23" H 7600 3650 50  0001 C CNN
-F 3 "http://www.onsemi.com/pub/Collateral/MMBT3904LT1-D.PDF" H 7400 3550 50  0001 C CNN
-F 4 "MMBT3904LT1GOSCT-ND" H 7400 3550 60  0001 C CNN "Part Number"
-	1    7400 3550
+P 7525 3600
+F 0 "Q1" H 7825 3650 50  0000 R CNN
+F 1 "Q_NPN_BEC" H 8125 3550 50  0000 R CNN
+F 2 "TO_SOT_Packages_SMD:SOT-23" H 7725 3700 50  0001 C CNN
+F 3 "http://www.onsemi.com/pub/Collateral/MMBT3904LT1-D.PDF" H 7525 3600 50  0001 C CNN
+F 4 "MMBT3904LT1GOSCT-ND" H 7525 3600 60  0001 C CNN "Part Number"
+	1    7525 3600
 	1    0    0    -1
 $EndComp
 $Comp
-L GND #PWR06
+L GND #PWR05
 U 1 1 59098AF9
-P 7500 3950
-F 0 "#PWR06" H 7500 3700 50  0001 C CNN
-F 1 "GND" H 7500 3800 50  0000 C CNN
-F 2 "" H 7500 3950 50  0000 C CNN
-F 3 "" H 7500 3950 50  0000 C CNN
-	1    7500 3950
+P 7625 4000
+F 0 "#PWR05" H 7625 3750 50  0001 C CNN
+F 1 "GND" H 7625 3850 50  0000 C CNN
+F 2 "" H 7625 4000 50  0000 C CNN
+F 3 "" H 7625 4000 50  0000 C CNN
+	1    7625 4000
 	1    0    0    -1
 $EndComp
-Text GLabel 6350 3550 0    60   Input ~ 0
+Text GLabel 6475 3600 0    60   Input ~ 0
 IR_TX
-Text Label 6600 3000 0    60   ~ 0
+Text Label 6925 4400 0    60   ~ 0
 IR-Transmit
 Wire Wire Line
-	6650 3550 6350 3550
+	6775 3600 6475 3600
 Wire Wire Line
-	7500 3750 7500 3950
+	7625 3800 7625 4000
 Wire Wire Line
-	6950 3550 7200 3550
+	7075 3600 7325 3600
 Wire Wire Line
-	7500 2300 7500 2450
+	7625 2350 7625 2500
 Wire Wire Line
-	4300 3400 4200 3400
+	7625 2800 7625 2950
 Wire Wire Line
-	5200 3400 5200 3300
-Wire Wire Line
-	5000 3400 5200 3400
-Wire Wire Line
-	5000 3300 5000 3400
-Wire Wire Line
-	4900 3300 4900 3450
-Wire Wire Line
-	4800 3400 4600 3400
-Wire Wire Line
-	4800 3300 4800 3400
-Wire Wire Line
-	7500 2750 7500 2900
-Wire Wire Line
-	7500 3200 7500 3350
-Text GLabel 7500 2300 1    60   Input ~ 0
+	7625 3250 7625 3400
+Text GLabel 7625 2350 1    60   Input ~ 0
 3V3
-Text GLabel 5200 3300 1    60   Input ~ 0
+Text GLabel 3525 3475 0    60   Input ~ 0
 3V3
 $Comp
 L R_1k R3
 U 1 1 59BA28B3
-P 4450 3400
-F 0 "R3" V 4450 3400 50  0000 C CNN
-F 1 "R_1k" V 4375 3400 50  0000 C CNN
-F 2 "Resistors_SMD:R_0603_HandSoldering" V 4380 3400 50  0001 C CNN
-F 3 "https://www.digikey.com/product-detail/en/yageo/RC0603JR-071KL/311-1.0KGRCT-ND/729624" V 4530 3400 50  0001 C CNN
-F 4 "RC0603JR-071KL" V 4630 3500 60  0001 C CNN "Part Number"
-	1    4450 3400
+P 4625 3550
+F 0 "R3" V 4625 3550 50  0000 C CNN
+F 1 "R_1k" V 4550 3550 50  0000 C CNN
+F 2 "Resistors_SMD:R_0603_HandSoldering" V 4555 3550 50  0001 C CNN
+F 3 "https://www.digikey.com/product-detail/en/yageo/RC0603JR-071KL/311-1.0KGRCT-ND/729624" V 4705 3550 50  0001 C CNN
+F 4 "RC0603JR-071KL" V 4805 3650 60  0001 C CNN "Part Number"
+	1    4625 3550
 	0    1    1    0
 $EndComp
@@
 L R_1k R4
 U 1 1 59BA28E7
-P 6800 3550
-F 0 "R4" V 6800 3550 50  0000 C CNN
-F 1 "R_1k" V 6725 3550 50  0000 C CNN
-F 2 "Resistors_SMD:R_0603_HandSoldering" V 6730 3550 50  0001 C CNN
-F 3 "https://www.digikey.com/product-detail/en/yageo/RC0603JR-071KL/311-1.0KGRCT-ND/729624" V 6880 3550 50  0001 C CNN
-F 4 "RC0603JR-071KL" V 6980 3650 60  0001 C CNN "Part Number"
-	1    6800 3550
+P 6925 3600
+F 0 "R4" V 6925 3600 50  0000 C CNN
+F 1 "R_1k" V 6850 3600 50  0000 C CNN
+F 2 "Resistors_SMD:R_0603_HandSoldering" V 6855 3600 50  0001 C CNN
+F 3 "https://www.digikey.com/product-detail/en/yageo/RC0603JR-071KL/311-1.0KGRCT-ND/729624" V 7005 3600 50  0001 C CNN
+F 4 "RC0603JR-071KL" V 7105 3700 60  0001 C CNN "Part Number"
+	1    6925 3600
 	0    1    1    0
 $EndComp
+Wire Wire Line
+	4875 3550 4775 3550
+Wire Wire Line
+	4475 3550 4400 3550
+Wire Wire Line
+	3525 3650 3525 3625
+Wire Wire Line
+	3525 3625 3575 3625
+Wire Wire Line
+	3525 3475 3575 3475
+$Comp
+L IR-RX-TSOP34438 U2
+U 1 1 5A1853BB
+P 3925 3150
+F 0 "U2" H 4125 2575 60  0000 C CNN
+F 1 "IR-RX-TSOP34438" H 3975 3000 60  0000 C CNN
+F 2 "open-automation:TSOP75338TR" H 3925 2500 60  0001 C CNN
+F 3 "https://www.digikey.com/product-detail/en/vishay-semiconductor-opto-division/TSOP75338TR/TSOP75338CT-ND/6596741" H 3950 2400 60  0001 C CNN
+F 4 "TSOP75338TR" H 3950 3100 60  0001 C CNN "Part Number"
+	1    3925 3150
+	1    0    0    -1
+$EndComp
 $EndSCHEMATC

Commit message: update
Parts:
- D1: symbol LED -> liger-rescue:LED
- Q1: symbol Q_NPN_BEC -> liger-rescue:Q_NPN_BEC
- R3, R4: symbol R_1k -> liger-rescue:R_1k
- R5: symbol R -> liger-rescue:R
- U2: symbol IR-RX-TSOP34438 -> liger-rescue:IR-RX-TSOP34438
Changed lines of the file:
@@
-EESchema Schematic File Version 2
-LIBS:power
-LIBS:device
-LIBS:transistors
-LIBS:conn
-LIBS:linear
-LIBS:regul
-LIBS:74xx
-LIBS:cmos4000
-LIBS:adc-dac
-LIBS:memory
-LIBS:xilinx
-LIBS:microcontrollers
-LIBS:dsp
-LIBS:microchip
-LIBS:analog_switches
-LIBS:motorola
-LIBS:texas
-LIBS:intel
-LIBS:audio
-LIBS:interface
-LIBS:digital-audio
-LIBS:philips
-LIBS:display
-LIBS:cypress
-LIBS:siliconi
-LIBS:opto
-LIBS:atmel
-LIBS:contrib
-LIBS:valves
-LIBS:open-automation
+EESchema Schematic File Version 4
 LIBS:liger-cache
-EELAYER 25 0
+EELAYER 26 0
 EELAYER END
 $Descr A4 11693 8268
@@
 IR-Receive
 $Comp
-L GND #PWR04
+L power:GND #PWR04
 U 1 1 59098AF2
 P 3525 3650
@@
 IR_RX
 $Comp
-L LED D1
+L liger-rescue:LED D1
 U 1 1 59098AF4
 P 7625 3100
@@
 $EndComp
 $Comp
-L R R5
+L liger-rescue:R R5
 U 1 1 59098AF5
 P 7625 2650
@@
 $EndComp
 $Comp
-L Q_NPN_BEC Q1
+L liger-rescue:Q_NPN_BEC Q1
 U 1 1 59098AF8
 P 7525 3600
@@
 $EndComp
 $Comp
-L GND #PWR05
+L power:GND #PWR05
 U 1 1 59098AF9
 P 7625 4000
@@
 3V3
 $Comp
-L R_1k R3
+L liger-rescue:R_1k R3
 U 1 1 59BA28B3
 P 4625 3550
@@
 $EndComp
 $Comp
-L R_1k R4
+L liger-rescue:R_1k R4
 U 1 1 59BA28E7
 P 6925 3600
@@
 	3525 3475 3575 3475
 $Comp
-L IR-RX-TSOP34438 U2
+L liger-rescue:IR-RX-TSOP34438 U2
 U 1 1 5A1853BB
 P 3925 3150

Commit message: updated schematic
Changed lines of the file:
@@
 	1    0    0    -1
 $EndComp
-Text GLabel 4875 3550 2    60   Input ~ 0
-IR_RX
 $Comp
 L liger-rescue:LED D1
@@
 	1    0    0    -1
 $EndComp
-Text GLabel 6475 3600 0    60   Input ~ 0
-IR_TX
 Text Label 6925 4400 0    60   ~ 0
 IR-Transmit
@@
 Wire Wire Line
 	7625 3250 7625 3400
-Text GLabel 7625 2350 1    60   Input ~ 0
-3V3
-Text GLabel 3525 3475 0    60   Input ~ 0
-3V3
 $Comp
 L liger-rescue:R_1k R3
@@
 	1    0    0    -1
 $EndComp
+Text HLabel 3525 3475 0    60   Input ~ 0
+3V3
+Text HLabel 4875 3550 2    60   Input ~ 0
+IR_RX
+Text HLabel 6475 3600 0    60   Input ~ 0
+IR_TX
+Text HLabel 7625 2350 1    60   Input ~ 0
+3V3
 $EndSCHEMATC

Commit message: update
Parts:
- D1: footprint LEDs:LED_D3.0mm -> LED_THT:LED_D3.0mm
- Q1: footprint TO_SOT_Packages_SMD:SOT-23 -> Package_TO_SOT_SMD:SOT-23
- R3, R4, R5: footprint Resistors_SMD:R_0603_HandSoldering -> Resistor_SMD:R_0603_1608Metric_Pad1.05x0.95mm_HandSolder
Changed lines of the file:
@@
 F 0 "D1" H 7625 3200 50  0000 C CNN
 F 1 "LED" H 7625 3000 50  0000 C CNN
-F 2 "LEDs:LED_D3.0mm" H 7625 3100 50  0001 C CNN
+F 2 "LED_THT:LED_D3.0mm" H 7625 3100 50  0001 C CNN
 F 3 "http://www.mouser.com/ds/2/149/QED123-890063.pdf" H 7625 3100 50  0001 C CNN
 F 4 "QED123" H 7625 3100 60  0001 C CNN "Part Number"
@@
 F 0 "R5" V 7705 2650 50  0000 C CNN
 F 1 "36" V 7625 2650 50  0000 C CNN
-F 2 "Resistors_SMD:R_0603_HandSoldering" V 7555 2650 50  0001 C CNN
+F 2 "Resistor_SMD:R_0603_1608Metric_Pad1.05x0.95mm_HandSolder" V 7555 2650 50  0001 C CNN
 F 3 "http://www.yageo.com.tw/exep/pages/download/literatures/PYu-R_INT-thick_7.pdf" H 7625 2650 50  0001 C CNN
 F 4 "RC0603JR-0736RL" V 7625 2650 60  0001 C CNN "Part Number"
@@
 F 0 "Q1" H 7825 3650 50  0000 R CNN
 F 1 "Q_NPN_BEC" H 8125 3550 50  0000 R CNN
-F 2 "TO_SOT_Packages_SMD:SOT-23" H 7725 3700 50  0001 C CNN
+F 2 "Package_TO_SOT_SMD:SOT-23" H 7725 3700 50  0001 C CNN
 F 3 "http://www.onsemi.com/pub/Collateral/MMBT3904LT1-D.PDF" H 7525 3600 50  0001 C CNN
 F 4 "MMBT3904LT1GOSCT-ND" H 7525 3600 60  0001 C CNN "Part Number"
@@
 F 0 "R3" V 4625 3550 50  0000 C CNN
 F 1 "R_1k" V 4550 3550 50  0000 C CNN
-F 2 "Resistors_SMD:R_0603_HandSoldering" V 4555 3550 50  0001 C CNN
+F 2 "Resistor_SMD:R_0603_1608Metric_Pad1.05x0.95mm_HandSolder" V 4555 3550 50  0001 C CNN
 F 3 "https://www.digikey.com/product-detail/en/yageo/RC0603JR-071KL/311-1.0KGRCT-ND/729624" V 4705 3550 50  0001 C CNN
 F 4 "RC0603JR-071KL" V 4805 3650 60  0001 C CNN "Part Number"
@@
 F 0 "R4" V 6925 3600 50  0000 C CNN
 F 1 "R_1k" V 6850 3600 50  0000 C CNN
-F 2 "Resistors_SMD:R_0603_HandSoldering" V 6855 3600 50  0001 C CNN
+F 2 "Resistor_SMD:R_0603_1608Metric_Pad1.05x0.95mm_HandSolder" V 6855 3600 50  0001 C CNN
 F 3 "https://www.digikey.com/product-detail/en/yageo/RC0603JR-071KL/311-1.0KGRCT-ND/729624" V 7005 3600 50  0001 C CNN
 F 4 "RC0603JR-071KL" V 7105 3700 60  0001 C CNN "Part Number"

Commit message: order complete
Parts:
- Q1: Part Number MMBT3904LT1GOSCT-ND -> MMBT3904-TP
- R3, R4: Part Number RC0603JR-071KL -> ESR03EZPJ102
Changed lines of the file:
@@
 F 2 "Package_TO_SOT_SMD:SOT-23" H 7725 3700 50  0001 C CNN
 F 3 "http://www.onsemi.com/pub/Collateral/MMBT3904LT1-D.PDF" H 7525 3600 50  0001 C CNN
-F 4 "MMBT3904LT1GOSCT-ND" H 7525 3600 60  0001 C CNN "Part Number"
+F 4 "MMBT3904-TP" H 7525 3600 60  0001 C CNN "Part Number"
 	1    7525 3600
 	1    0    0    -1
@@
 F 2 "Resistor_SMD:R_0603_1608Metric_Pad1.05x0.95mm_HandSolder" V 4555 3550 50  0001 C CNN
 F 3 "https://www.digikey.com/product-detail/en/yageo/RC0603JR-071KL/311-1.0KGRCT-ND/729624" V 4705 3550 50  0001 C CNN
-F 4 "RC0603JR-071KL" V 4805 3650 60  0001 C CNN "Part Number"
+F 4 "ESR03EZPJ102" V 4805 3650 60  0001 C CNN "Part Number"
 	1    4625 3550
 	0    1    1    0
@@
 F 2 "Resistor_SMD:R_0603_1608Metric_Pad1.05x0.95mm_HandSolder" V 6855 3600 50  0001 C CNN
 F 3 "https://www.digikey.com/product-detail/en/yageo/RC0603JR-071KL/311-1.0KGRCT-ND/729624" V 7005 3600 50  0001 C CNN
-F 4 "RC0603JR-071KL" V 7105 3700 60  0001 C CNN "Part Number"
+F 4 "ESR03EZPJ102" V 7105 3700 60  0001 C CNN "Part Number"
 	1    6925 3600
 	0    1    1    0

Commit message: 0.7.1
Parts:
- R5: Part Number RC0603JR-0736RL -> RMCF0603FT36R0
Changed lines of the file:
@@
 F 2 "Resistor_SMD:R_0603_1608Metric_Pad1.05x0.95mm_HandSolder" V 7555 2650 50  0001 C CNN
 F 3 "http://www.yageo.com.tw/exep/pages/download/literatures/PYu-R_INT-thick_7.pdf" H 7625 2650 50  0001 C CNN
-F 4 "RC0603JR-0736RL" V 7625 2650 60  0001 C CNN "Part Number"
+F 4 "RMCF0603FT36R0" V 7625 2650 60  0001 C CNN "Part Number"
 	1    7625 2650
 	1    0    0    -1
