File: hardware/speaker.sch (KiCad schematic (older format))
At the start: 9 parts, among them U11 OPA344

Commit message: update
Parts:
- C6, C7, C8: value 0.1u -> 100nF; Part Number C1608X7R1C224K080AC -> GRM188R71C104KA01D
- LS1: Part Number (none) -> CVS-1508
- R20, R21, R22, R23: Part Number RC0603JR-0710KL -> RC0603JR-07100KL
- U11: Part Number (none) -> 296-41475-1-ND
Changed lines of the file:
@@
 P 5000 3100
 F 0 "C7" V 4950 3150 50  0000 L CNN
-F 1 "0.1u" V 5150 3000 50  0000 L CNN
+F 1 "100nF" V 5150 3000 50  0000 L CNN
 F 2 "Capacitors_SMD:C_0603_HandSoldering" H 5115 3055 50  0001 L CNN
 F 3 "http://www.digikey.com/product-detail/en/tdk-corporation/C1608X7R1C224K080AC/445-1318-1-ND/567690" H 5115 2964 50  0001 L CNN
-F 4 "C1608X7R1C224K080AC" H 5000 3100 60  0001 C CNN "Part Number"
+F 4 "GRM188R71C104KA01D" H 5000 3100 60  0001 C CNN "Part Number"
 	1    5000 3100
 	0    1    1    0
@@
 F 1 "100K" V 5800 3900 50  0000 C CNN
 F 2 "Resistors_SMD:R_0603_HandSoldering" V 5730 3900 50  0001 C CNN
-F 3 "http://www.digikey.com/en/resources/datasheets/yageo/rc-series-l-suffix-datasheet" H 5800 3900 50  0001 C CNN
-F 4 "RC0603JR-0710KL" V 5800 3900 60  0001 C CNN "Part Number"
+F 3 "http://www.yageo.com/documents/recent/PYu-RC_Group_51_RoHS_L_7.pdf" H 5800 3900 50  0001 C CNN
+F 4 "RC0603JR-07100KL" V 5800 3900 60  0001 C CNN "Part Number"
 	1    5800 3900
 	0    -1   -1   0
@@
 P 6400 3200
 F 0 "C8" V 6350 3250 50  0000 L CNN
-F 1 "0.1u" V 6550 3100 50  0000 L CNN
+F 1 "100nF" V 6550 3100 50  0000 L CNN
 F 2 "Capacitors_SMD:C_0603_HandSoldering" H 6515 3155 50  0001 L CNN
 F 3 "http://www.digikey.com/product-detail/en/tdk-corporation/C1608X7R1C224K080AC/445-1318-1-ND/567690" H 6515 3064 50  0001 L CNN
-F 4 "C1608X7R1C224K080AC" H 6400 3200 60  0001 C CNN "Part Number"
+F 4 "GRM188R71C104KA01D" H 6400 3200 60  0001 C CNN "Part Number"
 	1    6400 3200
 	0    1    1    0
@@
 F 1 "100K" V 5250 3900 50  0000 C CNN
 F 2 "Resistors_SMD:R_0603_HandSoldering" V 5180 3900 50  0001 C CNN
-F 3 "http://www.digikey.com/en/resources/datasheets/yageo/rc-series-l-suffix-datasheet" H 5250 3900 50  0001 C CNN
-F 4 "RC0603JR-0710KL" V 5250 3900 60  0001 C CNN "Part Number"
+F 3 "http://www.yageo.com/documents/recent/PYu-RC_Group_51_RoHS_L_7.pdf" H 5250 3900 50  0001 C CNN
+F 4 "RC0603JR-07100KL" V 5250 3900 60  0001 C CNN "Part Number"
 	1    5250 3900
 	0    1    1    0
@@
 F 1 "100K" V 5450 2850 50  0000 C CNN
 F 2 "Resistors_SMD:R_0603_HandSoldering" V 5380 2850 50  0001 C CNN
-F 3 "http://www.digikey.com/en/resources/datasheets/yageo/rc-series-l-suffix-datasheet" H 5450 2850 50  0001 C CNN
-F 4 "RC0603JR-0710KL" V 5450 2850 60  0001 C CNN "Part Number"
+F 3 "http://www.yageo.com/documents/recent/PYu-RC_Group_51_RoHS_L_7.pdf" H 5450 2850 50  0001 C CNN
+F 4 "RC0603JR-07100KL" V 5450 2850 60  0001 C CNN "Part Number"
 	1    5450 2850
 	0    -1   -1   0
@@
 F 1 "100K" V 5250 3350 50  0000 C CNN
 F 2 "Resistors_SMD:R_0603_HandSoldering" V 5180 3350 50  0001 C CNN
-F 3 "http://www.digikey.com/en/resources/datasheets/yageo/rc-series-l-suffix-datasheet" H 5250 3350 50  0001 C CNN
-F 4 "RC0603JR-0710KL" V 5250 3350 60  0001 C CNN "Part Number"
+F 3 "http://www.yageo.com/documents/recent/PYu-RC_Group_51_RoHS_L_7.pdf" H 5250 3350 50  0001 C CNN
+F 4 "RC0603JR-07100KL" V 5250 3350 60  0001 C CNN "Part Number"
 	1    5250 3350
 	-1   0    0    1
@@
 P 4800 3900
 F 0 "C6" V 4750 3950 50  0000 L CNN
-F 1 "0.1u" V 4950 3800 50  0000 L CNN
+F 1 "100nF" V 4950 3800 50  0000 L CNN
 F 2 "Capacitors_SMD:C_0603_HandSoldering" H 4915 3855 50  0001 L CNN
 F 3 "http://www.digikey.com/product-detail/en/tdk-corporation/C1608X7R1C224K080AC/445-1318-1-ND/567690" H 4915 3764 50  0001 L CNN
-F 4 "C1608X7R1C224K080AC" H 4800 3900 60  0001 C CNN "Part Number"
+F 4 "GRM188R71C104KA01D" H 4800 3900 60  0001 C CNN "Part Number"
 	1    4800 3900
 	0    1    1    0
@@
 F 2 "footprints:speaker-1508" H 6850 3000 50  0001 C CNN
 F 3 "http://www.cui.com/product/resource/cvs-1508.pdf" H 6840 3150 50  0001 C CNN
+F 4 "CVS-1508" H 6850 3200 60  0001 C CNN "Part Number"
 	1    6850 3200
 	1    0    0    -1
@@
 F 2 "TO_SOT_Packages_SMD:SOT-23-5" H 5700 3250 50  0001 C CNN
 F 3 "http://www.ti.com/lit/ds/symlink/opa344.pdf" H 5800 3350 50  0001 C CNN
+F 4 "296-41475-1-ND" H 5800 3200 60  0001 C CNN "Part Number"
 	1    5800 3200
 	1    0    0    -1

Commit message: updatge
Parts:
- removed C8: 100nF, Capacitors_SMD:C_0603_HandSoldering, symbol C
- removed R22, R23: 100K, Resistors_SMD:R_0603_HandSoldering, symbol R
- removed U11: OPA344, TO_SOT_Packages_SMD:SOT-23-5, symbol OPA344
- added U8: Amplifier-D-TS4962IQT, Housings_DFN_QFN:DFN-8-1EP_3x3mm_Pitch0.65mm, symbol Amplifier-D-TS4962IQT
- C6, C7: value 100nF -> 4.7uF; Part Number GRM188R71C104KA01D -> CL10B475KQ8NQNC
- R20, R21: Part Number RC0603JR-07100KL -> RC0603JR-07150KL
Connections:
- net 5V: now also U8.1 (STBY), U8.6 (VCC)
- net GND: now also C6.1, U8.7 (GND); no longer C6.2, LS1.2, R20.1
- net IO25: now also C7.1; no longer C7.2
- net at R21.1: now also C7.2
- net at R20.2: now also U8.4 (IN-); no longer C7.1
- net SPEAKER-: now reaches LS1.1
- net SPEAKER-: now also U8.8 (OUT-)
- net at R21.2: now also U8.3 (IN+); no longer C6.1
- new net: C6.2, R20.1
- new net SPEAKER+: LS1.2, U8.5 (OUT+)
Other:
- moved on the sheet: LS1
