File: hardware/speaker.sch (KiCad schematic (older format))
At the start: 6 parts, among them U8 Amplifier-D-TS4962IQT

Commit message: update
Parts:
- U8: footprint Housings_DFN_QFN:DFN-8-1EP_3x3mm_Pitch0.65mm -> open-automation:Amplifier-D-TS4962IQT
Changed lines of the file:
@@
 LIBS:open-automation
 LIBS:liger-cache
-EELAYER 26 0
+EELAYER 25 0
 EELAYER END
 $Descr A4 11693 8268
@@
 F 0 "U8" H 6150 2950 60  0000 C CNN
 F 1 "Amplifier-D-TS4962IQT" H 5900 3500 60  0000 C CNN
-F 2 "Housings_DFN_QFN:DFN-8-1EP_3x3mm_Pitch0.65mm" H 5600 2800 60  0001 C CNN
+F 2 "open-automation:Amplifier-D-TS4962IQT" H 5600 2800 60  0001 C CNN
 F 3 "https://www.digikey.com/product-detail/en/stmicroelectronics/TS4962IQT/497-5993-1-ND/1578476" H 5600 2800 60  0001 C CNN
 F 4 "TS4962IQT" H 5900 3250 60  0001 C CNN "Part Number"

Commit message: update
Parts:
- removed R20, R21: 100K, Resistors_SMD:R_0603_HandSoldering, symbol R
- added R20, R21: R_100k, Resistors_SMD:R_0603, symbol R_100k
Connections:
- net at U8.3 (IN+): now also R21.1
- net at U8.4 (IN-): now also R20.1
- net at C7.2: now also R21.2
- net at C6.2: now also R20.2
- net 5V renamed V_USB
- net IO25 renamed SPEAKER_IN
Changed lines of the file:
@@
 $Descr A4 11693 8268
 encoding utf-8
-Sheet 8 8
+Sheet 7 10
 Title ""
 Date ""
@@
 $EndDescr
 Text GLabel 6700 4300 3    60   Input ~ 0
-IO25
+SPEAKER_IN
 Text Label 4050 2200 0    60   ~ 0
 speaker_driver
@@
 $EndComp
 $Comp
-L GND #PWR021
+L GND #PWR019
 U 1 1 590F73ED
 P 5400 3400
-F 0 "#PWR021" H 5400 3150 50  0001 C CNN
+F 0 "#PWR019" H 5400 3150 50  0001 C CNN
 F 1 "GND" H 5400 3250 50  0000 C CNN
 F 2 "" H 5400 3400 50  0000 C CNN
@@
 $EndComp
 Text GLabel 5350 3250 0    60   Input ~ 0
-5V
+V_USB
 $Comp
 L Amplifier-D-TS4962IQT U8
@@
 	1    5900 3250
 	1    0    0    -1
-$EndComp
-$Comp
-L R R21
-U 1 1 5981296E
-P 6700 3650
-F 0 "R21" H 6600 3600 50  0000 C CNN
-F 1 "100K" V 6700 3650 50  0000 C CNN
-F 2 "Resistors_SMD:R_0603_HandSoldering" V 6630 3650 50  0001 C CNN
-F 3 "http://www.yageo.com/documents/recent/PYu-RC_Group_51_RoHS_L_7.pdf" H 6700 3650 50  0001 C CNN
-F 4 "RC0603JR-07150KL" V 6700 3650 60  0001 C CNN "Part Number"
-	1    6700 3650
-	-1   0    0    1
 $EndComp
 $Comp
@@
 $EndComp
 $Comp
-L GND #PWR022
+L GND #PWR020
 U 1 1 59812E44
 P 6500 4300
-F 0 "#PWR022" H 6500 4050 50  0001 C CNN
+F 0 "#PWR020" H 6500 4050 50  0001 C CNN
 F 1 "GND" H 6500 4150 50  0000 C CNN
 F 2 "" H 6500 4300 50  0000 C CNN
@@
 	1    6500 4300
 	1    0    0    -1
-$EndComp
-$Comp
-L R R20
-U 1 1 598139C0
-P 6500 3650
-F 0 "R20" H 6600 3600 50  0000 C CNN
-F 1 "100K" V 6500 3650 50  0000 C CNN
-F 2 "Resistors_SMD:R_0603_HandSoldering" V 6430 3650 50  0001 C CNN
-F 3 "http://www.yageo.com/documents/recent/PYu-RC_Group_51_RoHS_L_7.pdf" H 6500 3650 50  0001 C CNN
-F 4 "RC0603JR-07150KL" V 6500 3650 60  0001 C CNN "Part Number"
-	1    6500 3650
-	-1   0    0    1
 $EndComp
 Text GLabel 6450 2650 1    60   Input ~ 0
@@
 	6600 2650 6600 3250
 Connection ~ 6600 3250
+$Comp
+L R_100k R21
+U 1 1 59BA2110
+P 6700 3650
+F 0 "R21" V 6700 3650 50  0000 C CNN
+F 1 "R_100k" V 6625 3650 50  0000 C CNN
+F 2 "Resistors_SMD:R_0603" V 6630 3650 50  0001 C CNN
+F 3 "https://www.digikey.com/product-detail/en/yageo/RC0603JR-07100KL/311-100KGRCT-ND/729645" V 6780 3650 50  0001 C CNN
+F 4 "RC0603JR-07100KL" V 6880 3750 60  0001 C CNN "Part Number"
+	1    6700 3650
+	1    0    0    -1
+$EndComp
+$Comp
+L R_100k R20
+U 1 1 59BA214E
+P 6500 3650
+F 0 "R20" V 6500 3650 50  0000 C CNN
+F 1 "R_100k" V 6425 3650 50  0000 C CNN
+F 2 "Resistors_SMD:R_0603" V 6430 3650 50  0001 C CNN
+F 3 "https://www.digikey.com/product-detail/en/yageo/RC0603JR-07100KL/311-100KGRCT-ND/729645" V 6580 3650 50  0001 C CNN
+F 4 "RC0603JR-07100KL" V 6680 3750 60  0001 C CNN "Part Number"
+	1    6500 3650
+	1    0    0    -1
+$EndComp
 $EndSCHEMATC

Commit message: update
Parts:
- C6, C7: footprint Capacitors_SMD:C_0603_HandSoldering -> Capacitors_SMD:C_0603
- LS1: footprint footprints:speaker-1508 -> open-automation:speaker-1508
Changed lines of the file:
@@
 F 0 "LS1" H 6900 3375 50  0000 R CNN
 F 1 "Speaker" H 6900 3300 50  0000 R CNN
-F 2 "footprints:speaker-1508" H 6850 2950 50  0001 C CNN
+F 2 "open-automation:speaker-1508" H 6850 2950 50  0001 C CNN
 F 3 "http://www.cui.com/product/resource/cvs-1508.pdf" H 6840 3100 50  0001 C CNN
 F 4 "CVS-1508" H 6850 3150 60  0001 C CNN "Part Number"
@@
 F 0 "C6" H 6500 4150 50  0000 L CNN
 F 1 "4.7uF" H 6550 3950 50  0000 L CNN
-F 2 "Capacitors_SMD:C_0603_HandSoldering" H 6615 4005 50  0001 L CNN
+F 2 "Capacitors_SMD:C_0603" H 6615 4005 50  0001 L CNN
 F 3 "https://www.digikey.com/product-detail/en/samsung-electro-mechanics-america-inc/CL10B475KQ8NQNC/1276-2087-1-ND/3890173" H 6615 3914 50  0001 L CNN
 F 4 "CL10B475KQ8NQNC" H 6500 4050 60  0001 C CNN "Part Number"
@@
 F 0 "C7" H 6600 4150 50  0000 L CNN
 F 1 "4.7uF" H 6500 3950 50  0000 L CNN
-F 2 "Capacitors_SMD:C_0603_HandSoldering" H 6815 4005 50  0001 L CNN
+F 2 "Capacitors_SMD:C_0603" H 6815 4005 50  0001 L CNN
 F 3 "https://www.digikey.com/product-detail/en/samsung-electro-mechanics-america-inc/CL10B475KQ8NQNC/1276-2087-1-ND/3890173" H 6815 3914 50  0001 L CNN
 F 4 "CL10B475KQ8NQNC" H 6700 4050 60  0001 C CNN "Part Number"

Commit message: update
Connections:
- net V_USB renamed 3V3
Changed lines of the file:
@@
 $EndComp
 $Comp
-L GND #PWR016
+L GND #PWR021
 U 1 1 590F73ED
 P 5400 3400
-F 0 "#PWR016" H 5400 3150 50  0001 C CNN
+F 0 "#PWR021" H 5400 3150 50  0001 C CNN
 F 1 "GND" H 5400 3250 50  0000 C CNN
 F 2 "" H 5400 3400 50  0000 C CNN
@@
 $EndComp
 Text GLabel 5350 3250 0    60   Input ~ 0
-V_USB
+3V3
 $Comp
 L Amplifier-D-TS4962IQT U8
@@
 $EndComp
 $Comp
-L GND #PWR017
+L GND #PWR022
 U 1 1 59812E44
 P 6500 4300
-F 0 "#PWR017" H 6500 4050 50  0001 C CNN
+F 0 "#PWR022" H 6500 4050 50  0001 C CNN
 F 1 "GND" H 6500 4150 50  0000 C CNN
 F 2 "" H 6500 4300 50  0000 C CNN

Commit message: update
Parts:
- removed C6, C7: 4.7uF, Capacitors_SMD:C_0603, symbol C
- removed LS1: Speaker, open-automation:speaker-1508, symbol Speaker
- removed R21: R_100k, Resistors_SMD:R_0603, symbol R_100k
- removed U8: Amplifier-D-TS4962IQT, open-automation:Amplifier-D-TS4962IQT, symbol Amplifier-D-TS4962IQT
- added C6: C_1uF, Capacitors_SMD:C_0603_HandSoldering, symbol C_1uF
- added LS1: speaker-CVS-1508, open-automation:speaker-1508, symbol speaker-CVS-1508
- added U5: MAX98357AETE+T, open-automation:MAX98357A, symbol MAX98357AETE+T
- R20: footprint Resistors_SMD:R_0603 -> Resistors_SMD:R_0603_HandSoldering
Connections:
- net 3V3: now also C6.1, U5.4 (~SD_MODE), U5.7 (VDD)
- net GND: now also R20.2, C6.2, U5.3 (GND)
- net at R20.1: now also U5.2 (GAIN_SLOT)
- new net: LS1.2, U5.10 (OUTN)
- new net: LS1.1, U5.9 (OUTP)
- new net I2S_BCLK: U5.16 (BCLK)
- new net I2S_DATA_OUT: U5.1 (DIN)
- new net I2S_WS: U5.14 (LRCLK)
Other:
- moved on the sheet: R20
Changed lines of the file:
@@
 Comment4 ""
 $EndDescr
-Text GLabel 6700 4300 3    60   Input ~ 0
-SPEAKER_IN
-Text Label 4050 2200 0    60   ~ 0
-speaker_driver
+Text Label 3600 1575 0    394  ~ 0
+Speaker-Driver
 $Comp
-L Speaker LS1
-U 1 1 590F705D
-P 6850 3150
-F 0 "LS1" H 6900 3375 50  0000 R CNN
-F 1 "Speaker" H 6900 3300 50  0000 R CNN
-F 2 "open-automation:speaker-1508" H 6850 2950 50  0001 C CNN
-F 3 "http://www.cui.com/product/resource/cvs-1508.pdf" H 6840 3100 50  0001 C CNN
-F 4 "CVS-1508" H 6850 3150 60  0001 C CNN "Part Number"
-	1    6850 3150
-	1    0    0    -1
+L R_100k R20
+U 1 1 59BA214E
+P 5525 3100
+F 0 "R20" V 5525 3100 50  0000 C CNN
+F 1 "R_100k" V 5450 3100 50  0000 C CNN
+F 2 "Resistors_SMD:R_0603_HandSoldering" V 5455 3100 50  0001 C CNN
+F 3 "https://www.digikey.com/product-detail/en/yageo/RC0603JR-07100KL/311-100KGRCT-ND/729645" V 5605 3100 50  0001 C CNN
+F 4 "RC0603JR-07100KL" V 5705 3200 60  0001 C CNN "Part Number"
+	1    5525 3100
+	0    1    1    0
 $EndComp
 $Comp
 L GND #PWR021
-U 1 1 590F73ED
-P 5400 3400
-F 0 "#PWR021" H 5400 3150 50  0001 C CNN
-F 1 "GND" H 5400 3250 50  0000 C CNN
-F 2 "" H 5400 3400 50  0000 C CNN
-F 3 "" H 5400 3400 50  0000 C CNN
-	1    5400 3400
+U 1 1 59EB6805
+P 5750 3325
+F 0 "#PWR021" H 5750 3075 50  0001 C CNN
+F 1 "GND" H 5750 3175 50  0000 C CNN
+F 2 "" H 5750 3325 50  0000 C CNN
+F 3 "" H 5750 3325 50  0000 C CNN
+	1    5750 3325
 	1    0    0    -1
 $EndComp
-Text GLabel 5350 3250 0    60   Input ~ 0
+Text GLabel 5700 2925 0    60   Input ~ 0
+I2S_DATA_OUT
+Text GLabel 5425 3225 0    60   Input ~ 0
 3V3
+Wire Wire Line
+	5750 3325 5750 3300
+Wire Wire Line
+	5750 3300 5775 3300
+Wire Wire Line
+	5425 3225 5775 3225
+Wire Wire Line
+	5700 2925 5775 2925
+Wire Wire Line
+	6875 2925 7025 2925
+Wire Wire Line
+	6875 3025 7100 3025
+Text GLabel 6975 3125 2    60   Input ~ 0
+I2S_WS
+Text GLabel 6975 3225 2    60   Input ~ 0
+I2S_BCLK
+Wire Wire Line
+	6975 3225 6875 3225
+Wire Wire Line
+	6975 3125 6875 3125
 $Comp
-L Amplifier-D-TS4962IQT U8
-U 1 1 59812510
-P 5900 3250
-F 0 "U8" H 6150 2950 60  0000 C CNN
-F 1 "Amplifier-D-TS4962IQT" H 5900 3500 60  0000 C CNN
-F 2 "open-automation:Amplifier-D-TS4962IQT" H 5600 2800 60  0001 C CNN
-F 3 "https://www.digikey.com/product-detail/en/stmicroelectronics/TS4962IQT/497-5993-1-ND/1578476" H 5600 2800 60  0001 C CNN
-F 4 "TS4962IQT" H 5900 3250 60  0001 C CNN "Part Number"
-	1    5900 3250
+L MAX98357AETE+T U5
+U 1 1 59EB8FEC
+P 6125 3050
+F 0 "U5" H 6575 2700 60  0000 C CNN
+F 1 "MAX98357AETE+T" H 6325 3275 60  0000 C CNN
+F 2 "open-automation:MAX98357A" H 6475 2600 60  0001 C CNN
+F 3 "https://www.digikey.com/product-detail/en/maxim-integrated/MAX98357AETE-T/MAX98357AETE-TCT-ND/7603777" H 6300 2625 60  0001 C CNN
+F 4 "MAX98357AETE+T" H 6325 3350 60  0000 C CNN "Part Number"
+	1    6125 3050
 	1    0    0    -1
 $EndComp
-$Comp
-L C C6
-U 1 1 59812A7F
-P 6500 4050
-F 0 "C6" H 6500 4150 50  0000 L CNN
-F 1 "4.7uF" H 6550 3950 50  0000 L CNN
-F 2 "Capacitors_SMD:C_0603" H 6615 4005 50  0001 L CNN
-F 3 "https://www.digikey.com/product-detail/en/samsung-electro-mechanics-america-inc/CL10B475KQ8NQNC/1276-2087-1-ND/3890173" H 6615 3914 50  0001 L CNN
-F 4 "CL10B475KQ8NQNC" H 6500 4050 60  0001 C CNN "Part Number"
-	1    6500 4050
-	-1   0    0    1
-$EndComp
-$Comp
-L C C7
-U 1 1 59812D76
-P 6700 4050
-F 0 "C7" H 6600 4150 50  0000 L CNN
-F 1 "4.7uF" H 6500 3950 50  0000 L CNN
-F 2 "Capacitors_SMD:C_0603" H 6815 4005 50  0001 L CNN
-F 3 "https://www.digikey.com/product-detail/en/samsung-electro-mechanics-america-inc/CL10B475KQ8NQNC/1276-2087-1-ND/3890173" H 6815 3914 50  0001 L CNN
-F 4 "CL10B475KQ8NQNC" H 6700 4050 60  0001 C CNN "Part Number"
-	1    6700 4050
-	-1   0    0    1
-$EndComp
+Wire Wire Line
+	5775 3125 5725 3125
+Wire Wire Line
+	5725 3125 5725 3225
+Connection ~ 5725 3225
 $Comp
 L GND #PWR022
-U 1 1 59812E44
-P 6500 4300
-F 0 "#PWR022" H 6500 4050 50  0001 C CNN
-F 1 "GND" H 6500 4150 50  0000 C CNN
-F 2 "" H 6500 4300 50  0000 C CNN
-F 3 "" H 6500 4300 50  0000 C CNN
-	1    6500 4300
+U 1 1 59EB98C9
+P 5275 3100
+F 0 "#PWR022" H 5275 2850 50  0001 C CNN
+F 1 "GND" V 5225 2925 50  0000 C CNN
+F 2 "" H 5275 3100 50  0000 C CNN
+F 3 "" H 5275 3100 50  0000 C CNN
+	1    5275 3100
+	0    1    1    0
+$EndComp
+Wire Wire Line
+	5275 3100 5375 3100
+Wire Wire Line
+	5675 3100 5700 3100
+Wire Wire Line
+	5700 3100 5700 3025
+Wire Wire Line
+	5700 3025 5775 3025
+$Comp
+L C_1uF C6
+U 1 1 59EB9DF5
+P 5525 3400
+F 0 "C6" H 5550 3500 50  0000 L CNN
+F 1 "C_1uF" H 5300 3300 50  0000 L CNN
+F 2 "Capacitors_SMD:C_0603_HandSoldering" H 5625 3700 50  0001 C CNN
+F 3 "https://www.digikey.com/product-detail/en/yageo/CC0603ZRY5V7BB105/311-1372-1-ND/2103156" H 5525 3150 50  0001 C CNN
+F 4 "CC0603ZRY5V7BB105" H 5650 3600 60  0001 C CNN "Part Number"
+	1    5525 3400
 	1    0    0    -1
 $EndComp
-Text GLabel 6450 2650 1    60   Input ~ 0
-SPEAKER-
-Text GLabel 6600 2650 1    60   Input ~ 0
-SPEAKER+
 Wire Wire Line
-	5450 3350 5400 3350
-Wire Wire Line
-	5400 3350 5400 3400
-Wire Wire Line
-	5350 3250 5450 3250
-Wire Wire Line
-	5450 3150 5400 3150
-Wire Wire Line
-	5400 3150 5400 3250
-Connection ~ 5400 3250
-Wire Wire Line
-	6400 3150 6650 3150
-Wire Wire Line
-	6400 3250 6650 3250
-Wire Wire Line
-	6400 3450 6500 3450
-Wire Wire Line
-	6400 3350 6700 3350
-Wire Wire Line
-	6700 3800 6700 3900
-Wire Wire Line
-	6500 3800 6500 3900
-Wire Wire Line
-	6700 4200 6700 4300
-Wire Wire Line
-	6500 4200 6500 4300
-Wire Wire Line
-	6500 3450 6500 3500
-Wire Wire Line
-	6700 3350 6700 3500
-Wire Wire Line
-	6450 2650 6450 3150
-Connection ~ 6450 3150
-Wire Wire Line
-	6600 2650 6600 3250
-Connection ~ 6600 3250
+	5525 3250 5525 3225
+Connection ~ 5525 3225
 $Comp
-L R_100k R21
-U 1 1 59BA2110
-P 6700 3650
-F 0 "R21" V 6700 3650 50  0000 C CNN
-F 1 "R_100k" V 6625 3650 50  0000 C CNN
-F 2 "Resistors_SMD:R_0603" V 6630 3650 50  0001 C CNN
-F 3 "https://www.digikey.com/product-detail/en/yageo/RC0603JR-07100KL/311-100KGRCT-ND/729645" V 6780 3650 50  0001 C CNN
-F 4 "RC0603JR-07100KL" V 6880 3750 60  0001 C CNN "Part Number"
-	1    6700 3650
+L GND #PWR023
+U 1 1 59EB9E7A
+P 5525 3600
+F 0 "#PWR023" H 5525 3350 50  0001 C CNN
+F 1 "GND" H 5525 3450 50  0000 C CNN
+F 2 "" H 5525 3600 50  0000 C CNN
+F 3 "" H 5525 3600 50  0000 C CNN
+	1    5525 3600
 	1    0    0    -1
 $EndComp
+Wire Wire Line
+	5525 3600 5525 3550
 $Comp
-L R_100k R20
-U 1 1 59BA214E
-P 6500 3650
-F 0 "R20" V 6500 3650 50  0000 C CNN
-F 1 "R_100k" V 6425 3650 50  0000 C CNN
-F 2 "Resistors_SMD:R_0603" V 6430 3650 50  0001 C CNN
-F 3 "https://www.digikey.com/product-detail/en/yageo/RC0603JR-07100KL/311-100KGRCT-ND/729645" V 6580 3650 50  0001 C CNN
-F 4 "RC0603JR-07100KL" V 6680 3750 60  0001 C CNN "Part Number"
-	1    6500 3650
+L speaker-CVS-1508 LS1
+U 1 1 59EB9CC6
+P 7350 2725
+F 0 "LS1" H 7350 2850 50  0000 R CNN
+F 1 "speaker-CVS-1508" H 7400 2875 50  0001 R CNN
+F 2 "open-automation:speaker-1508" H 7350 2525 50  0001 C CNN
+F 3 "http://www.cui.com/product/resource/cvs-1508.pdf" H 7340 2675 50  0001 C CNN
+F 4 "CVS-1508" H 7500 3050 60  0001 C CNN "Part Number"
+	1    7350 2725
 	1    0    0    -1
 $EndComp
+Wire Wire Line
+	7025 2925 7025 2725
+Wire Wire Line
+	7025 2725 7150 2725
+Wire Wire Line
+	7100 3025 7100 2825
+Wire Wire Line
+	7100 2825 7150 2825
 $EndSCHEMATC

Commit message: update
Connections:
- net 3V3 renamed V_IN
Changed lines of the file:
@@
 I2S_DATA_OUT
 Text GLabel 5425 3225 0    60   Input ~ 0
-3V3
+V_IN
 Wire Wire Line
 	5750 3325 5750 3300
