File: hardware/microphone.sch (KiCad schematic (older format))
At the start: 9 parts, among them U3 MEMS-SPM0408LE5H, U4 OPA344

Commit message: update
Parts:
- C1: value 4.7uf -> 4.7uF
- U4: Part Number (none) -> 296-41475-1-ND
Changed lines of the file:
@@
 F 2 "TO_SOT_Packages_SMD:SOT-23-5" H 6500 3850 50  0001 C CNN
 F 3 "http://www.digikey.com/product-detail/en/texas-instruments/OPA344NA-3K/296-41475-1-ND/5222851" H 6600 3950 50  0001 C CNN
+F 4 "296-41475-1-ND" H 6600 3800 60  0001 C CNN "Part Number"
 	1    6600 3800
 	1    0    0    -1
@@
 P 5550 4400
 F 0 "C1" V 5500 4450 50  0000 L CNN
-F 1 "4.7uf" V 5700 4300 50  0000 L CNN
+F 1 "4.7uF" V 5700 4300 50  0000 L CNN
 F 2 "Capacitors_SMD:C_0603_HandSoldering" H 5665 4355 50  0001 L CNN
 F 3 "http://www.digikey.com/product-detail/en/samsung-electro-mechanics-america-inc/CL10B475KQ8NQNC/1276-2087-1-ND/3890173" H 5665 4264 50  0001 L CNN

Commit message: updatE
Parts:
- removed R8: 1K, Resistors_SMD:R_0603_HandSoldering, symbol R
- C2: value 220nF -> 4.7uF; Part Number C1608X7R1C224K080AC -> CL10B475KQ8NQNC
- R10: value 10K -> 2.2K
- R6: value 6.65K -> 100K; Part Number RC0603FR-076K65L -> RC0603JR-07100KL
- R7: value 1K -> 3.2K; Part Number RC0603JR-071KL -> RC0402FR-073K24L
Connections:
- net 3V3: now also R6.1; no longer R6.2
- net GND: now also R7.1, R9.2; no longer R7.2
- net at U4.3 (+): now also C2.2, R6.2, R7.2
- net at C2.1: now also U3.1 (OUTPUT); no longer R9.2
Other:
- moved on the sheet: C1, R10, R9, U3, U4A

Commit message: update
Connections:
- net IO19 renamed IO34
Changed lines of the file:
@@
 $EndComp
 Text GLabel 8400 3550 2    60   Input ~ 0
-IO19
+IO34
 Text Label 4050 2900 0    60   ~ 0
 Mic_pre-amp

Commit message: update
Parts:
- R10: Part Number RC0603JR-0710KL -> RC0603JR-072K2L
Changed lines of the file:
@@
 LIBS:open-automation
 LIBS:liger-cache
-EELAYER 26 0
+EELAYER 25 0
 EELAYER END
 $Descr A4 11693 8268
@@
 F 1 "2.2K" V 7900 4300 50  0000 C CNN
 F 2 "Resistors_SMD:R_0603_HandSoldering" V 7830 4300 50  0001 C CNN
-F 3 "http://www.digikey.com/en/resources/datasheets/yageo/rc-series-l-suffix-datasheet" H 7900 4300 50  0001 C CNN
-F 4 "RC0603JR-0710KL" V 7900 4300 60  0001 C CNN "Part Number"
+F 3 "https://www.digikey.com/product-detail/en/yageo/RC0603JR-072K2L/311-2.2KGRCT-ND/729676" H 7900 4300 50  0001 C CNN
+F 4 "RC0603JR-072K2L" V 7900 4300 60  0001 C CNN "Part Number"
 	1    7900 4300
 	0    -1   -1   0
