File: hardware/microphone.sch (KiCad schematic (older format))
At the start: 8 parts, among them U3 MEMS-SPM0408LE5H, U4 OPA344

Commit message: update
Parts:
- R10: Part Number RC0603JR-072K2L -> RC0603JR-0710KL
- R7: Part Number RC0402FR-073K24L -> RC0603FR-073K24L
Changed lines of the file:
@@
 LIBS:open-automation
 LIBS:liger-cache
-EELAYER 25 0
+EELAYER 26 0
 EELAYER END
 $Descr A4 11693 8268
@@
 F 1 "2.2K" V 7900 4300 50  0000 C CNN
 F 2 "Resistors_SMD:R_0603_HandSoldering" V 7830 4300 50  0001 C CNN
-F 3 "https://www.digikey.com/product-detail/en/yageo/RC0603JR-072K2L/311-2.2KGRCT-ND/729676" H 7900 4300 50  0001 C CNN
-F 4 "RC0603JR-072K2L" V 7900 4300 60  0001 C CNN "Part Number"
+F 3 "http://www.digikey.com/en/resources/datasheets/yageo/rc-series-l-suffix-datasheet" H 7900 4300 50  0001 C CNN
+F 4 "RC0603JR-0710KL" V 7900 4300 60  0001 C CNN "Part Number"
 	1    7900 4300
 	0    -1   -1   0
@@
 F 1 "3.2K" V 6800 3700 50  0000 C CNN
 F 2 "Resistors_SMD:R_0603_HandSoldering" V 6730 3700 50  0001 C CNN
-F 3 "https://www.digikey.com/product-detail/en/yageo/RC0402FR-073K24L/YAG3147CT-ND/5282012" H 6800 3700 50  0001 C CNN
-F 4 "RC0402FR-073K24L" V 6800 3700 60  0001 C CNN "Part Number"
+F 3 "https://www.digikey.com/product-detail/en/yageo/RC0603FR-073K24L/311-3.24KHRCT-ND/730072" H 6800 3700 50  0001 C CNN
+F 4 "RC0603FR-073K24L" V 6800 3700 60  0001 C CNN "Part Number"
 	1    6800 3700
 	-1   0    0    1

Commit message: update
Parts:
- removed C1, C2: 4.7uF, Capacitors_SMD:C_0603_HandSoldering, symbol C
- removed R10: 2.2K, Resistors_SMD:R_0603_HandSoldering, symbol R
- removed R6: 100K, Resistors_SMD:R_0603_HandSoldering, symbol R
- removed R7: 3.2K, Resistors_SMD:R_0603_HandSoldering, symbol R
- removed R9: 1K, Resistors_SMD:R_0603_HandSoldering, symbol R
- removed U3: MEMS-SPM0408LE5H, footprints:mems-mic, symbol MEMS-SPM0408LE5H
- removed U4: OPA344, TO_SOT_Packages_SMD:SOT-23-5, symbol OPA344
- added C1: C_0.1uF, Capacitors_SMD:C_0603, symbol C_0.1uF
- added R9: R_10k, Resistors_SMD:R_0603, symbol R_10k
- added U3: SPH0645LM4H-B, open-automation:SPH0645LM4H-B, symbol SPH0645LM4H-B
Connections:
- net labels added: I2S_BCLK, I2S_DATA, I2S_WS, Microphone, VCC_I2S
- net labels removed: 3V3, IO34, Mic_pre-amp
- wire segments 22 -> 11

Commit message: update
Parts:
- added C10, C9: C_0.1uF, Capacitors_SMD:C_0603, symbol C_0.1uF
- added C2: C_100uF, Capacitors_SMD:C_1206, symbol C_100uF
- added C8: C_1uF, Capacitors_SMD:C_0603, symbol C_1uF
- added R11: R_10, Resistors_SMD:R_0603, symbol R_10
Connections:
- net GND: now also C10.2, C2.2, C8.2, C9.2
- new net 3V3: R11.2
- new net VCC_PIR1: C10.1, C2.1, C8.1, C9.1, R11.1
Other:
- note added: "PIR1 ByPass CAPs"
- note added: "PIR1 OPAMP"
- moved on the sheet: C1, R9, U3
Changed lines of the file:
@@
 Comment4 ""
 $EndDescr
-Text Label 4600 1450 0    197  ~ 0
+Text Label 4500 950  0    197  ~ 0
 Microphone
 $Comp
 L SPH0645LM4H-B U3
 U 1 1 59AB3A7D
-P 5350 2150
-F 0 "U3" H 5550 1850 60  0000 C CNN
-F 1 "SPH0645LM4H-B" H 5350 2350 60  0000 C CNN
-F 2 "open-automation:SPH0645LM4H-B" H 5350 1750 60  0001 C CNN
-F 3 "https://www.digikey.com/product-detail/en/knowles/SPH0645LM4H-B/423-1405-6-ND/5332436" H 5300 1650 60  0001 C CNN
-F 4 "SPH0645LM4H-B" H 5350 2450 60  0001 C CNN "Part Number"
-	1    5350 2150
-	1    0    0    -1
-$EndComp
-$Comp
-L GND #PWR04
+P 5250 1650
+F 0 "U3" H 5450 1350 60  0000 C CNN
+F 1 "SPH0645LM4H-B" H 5250 1850 60  0000 C CNN
+F 2 "open-automation:SPH0645LM4H-B" H 5250 1250 60  0001 C CNN
+F 3 "https://www.digikey.com/product-detail/en/knowles/SPH0645LM4H-B/423-1405-6-ND/5332436" H 5200 1150 60  0001 C CNN
+F 4 "SPH0645LM4H-B" H 5250 1950 60  0001 C CNN "Part Number"
+	1    5250 1650
+	1    0    0    -1
+$EndComp
+$Comp
+L GND #PWR5
 U 1 1 59AB3AE9
-P 4900 2400
-F 0 "#PWR04" H 4900 2150 50  0001 C CNN
-F 1 "GND" H 4900 2250 50  0000 C CNN
-F 2 "" H 4900 2400 50  0000 C CNN
-F 3 "" H 4900 2400 50  0000 C CNN
-	1    4900 2400
-	1    0    0    -1
-$EndComp
-Text GLabel 4500 2100 0    60   Input ~ 0
+P 4800 1900
+F 0 "#PWR5" H 4800 1650 50  0001 C CNN
+F 1 "GND" H 4800 1750 50  0000 C CNN
+F 2 "" H 4800 1900 50  0000 C CNN
+F 3 "" H 4800 1900 50  0000 C CNN
+	1    4800 1900
+	1    0    0    -1
+$EndComp
+Text GLabel 4400 1600 0    60   Input ~ 0
 VCC_I2S
-Text GLabel 5850 2300 2    60   Input ~ 0
+Text GLabel 5750 1800 2    60   Input ~ 0
 I2S_BCLK
-Text GLabel 6300 2000 2    60   Input ~ 0
+Text GLabel 6200 1500 2    60   Input ~ 0
 I2S_DATA
 Wire Wire Line
-	5750 2300 5850 2300
-Wire Wire Line
-	5850 2200 5750 2200
-Wire Wire Line
-	4950 2350 4900 2350
-Wire Wire Line
-	4900 2200 4900 2400
-Wire Wire Line
-	4950 2200 4900 2200
-Connection ~ 4900 2350
+	5650 1800 5750 1800
+Wire Wire Line
+	5750 1700 5650 1700
+Wire Wire Line
+	4850 1850 4800 1850
+Wire Wire Line
+	4800 1700 4800 1900
+Wire Wire Line
+	4850 1700 4800 1700
+Connection ~ 4800 1850
 $Comp
 L R_10k R9
 U 1 1 59B93093
-P 6000 2000
-F 0 "R9" V 6000 2000 50  0000 C CNN
-F 1 "R_10k" V 5900 2000 50  0000 C CNN
-F 2 "Resistors_SMD:R_0603" V 5930 2000 50  0001 C CNN
-F 3 "https://www.digikey.com/product-detail/en/yageo/RC0603JR-0710KL/311-10KGRCT-ND/729647" V 6080 2000 50  0001 C CNN
-F 4 "RC0603JR-0710KL" V 6180 2100 60  0001 C CNN "Part Number"
-	1    6000 2000
+P 5900 1500
+F 0 "R9" V 5900 1500 50  0000 C CNN
+F 1 "R_10k" V 5800 1500 50  0000 C CNN
+F 2 "Resistors_SMD:R_0603" V 5830 1500 50  0001 C CNN
+F 3 "https://www.digikey.com/product-detail/en/yageo/RC0603JR-0710KL/311-10KGRCT-ND/729647" V 5980 1500 50  0001 C CNN
+F 4 "RC0603JR-0710KL" V 6080 1600 60  0001 C CNN "Part Number"
+	1    5900 1500
 	0    1    1    0
 $EndComp
-Text GLabel 5850 2200 2    60   Input ~ 0
+Text GLabel 5750 1700 2    60   Input ~ 0
 I2S_WS
 Wire Wire Line
-	4500 2100 4950 2100
+	4400 1600 4850 1600
 $Comp
 L C_0.1uF C1
 U 1 1 59B9ACE4
-P 4650 2400
-F 0 "C1" H 4675 2500 50  0000 L CNN
-F 1 "C_0.1uF" H 4325 2300 50  0000 L CNN
-F 2 "Capacitors_SMD:C_0603" H 4750 2700 50  0001 C CNN
-F 3 "https://www.digikey.com/product-detail/en/kemet/C0603C104K5RACTU/399-5089-1-ND/1465623" H 4650 2150 50  0001 C CNN
-F 4 "C0603C104K5RACTU" H 4775 2600 60  0001 C CNN "Part Number"
-	1    4650 2400
-	1    0    0    -1
-$EndComp
-Wire Wire Line
-	4650 2250 4650 2100
-Connection ~ 4650 2100
-$Comp
-L GND #PWR05
+P 4550 1900
+F 0 "C1" H 4575 2000 50  0000 L CNN
+F 1 "C_0.1uF" H 4225 1800 50  0000 L CNN
+F 2 "Capacitors_SMD:C_0603" H 4650 2200 50  0001 C CNN
+F 3 "https://www.digikey.com/product-detail/en/kemet/C0603C104K5RACTU/399-5089-1-ND/1465623" H 4550 1650 50  0001 C CNN
+F 4 "C0603C104K5RACTU" H 4675 2100 60  0001 C CNN "Part Number"
+	1    4550 1900
+	1    0    0    -1
+$EndComp
+Wire Wire Line
+	4550 1750 4550 1600
+Connection ~ 4550 1600
+$Comp
+L GND #PWR4
 U 1 1 59B9AD4C
-P 4650 2600
-F 0 "#PWR05" H 4650 2350 50  0001 C CNN
-F 1 "GND" H 4650 2450 50  0000 C CNN
-F 2 "" H 4650 2600 50  0000 C CNN
-F 3 "" H 4650 2600 50  0000 C CNN
-	1    4650 2600
-	1    0    0    -1
-$EndComp
-Wire Wire Line
-	4650 2550 4650 2600
-Wire Wire Line
-	5750 2100 5850 2100
-Wire Wire Line
-	6150 2000 6300 2000
-Wire Wire Line
-	5850 2100 5850 2000
+P 4550 2100
+F 0 "#PWR4" H 4550 1850 50  0001 C CNN
+F 1 "GND" H 4550 1950 50  0000 C CNN
+F 2 "" H 4550 2100 50  0000 C CNN
+F 3 "" H 4550 2100 50  0000 C CNN
+	1    4550 2100
+	1    0    0    -1
+$EndComp
+Wire Wire Line
+	4550 2050 4550 2100
+Wire Wire Line
+	5650 1600 5750 1600
+Wire Wire Line
+	6050 1500 6200 1500
+Wire Wire Line
+	5750 1600 5750 1500
+Text GLabel 6000 3500 2    60   Input ~ 0
+VCC_PIR1
+$Comp
+L R_10 R11
+U 1 1 59B80153
+P 4200 3500
+F 0 "R11" V 4280 3500 50  0000 C CNN
+F 1 "R_10" V 4200 3500 50  0000 C CNN
+F 2 "Resistors_SMD:R_0603" V 4130 3500 50  0001 C CNN
+F 3 "https://www.digikey.com/product-detail/en/te-connectivity-passive-product/CPF0603B10RE/A119908CT-ND/4966506" V 4280 3500 50  0001 C CNN
+F 4 "CPF0603B10RE" V 4380 3600 60  0001 C CNN "Part Number"
+	1    4200 3500
+	0    1    1    0
+$EndComp
+$Comp
+L C_1uF C8
+U 1 1 59B80154
+P 4900 3700
+F 0 "C8" H 4900 3800 50  0000 L CNN
+F 1 "C_1uF" H 4650 3600 50  0000 L CNN
+F 2 "Capacitors_SMD:C_0603" H 5000 4000 50  0001 C CNN
+F 3 "https://www.digikey.com/product-detail/en/yageo/CC0603ZRY5V7BB105/311-1372-1-ND/2103156" H 4900 3450 50  0001 C CNN
+F 4 "CC0603ZRY5V7BB105" H 5025 3900 60  0001 C CNN "Part Number"
+	1    4900 3700
+	1    0    0    -1
+$EndComp
+$Comp
+L C_0.1uF C9
+U 1 1 59B80155
+P 5300 3700
+F 0 "C9" H 5300 3800 50  0000 L CNN
+F 1 "C_0.1uF" H 5000 3600 50  0000 L CNN
+F 2 "Capacitors_SMD:C_0603" H 5400 4000 50  0001 C CNN
+F 3 "https://www.digikey.com/product-detail/en/kemet/C0603C104K5RACTU/399-5089-1-ND/1465623" H 5300 3450 50  0001 C CNN
+F 4 "C0603C104K5RACTU" H 5425 3900 60  0001 C CNN "Part Number"
+	1    5300 3700
+	1    0    0    -1
+$EndComp
+$Comp
+L C_100uF C2
+U 1 1 59B80156
+P 4500 3700
+F 0 "C2" H 4525 3800 50  0000 L CNN
+F 1 "C_100uF" H 4150 3600 50  0000 L CNN
+F 2 "Capacitors_SMD:C_1206" H 4600 4000 50  0001 C CNN
+F 3 "https://www.digikey.com/product-detail/en/kemet/C0603C104K5RACTU/399-5089-1-ND/1465623" H 4500 3450 50  0001 C CNN
+F 4 "C3216X5R1A107M160AC" H 4625 3900 60  0001 C CNN "Part Number"
+	1    4500 3700
+	1    0    0    -1
+$EndComp
+$Comp
+L GND #PWR6
+U 1 1 59B80157
+P 4900 3950
+F 0 "#PWR6" H 4900 3700 50  0001 C CNN
+F 1 "GND" H 4900 3800 50  0000 C CNN
+F 2 "" H 4900 3950 50  0000 C CNN
+F 3 "" H 4900 3950 50  0000 C CNN
+	1    4900 3950
+	1    0    0    -1
+$EndComp
+Text GLabel 3950 3500 0    60   Input ~ 0
+3V3
+$Comp
+L C_0.1uF C10
+U 1 1 59B80158
+P 5850 3700
+F 0 "C10" H 5850 3800 50  0000 L CNN
+F 1 "C_0.1uF" H 5550 3600 50  0000 L CNN
+F 2 "Capacitors_SMD:C_0603" H 5950 4000 50  0001 C CNN
+F 3 "https://www.digikey.com/product-detail/en/kemet/C0603C104K5RACTU/399-5089-1-ND/1465623" H 5850 3450 50  0001 C CNN
+F 4 "C0603C104K5RACTU" H 5975 3900 60  0001 C CNN "Part Number"
+	1    5850 3700
+	1    0    0    -1
+$EndComp
+Text Notes 4300 4300 0    60   ~ 0
+PIR1 ByPass CAPs
+Text Notes 5650 4300 0    60   ~ 0
+PIR1 OPAMP
+Wire Wire Line
+	4500 3850 4500 3900
+Wire Wire Line
+	4500 3900 5850 3900
+Wire Wire Line
+	5300 3900 5300 3850
+Wire Wire Line
+	4900 3850 4900 3950
+Connection ~ 4900 3900
+Wire Wire Line
+	4350 3500 6000 3500
+Wire Wire Line
+	5300 3550 5300 3500
+Connection ~ 5300 3500
+Wire Wire Line
+	4900 3550 4900 3500
+Connection ~ 4900 3500
+Wire Wire Line
+	4500 3550 4500 3500
+Connection ~ 4500 3500
+Wire Wire Line
+	3950 3500 4050 3500
+Wire Wire Line
+	5850 3550 5850 3500
+Connection ~ 5850 3500
+Wire Wire Line
+	5850 3900 5850 3850
+Connection ~ 5300 3900
+Wire Notes Line
+	3650 4200 5550 4200
+Wire Notes Line
+	5550 4200 5550 3350
+Wire Notes Line
+	5550 3350 3650 3350
+Wire Notes Line
+	5750 3350 5750 4200
+Wire Notes Line
+	5750 4200 6550 4200
+Wire Notes Line
+	5750 3350 6550 3350
+Wire Notes Line
+	3650 3350 3650 4200
+Wire Notes Line
+	6550 3350 6550 4200
 $EndSCHEMATC

Commit message: update
Parts:
- removed R9: R_10k, Resistors_SMD:R_0603, symbol R_10k
- added R47: R_47.5, Resistors_SMD:R_0603, symbol R_47.5
- added R9: R_100k, Resistors_SMD:R_0603, symbol R_100k
Connections:
- net GND: now also R9.1
- net I2S_DATA: now also R47.1
- net at U3.6 (DATA): now also R47.2, R9.2
Other:
- moved on the sheet: C1, U3
Changed lines of the file:
@@
 L SPH0645LM4H-B U3
 U 1 1 59AB3A7D
-P 5250 1650
-F 0 "U3" H 5450 1350 60  0000 C CNN
-F 1 "SPH0645LM4H-B" H 5250 1850 60  0000 C CNN
-F 2 "open-automation:SPH0645LM4H-B" H 5250 1250 60  0001 C CNN
-F 3 "https://www.digikey.com/product-detail/en/knowles/SPH0645LM4H-B/423-1405-6-ND/5332436" H 5200 1150 60  0001 C CNN
-F 4 "SPH0645LM4H-B" H 5250 1950 60  0001 C CNN "Part Number"
-	1    5250 1650
-	1    0    0    -1
-$EndComp
-$Comp
-L GND #PWR5
+P 5300 2100
+F 0 "U3" H 5500 1800 60  0000 C CNN
+F 1 "SPH0645LM4H-B" H 5300 2300 60  0000 C CNN
+F 2 "open-automation:SPH0645LM4H-B" H 5300 1700 60  0001 C CNN
+F 3 "https://www.digikey.com/product-detail/en/knowles/SPH0645LM4H-B/423-1405-6-ND/5332436" H 5250 1600 60  0001 C CNN
+F 4 "SPH0645LM4H-B" H 5300 2400 60  0001 C CNN "Part Number"
+	1    5300 2100
+	1    0    0    -1
+$EndComp
+$Comp
+L GND #PWR04
 U 1 1 59AB3AE9
-P 4800 1900
-F 0 "#PWR5" H 4800 1650 50  0001 C CNN
-F 1 "GND" H 4800 1750 50  0000 C CNN
-F 2 "" H 4800 1900 50  0000 C CNN
-F 3 "" H 4800 1900 50  0000 C CNN
-	1    4800 1900
-	1    0    0    -1
-$EndComp
-Text GLabel 4400 1600 0    60   Input ~ 0
+P 4850 2350
+F 0 "#PWR04" H 4850 2100 50  0001 C CNN
+F 1 "GND" H 4850 2200 50  0000 C CNN
+F 2 "" H 4850 2350 50  0000 C CNN
+F 3 "" H 4850 2350 50  0000 C CNN
+	1    4850 2350
+	1    0    0    -1
+$EndComp
+Text GLabel 4450 2050 0    60   Input ~ 0
 VCC_I2S
-Text GLabel 5750 1800 2    60   Input ~ 0
+Text GLabel 5800 2250 2    60   Input ~ 0
 I2S_BCLK
-Text GLabel 6200 1500 2    60   Input ~ 0
+Text GLabel 6250 1950 2    60   Input ~ 0
 I2S_DATA
 Wire Wire Line
-	5650 1800 5750 1800
-Wire Wire Line
-	5750 1700 5650 1700
-Wire Wire Line
-	4850 1850 4800 1850
-Wire Wire Line
-	4800 1700 4800 1900
-Wire Wire Line
-	4850 1700 4800 1700
-Connection ~ 4800 1850
-$Comp
-L R_10k R9
-U 1 1 59B93093
-P 5900 1500
-F 0 "R9" V 5900 1500 50  0000 C CNN
-F 1 "R_10k" V 5800 1500 50  0000 C CNN
-F 2 "Resistors_SMD:R_0603" V 5830 1500 50  0001 C CNN
-F 3 "https://www.digikey.com/product-detail/en/yageo/RC0603JR-0710KL/311-10KGRCT-ND/729647" V 5980 1500 50  0001 C CNN
-F 4 "RC0603JR-0710KL" V 6080 1600 60  0001 C CNN "Part Number"
-	1    5900 1500
-	0    1    1    0
-$EndComp
-Text GLabel 5750 1700 2    60   Input ~ 0
+	5700 2250 5800 2250
+Wire Wire Line
+	5800 2150 5700 2150
+Wire Wire Line
+	4900 2300 4850 2300
+Wire Wire Line
+	4850 2150 4850 2350
+Wire Wire Line
+	4900 2150 4850 2150
+Connection ~ 4850 2300
+Text GLabel 5800 2150 2    60   Input ~ 0
 I2S_WS
 Wire Wire Line
-	4400 1600 4850 1600
+	4450 2050 4900 2050
 $Comp
 L C_0.1uF C1
 U 1 1 59B9ACE4
-P 4550 1900
-F 0 "C1" H 4575 2000 50  0000 L CNN
-F 1 "C_0.1uF" H 4225 1800 50  0000 L CNN
-F 2 "Capacitors_SMD:C_0603" H 4650 2200 50  0001 C CNN
-F 3 "https://www.digikey.com/product-detail/en/kemet/C0603C104K5RACTU/399-5089-1-ND/1465623" H 4550 1650 50  0001 C CNN
-F 4 "C0603C104K5RACTU" H 4675 2100 60  0001 C CNN "Part Number"
-	1    4550 1900
-	1    0    0    -1
-$EndComp
-Wire Wire Line
-	4550 1750 4550 1600
-Connection ~ 4550 1600
-$Comp
-L GND #PWR4
+P 4600 2350
+F 0 "C1" H 4625 2450 50  0000 L CNN
+F 1 "C_0.1uF" H 4275 2250 50  0000 L CNN
+F 2 "Capacitors_SMD:C_0603" H 4700 2650 50  0001 C CNN
+F 3 "https://www.digikey.com/product-detail/en/kemet/C0603C104K5RACTU/399-5089-1-ND/1465623" H 4600 2100 50  0001 C CNN
+F 4 "C0603C104K5RACTU" H 4725 2550 60  0001 C CNN "Part Number"
+	1    4600 2350
+	1    0    0    -1
+$EndComp
+Wire Wire Line
+	4600 2200 4600 2050
+Connection ~ 4600 2050
+$Comp
+L GND #PWR05
 U 1 1 59B9AD4C
-P 4550 2100
-F 0 "#PWR4" H 4550 1850 50  0001 C CNN
-F 1 "GND" H 4550 1950 50  0000 C CNN
-F 2 "" H 4550 2100 50  0000 C CNN
-F 3 "" H 4550 2100 50  0000 C CNN
-	1    4550 2100
-	1    0    0    -1
-$EndComp
-Wire Wire Line
-	4550 2050 4550 2100
-Wire Wire Line
-	5650 1600 5750 1600
-Wire Wire Line
-	6050 1500 6200 1500
-Wire Wire Line
-	5750 1600 5750 1500
+P 4600 2550
+F 0 "#PWR05" H 4600 2300 50  0001 C CNN
+F 1 "GND" H 4600 2400 50  0000 C CNN
+F 2 "" H 4600 2550 50  0000 C CNN
+F 3 "" H 4600 2550 50  0000 C CNN
+	1    4600 2550
+	1    0    0    -1
+$EndComp
+Wire Wire Line
+	4600 2500 4600 2550
+Wire Wire Line
+	6100 1950 6250 1950
 Text GLabel 6000 3500 2    60   Input ~ 0
 VCC_PIR1
@@
 $EndComp
 $Comp
-L GND #PWR6
+L GND #PWR06
 U 1 1 59B80157
 P 4900 3950
-F 0 "#PWR6" H 4900 3700 50  0001 C CNN
+F 0 "#PWR06" H 4900 3700 50  0001 C CNN
 F 1 "GND" H 4900 3800 50  0000 C CNN
 F 2 "" H 4900 3950 50  0000 C CNN
@@
 Wire Notes Line
 	6550 3350 6550 4200
+$Comp
+L R_47.5 R47
+U 1 1 59B81820
+P 5950 1950
+F 0 "R47" V 5950 1950 50  0000 C CNN
+F 1 "R_47.5" V 5875 1950 50  0000 C CNN
+F 2 "Resistors_SMD:R_0603" V 5880 1950 50  0001 C CNN
+F 3 "https://www.digikey.com/product-detail/en/yageo/RC0603FR-0747R5L/311-47.5HRCT-ND/730201" V 6030 1950 50  0001 C CNN
+F 4 "RC0603FR-0747R5L" V 6130 2050 60  0001 C CNN "Part Number"
+	1    5950 1950
+	0    1    1    0
+$EndComp
+$Comp
+L R_100k R9
+U 1 1 59B82082
+P 5950 1750
+F 0 "R9" V 5950 1750 50  0000 C CNN
+F 1 "R_100k" V 5850 1750 50  0000 C CNN
+F 2 "Resistors_SMD:R_0603" V 5880 1750 50  0001 C CNN
+F 3 "https://www.digikey.com/product-detail/en/yageo/RC0603JR-07100KL/311-100KGRCT-ND/729645" V 6030 1750 50  0001 C CNN
+F 4 "RC0603JR-07100KL" V 6130 1850 60  0001 C CNN "Part Number"
+	1    5950 1750
+	0    1    1    0
+$EndComp
+$Comp
+L GND #PWR07
+U 1 1 59B820C6
+P 6150 1750
+F 0 "#PWR07" H 6150 1500 50  0001 C CNN
+F 1 "GND" H 6150 1600 50  0000 C CNN
+F 2 "" H 6150 1750 50  0000 C CNN
+F 3 "" H 6150 1750 50  0000 C CNN
+	1    6150 1750
+	0    -1   -1   0
+$EndComp
+Wire Wire Line
+	6100 1750 6150 1750
+Wire Wire Line
+	5750 2050 5700 2050
+Wire Wire Line
+	5750 1750 5750 2050
+Wire Wire Line
+	5750 1950 5800 1950
+Wire Wire Line
+	5800 1750 5750 1750
+Connection ~ 5750 1950
 $EndSCHEMATC

Commit message: update
Parts:
- removed C10, C9: C_0.1uF, Capacitors_SMD:C_0603, symbol C_0.1uF
Connections:
- net VCC_PIR1 is gone; now on net VCC_I2S: C2.1, C8.1, R11.1
Other:
- note removed: "PIR1 OPAMP"
Changed lines of the file:
@@
 $EndComp
 $Comp
-L GND #PWR04
+L GND #PWR08
 U 1 1 59AB3AE9
 P 4850 2350
-F 0 "#PWR04" H 4850 2100 50  0001 C CNN
+F 0 "#PWR08" H 4850 2100 50  0001 C CNN
 F 1 "GND" H 4850 2200 50  0000 C CNN
 F 2 "" H 4850 2350 50  0000 C CNN
@@
 	1    0    0    -1
 $EndComp
-Text GLabel 4450 2050 0    60   Input ~ 0
-VCC_I2S
 Text GLabel 5800 2250 2    60   Input ~ 0
 I2S_BCLK
 Text GLabel 6250 1950 2    60   Input ~ 0
 I2S_DATA
-Wire Wire Line
-	5700 2250 5800 2250
-Wire Wire Line
-	5800 2150 5700 2150
-Wire Wire Line
-	4900 2300 4850 2300
-Wire Wire Line
-	4850 2150 4850 2350
-Wire Wire Line
-	4900 2150 4850 2150
-Connection ~ 4850 2300
 Text GLabel 5800 2150 2    60   Input ~ 0
 I2S_WS
-Wire Wire Line
-	4450 2050 4900 2050
 $Comp
 L C_0.1uF C1
@@
 	1    0    0    -1
 $EndComp
-Wire Wire Line
-	4600 2200 4600 2050
-Connection ~ 4600 2050
 $Comp
-L GND #PWR05
+L GND #PWR09
 U 1 1 59B9AD4C
 P 4600 2550
-F 0 "#PWR05" H 4600 2300 50  0001 C CNN
+F 0 "#PWR09" H 4600 2300 50  0001 C CNN
 F 1 "GND" H 4600 2400 50  0000 C CNN
 F 2 "" H 4600 2550 50  0000 C CNN
@@
 	1    0    0    -1
 $EndComp
-Wire Wire Line
-	4600 2500 4600 2550
-Wire Wire Line
-	6100 1950 6250 1950
-Text GLabel 6000 3500 2    60   Input ~ 0
-VCC_PIR1
 $Comp
 L R_10 R11
@@
 $EndComp
 $Comp
-L C_0.1uF C9
-U 1 1 59B80155
-P 5300 3700
-F 0 "C9" H 5300 3800 50  0000 L CNN
-F 1 "C_0.1uF" H 5000 3600 50  0000 L CNN
-F 2 "Capacitors_SMD:C_0603" H 5400 4000 50  0001 C CNN
-F 3 "https://www.digikey.com/product-detail/en/kemet/C0603C104K5RACTU/399-5089-1-ND/1465623" H 5300 3450 50  0001 C CNN
-F 4 "C0603C104K5RACTU" H 5425 3900 60  0001 C CNN "Part Number"
-	1    5300 3700
-	1    0    0    -1
-$EndComp
-$Comp
 L C_100uF C2
 U 1 1 59B80156
@@
 $EndComp
 $Comp
-L GND #PWR06
+L GND #PWR010
 U 1 1 59B80157
-P 4900 3950
-F 0 "#PWR06" H 4900 3700 50  0001 C CNN
-F 1 "GND" H 4900 3800 50  0000 C CNN
-F 2 "" H 4900 3950 50  0000 C CNN
-F 3 "" H 4900 3950 50  0000 C CNN
-	1    4900 3950
+P 4675 3950
+F 0 "#PWR010" H 4675 3700 50  0001 C CNN
+F 1 "GND" H 4675 3800 50  0000 C CNN
+F 2 "" H 4675 3950 50  0000 C CNN
+F 3 "" H 4675 3950 50  0000 C CNN
+	1    4675 3950
 	1    0    0    -1
 $EndComp
 Text GLabel 3950 3500 0    60   Input ~ 0
 3V3
-$Comp
-L C_0.1uF C10
-U 1 1 59B80158
-P 5850 3700
-F 0 "C10" H 5850 3800 50  0000 L CNN
-F 1 "C_0.1uF" H 5550 3600 50  0000 L CNN
-F 2 "Capacitors_SMD:C_0603" H 5950 4000 50  0001 C CNN
-F 3 "https://www.digikey.com/product-detail/en/kemet/C0603C104K5RACTU/399-5089-1-ND/1465623" H 5850 3450 50  0001 C CNN
-F 4 "C0603C104K5RACTU" H 5975 3900 60  0001 C CNN "Part Number"
-	1    5850 3700
-	1    0    0    -1
-$EndComp
 Text Notes 4300 4300 0    60   ~ 0
 PIR1 ByPass CAPs
-Text Notes 5650 4300 0    60   ~ 0
-PIR1 OPAMP
-Wire Wire Line
-	4500 3850 4500 3900
-Wire Wire Line
-	4500 3900 5850 3900
-Wire Wire Line
-	5300 3900 5300 3850
-Wire Wire Line
-	4900 3850 4900 3950
-Connection ~ 4900 3900
-Wire Wire Line
-	4350 3500 6000 3500
-Wire Wire Line
-	5300 3550 5300 3500
-Connection ~ 5300 3500
-Wire Wire Line
-	4900 3550 4900 3500
-Connection ~ 4900 3500
-Wire Wire Line
-	4500 3550 4500 3500
-Connection ~ 4500 3500
-Wire Wire Line
-	3950 3500 4050 3500
-Wire Wire Line
-	5850 3550 5850 3500
-Connection ~ 5850 3500
-Wire Wire Line
-	5850 3900 5850 3850
-Connection ~ 5300 3900
-Wire Notes Line
-	3650 4200 5550 4200
-Wire Notes Line
-	5550 4200 5550 3350
-Wire Notes Line
-	5550 3350 3650 3350
-Wire Notes Line
-	5750 3350 5750 4200
-Wire Notes Line
-	5750 4200 6550 4200
-Wire Notes Line
-	5750 3350 6550 3350
-Wire Notes Line
-	3650 3350 3650 4200
-Wire Notes Line
-	6550 3350 6550 4200
 $Comp
 L R_47.5 R47
@@
 $EndComp
 $Comp
-L GND #PWR07
+L GND #PWR011
 U 1 1 59B820C6
 P 6150 1750
-F 0 "#PWR07" H 6150 1500 50  0001 C CNN
+F 0 "#PWR011" H 6150 1500 50  0001 C CNN
 F 1 "GND" H 6150 1600 50  0000 C CNN
 F 2 "" H 6150 1750 50  0000 C CNN
@@
 	0    -1   -1   0
 $EndComp
+Text GLabel 4450 2050 0    60   Input ~ 0
+VCC_I2S
+Text GLabel 5100 3500 2    60   Input ~ 0
+VCC_I2S
+Connection ~ 4675 3925
 Wire Wire Line
-	6100 1750 6150 1750
+	4675 3950 4675 3925
+Wire Wire Line
+	4900 3925 4500 3925
+Wire Wire Line
+	4900 3850 4900 3925
+Wire Wire Line
+	4350 3500 5100 3500
+Connection ~ 5750 1950
+Wire Wire Line
+	5800 1750 5750 1750
+Wire Wire Line
+	5750 1950 5800 1950
+Wire Wire Line
+	5750 1750 5750 2050
 Wire Wire Line
 	5750 2050 5700 2050
 Wire Wire Line
-	5750 1750 5750 2050
+	6100 1750 6150 1750
+Wire Notes Line
+	3650 3350 3650 4200
+Wire Notes Line
+	5550 3350 3650 3350
+Wire Notes Line
+	5550 4200 5550 3350
+Wire Notes Line
+	3650 4200 5550 4200
 Wire Wire Line
-	5750 1950 5800 1950
+	3950 3500 4050 3500
+Connection ~ 4500 3500
 Wire Wire Line
-	5800 1750 5750 1750
-Connection ~ 5750 1950
+	4500 3550 4500 3500
+Connection ~ 4900 3500
+Wire Wire Line
+	4900 3550 4900 3500
+Wire Wire Line
+	4500 3925 4500 3850
+Wire Wire Line
+	6100 1950 6250 1950
+Wire Wire Line
+	4600 2500 4600 2550
+Connection ~ 4600 2050
+Wire Wire Line
+	4600 2200 4600 2050
+Wire Wire Line
+	4450 2050 4900 2050
+Connection ~ 4850 2300
+Wire Wire Line
+	4900 2150 4850 2150
+Wire Wire Line
+	4850 2150 4850 2350
+Wire Wire Line
+	4900 2300 4850 2300
+Wire Wire Line
+	5800 2150 5700 2150
+Wire Wire Line
+	5700 2250 5800 2250
 $EndSCHEMATC
