File: hardware/microphone.sch (KiCad schematic (older format))
At the start: 7 parts, among them U3 SPH0645LM4H-B

Commit message: update
Parts:
- C1, C8: footprint Capacitors_SMD:C_0603 -> Capacitors_SMD:C_0603_HandSoldering
- C2: footprint Capacitors_SMD:C_1206 -> Capacitors_SMD:C_1206_HandSoldering
- R11: footprint Resistors_SMD:R_0603 -> Resistors_SMD:R_0805_HandSoldering; Part Number CPF0603B10RE -> ERJ-P06J100V
- R47, R9: footprint Resistors_SMD:R_0603 -> Resistors_SMD:R_0603_HandSoldering
Connections:
- net 3V3: now also R11.1; no longer R11.2
- net VCC_I2S: now also R11.2; no longer R11.1
- net I2S_DATA renamed I2S_DATA_IN
Changed lines of the file:
@@
 $EndComp
 $Comp
-L GND #PWR08
+L GND #PWR07
 U 1 1 59AB3AE9
 P 4850 2350
-F 0 "#PWR08" H 4850 2100 50  0001 C CNN
+F 0 "#PWR07" H 4850 2100 50  0001 C CNN
 F 1 "GND" H 4850 2200 50  0000 C CNN
 F 2 "" H 4850 2350 50  0000 C CNN
@@
 I2S_BCLK
 Text GLabel 6250 1950 2    60   Input ~ 0
-I2S_DATA
+I2S_DATA_IN
 Text GLabel 5800 2150 2    60   Input ~ 0
 I2S_WS
@@
 F 0 "C1" H 4625 2450 50  0000 L CNN
 F 1 "C_0.1uF" H 4275 2250 50  0000 L CNN
-F 2 "Capacitors_SMD:C_0603" H 4700 2650 50  0001 C CNN
+F 2 "Capacitors_SMD:C_0603_HandSoldering" H 4700 2650 50  0001 C CNN
 F 3 "https://www.digikey.com/product-detail/en/kemet/C0603C104K5RACTU/399-5089-1-ND/1465623" H 4600 2100 50  0001 C CNN
 F 4 "C0603C104K5RACTU" H 4725 2550 60  0001 C CNN "Part Number"
@@
 $EndComp
 $Comp
-L GND #PWR09
+L GND #PWR08
 U 1 1 59B9AD4C
 P 4600 2550
-F 0 "#PWR09" H 4600 2300 50  0001 C CNN
+F 0 "#PWR08" H 4600 2300 50  0001 C CNN
 F 1 "GND" H 4600 2400 50  0000 C CNN
 F 2 "" H 4600 2550 50  0000 C CNN
@@
 $EndComp
 $Comp
-L R_10 R11
-U 1 1 59B80153
-P 4200 3500
-F 0 "R11" V 4280 3500 50  0000 C CNN
-F 1 "R_10" V 4200 3500 50  0000 C CNN
-F 2 "Resistors_SMD:R_0603" V 4130 3500 50  0001 C CNN
-F 3 "https://www.digikey.com/product-detail/en/te-connectivity-passive-product/CPF0603B10RE/A119908CT-ND/4966506" V 4280 3500 50  0001 C CNN
-F 4 "CPF0603B10RE" V 4380 3600 60  0001 C CNN "Part Number"
-	1    4200 3500
-	0    1    1    0
-$EndComp
-$Comp
 L C_1uF C8
 U 1 1 59B80154
@@
 F 0 "C8" H 4900 3800 50  0000 L CNN
 F 1 "C_1uF" H 4650 3600 50  0000 L CNN
-F 2 "Capacitors_SMD:C_0603" H 5000 4000 50  0001 C CNN
+F 2 "Capacitors_SMD:C_0603_HandSoldering" H 5000 4000 50  0001 C CNN
 F 3 "https://www.digikey.com/product-detail/en/yageo/CC0603ZRY5V7BB105/311-1372-1-ND/2103156" H 4900 3450 50  0001 C CNN
 F 4 "CC0603ZRY5V7BB105" H 5025 3900 60  0001 C CNN "Part Number"
@@
 F 0 "C2" H 4525 3800 50  0000 L CNN
 F 1 "C_100uF" H 4150 3600 50  0000 L CNN
-F 2 "Capacitors_SMD:C_1206" H 4600 4000 50  0001 C CNN
+F 2 "Capacitors_SMD:C_1206_HandSoldering" H 4600 4000 50  0001 C CNN
 F 3 "https://www.digikey.com/product-detail/en/kemet/C0603C104K5RACTU/399-5089-1-ND/1465623" H 4500 3450 50  0001 C CNN
 F 4 "C3216X5R1A107M160AC" H 4625 3900 60  0001 C CNN "Part Number"
@@
 $EndComp
 $Comp
-L GND #PWR010
+L GND #PWR09
 U 1 1 59B80157
 P 4675 3950
-F 0 "#PWR010" H 4675 3700 50  0001 C CNN
+F 0 "#PWR09" H 4675 3700 50  0001 C CNN
 F 1 "GND" H 4675 3800 50  0000 C CNN
 F 2 "" H 4675 3950 50  0000 C CNN
@@
 F 0 "R47" V 5950 1950 50  0000 C CNN
 F 1 "R_47.5" V 5875 1950 50  0000 C CNN
-F 2 "Resistors_SMD:R_0603" V 5880 1950 50  0001 C CNN
+F 2 "Resistors_SMD:R_0603_HandSoldering" V 5880 1950 50  0001 C CNN
 F 3 "https://www.digikey.com/product-detail/en/yageo/RC0603FR-0747R5L/311-47.5HRCT-ND/730201" V 6030 1950 50  0001 C CNN
 F 4 "RC0603FR-0747R5L" V 6130 2050 60  0001 C CNN "Part Number"
@@
 F 0 "R9" V 5950 1750 50  0000 C CNN
 F 1 "R_100k" V 5850 1750 50  0000 C CNN
-F 2 "Resistors_SMD:R_0603" V 5880 1750 50  0001 C CNN
+F 2 "Resistors_SMD:R_0603_HandSoldering" V 5880 1750 50  0001 C CNN
 F 3 "https://www.digikey.com/product-detail/en/yageo/RC0603JR-07100KL/311-100KGRCT-ND/729645" V 6030 1750 50  0001 C CNN
 F 4 "RC0603JR-07100KL" V 6130 1850 60  0001 C CNN "Part Number"
@@
 $EndComp
 $Comp
-L GND #PWR011
+L GND #PWR010
 U 1 1 59B820C6
 P 6150 1750
-F 0 "#PWR011" H 6150 1500 50  0001 C CNN
+F 0 "#PWR010" H 6150 1500 50  0001 C CNN
 F 1 "GND" H 6150 1600 50  0000 C CNN
 F 2 "" H 6150 1750 50  0000 C CNN
@@
 Wire Wire Line
 	5700 2250 5800 2250
+$Comp
+L R_10 R11
+U 1 1 59EBEDAE
+P 4200 3500
+F 0 "R11" V 4200 3500 50  0000 C CNN
+F 1 "R_10" V 4125 3500 50  0000 C CNN
+F 2 "Resistors_SMD:R_0805_HandSoldering" V 4130 3500 50  0001 C CNN
+F 3 "https://www.digikey.com/product-detail/en/panasonic-electronic-components/ERJ-P06J100V/P10ADCT-ND/525435" V 4280 3500 50  0001 C CNN
+F 4 "ERJ-P06J100V" V 4380 3600 60  0001 C CNN "Part Number"
+	1    4200 3500
+	0    -1   -1   0
+$EndComp
 $EndSCHEMATC

Commit message: update
Parts:
- removed C2: C_100uF, Capacitors_SMD:C_1206_HandSoldering, symbol C_100uF
- removed C8: C_1uF, Capacitors_SMD:C_0603_HandSoldering, symbol C_1uF
- removed R11: R_10, Resistors_SMD:R_0805_HandSoldering, symbol R_10
- added C?: C_1uF, Capacitors_SMD:C_0603_HandSoldering, symbol C_1uF
- added LS?: speaker-CVS-1508, open-automation:speaker-1508, symbol speaker-CVS-1508
- added R?: R_100k, Resistors_SMD:R_0603_HandSoldering, symbol R_100k
- added U?: MAX98357AETE+T, open-automation:MAX98357A, symbol MAX98357AETE+T
Connections:
- net VCC_I2S is gone; now on net 3V3: C1.1, U3.5 (Vin)
- net GND: now also C?.2, R?.2, U?.3 (GND)
- net I2S_BCLK: now also U?.16 (BCLK)
- net I2S_WS: now also U?.14 (LRCLK)
- new net: R?.1, U?.2 (GAIN_SLOT)
- new net: LS?.2, U?.10 (OUTN)
- new net: LS?.1, U?.9 (OUTP)
- new net I2S_DATA_OUT: U?.1 (DIN)
- new net V_IN: C?.1, U?.4 (~SD_MODE), U?.7 (VDD)
Other:
- note removed: "PIR1 ByPass CAPs"
- moved on the sheet: C1, R47, R9, U3
