File: hardware/climate.sch (KiCad schematic (older format))
At the start: 2 parts, among them P6 CONN_01X04

Commit message: update
Parts:
- P6: footprint Pin_Headers:Pin_Header_Angled_1x04_Pitch2.54mm -> open-automation:Pin_Header_Angled_1x04_Pitch2.54mm_CORRECTED
Connections:
- net IO17 renamed IO21
Changed lines of the file:
@@
 LIBS:open-automation
 LIBS:liger-cache
-EELAYER 26 0
+EELAYER 25 0
 EELAYER END
 $Descr A4 11693 8268
 encoding utf-8
-Sheet 9 8
+Sheet 8 8
 Title ""
 Date ""
@@
 $EndDescr
 Text GLabel 5400 2800 0    60   Input ~ 0
-IO17
+IO21
 $Comp
 L GND #PWR023
@@
 F 0 "P6" H 6150 3100 50  0000 C CNN
 F 1 "CONN_01X04" V 6250 2850 50  0000 C CNN
-F 2 "Pin_Headers:Pin_Header_Angled_1x04_Pitch2.54mm" H 6150 2850 50  0001 C CNN
+F 2 "open-automation:Pin_Header_Angled_1x04_Pitch2.54mm_CORRECTED" H 6150 2850 50  0001 C CNN
 F 3 "" H 6150 2850 50  0000 C CNN
 	1    6150 2850
