File: hardware/microcontroller.sch (KiCad schematic (older format))
At the start: 5 parts, among them P1 CONN_01X20, P2 CONN_01X20, U1 ESP-WROOM-32

Commit message: updatge
Connections:
- net CLK: no longer P1.20 (P20)
- net CMD: no longer P1.19 (P19)
- new net SPEAKER+: P1.19 (P19)
- new net SPEAKER-: P1.20 (P20)
Changed lines of the file:
@@
 $EndDescr
 $Comp
-L GND #PWR3
+L GND #PWR01
 U 1 1 59097974
 P 5050 2400
-F 0 "#PWR3" H 5050 2150 50  0001 C CNN
+F 0 "#PWR01" H 5050 2150 50  0001 C CNN
 F 1 "GND" H 5050 2250 50  0000 C CNN
 F 2 "" H 5050 2400 50  0000 C CNN
@@
 $EndComp
 $Comp
-L GND #PWR1
+L GND #PWR02
 U 1 1 590979AD
 P 2200 4000
-F 0 "#PWR1" H 2200 3750 50  0001 C CNN
+F 0 "#PWR02" H 2200 3750 50  0001 C CNN
 F 1 "GND" H 2200 3850 50  0000 C CNN
 F 2 "" H 2200 4000 50  0000 C CNN
@@
 IO17
 $Comp
-L GND #PWR2
+L GND #PWR03
 U 1 1 590979B0
 P 3650 2350
-F 0 "#PWR2" H 3650 2100 50  0001 C CNN
+F 0 "#PWR03" H 3650 2100 50  0001 C CNN
 F 1 "GND" H 3650 2200 50  0000 C CNN
 F 2 "" H 3650 2350 50  0000 C CNN
@@
 SD3
 Text GLabel 3650 4200 0    60   Input ~ 0
-CMD
-Text GLabel 3650 4300 0    60   Input ~ 0
-CLK
+SPEAKER+
 Text GLabel 3650 2600 0    60   Input ~ 0
 3v3
@@
 IO17
 $Comp
-L GND #PWR4
+L GND #PWR04
 U 1 1 590979B2
 P 8250 2300
-F 0 "#PWR4" H 8250 2050 50  0001 C CNN
+F 0 "#PWR04" H 8250 2050 50  0001 C CNN
 F 1 "GND" H 8250 2150 50  0000 C CNN
 F 2 "" H 8250 2300 50  0000 C CNN
@@
 Wire Wire Line
 	8200 2550 8300 2550
+Text GLabel 3650 4300 0    60   Input ~ 0
+SPEAKER-
 $EndSCHEMATC

Commit message: update
Parts:
- removed R2: 10K, Resistors_SMD:R_0603_HandSoldering, symbol R
Changed lines of the file:
@@
 LIBS:contrib
 LIBS:valves
-LIBS:open-automation
 LIBS:liger-cache
-EELAYER 25 0
+EELAYER 26 0
 EELAYER END
 $Descr A4 11693 8268
@@
 Text GLabel 6300 4400 3    60   Input ~ 0
 IO15
-Text GLabel 2450 4000 3    60   Input ~ 0
-IO2
-$Comp
-L R R2
-U 1 1 590979AE
-P 2450 3750
-F 0 "R2" V 2530 3750 50  0000 C CNN
-F 1 "10K" V 2450 3750 50  0000 C CNN
-F 2 "Resistors_SMD:R_0603_HandSoldering" V 2380 3750 50  0001 C CNN
-F 3 "http://www.digikey.com/en/resources/datasheets/yageo/rc-series-l-suffix-datasheet" H 2450 3750 50  0001 C CNN
-F 4 "RC0603JR-0710KL" V 2450 3750 60  0001 C CNN "Part Number"
-	1    2450 3750
-	1    0    0    -1
-$EndComp
-Text GLabel 2450 3400 1    60   Input ~ 0
-3v3
 $Comp
 L ESP-WROOM-32 U1
@@
 	2200 3900 2200 4000
 Wire Wire Line
-	2450 4000 2450 3900
-Wire Wire Line
-	2450 3400 2450 3600
-Wire Wire Line
 	5050 2400 5050 2450

Commit message: update
Connections:
- net 3v3 renamed 3V3
Changed lines of the file:
@@
 LIBS:open-automation
 LIBS:liger-cache
-EELAYER 25 0
+EELAYER 26 0
 EELAYER END
 $Descr A4 11693 8268
@@
 IO2
 Text GLabel 5000 2550 0    60   Input ~ 0
-3v3
+3V3
 $Comp
 L R R1
@@
 SPEAKER+
 Text GLabel 3650 2600 0    60   Input ~ 0
-3v3
+3V3
 Text GLabel 8300 3450 2    60   Input ~ 0
 IO5

Commit message: update
Parts:
- P1, P2: footprint Pin_Headers:Pin_Header_Straight_1x20_Pitch2.54mm -> open-automation:Pin_Header_Straight_1x20_Pitch2.54mm_CORRECTED
Connections:
- net 3V3: now also P1.19 (P19), P1.20 (P20); no longer P1.3 (P3), P1.4 (P4)
- net SD2: no longer P1.17 (P17)
- net SD3: no longer P1.18 (P18)
- net SPEAKER+: now also P1.4 (P4); no longer P1.19 (P19)
- net SPEAKER-: now also P1.3 (P3); no longer P1.20 (P20)
Changed lines of the file:
@@
 LIBS:open-automation
 LIBS:liger-cache
-EELAYER 26 0
+EELAYER 25 0
 EELAYER END
 $Descr A4 11693 8268
@@
 F 1 "ESP-WROOM-32" H 6000 3900 60  0000 C CNN
 F 2 "footprints:ESP-WROOM-32" H 5650 3700 60  0001 C CNN
-F 3 "https://www.espressif.com/sites/default/files/documentation/esp_wroom_32_datasheet_en.pdf" H 5650 3700 60  0001 C CNN
+F 3 "http://espressif.com/sites/default/files/documentation/esp-wroom-32_datasheet_en.pdf" H 5650 3700 60  0001 C CNN
 	1    6000 3100
 	1    0    0    -1
@@
 Text GLabel 3650 3900 0    60   Input ~ 0
 IO13
-Text GLabel 3650 4000 0    60   Input ~ 0
-SD2
 $Comp
 L CONN_01X20 P1
@@
 F 0 "P1" H 3950 4400 50  0000 C CNN
 F 1 "CONN_01X20" V 4050 3350 50  0000 C CNN
-F 2 "Pin_Headers:Pin_Header_Straight_1x20_Pitch2.54mm" H 3950 3350 50  0001 C CNN
+F 2 "open-automation:Pin_Header_Straight_1x20_Pitch2.54mm_CORRECTED" H 3950 3350 50  0001 C CNN
 F 3 "" H 3950 3350 50  0000 C CNN
 	1    3950 3350
 	1    0    0    -1
 $EndComp
-Text GLabel 3650 4100 0    60   Input ~ 0
-SD3
 Text GLabel 3650 4200 0    60   Input ~ 0
-SPEAKER+
-Text GLabel 3650 2600 0    60   Input ~ 0
 3V3
 Text GLabel 8300 3450 2    60   Input ~ 0
@@
 F 0 "P2" H 8000 4350 50  0000 C CNN
 F 1 "CONN_01X20" V 8100 3300 50  0000 C CNN
-F 2 "Pin_Headers:Pin_Header_Straight_1x20_Pitch2.54mm" H 8000 3300 50  0001 C CNN
+F 2 "open-automation:Pin_Header_Straight_1x20_Pitch2.54mm_CORRECTED" H 8000 3300 50  0001 C CNN
 F 3 "" H 8000 3300 50  0000 C CNN
 	1    8000 3300
@@
 	3650 2900 3750 2900
 Wire Wire Line
-	3650 2600 3750 2600
-Wire Wire Line
 	3650 3800 3750 3800
 Wire Wire Line
 	3750 3900 3650 3900
 Wire Wire Line
-	3650 4100 3750 4100
-Wire Wire Line
-	3750 4000 3650 4000
-Wire Wire Line
-	3750 2700 3700 2700
-Wire Wire Line
-	3700 2700 3700 2600
-Connection ~ 3700 2600
-Wire Wire Line
 	3650 4200 3750 4200
-Wire Wire Line
-	3750 4300 3650 4300
 Wire Wire Line
 	8200 3850 8300 3850
@@
 Wire Wire Line
 	8200 2550 8300 2550
-Text GLabel 3650 4300 0    60   Input ~ 0
+Text GLabel 3650 2700 0    60   Input ~ 0
+SPEAKER+
+Text GLabel 3650 2600 0    60   Input ~ 0
 SPEAKER-
+Wire Wire Line
+	3750 4300 3700 4300
+Wire Wire Line
+	3700 4300 3700 4200
+Connection ~ 3700 4200
+Wire Wire Line
+	3650 2600 3750 2600
+Wire Wire Line
+	3750 2700 3650 2700
 $EndSCHEMATC
