File: hardware/microcontroller.sch (KiCad schematic (older format))
At the start: 4 parts, among them P1 CONN_01X20, P2 CONN_01X20, U1 ESP-WROOM-32

Commit message: update
Parts:
- removed P1, P2: CONN_01X20, open-automation:Pin_Header_Straight_1x20_Pitch2.54mm_CORRECTED, symbol CONN_01X20
- removed R1: 10K, Resistors_SMD:R_0603_HandSoldering, symbol R
- added R1, R2, R47, R6, R7: R_10k, Resistors_SMD:R_0603, symbol R_10k
Connections:
- net labels added: I2S_BCLK, I2S_DATA, I2S_WS, IR_RX, IR_TX, LED_B, LED_G, LED_R, PIR1_ADC, PIR2_ADC, PIR_HI, PIR_LO, RELAY, SCL, SDA, SPEAKER_IN, T_DOWN, T_LEFT, T_RIGHT, T_UP
- net labels removed: 5V, IO14, IO15, IO16, IO17, IO18, IO19, IO21, IO22, IO23, IO25, IO26, IO27, IO32, IO33, IO34, IO35, IO4, IO5, SD0, SD1, SPEAKER+, SPEAKER-
- wire segments 80 -> 45

Commit message: update
Parts:
- removed R1, R2, R47: R_10k, Resistors_SMD:R_0603, symbol R_10k
- added R1, R2: R_47.5, Resistors_SMD:R_0603, symbol R_47.5
Connections:
- net I2S_BCLK: now also R1.2
- net I2S_WS: now also R2.1
- net at U1.11 (IO26): now also R1.1
- net at U1.37 (IO23): now also R2.2
Other:
- moved on the sheet: R6, R7, U1

Commit message: update
Parts:
- U1: footprint footprints:ESP-WROOM-32 -> open-automation:ESP-WROOM-32
Changed lines of the file:
@@
 F 0 "U1" H 6000 1550 60  0000 C CNN
 F 1 "ESP-WROOM-32" H 5450 3450 60  0000 C CNN
-F 2 "footprints:ESP-WROOM-32" H 5100 3250 60  0001 C CNN
+F 2 "open-automation:ESP-WROOM-32" H 5100 3250 60  0001 C CNN
 F 3 "http://espressif.com/sites/default/files/documentation/esp-wroom-32_datasheet_en.pdf" H 5100 3250 60  0001 C CNN
 	1    5450 2650

Commit message: update
Parts:
- added C41: C_100uF, Capacitors_SMD:C_1206, symbol C_100uF
- added C42: C_1uF, Capacitors_SMD:C_0603, symbol C_1uF
- added J1: Conn_02x05_Odd_Even, Pin_Headers:Pin_Header_Straight_2x05_Pitch2.54mm, symbol Conn_02x05_Odd_Even
- added R48: R_10, Resistors_SMD:R_0603, symbol R_10
- added R49: R_10k, Resistors_SMD:R_0603, symbol R_10k
Connections:
- net IO12 is gone; now on net T_DOWN: U1.14 (IO12)
- net 3V3: now also J1.3 (Pin_3), R48.2
- net GND: now also C41.2, C42.2, J1.1 (Pin_1), J1.2 (Pin_2), J1.9 (Pin_9), R49.1
- net RXD: now also J1.8 (Pin_8)
- net TXD: now also J1.6 (Pin_6)
- net T_DOWN: no longer U1.13 (IO14)
- net CLK: no longer names the net of U1.20 (CLK)
- net CMD: no longer names the net of U1.19 (CMD)
- net IO0 renamed PROG
- net PROG: now also J1.7 (Pin_7)
- net IO13: no longer names the net of U1.16 (IO13)
- net IO2: no longer names the net of U1.24 (IO2)
- net IO2: now also R49.2
- net SD2: no longer names the net of U1.17 (SD2)
- net SD3: no longer names the net of U1.18 (SD3)
- net SENSOR_VN: no longer names the net of U1.5 (SENSOR_VN)
- net SENSOR_VP: no longer names the net of U1.4 (SENSOR_VP)
- new net FACTORY: J1.5 (Pin_5), U1.13 (IO14)
- new net VCC_I2C: C41.1, C42.1, R48.1
- new net V_BAT: J1.10 (Pin_10)
- new net V_USB: J1.4 (Pin_4)
Other:
- note added: "I2C ByPass CAPs"
- moved on the sheet: R1, R2, R6, R7, U1

Commit message: update
Parts:
- removed J1: Conn_02x05_Odd_Even, Pin_Headers:Pin_Header_Straight_2x05_Pitch2.54mm, symbol Conn_02x05_Odd_Even
- removed R48: R_10, Resistors_SMD:R_0603, symbol R_10
- removed R49: R_10k, Resistors_SMD:R_0603, symbol R_10k
- added J1: Conn_02x08_Odd_Even, Pin_Headers:Pin_Header_Straight_2x08_Pitch2.54mm, symbol Conn_02x08_Odd_Even
- C41: footprint Capacitors_SMD:C_1206 -> Capacitors_SMD:C_1206_HandSoldering
- C42: footprint Capacitors_SMD:C_0603 -> Capacitors_SMD:C_0603_HandSoldering
- R1, R2, R6, R7: footprint Resistors_SMD:R_0603 -> Resistors_SMD:R_0603_HandSoldering
Connections:
- net VCC_I2C is gone; now on net 3V3: C41.1, C42.1
- net 3V3: now also J1.3 (Pin_3)
- net FACTORY: now also J1.5 (Pin_5)
- net GND: now also J1.1 (Pin_1), J1.2 (Pin_2)
- net I2S_BCLK: now also J1.13 (Pin_13)
- net I2S_WS: now also J1.11 (Pin_11)
- net PIR_HI: now also U1.23 (IO15); no longer U1.33 (IO21)
- net PIR_LO: now also U1.16 (IO13); no longer U1.31 (IO19)
- net PROG: now also J1.7 (Pin_7)
- net RELAY: now also U1.24 (IO2), J1.15 (Pin_15); no longer U1.23 (IO15)
- net RXD: now also J1.8 (Pin_8)
- net SCL: now also U1.33 (IO21), J1.9 (Pin_9); no longer U1.22 (SD1)
- net SDA: now also U1.31 (IO19), J1.10 (Pin_10); no longer U1.21 (SD0)
- net TXD: now also J1.6 (Pin_6)
- net V_BAT: now also J1.16 (Pin_16)
- net V_USB: now also J1.4 (Pin_4)
- net I2S_DATA renamed I2S_DATA_IN
- net I2S_DATA_IN: now also J1.12 (Pin_12)
- net SPEAKER_IN renamed I2S_DATA_OUT
- net I2S_DATA_OUT: now also J1.14 (Pin_14)

Commit message: update
Parts:
- removed C41: C_100uF, Capacitors_SMD:C_1206_HandSoldering, symbol C_100uF
- removed J1: Conn_02x08_Odd_Even, Pin_Headers:Pin_Header_Straight_2x08_Pitch2.54mm, symbol Conn_02x08_Odd_Even
- added C1, C6: C_10uF, Capacitors_SMD:C_0603_HandSoldering, symbol C_10uF
- added C2: C_1uF, Capacitors_SMD:C_0603_HandSoldering, symbol C_1uF
Connections:
- net 3V3: now also C1.1, C2.1, C6.1
- net GND: now also C1.2, C2.2, C6.2
- net PIR1_ADC renamed V_IN
- net PIR2_ADC: no longer names the net of U1.7 (IO35)
- net PIR_HI renamed PIR
- net PIR_LO: no longer names the net of U1.16 (IO13)
Other:
- note added: "I2C PULL-UP"
- note added: "I2S ByPass CAPs"
- moved on the sheet: C42, R1, R2, R6, R7, U1

Commit message: update
Parts:
- C1, C6: symbol C_10uF -> liger-rescue:C_10uF
- C2, C42: symbol C_1uF -> liger-rescue:C_1uF
- R1, R2: symbol R_47.5 -> liger-rescue:R_47.5
- R6, R7: symbol R_10k -> liger-rescue:R_10k
- U1: symbol ESP-WROOM-32 -> liger-rescue:ESP-WROOM-32
Connections:
- net EN is gone; now on net 3V3: U1.3 (EN)
- net IR_RX: now also U1.27 (IO16); no longer U1.26 (IO4)
- net IR_TX: now also U1.26 (IO4); no longer U1.27 (IO16)
- net FACTORY renamed FACTORY_RST
- net V_IN: no longer names the net of U1.6 (IO34)
Changed lines of the file:
@@
-EESchema Schematic File Version 2
-LIBS:power
-LIBS:device
-LIBS:transistors
-LIBS:conn
-LIBS:linear
-LIBS:regul
-LIBS:74xx
-LIBS:cmos4000
-LIBS:adc-dac
-LIBS:memory
-LIBS:xilinx
-LIBS:microcontrollers
-LIBS:dsp
-LIBS:microchip
-LIBS:analog_switches
-LIBS:motorola
-LIBS:texas
-LIBS:intel
-LIBS:audio
-LIBS:interface
-LIBS:digital-audio
-LIBS:philips
-LIBS:display
-LIBS:cypress
-LIBS:siliconi
-LIBS:opto
-LIBS:atmel
-LIBS:contrib
-LIBS:valves
-LIBS:open-automation
+EESchema Schematic File Version 4
 LIBS:liger-cache
-EELAYER 25 0
+EELAYER 26 0
 EELAYER END
 $Descr A4 11693 8268
@@
 $EndDescr
 $Comp
-L GND #PWR01
+L power:GND #PWR01
 U 1 1 59097974
 P 5000 1800
@@
 	-1   0    0    1
 $EndComp
-Text GLabel 4950 3250 0    60   Input ~ 0
-T_DOWN
-Text GLabel 6900 2100 2    60   Input ~ 0
-RXD
-Text GLabel 6900 2750 2    60   Input ~ 0
-LED_G
-Text GLabel 6900 3050 2    60   Input ~ 0
-IR_RX
-Text GLabel 6900 2000 2    60   Input ~ 0
-TXD
-Text GLabel 6900 2950 2    60   Input ~ 0
-IR_TX
-Text GLabel 4950 1950 0    60   Input ~ 0
-3V3
-Text GLabel 6350 3800 3    60   Input ~ 0
-RELAY
-$Comp
-L ESP-WROOM-32 U1
+$Comp
+L liger-rescue:ESP-WROOM-32 U1
 U 1 1 590979AF
 P 5950 2500
@@
 	1    0    0    -1
 $EndComp
-Text GLabel 4950 3050 0    60   Input ~ 0
-T_UP
-Text GLabel 4250 2950 0    60   Input ~ 0
-I2S_BCLK
-Text GLabel 7550 2250 2    60   Input ~ 0
-I2S_WS
-Text GLabel 4950 2750 0    60   Input ~ 0
-T_RIGHT
-Text GLabel 4950 2650 0    60   Input ~ 0
-T_LEFT
-Text GLabel 4950 2450 0    60   Input ~ 0
-V_IN
-Text GLabel 6900 2550 2    60   Input ~ 0
-SDA
-Text GLabel 6900 2450 2    60   Input ~ 0
-SCL
-Text GLabel 6900 2650 2    60   Input ~ 0
-LED_R
-Text GLabel 6900 2350 2    60   Input ~ 0
-I2S_DATA_IN
-Text GLabel 6250 3800 3    60   Input ~ 0
-PIR
-Text GLabel 6900 2850 2    60   Input ~ 0
-LED_B
-Text GLabel 4950 2050 0    60   Input ~ 0
-EN
-Text GLabel 4950 2850 0    60   Input ~ 0
-I2S_DATA_OUT
-$Comp
-L R_10k R6
+$Comp
+L liger-rescue:R_10k R6
 U 1 1 59B92EE3
 P 7050 5175
@@
 $EndComp
 $Comp
-L R_10k R7
+L liger-rescue:R_10k R7
 U 1 1 59B92EEA
 P 6800 5175
@@
 	-1   0    0    1
 $EndComp
-Text GLabel 7050 4875 1    60   Input ~ 0
-3V3
-Text GLabel 7050 5475 3    60   Input ~ 0
-SDA
-Text GLabel 6800 5475 3    60   Input ~ 0
-SCL
-$Comp
-L R_47.5 R2
+$Comp
+L liger-rescue:R_47.5 R2
 U 1 1 59B81C1C
 P 7300 2250
@@
 $EndComp
 $Comp
-L R_47.5 R1
+L liger-rescue:R_47.5 R1
 U 1 1 59B81C70
 P 4500 2950
 F 0 "R1" V 4500 2950 50  0000 C CNN
-F 1 "R_47.5" V 4600 2950 50  0000 C CNN
+F 1 "R_47.5" V 4600 2850 50  0000 C CNN
 F 2 "Resistors_SMD:R_0603_HandSoldering" V 4430 2950 50  0001 C CNN
 F 3 "https://www.digikey.com/product-detail/en/yageo/RC0603FR-0747R5L/311-47.5HRCT-ND/730201" V 4580 2950 50  0001 C CNN
@@
 	0    1    1    0
 $EndComp
-Text GLabel 4950 3150 0    60   Input ~ 0
-FACTORY
-Text GLabel 6900 3150 2    60   Input ~ 0
-PROG
 Text Label 4800 1075 0    197  ~ 0
 Microcontroller
 $Comp
-L C_1uF C42
+L liger-rescue:C_1uF C42
 U 1 1 59C84AF9
 P 6150 5175
@@
 $EndComp
 $Comp
-L GND #PWR02
+L power:GND #PWR02
 U 1 1 59C84AFB
 P 5950 5425
@@
 	1    0    0    -1
 $EndComp
-Text GLabel 5975 4875 1    60   Input ~ 0
-3V3
 Text Notes 5575 5725 0    60   ~ 0
 I2C ByPass CAPs
@@
 	6150 5375 6150 5325
 Wire Wire Line
-	5750 5375 6150 5375
+	5750 5375 5950 5375
 Wire Wire Line
 	5750 5325 5750 5375
@@
 	6250 3700 6250 3800
 Wire Wire Line
-	4950 2450 5050 2450
-Wire Wire Line
 	4950 2650 5050 2650
 Wire Wire Line
@@
 	6800 3150 6900 3150
 Wire Wire Line
-	4950 2050 5050 2050
-Wire Wire Line
-	5050 1950 4950 1950
+	5050 1950 5025 1950
 Wire Wire Line
 	5000 1850 5050 1850
@@
 	5000 1800 5000 1850
 $Comp
-L C_1uF C2
+L liger-rescue:C_1uF C2
 U 1 1 5A1695ED
 P 5075 5175
@@
 $EndComp
 $Comp
-L GND #PWR03
+L power:GND #PWR03
 U 1 1 5A1695EE
 P 4850 5425
@@
 	1    0    0    -1
 $EndComp
-Text GLabel 4875 4875 1    60   Input ~ 0
-3V3
 Text Notes 4475 5775 0    60   ~ 0
 I2S ByPass CAPs
@@
 	4850 5425 4850 5400
 Wire Wire Line
-	5075 5400 4675 5400
+	5075 5400 4850 5400
 Wire Wire Line
 	5075 5325 5075 5400
@@
 	4675 5400 4675 5325
 $Comp
-L C_10uF C1
+L liger-rescue:C_10uF C1
 U 1 1 5A1695F2
 P 4675 5175
@@
 	5075 5025 5075 4950
 Wire Wire Line
-	5075 4950 4675 4950
+	5075 4950 4875 4950
 Wire Wire Line
 	4675 4950 4675 5025
@@
 	5750 5025 5750 4950
 Wire Wire Line
-	5750 4950 6150 4950
+	5750 4950 5975 4950
 Wire Wire Line
 	6150 4950 6150 5025
@@
 Connection ~ 5975 4950
 $Comp
-L C_10uF C6
+L liger-rescue:C_10uF C6
 U 1 1 5A169F88
 P 5750 5175
@@
 Wire Notes Line
 	6400 4625 6400 5750
-Text GLabel 6800 4875 1    60   Input ~ 0
-3V3
 Text Notes 6600 5825 0    60   ~ 0
 I2C PULL-UP
@@
 Wire Notes Line
 	7300 4625 7300 5850
+Wire Wire Line
+	5950 5375 6150 5375
+Wire Wire Line
+	4850 5400 4675 5400
+Wire Wire Line
+	4875 4950 4675 4950
+Wire Wire Line
+	5975 4950 6150 4950
+Text HLabel 4950 1950 0    60   Input ~ 0
+3V3
+Wire Wire Line
+	5050 2050 5025 2050
+Wire Wire Line
+	5025 2050 5025 1950
+Connection ~ 5025 1950
+Wire Wire Line
+	5025 1950 4950 1950
+Text HLabel 4950 2650 0    60   Input ~ 0
+T_LEFT
+Text HLabel 4950 2750 0    60   Input ~ 0
+T_RIGHT
+Text HLabel 4950 2850 0    60   Input ~ 0
+I2S_DATA_OUT
+Text HLabel 4250 2950 0    60   Input ~ 0
+I2S_BCLK
+Text HLabel 4950 3050 0    60   Input ~ 0
+T_UP
+Text HLabel 4950 3150 0    60   Input ~ 0
+FACTORY_RST
+Text HLabel 4950 3250 0    60   Input ~ 0
+T_DOWN
+Text HLabel 6250 3800 3    60   Input ~ 0
+PIR
+Text HLabel 6350 3800 3    60   Input ~ 0
+RELAY
+Text HLabel 6900 3150 2    60   Input ~ 0
+PROG
+Text HLabel 6900 3050 2    60   Output ~ 0
+IR_TX
+Text HLabel 6900 2950 2    60   Input ~ 0
+IR_RX
+Text HLabel 6900 2850 2    60   Output ~ 0
+LED_B
+Text HLabel 6900 2750 2    60   Output ~ 0
+LED_G
+Text HLabel 6900 2650 2    60   Output ~ 0
+LED_R
+Text HLabel 6900 2550 2    60   BiDi ~ 0
+SDA
+Text HLabel 6900 2450 2    60   Output ~ 0
+SCL
+Text HLabel 6900 2350 2    60   Input ~ 0
+I2S_DATA_IN
+Text HLabel 7550 2250 2    60   Input ~ 0
+I2S_WS
+Text HLabel 6900 2100 2    60   Input ~ 0
+RXD
+Text HLabel 6900 2000 2    60   Input ~ 0
+TXD
+Text HLabel 4875 4875 1    60   Input ~ 0
+3V3
+Text HLabel 5975 4875 1    60   Input ~ 0
+3V3
+Text HLabel 6800 4875 1    60   Input ~ 0
+3V3
+Text HLabel 7050 4875 1    60   Input ~ 0
+3V3
+Text HLabel 6800 5475 3    60   Output ~ 0
+SCL
+Text HLabel 7050 5475 3    60   BiDi ~ 0
+SDA
 $EndSCHEMATC
