File: hardware/power.sch (KiCad schematic (older format))
At the start: 5 parts, among them P4 CONN_01X03, U5 SPX3819

Commit message: update
Parts:
- C3, C4: value 1uf -> 1uF
- U5: Part Number SPX3819 -> 1016-1873-1-ND
Changed lines of the file:
@@
 F 1 "SPX3819" H 6350 4050 50  0000 C CNN
 F 2 "TO_SOT_Packages_SMD:SOT-23-5" H 6200 3300 50  0001 C CIN
-F 3 "http://www.mouser.com/ds/2/146/SPX3819_DS_R200_082312-17072.pdf" H 6250 3200 50  0001 C CNN
-F 4 "SPX3819" H 6200 3700 60  0001 C CNN "Part Number"
+F 3 "https://www.exar.com/content/document.ashx?id=22106" H 6250 3200 50  0001 C CNN
+F 4 "1016-1873-1-ND" H 6200 3700 60  0001 C CNN "Part Number"
 	1    6200 3700
 	1    0    0    -1
@@
 P 4650 3950
 F 0 "C3" H 4675 4050 50  0000 L CNN
-F 1 "1uf" H 4675 3850 50  0000 L CNN
+F 1 "1uF" H 4675 3850 50  0000 L CNN
 F 2 "Capacitors_SMD:C_0603_HandSoldering" H 4688 3800 50  0001 C CNN
 F 3 "http://www.yageo.com/documents/recent/UPY-GPHC_Y5V_6.3V-to-50V_6.pdf" H 4650 3950 50  0001 C CNN
@@
 P 6700 3700
 F 0 "C4" H 6725 3800 50  0000 L CNN
-F 1 "1uf" H 6725 3600 50  0000 L CNN
+F 1 "1uF" H 6725 3600 50  0000 L CNN
 F 2 "Capacitors_SMD:C_0603_HandSoldering" H 6738 3550 50  0001 C CNN
 F 3 "http://www.yageo.com/documents/recent/UPY-GPHC_Y5V_6.3V-to-50V_6.pdf" H 6700 3700 50  0001 C CNN

Commit message: updatge
Parts:
- P4: footprint footprints:connector_3pos_KR -> Pin_Headers:Pin_Header_Straight_1x03_Pitch2.54mm
Changed lines of the file:
@@
 $EndComp
 $Comp
-L GND #PWR16
+L GND #PWR015
 U 1 1 5909DD65
 P 5200 4250
-F 0 "#PWR16" H 5200 4000 50  0001 C CNN
+F 0 "#PWR015" H 5200 4000 50  0001 C CNN
 F 1 "GND" H 5200 4100 50  0000 C CNN
 F 2 "" H 5200 4250 50  0000 C CNN
@@
 $EndComp
 $Comp
-L GND #PWR15
+L GND #PWR016
 U 1 1 5909DD66
 P 4650 4300
-F 0 "#PWR15" H 4650 4050 50  0001 C CNN
+F 0 "#PWR016" H 4650 4050 50  0001 C CNN
 F 1 "GND" H 4650 4150 50  0000 C CNN
 F 2 "" H 4650 4300 50  0000 C CNN
@@
 $EndComp
 $Comp
-L GND #PWR18
+L GND #PWR017
 U 1 1 5909DD67
 P 6700 4050
-F 0 "#PWR18" H 6700 3800 50  0001 C CNN
+F 0 "#PWR017" H 6700 3800 50  0001 C CNN
 F 1 "GND" H 6700 3900 50  0000 C CNN
 F 2 "" H 6700 4050 50  0000 C CNN
@@
 F 0 "P4" H 6100 4700 50  0000 L CNN
 F 1 "CONN_01X03" V 6300 4250 50  0001 L CNN
-F 2 "footprints:connector_3pos_KR" H 6200 4500 50  0001 C CNN
+F 2 "Pin_Headers:Pin_Header_Straight_1x03_Pitch2.54mm" H 6200 4500 50  0001 C CNN
 F 3 "http://www.digikey.com/product-detail/en/hirose-electric-co-ltd/DF13C-3P-1.25V(21)/H121960CT-ND/3907735" H 6200 4500 50  0001 C CNN
 F 4 "A04KR04DA28W51B" H 6200 4500 60  0001 C CNN "Part Number"
@@
 $EndComp
 $Comp
-L GND #PWR17
+L GND #PWR018
 U 1 1 5909DD7D
 P 5950 4350
-F 0 "#PWR17" H 5950 4100 50  0001 C CNN
+F 0 "#PWR018" H 5950 4100 50  0001 C CNN
 F 1 "GND" H 5950 4200 50  0000 C CNN
 F 2 "" H 5950 4350 50  0000 C CNN

Commit message: update
Parts:
- removed R11: 10K, Resistors_SMD:R_0603_HandSoldering, symbol R
- removed U5: SPX3819, TO_SOT_Packages_SMD:SOT-23-5, symbol SPX3819
- added U11: SPX1117M3-L-3-3/TR, open-automation:SOT-223_CORRECTED, symbol SPX1117M3-L-3-3/TR
- P4: footprint Pin_Headers:Pin_Header_Straight_1x03_Pitch2.54mm -> open-automation:Pin_Header_Straight_1x03_Pitch2.54mm_CORRECTED
Connections:
- net 3V3: now also U11.2 (Vout)
- net 5V: now also U11.3 (Vin)
- net GND: now also U11.1 (GND)
Other:
- moved on the sheet: C3, C4
Changed lines of the file:
@@
 LIBS:open-automation
 LIBS:liger-cache
-EELAYER 26 0
+EELAYER 25 0
 EELAYER END
 $Descr A4 11693 8268
@@
 $EndDescr
 $Comp
-L SPX3819 U5
-U 1 1 5909DD63
-P 6200 3700
-F 0 "U5" H 5950 4050 50  0000 C CNN
-F 1 "SPX3819" H 6350 4050 50  0000 C CNN
-F 2 "TO_SOT_Packages_SMD:SOT-23-5" H 6200 3300 50  0001 C CIN
-F 3 "https://www.exar.com/content/document.ashx?id=22106" H 6250 3200 50  0001 C CNN
-F 4 "1016-1873-1-ND" H 6200 3700 60  0001 C CNN "Part Number"
-	1    6200 3700
-	1    0    0    -1
-$EndComp
-$Comp
 L C C3
 U 1 1 5909DD64
-P 4650 3950
-F 0 "C3" H 4675 4050 50  0000 L CNN
-F 1 "1uF" H 4675 3850 50  0000 L CNN
-F 2 "Capacitors_SMD:C_0603_HandSoldering" H 4688 3800 50  0001 C CNN
-F 3 "http://www.yageo.com/documents/recent/UPY-GPHC_Y5V_6.3V-to-50V_6.pdf" H 4650 3950 50  0001 C CNN
-F 4 "CC0603ZRY5V7BB105" H 4650 3950 60  0001 C CNN "Part Number"
-	1    4650 3950
+P 4950 3150
+F 0 "C3" H 4975 3250 50  0000 L CNN
+F 1 "1uF" H 4975 3050 50  0000 L CNN
+F 2 "Capacitors_SMD:C_0603_HandSoldering" H 4988 3000 50  0001 C CNN
+F 3 "http://www.yageo.com/documents/recent/UPY-GPHC_Y5V_6.3V-to-50V_6.pdf" H 4950 3150 50  0001 C CNN
+F 4 "CC0603ZRY5V7BB105" H 4950 3150 60  0001 C CNN "Part Number"
+	1    4950 3150
 	1    0    0    -1
 $EndComp
 $Comp
 L GND #PWR015
-U 1 1 5909DD65
-P 5200 4250
-F 0 "#PWR015" H 5200 4000 50  0001 C CNN
-F 1 "GND" H 5200 4100 50  0000 C CNN
-F 2 "" H 5200 4250 50  0000 C CNN
-F 3 "" H 5200 4250 50  0000 C CNN
-	1    5200 4250
+U 1 1 5909DD67
+P 6150 3400
+F 0 "#PWR015" H 6150 3150 50  0001 C CNN
+F 1 "GND" H 6150 3250 50  0000 C CNN
+F 2 "" H 6150 3400 50  0000 C CNN
+F 3 "" H 6150 3400 50  0000 C CNN
+	1    6150 3400
 	1    0    0    -1
-$EndComp
-$Comp
-L GND #PWR016
-U 1 1 5909DD66
-P 4650 4300
-F 0 "#PWR016" H 4650 4050 50  0001 C CNN
-F 1 "GND" H 4650 4150 50  0000 C CNN
-F 2 "" H 4650 4300 50  0000 C CNN
-F 3 "" H 4650 4300 50  0000 C CNN
-	1    4650 4300
-	1    0    0    -1
-$EndComp
-$Comp
-L GND #PWR017
-U 1 1 5909DD67
-P 6700 4050
-F 0 "#PWR017" H 6700 3800 50  0001 C CNN
-F 1 "GND" H 6700 3900 50  0000 C CNN
-F 2 "" H 6700 4050 50  0000 C CNN
-F 3 "" H 6700 4050 50  0000 C CNN
-	1    6700 4050
-	1    0    0    -1
-$EndComp
-Text Label 5550 3000 0    60   ~ 0
-Regulator
-$Comp
-L R R11
-U 1 1 5909DD71
-P 5050 3950
-F 0 "R11" V 5130 3950 50  0000 C CNN
-F 1 "10K" V 5050 3950 50  0000 C CNN
-F 2 "Resistors_SMD:R_0603_HandSoldering" V 4980 3950 50  0001 C CNN
-F 3 "http://www.digikey.com/en/resources/datasheets/yageo/rc-series-l-suffix-datasheet" H 5050 3950 50  0001 C CNN
-F 4 "RC0603JR-0710KL" V 5050 3950 60  0001 C CNN "Part Number"
-	1    5050 3950
-	-1   0    0    1
 $EndComp
 $Comp
 L C C4
 U 1 1 5909DD72
-P 6700 3700
-F 0 "C4" H 6725 3800 50  0000 L CNN
-F 1 "1uF" H 6725 3600 50  0000 L CNN
-F 2 "Capacitors_SMD:C_0603_HandSoldering" H 6738 3550 50  0001 C CNN
-F 3 "http://www.yageo.com/documents/recent/UPY-GPHC_Y5V_6.3V-to-50V_6.pdf" H 6700 3700 50  0001 C CNN
-F 4 "CC0603ZRY5V7BB105" H 6700 3700 60  0001 C CNN "Part Number"
-	1    6700 3700
+P 6150 3200
+F 0 "C4" H 6175 3300 50  0000 L CNN
+F 1 "1uF" H 6175 3100 50  0000 L CNN
+F 2 "Capacitors_SMD:C_0603_HandSoldering" H 6188 3050 50  0001 C CNN
+F 3 "http://www.yageo.com/documents/recent/UPY-GPHC_Y5V_6.3V-to-50V_6.pdf" H 6150 3200 50  0001 C CNN
+F 4 "CC0603ZRY5V7BB105" H 6150 3200 60  0001 C CNN "Part Number"
+	1    6150 3200
 	1    0    0    -1
 $EndComp
@@
 F 0 "P4" H 6100 4700 50  0000 L CNN
 F 1 "CONN_01X03" V 6300 4250 50  0001 L CNN
-F 2 "Pin_Headers:Pin_Header_Straight_1x03_Pitch2.54mm" H 6200 4500 50  0001 C CNN
+F 2 "open-automation:Pin_Header_Straight_1x03_Pitch2.54mm_CORRECTED" H 6200 4500 50  0001 C CNN
 F 3 "http://www.digikey.com/product-detail/en/hirose-electric-co-ltd/DF13C-3P-1.25V(21)/H121960CT-ND/3907735" H 6200 4500 50  0001 C CNN
 F 4 "A04KR04DA28W51B" H 6200 4500 60  0001 C CNN "Part Number"
@@
 $EndComp
 $Comp
-L GND #PWR018
+L GND #PWR016
 U 1 1 5909DD7D
 P 5950 4350
-F 0 "#PWR018" H 5950 4100 50  0001 C CNN
+F 0 "#PWR016" H 5950 4100 50  0001 C CNN
 F 1 "GND" H 5950 4200 50  0000 C CNN
 F 2 "" H 5950 4350 50  0000 C CNN
@@
 Text GLabel 5900 4500 0    60   Input ~ 0
 IO15
-Wire Wire Line
-	6700 3850 6700 4050
-Wire Wire Line
-	4650 4100 4650 4300
-Connection ~ 5650 3500
-Wire Wire Line
-	5650 3500 5650 3900
-Wire Wire Line
-	5650 3900 5800 3900
-Connection ~ 5200 4200
-Wire Wire Line
-	5200 4200 5200 4250
-Wire Wire Line
-	5050 4200 5050 4100
-Wire Wire Line
-	5050 4200 5400 4200
-Wire Wire Line
-	5400 4200 5400 3700
-Wire Wire Line
-	5400 3700 5800 3700
-Connection ~ 4650 3500
-Connection ~ 5050 3500
-Wire Wire Line
-	5050 3800 5050 3500
-Wire Wire Line
-	4650 3500 5800 3500
-Connection ~ 6700 3500
-Wire Wire Line
-	6700 3300 6700 3550
-Wire Wire Line
-	4650 3250 4650 3800
+Text GLabel 6350 3050 2    60   Input ~ 0
+3V3
+Text GLabel 5950 4650 3    60   Input ~ 0
+5V
+$Comp
+L SPX1117M3-L-3-3/TR U11
+U 1 1 59A4B87F
+P 5650 3050
+F 0 "U11" H 5750 2750 50  0000 C CNN
+F 1 "SPX1117M3-L-3-3/TR" H 5650 3300 50  0000 C CNN
+F 2 "open-automation:SOT-223_CORRECTED" H 5650 2650 50  0001 C CIN
+F 3 "https://www.digikey.com/product-detail/en/exar-corporation/SPX1117M3-L-3-3-TR/1016-1848-1-ND/3586565" H 5700 2550 50  0001 C CNN
+F 4 "SPX1117M3-L-3-3/TR" H 5850 2850 60  0001 C CNN "Part Number"
+	1    5650 3050
+	1    0    0    -1
+$EndComp
+$Comp
+L GND #PWR017
+U 1 1 59A4BA1C
+P 5200 3200
+F 0 "#PWR017" H 5200 2950 50  0001 C CNN
+F 1 "GND" H 5200 3050 50  0000 C CNN
+F 2 "" H 5200 3200 50  0000 C CNN
+F 3 "" H 5200 3200 50  0000 C CNN
+	1    5200 3200
+	1    0    0    -1
+$EndComp
+$Comp
+L GND #PWR018
+U 1 1 59A4BAA9
+P 4950 3350
+F 0 "#PWR018" H 4950 3100 50  0001 C CNN
+F 1 "GND" H 4950 3200 50  0000 C CNN
+F 2 "" H 4950 3350 50  0000 C CNN
+F 3 "" H 4950 3350 50  0000 C CNN
+	1    4950 3350
+	1    0    0    -1
+$EndComp
+Text Label 4600 2450 0    60   ~ 0
+Regulator
 Wire Wire Line
 	5950 4350 5950 4400
@@
 	5900 4500 6000 4500
 Wire Wire Line
-	6600 3500 6700 3500
-Text GLabel 4650 3250 1    60   Input ~ 0
+	6000 3050 6350 3050
+Wire Wire Line
+	6150 3400 6150 3350
+Wire Wire Line
+	5200 3200 5200 3150
+Wire Wire Line
+	5200 3150 5250 3150
+Wire Wire Line
+	4950 3000 4950 2950
+Wire Wire Line
+	4800 2950 5250 2950
+Wire Wire Line
+	4950 3350 4950 3300
+Connection ~ 6150 3050
+Text GLabel 4800 2950 0    60   Input ~ 0
 5V
-Text GLabel 6700 3300 1    60   Input ~ 0
-3V3
-Text GLabel 5950 4650 3    60   Input ~ 0
-5V
+Connection ~ 4950 2950
 $EndSCHEMATC

Commit message: update
Parts:
- removed C3, C4: 1uF, Capacitors_SMD:C_0603_HandSoldering, symbol C
- removed P4: CONN_01X03, open-automation:Pin_Header_Straight_1x03_Pitch2.54mm_CORRECTED, symbol CONN_01X03
- removed U11: SPX1117M3-L-3-3/TR, open-automation:SOT-223_CORRECTED, symbol SPX1117M3-L-3-3/TR
- added BT1: 18650_Battery_Cell_1043, symbol 18650_Battery_Cell_1043
- added C10, C11, C12, C19, C3, C4: C_1uF, Capacitors_SMD:C_0603, symbol C_1uF
- added C13, C14, C15, C16, C18, C20, C21, C22: C_0.1uF, Capacitors_SMD:C_0603, symbol C_0.1uF
- added C17, C2, C8, C9: C_100uF, Capacitors_SMD:C_1206, symbol C_100uF
- added D3: LED-GREEN-LTST-C191GKT, LEDs:LED_0603, symbol LED-GREEN-LTST-C191GKT
- added Q4: PMOS-DMG3413L, TO_SOT_Packages_SMD:SOT-23, symbol PMOS-DMG3413L
- added R10: R_1k, Resistors_SMD:R_0603, symbol R_1k
- added R11, R17, R18, R23, R24: R_10, Resistors_SMD:R_0603, symbol R_10
- added R19: R_2k, Resistors_SMD:R_0603, symbol R_2k
- added R22: R_10k, Resistors_SMD:R_0603, symbol R_10k
- added U18: AZ1117E, TO_SOT_Packages_SMD:SOT-223, symbol AZ1117E
- added U4: MCP73831T, TO_SOT_Packages_SMD:SOT-23-5, symbol MCP73831T
Connections:
- net 3V3: now also C4.1, R11.2, R17.2, R18.2, R23.2, R24.2, U18.2 (Vout)
- net GND: now also BT1.2 (-), C10.2, C11.2, C12.2, C13.2, C14.2, C15.2, C16.2, C17.2, C18.2, C19.2, C2.2, C20.2, C21.2, C22.2, C3.2, C4.2, C8.2, C9.2, R19.1, R22.2, U18.1 (GND), U4.2 (GND)
- new net: D3.2 (A), R10.2
- new net: D3.1 (K), U4.1 (STAT)
- new net: R19.2, U4.5 (PROG)
- new net VCC_COMP: C18.1, C20.1, C21.1, C22.1, R23.1
- new net VCC_I2C: C12.1, C9.1, R18.1
- new net VCC_I2S: C17.1, C19.1, R24.1
- new net VCC_PIR1: C10.1, C13.1, C15.1, C2.1, R11.1
- new net VCC_PIR2: C11.1, C14.1, C16.1, C8.1, R17.1
- new net V_BAT: BT1.1 (+), Q4.2 (S), U4.3 (Vbat)
- new net V_USB: C3.1, Q4.1 (G), Q4.3 (D), R10.1, R22.1, U18.3 (Vin), U4.4 (Vin)
Other:
- note added: "ByPass CAPs for comparator OPAMPs"
- note added: "I2C ByPass CAPs"
- note added: "I2S ByPass CAPs"
- note added: "PIR1 ByPass CAPs"
- note added: "PIR1 OPAMP"
- note added: "PIR2 ByPass CAPs"
- note added: "PIR2 OPAMP"
