File: hardware/power.sch (KiCad schematic (older format))
At the start: 31 parts, among them Q4 PMOS-DMG3413L, U18 AZ1117E, U4 MCP73831T

Commit message: update
Parts:
- removed C10, C11, C12, C19: C_1uF, Capacitors_SMD:C_0603, symbol C_1uF
- removed C13, C14, C15, C16, C18, C20, C21, C22: C_0.1uF, Capacitors_SMD:C_0603, symbol C_0.1uF
- removed C17, C2, C8, C9: C_100uF, Capacitors_SMD:C_1206, symbol C_100uF
- removed R11, R17, R18, R23, R24: R_10, Resistors_SMD:R_0603, symbol R_10
Other:
- note removed: "ByPass CAPs for comparator OPAMPs"
- note removed: "I2C ByPass CAPs"
- note removed: "I2S ByPass CAPs"
- note removed: "PIR1 ByPass CAPs"
- note removed: "PIR1 OPAMP"
- note removed: "PIR2 ByPass CAPs"
- note removed: "PIR2 OPAMP"
- moved on the sheet: BT1, C3, C4, D3, Q4, R10, R19, R22, U18, U4

Commit message: update
Parts:
- U18: footprint TO_SOT_Packages_SMD:SOT-223 -> open-automation:SPX1117M3
- U4: Part Number MCP73831T -> MCP73831T-2ACI/OT
Changed lines of the file:
@@
 $EndDescr
 $Comp
-L GND #PWR08
+L GND #PWR012
 U 1 1 5909DD67
 P 7950 4400
-F 0 "#PWR08" H 7950 4150 50  0001 C CNN
+F 0 "#PWR012" H 7950 4150 50  0001 C CNN
 F 1 "GND" H 7950 4250 50  0000 C CNN
 F 2 "" H 7950 4400 50  0000 C CNN
@@
 3V3
 $Comp
-L GND #PWR09
+L GND #PWR013
 U 1 1 59A4BA1C
 P 7000 4100
-F 0 "#PWR09" H 7000 3850 50  0001 C CNN
+F 0 "#PWR013" H 7000 3850 50  0001 C CNN
 F 1 "GND" H 7000 3950 50  0000 C CNN
 F 2 "" H 7000 4100 50  0000 C CNN
@@
 $EndComp
 $Comp
-L GND #PWR010
+L GND #PWR014
 U 1 1 59A4BAA9
 P 6750 4250
-F 0 "#PWR010" H 6750 4000 50  0001 C CNN
+F 0 "#PWR014" H 6750 4000 50  0001 C CNN
 F 1 "GND" H 6750 4100 50  0000 C CNN
 F 2 "" H 6750 4250 50  0000 C CNN
@@
 F 2 "TO_SOT_Packages_SMD:SOT-23-5" H 3500 3500 60  0001 C CNN
 F 3 "https://www.digikey.com/product-detail/en/microchip-technology/MCP73831T-2ACI-OT/MCP73831T-2ACI-OTCT-ND/1979802" H 3750 3400 60  0001 C CNN
-F 4 "MCP73831T" H 3200 4100 60  0001 C CNN "Part Number"
+F 4 "MCP73831T-2ACI/OT" H 3200 4100 60  0001 C CNN "Part Number"
 	1    3250 3800
 	1    0    0    -1
 $EndComp
 $Comp
-L GND #PWR011
+L GND #PWR015
 U 1 1 59B41D6D
 P 3900 4200
-F 0 "#PWR011" H 3900 3950 50  0001 C CNN
+F 0 "#PWR015" H 3900 3950 50  0001 C CNN
 F 1 "GND" H 3900 4050 50  0000 C CNN
 F 2 "" H 3900 4200 50  0000 C CNN
@@
 $EndComp
 $Comp
-L GND #PWR012
+L GND #PWR016
 U 1 1 59B57C4B
 P 4200 4200
-F 0 "#PWR012" H 4200 3950 50  0001 C CNN
+F 0 "#PWR016" H 4200 3950 50  0001 C CNN
 F 1 "GND" H 4200 4050 50  0000 C CNN
 F 2 "" H 4200 4200 50  0000 C CNN
@@
 V_USB
 $Comp
-L GND #PWR013
+L GND #PWR017
 U 1 1 59B58DE3
 P 4950 4200
-F 0 "#PWR013" H 4950 3950 50  0001 C CNN
+F 0 "#PWR017" H 4950 3950 50  0001 C CNN
 F 1 "GND" H 4950 4050 50  0000 C CNN
 F 2 "" H 4950 4200 50  0000 C CNN
@@
 	3700 3800 3900 3800
 $Comp
-L AZ1117E U18
-U 1 1 59B9CD6B
-P 7450 3950
-F 0 "U18" H 7600 3750 50  0000 C CNN
-F 1 "AZ1117E" H 7400 4150 50  0000 C CNN
-F 2 "TO_SOT_Packages_SMD:SOT-223" H 7450 3550 50  0001 C CIN
-F 3 "https://www.digikey.com/product-detail/en/diodes-incorporated/AZ1117EH-3.3TRG1/AZ1117EH-3.3TRG1DICT-ND/5001336" H 7500 3450 50  0001 C CNN
-F 4 "AZ1117EH-3.3TRG1" H 7650 3750 60  0001 C CNN "Part Number"
-	1    7450 3950
-	1    0    0    -1
-$EndComp
-$Comp
 L C_1uF C3
 U 1 1 59BA119E
@@
 	1    0    0    -1
 $EndComp
+$Comp
+L AZ1117E U18
+U 1 1 59C9F39B
+P 7450 3950
+F 0 "U18" H 7550 3650 50  0000 C CNN
+F 1 "AZ1117E" H 7400 4150 50  0000 C CNN
+F 2 "open-automation:SPX1117M3" H 7450 3550 50  0001 C CIN
+F 3 "https://www.digikey.com/product-detail/en/diodes-incorporated/AZ1117EH-3.3TRG1/AZ1117EH-3.3TRG1DICT-ND/5001336" H 7500 3450 50  0001 C CNN
+F 4 "AZ1117EH-3.3TRG1" H 7650 3750 60  0001 C CNN "Part Number"
+	1    7450 3950
+	1    0    0    -1
+$EndComp

Commit message: update
Parts:
- added C5: C_1uF, Capacitors_SMD:C_0603_HandSoldering, symbol C_1uF
- added D6: D_Schottky-BAT20JFILM, Diodes_SMD:D_SOD-323_HandSoldering, symbol D_Schottky-BAT20JFILM
- C3, C4: footprint Capacitors_SMD:C_0603 -> Capacitors_SMD:C_0603_HandSoldering
- D3: footprint LEDs:LED_0603 -> LEDs:LED_0603_HandSoldering
- R10, R19, R22: footprint Resistors_SMD:R_0603 -> Resistors_SMD:R_0603_HandSoldering
Connections:
- net GND: now also C5.2
- net V_BAT: now also Q4.3 (D), C5.1; no longer Q4.2 (S)
- net V_USB: now also D6.2 (A); no longer C3.1, Q4.3 (D), U18.3 (Vin)
- new net V_IN: C3.1, D6.1 (K), Q4.2 (S), U18.3 (Vin)
Other:
- moved on the sheet: BT1, C3, C4, D3, Q4, R10, R19, R22, U18, U4

Commit message: update
Parts:
- removed U18: AZ1117E, open-automation:SPX1117M3, symbol AZ1117E
- added U9: AP2112, TO_SOT_Packages_SMD:SOT-23-5, symbol AP2112
Connections:
- net 3V3: now also U9.5 (VOUT)
- net GND: now also U9.2 (GND)
- net V_IN: now also U9.1 (Vin), U9.3 (EN)
Other:
- moved on the sheet: BT1, C3, C4, C5, D3, D6, Q4, R10, R19, R22, U4

Commit message: update
Parts:
- BT1: symbol 18650_Battery_Cell_1043 -> liger-rescue:18650_Battery_Cell_1043
- C3, C4, C5: symbol C_1uF -> liger-rescue:C_1uF
- D3: symbol LED-GREEN-LTST-C191GKT -> liger-rescue:LED-GREEN-LTST-C191GKT
- D6: symbol D_Schottky-BAT20JFILM -> liger-rescue:D_Schottky-BAT20JFILM
- Q4: symbol PMOS-DMG3413L -> liger-rescue:PMOS-DMG3413L
- R10: symbol R_1k -> liger-rescue:R_1k
- R19: symbol R_2k -> liger-rescue:R_2k
- R22: symbol R_10k -> liger-rescue:R_10k
- U4: symbol MCP73831T -> liger-rescue:MCP73831T
- U9: symbol AP2112 -> liger-rescue:AP2112
Changed lines of the file:
@@
-EESchema Schematic File Version 2
-LIBS:power
-LIBS:device
-LIBS:transistors
-LIBS:conn
-LIBS:linear
-LIBS:regul
-LIBS:74xx
-LIBS:cmos4000
-LIBS:adc-dac
-LIBS:memory
-LIBS:xilinx
-LIBS:microcontrollers
-LIBS:dsp
-LIBS:microchip
-LIBS:analog_switches
-LIBS:motorola
-LIBS:texas
-LIBS:intel
-LIBS:audio
-LIBS:interface
-LIBS:digital-audio
-LIBS:philips
-LIBS:display
-LIBS:cypress
-LIBS:siliconi
-LIBS:opto
-LIBS:atmel
-LIBS:contrib
-LIBS:valves
-LIBS:open-automation
+EESchema Schematic File Version 4
 LIBS:liger-cache
-EELAYER 25 0
+EELAYER 26 0
 EELAYER END
 $Descr A4 11693 8268
@@
 $EndDescr
 $Comp
-L GND #PWR012
+L power:GND #PWR012
 U 1 1 5909DD67
 P 5125 3875
@@
 $EndComp
 $Comp
-L GND #PWR013
+L power:GND #PWR013
 U 1 1 59A4BAA9
 P 3500 3850
@@
 Power
 $Comp
-L R_1k R10
+L liger-rescue:R_1k R10
 U 1 1 59B41A3B
 P 6575 3450
@@
 $EndComp
 $Comp
-L MCP73831T U4
+L liger-rescue:MCP73831T U4
 U 1 1 59B41D1D
 P 7325 3550
@@
 $EndComp
 $Comp
-L GND #PWR014
+L power:GND #PWR014
 U 1 1 59B41D6D
 P 7975 3950
@@
 	1    0    0    -1
 $EndComp
-Text GLabel 8125 3250 1    60   Input ~ 0
-V_BAT
-$Comp
-L PMOS-DMG3413L Q4
+$Comp
+L liger-rescue:PMOS-DMG3413L Q4
 U 1 1 59B57188
 P 3400 3125
@@
 $EndComp
 $Comp
-L GND #PWR015
+L power:GND #PWR015
 U 1 1 59B57C4B
 P 8275 3950
@@
 $EndComp
 $Comp
-L LED-GREEN-LTST-C191GKT D3
+L liger-rescue:LED-GREEN-LTST-C191GKT D3
 U 1 1 59B58167
 P 6375 3650
@@
 	0    -1   -1   0
 $EndComp
-Text GLabel 6775 3150 1    60   Input ~ 0
-V_USB
-$Comp
-L GND #PWR016
+$Comp
+L power:GND #PWR016
 U 1 1 59B58DE3
 P 2975 3925
@@
 $EndComp
 $Comp
-L R_10k R22
+L liger-rescue:R_10k R22
 U 1 1 59B5A0F4
 P 2975 3700
@@
 $EndComp
 $Comp
-L R_2k R19
+L liger-rescue:R_2k R19
 U 1 1 59B5A181
 P 7975 3700
@@
 	-1   0    0    1
 $EndComp
-Text GLabel 2775 3450 0    60   Input ~ 0
-V_USB
-$Comp
-L C_1uF C3
+$Comp
+L liger-rescue:C_1uF C3
 U 1 1 59BA119E
 P 3500 3650
@@
 $EndComp
 $Comp
-L C_1uF C4
+L liger-rescue:C_1uF C4
 U 1 1 59BA1591
 P 5125 3675
@@
 $EndComp
 $Comp
-L 18650_Battery_Cell_1043 BT1
+L liger-rescue:18650_Battery_Cell_1043 BT1
 U 1 1 59BA3E14
 P 8275 3750
+AR Path="/59BA3E14" Ref="BT1"  Part="1"
+AR Path="/5909D8E3/59BA3E14" Ref="BT1"  Part="1"
 F 0 "BT1" H 8375 3850 50  0000 L CNN
 F 1 "18650_Battery_Cell_1043" H 8375 3750 50  0001 L CNN
@@
 $EndComp
 $Comp
-L D_Schottky-BAT20JFILM D6
+L liger-rescue:D_Schottky-BAT20JFILM D6
 U 1 1 59EBB5BE
 P 3200 3450
@@
 	-1   0    0    1
 $EndComp
-Text GLabel 3500 2800 1    60   Input ~ 0
-V_BAT
 Wire Wire Line
 	3500 2800 3500 2925
 Connection ~ 2975 3450
 Wire Wire Line
-	2775 3450 3050 3450
+	2775 3450 2975 3450
 Wire Wire Line
 	2975 3925 2975 3850
@@
 	7825 3900 7975 3900
 Wire Wire Line
-	7975 3850 7975 3950
+	7975 3850 7975 3900
 Connection ~ 8125 3450
 Connection ~ 6775 3450
@@
 	6425 3450 6375 3450
 Wire Wire Line
-	6825 3450 6725 3450
+	6825 3450 6775 3450
 Wire Wire Line
 	8125 3250 8125 3450
 Wire Wire Line
-	7775 3450 8700 3450
+	7775 3450 8125 3450
 Wire Wire Line
 	6725 3650 6825 3650
@@
 	3500 3850 3500 3800
 Wire Wire Line
-	3350 3450 3900 3450
-Wire Wire Line
-	3500 3325 3500 3500
+	3350 3450 3500 3450
+Wire Wire Line
+	3500 3325 3500 3450
 Wire Wire Line
 	5125 3875 5125 3825
 $Comp
-L C_1uF C5
+L liger-rescue:C_1uF C5
 U 1 1 59EBD4F3
 P 8700 3700
@@
 Connection ~ 8275 3450
 $Comp
-L GND #PWR017
+L power:GND #PWR017
 U 1 1 59EBD5C7
 P 8700 3950
@@
 Wire Wire Line
 	8700 3950 8700 3850
-Text GLabel 3075 3125 0    60   Input ~ 0
-V_USB
 Wire Wire Line
 	3075 3125 3200 3125
@@
 	2975 3550 2975 3450
 $Comp
-L AP2112 U9
+L liger-rescue:AP2112 U9
 U 1 1 5A164E45
 P 4350 3525
@@
 $EndComp
 $Comp
-L GND #PWR018
+L power:GND #PWR018
 U 1 1 5A1650D9
 P 4850 3650
@@
 	5125 3450 5125 3525
 Wire Wire Line
-	4800 3450 5250 3450
+	4800 3450 5125 3450
 Wire Wire Line
 	3850 3600 3900 3600
 Wire Wire Line
-	3850 3300 3850 3600
+	3850 3300 3850 3450
 Connection ~ 3850 3450
-Text GLabel 5250 3450 2    60   Input ~ 0
+Connection ~ 5125 3450
+Wire Wire Line
+	2975 3450 3050 3450
+Wire Wire Line
+	7975 3900 7975 3950
+Wire Wire Line
+	8125 3450 8275 3450
+Wire Wire Line
+	6775 3450 6725 3450
+Wire Wire Line
+	3500 3450 3850 3450
+Wire Wire Line
+	3500 3450 3500 3500
+Wire Wire Line
+	8275 3450 8700 3450
+Wire Wire Line
+	3850 3450 3850 3600
+Wire Wire Line
+	3850 3450 3900 3450
+Wire Wire Line
+	5125 3450 5250 3450
+Text HLabel 3500 2800 1    60   Input ~ 0
+V_BAT
+Text HLabel 3075 3125 0    60   Input ~ 0
+V_USB
+Text HLabel 2775 3450 0    60   Input ~ 0
+V_USB
+Text HLabel 3850 3300 1    60   Input ~ 0
+V_IN
+Text HLabel 5250 3450 2    60   Output ~ 0
 3V3
-Connection ~ 5125 3450
-Text GLabel 3850 3300 1    60   Input ~ 0
-V_IN
+Text HLabel 6775 3150 1    60   Input ~ 0
+V_USB
+Text HLabel 8125 3250 1    60   Input ~ 0
+V_BAT
 $EndSCHEMATC

Commit message: updated schematic
Parts:
- removed C3, C4, C5: C_1uF, Capacitors_SMD:C_0603_HandSoldering, symbol liger-rescue:C_1uF
- added C7, C8, C9: C_1uF, Capacitor_SMD:C_0603_1608Metric_Pad0.99x1.00mm_HandSolder, symbol open-automation:C_1uF
- BT1: footprint (none) -> Battery:BatteryHolder_Keystone_1042_1x18650
Connections:
- net 3V3: now also C8.1
- net GND: now also C7.2, C8.2, C9.2
- net V_BAT: now also C9.1
- net V_IN: now also C7.1
Changed lines of the file:
@@
-$EndComp
-$Comp
-L liger-rescue:C_1uF C3
-U 1 1 59BA119E
-P 3500 3650
-F 0 "C3" H 3525 3750 50  0000 L CNN
-F 1 "C_1uF" H 3250 3550 50  0000 L CNN
-F 2 "Capacitors_SMD:C_0603_HandSoldering" H 3600 3950 50  0001 C CNN
-F 3 "https://www.digikey.com/product-detail/en/yageo/CC0603ZRY5V7BB105/311-1372-1-ND/2103156" H 3500 3400 50  0001 C CNN
-F 4 "CC0603ZRY5V7BB105" H 3625 3850 60  0001 C CNN "Part Number"
-	1    3500 3650
-	1    0    0    -1
-$EndComp
-$Comp
-L liger-rescue:C_1uF C4
-U 1 1 59BA1591
-P 5125 3675
-F 0 "C4" H 5150 3775 50  0000 L CNN
-F 1 "C_1uF" H 5150 3600 50  0000 L CNN
-F 2 "Capacitors_SMD:C_0603_HandSoldering" H 5225 3975 50  0001 C CNN
-F 3 "https://www.digikey.com/product-detail/en/yageo/CC0603ZRY5V7BB105/311-1372-1-ND/2103156" H 5125 3425 50  0001 C CNN
-F 4 "CC0603ZRY5V7BB105" H 5250 3875 60  0001 C CNN "Part Number"
-	1    5125 3675
-	1    0    0    -1
 $EndComp
 $Comp
@@
 F 0 "BT1" H 8375 3850 50  0000 L CNN
 F 1 "18650_Battery_Cell_1043" H 8375 3750 50  0001 L CNN
-F 2 "" V 8275 3810 50  0001 C CNN
+F 2 "Battery:BatteryHolder_Keystone_1042_1x18650" V 8275 3810 50  0001 C CNN
 F 3 "https://www.digikey.com/product-detail/en/keystone-electronics/1043/36-1043-ND/2745669" V 8275 3810 50  0001 C CNN
 F 4 "36-1043-ND" H 8475 3950 60  0001 C CNN "Part Number"
@@
 Wire Wire Line
 	5125 3875 5125 3825
-$Comp
-L liger-rescue:C_1uF C5
-U 1 1 59EBD4F3
-P 8700 3700
-F 0 "C5" H 8725 3800 50  0000 L CNN
-F 1 "C_1uF" H 8475 3600 50  0000 L CNN
-F 2 "Capacitors_SMD:C_0603_HandSoldering" H 8800 4000 50  0001 C CNN
-F 3 "https://www.digikey.com/product-detail/en/yageo/CC0603ZRY5V7BB105/311-1372-1-ND/2103156" H 8700 3450 50  0001 C CNN
-F 4 "CC0603ZRY5V7BB105" H 8825 3900 60  0001 C CNN "Part Number"
-	1    8700 3700
-	1    0    0    -1
-$EndComp
 Wire Wire Line
 	8700 3450 8700 3550
@@
 Text HLabel 8125 3250 1    60   Input ~ 0
 V_BAT
+$Comp
+L open-automation:C_1uF C8
+U 1 1 5B1EEF77
+P 5125 3675
+F 0 "C8" H 5240 3721 50  0000 L CNN
+F 1 "C_1uF" H 5240 3630 50  0000 L CNN
+F 2 "Capacitor_SMD:C_0603_1608Metric_Pad0.99x1.00mm_HandSolder" H 5225 3975 50  0001 C CNN
+F 3 "https://www.digikey.com/product-detail/en/tdk-corporation/CGA3E1X7R1C105M080AC/445-12540-1-ND/3954206" H 5125 3425 50  0001 C CNN
+F 4 "CGA3E1X7R1C105M080AC" H 5250 3875 60  0001 C CNN "Part Number"
+	1    5125 3675
+	1    0    0    -1
+$EndComp
+$Comp
+L open-automation:C_1uF C7
+U 1 1 5B1EF368
+P 3500 3650
+F 0 "C7" H 3615 3696 50  0000 L CNN
+F 1 "C_1uF" H 3615 3605 50  0000 L CNN
+F 2 "Capacitor_SMD:C_0603_1608Metric_Pad0.99x1.00mm_HandSolder" H 3600 3950 50  0001 C CNN
+F 3 "https://www.digikey.com/product-detail/en/tdk-corporation/CGA3E1X7R1C105M080AC/445-12540-1-ND/3954206" H 3500 3400 50  0001 C CNN
+F 4 "CGA3E1X7R1C105M080AC" H 3625 3850 60  0001 C CNN "Part Number"
+	1    3500 3650
+	1    0    0    -1
+$EndComp
+$Comp
+L open-automation:C_1uF C9
+U 1 1 5B1EF9E4
+P 8700 3700
+F 0 "C9" H 8815 3746 50  0000 L CNN
+F 1 "C_1uF" H 8815 3655 50  0000 L CNN
+F 2 "Capacitor_SMD:C_0603_1608Metric_Pad0.99x1.00mm_HandSolder" H 8800 4000 50  0001 C CNN
+F 3 "https://www.digikey.com/product-detail/en/tdk-corporation/CGA3E1X7R1C105M080AC/445-12540-1-ND/3954206" H 8700 3450 50  0001 C CNN
+F 4 "CGA3E1X7R1C105M080AC" H 8825 3900 60  0001 C CNN "Part Number"
+	1    8700 3700
+	1    0    0    -1
+$EndComp
 $EndSCHEMATC

Commit message: update
Parts:
- C7, C8, C9: footprint Capacitor_SMD:C_0603_1608Metric_Pad0.99x1.00mm_HandSolder -> Capacitor_SMD:C_0603_1608Metric_Pad1.05x0.95mm_HandSolder
- D3: footprint LEDs:LED_0603_HandSoldering -> LED_SMD:LED_0603_1608Metric_Pad1.05x0.95mm_HandSolder
- D6: footprint Diodes_SMD:D_SOD-323_HandSoldering -> Diode_SMD:D_SOD-323_HandSoldering
- Q4: footprint TO_SOT_Packages_SMD:SOT-23 -> Package_TO_SOT_SMD:SOT-23
- R10, R19, R22: footprint Resistors_SMD:R_0603_HandSoldering -> Resistor_SMD:R_0603_1608Metric_Pad1.05x0.95mm_HandSolder
- U4, U9: footprint TO_SOT_Packages_SMD:SOT-23-5 -> Package_TO_SOT_SMD:SOT-23-5_HandSoldering
Changed lines of the file:
@@
 F 0 "R10" V 6655 3450 50  0000 C CNN
 F 1 "R_1k" V 6575 3450 50  0000 C CNN
-F 2 "Resistors_SMD:R_0603_HandSoldering" V 6505 3450 50  0001 C CNN
+F 2 "Resistor_SMD:R_0603_1608Metric_Pad1.05x0.95mm_HandSolder" V 6505 3450 50  0001 C CNN
 F 3 "https://www.digikey.com/product-detail/en/yageo/RC0603JR-071KL/311-1.0KGRCT-ND/729624" V 6655 3450 50  0001 C CNN
 F 4 "RC0603JR-071KL" V 6755 3550 60  0001 C CNN "Part Number"
@@
 F 0 "U4" H 7325 3350 60  0000 C CNN
 F 1 "MCP73831T" H 7275 3750 60  0000 C CNN
-F 2 "TO_SOT_Packages_SMD:SOT-23-5" H 7575 3250 60  0001 C CNN
+F 2 "Package_TO_SOT_SMD:SOT-23-5_HandSoldering" H 7575 3250 60  0001 C CNN
 F 3 "https://www.digikey.com/product-detail/en/microchip-technology/MCP73831T-2ACI-OT/MCP73831T-2ACI-OTCT-ND/1979802" H 7825 3150 60  0001 C CNN
 F 4 "MCP73831T-2ACI/OT" H 7275 3850 60  0001 C CNN "Part Number"
@@
 F 0 "Q4" H 3550 3275 50  0000 L CNN
 F 1 "PMOS-DMG3413L" H 3150 2975 50  0001 L CNN
-F 2 "TO_SOT_Packages_SMD:SOT-23" H 3600 3050 50  0001 L CIN
+F 2 "Package_TO_SOT_SMD:SOT-23" H 3600 3050 50  0001 L CIN
 F 3 "https://www.digikey.com/product-detail/en/diodes-incorporated/DMG3413L-7/DMG3413L-7DICT-ND/5218387" H 3600 3200 50  0001 L CNN
 F 4 "DMG3413L-7" H 3700 3300 60  0001 C CNN "Part Number"
@@
 F 0 "D3" H 6375 3750 50  0000 C CNN
 F 1 "LED-GREEN-LTST-C191GKT" H 6375 3850 50  0001 C CNN
-F 2 "LEDs:LED_0603_HandSoldering" H 6275 3650 50  0001 C CNN
+F 2 "LED_SMD:LED_0603_1608Metric_Pad1.05x0.95mm_HandSolder" H 6275 3650 50  0001 C CNN
 F 3 "https://www.digikey.com/product-detail/en/lite-on-inc/LTST-C191GKT/160-1443-1-ND/386828" H 6375 3750 50  0001 C CNN
 F 4 "LTST-C191GKT" H 6475 3850 60  0001 C CNN "Part Number"
@@
 F 0 "R22" V 2975 3700 50  0000 C CNN
 F 1 "R_10k" V 2875 3700 50  0000 C CNN
-F 2 "Resistors_SMD:R_0603_HandSoldering" V 2905 3700 50  0001 C CNN
+F 2 "Resistor_SMD:R_0603_1608Metric_Pad1.05x0.95mm_HandSolder" V 2905 3700 50  0001 C CNN
 F 3 "https://www.digikey.com/product-detail/en/yageo/RC0603JR-0710KL/311-10KGRCT-ND/729647" V 3055 3700 50  0001 C CNN
 F 4 "RC0603JR-0710KL" V 3155 3800 60  0001 C CNN "Part Number"
@@
 F 0 "R19" V 7975 3700 50  0000 C CNN
 F 1 "R_2k" V 7875 3700 50  0000 C CNN
-F 2 "Resistors_SMD:R_0603_HandSoldering" V 7905 3700 50  0001 C CNN
+F 2 "Resistor_SMD:R_0603_1608Metric_Pad1.05x0.95mm_HandSolder" V 7905 3700 50  0001 C CNN
 F 3 "https://www.digikey.com/product-detail/en/yageo/RC0603JR-072KL/311-2.0KGRCT-ND/729673" V 8055 3700 50  0001 C CNN
 F 4 "RC0603JR-072KL" V 8155 3800 60  0001 C CNN "Part Number"
@@
 F 0 "D6" H 3200 3550 50  0000 C CNN
 F 1 "D_Schottky-BAT20JFILM" H 3200 3350 50  0001 C CNN
-F 2 "Diodes_SMD:D_SOD-323_HandSoldering" H 3200 3275 50  0001 C CNN
+F 2 "Diode_SMD:D_SOD-323_HandSoldering" H 3200 3275 50  0001 C CNN
 F 3 "https://www.digikey.com/product-detail/en/stmicroelectronics/BAT20JFILM/497-3381-1-ND/669138" H 3200 3200 50  0001 C CNN
 F 4 "BAT20JFILM" H 3250 3625 60  0001 C CNN "Part Number"
@@
 F 0 "U9" H 4525 3350 60  0000 C CNN
 F 1 "AP2112" H 4350 3725 60  0000 C CNN
-F 2 "TO_SOT_Packages_SMD:SOT-23-5" H 4350 3200 60  0001 C CNN
+F 2 "Package_TO_SOT_SMD:SOT-23-5_HandSoldering" H 4350 3200 60  0001 C CNN
 F 3 "https://www.digikey.com/product-detail/en/diodes-incorporated/AP2112K-3.3TRG1/AP2112K-3.3TRG1DICT-ND/4505257" H 4350 3100 60  0001 C CNN
 F 4 "AP2112K-3.3TRG1" H 4350 3825 60  0001 C CNN "Part Number"
@@
 F 0 "C8" H 5240 3721 50  0000 L CNN
 F 1 "C_1uF" H 5240 3630 50  0000 L CNN
-F 2 "Capacitor_SMD:C_0603_1608Metric_Pad0.99x1.00mm_HandSolder" H 5225 3975 50  0001 C CNN
+F 2 "Capacitor_SMD:C_0603_1608Metric_Pad1.05x0.95mm_HandSolder" H 5225 3975 50  0001 C CNN
 F 3 "https://www.digikey.com/product-detail/en/tdk-corporation/CGA3E1X7R1C105M080AC/445-12540-1-ND/3954206" H 5125 3425 50  0001 C CNN
 F 4 "CGA3E1X7R1C105M080AC" H 5250 3875 60  0001 C CNN "Part Number"
@@
 F 0 "C7" H 3615 3696 50  0000 L CNN
 F 1 "C_1uF" H 3615 3605 50  0000 L CNN
-F 2 "Capacitor_SMD:C_0603_1608Metric_Pad0.99x1.00mm_HandSolder" H 3600 3950 50  0001 C CNN
+F 2 "Capacitor_SMD:C_0603_1608Metric_Pad1.05x0.95mm_HandSolder" H 3600 3950 50  0001 C CNN
 F 3 "https://www.digikey.com/product-detail/en/tdk-corporation/CGA3E1X7R1C105M080AC/445-12540-1-ND/3954206" H 3500 3400 50  0001 C CNN
 F 4 "CGA3E1X7R1C105M080AC" H 3625 3850 60  0001 C CNN "Part Number"
@@
 F 0 "C9" H 8815 3746 50  0000 L CNN
 F 1 "C_1uF" H 8815 3655 50  0000 L CNN
-F 2 "Capacitor_SMD:C_0603_1608Metric_Pad0.99x1.00mm_HandSolder" H 8800 4000 50  0001 C CNN
+F 2 "Capacitor_SMD:C_0603_1608Metric_Pad1.05x0.95mm_HandSolder" H 8800 4000 50  0001 C CNN
 F 3 "https://www.digikey.com/product-detail/en/tdk-corporation/CGA3E1X7R1C105M080AC/445-12540-1-ND/3954206" H 8700 3450 50  0001 C CNN
 F 4 "CGA3E1X7R1C105M080AC" H 8825 3900 60  0001 C CNN "Part Number"
