File: hardware/power.sch (KiCad schematic (older format))
At the start: 12 parts, among them Q4 PMOS-DMG3413L, U4 MCP73831T, U9 AP2112

Commit message: order complete
Parts:
- C7, C8, C9: Part Number CGA3E1X7R1C105M080AC -> CL10B105KP8NNNC
- R10: Part Number RC0603JR-071KL -> ESR03EZPJ102
- R19: Part Number RC0603JR-072KL -> ERA-3AEB202V
- R22: Part Number RC0603JR-0710KL -> MCT06030C1002FP500
Changed lines of the file:
@@
 F 2 "Resistor_SMD:R_0603_1608Metric_Pad1.05x0.95mm_HandSolder" V 6505 3450 50  0001 C CNN
 F 3 "https://www.digikey.com/product-detail/en/yageo/RC0603JR-071KL/311-1.0KGRCT-ND/729624" V 6655 3450 50  0001 C CNN
-F 4 "RC0603JR-071KL" V 6755 3550 60  0001 C CNN "Part Number"
+F 4 "ESR03EZPJ102" V 6755 3550 60  0001 C CNN "Part Number"
 	1    6575 3450
 	0    1    1    0
@@
 F 2 "Resistor_SMD:R_0603_1608Metric_Pad1.05x0.95mm_HandSolder" V 2905 3700 50  0001 C CNN
 F 3 "https://www.digikey.com/product-detail/en/yageo/RC0603JR-0710KL/311-10KGRCT-ND/729647" V 3055 3700 50  0001 C CNN
-F 4 "RC0603JR-0710KL" V 3155 3800 60  0001 C CNN "Part Number"
+F 4 "MCT06030C1002FP500" V 3155 3800 60  0001 C CNN "Part Number"
 	1    2975 3700
 	1    0    0    -1
@@
 F 2 "Resistor_SMD:R_0603_1608Metric_Pad1.05x0.95mm_HandSolder" V 7905 3700 50  0001 C CNN
 F 3 "https://www.digikey.com/product-detail/en/yageo/RC0603JR-072KL/311-2.0KGRCT-ND/729673" V 8055 3700 50  0001 C CNN
-F 4 "RC0603JR-072KL" V 8155 3800 60  0001 C CNN "Part Number"
+F 4 "ERA-3AEB202V" V 8155 3800 60  0001 C CNN "Part Number"
 	1    7975 3700
 	-1   0    0    1
@@
 F 2 "Capacitor_SMD:C_0603_1608Metric_Pad1.05x0.95mm_HandSolder" H 5225 3975 50  0001 C CNN
 F 3 "https://www.digikey.com/product-detail/en/tdk-corporation/CGA3E1X7R1C105M080AC/445-12540-1-ND/3954206" H 5125 3425 50  0001 C CNN
-F 4 "CGA3E1X7R1C105M080AC" H 5250 3875 60  0001 C CNN "Part Number"
+F 4 "CL10B105KP8NNNC" H 5250 3875 60  0001 C CNN "Part Number"
 	1    5125 3675
 	1    0    0    -1
@@
 F 2 "Capacitor_SMD:C_0603_1608Metric_Pad1.05x0.95mm_HandSolder" H 3600 3950 50  0001 C CNN
 F 3 "https://www.digikey.com/product-detail/en/tdk-corporation/CGA3E1X7R1C105M080AC/445-12540-1-ND/3954206" H 3500 3400 50  0001 C CNN
-F 4 "CGA3E1X7R1C105M080AC" H 3625 3850 60  0001 C CNN "Part Number"
+F 4 "CL10B105KP8NNNC" H 3625 3850 60  0001 C CNN "Part Number"
 	1    3500 3650
 	1    0    0    -1
@@
 F 2 "Capacitor_SMD:C_0603_1608Metric_Pad1.05x0.95mm_HandSolder" H 8800 4000 50  0001 C CNN
 F 3 "https://www.digikey.com/product-detail/en/tdk-corporation/CGA3E1X7R1C105M080AC/445-12540-1-ND/3954206" H 8700 3450 50  0001 C CNN
-F 4 "CGA3E1X7R1C105M080AC" H 8825 3900 60  0001 C CNN "Part Number"
+F 4 "CL10B105KP8NNNC" H 8825 3900 60  0001 C CNN "Part Number"
 	1    8700 3700
 	1    0    0    -1

Commit message: 0.7.1
Parts:
- removed D3: LED-GREEN-LTST-C191GKT, LED_SMD:LED_0603_1608Metric_Pad1.05x0.95mm_HandSolder, symbol liger-rescue:LED-GREEN-LTST-C191GKT
- added D3: LED-0603-G, LED_SMD:LED_0603_1608Metric_Pad1.05x0.95mm_HandSolder, symbol open-automation:LED-0603-G
Connections:
- net at R10.2: now also D3.2 (A)
- net at U4.1 (STAT): now also D3.1 (K)
Changed lines of the file:
@@
-$EndComp
-$Comp
-L liger-rescue:LED-GREEN-LTST-C191GKT D3
-U 1 1 59B58167
-P 6375 3650
-F 0 "D3" H 6375 3750 50  0000 C CNN
-F 1 "LED-GREEN-LTST-C191GKT" H 6375 3850 50  0001 C CNN
-F 2 "LED_SMD:LED_0603_1608Metric_Pad1.05x0.95mm_HandSolder" H 6275 3650 50  0001 C CNN
-F 3 "https://www.digikey.com/product-detail/en/lite-on-inc/LTST-C191GKT/160-1443-1-ND/386828" H 6375 3750 50  0001 C CNN
-F 4 "LTST-C191GKT" H 6475 3850 60  0001 C CNN "Part Number"
-	1    6375 3650
-	0    -1   -1   0
 $EndComp
 $Comp
@@
 	1    0    0    -1
 $EndComp
+$Comp
+L open-automation:LED-0603-G D?
+U 1 1 5BBE79A0
+P 6375 3650
+AR Path="/59092AD4/5BBE79A0" Ref="D?"  Part="1"
+AR Path="/5909D8E3/5BBE79A0" Ref="D3"  Part="1"
+F 0 "D3" V 6350 3800 50  0000 R CNN
+F 1 "LED-0603-G" V 6175 3950 50  0000 R CNN
+F 2 "LED_SMD:LED_0603_1608Metric_Pad1.05x0.95mm_HandSolder" H 6275 3650 50  0001 C CNN
+F 3 "https://www.digikey.com/product-detail/en/rohm-semiconductor/SML-D12M8WT86/511-1578-1-ND/1641810" H 6375 3750 50  0001 C CNN
+F 4 "SML-D12M8WT86" H 6475 3850 50  0001 C CNN "Part Number"
+	1    6375 3650
+	0    -1   -1   0
+$EndComp
 $EndSCHEMATC
