File: hardware/switches.sch (KiCad schematic (older format))
At the start: 15 parts, among them Q2 Q_NMOS_GSD, Q3 Q_PMOS_GSD, SW1 LED-switch, U10 touchpad, U7 touchpad, U8 touchpad, U9 touchpad

Commit message: update
Parts:
- D2: Part Number LS Q976-NR-1 -> 475-2512-2-ND
- Q3: Part Number BSS84LT1G -> BSS84
- SW1: Part Number (none) -> CKN10530TR-ND
Changed lines of the file:
@@
 F 1 "Q_PMOS_GSD" H 6150 3700 50  0000 R CNN
 F 2 "TO_SOT_Packages_SMD:SOT-23" H 6050 4000 50  0001 C CNN
-F 3 "http://www.mouser.com/ds/2/308/BSS84LT1-D-105913.pdf" H 5850 3900 50  0001 C CNN
-F 4 "BSS84LT1G" H 5850 3900 60  0001 C CNN "Part Number"
+F 3 "https://www.fairchildsemi.com/datasheets/BS/BSS84.pdf" H 5850 3900 50  0001 C CNN
+F 4 "BSS84" H 5850 3900 60  0001 C CNN "Part Number"
 	1    5850 3900
 	-1   0    0    1
@@
 F 2 "LEDs:LED_0603" H 6200 3200 50  0001 C CNN
 F 3 "http://www.osram-os.com/Graphics/XPic9/00128792_0.pdf" H 6200 3200 50  0001 C CNN
-F 4 "LS Q976-NR-1" H 6200 3200 60  0001 C CNN "Part Number"
+F 4 "475-2512-2-ND" H 6200 3200 60  0001 C CNN "Part Number"
 	1    6200 3200
 	0    -1   -1   0
@@
 F 1 "LED-switch" H 3350 3750 60  0000 C CNN
 F 2 "footprints:SMT-led-switch" H 3400 4050 60  0001 C CNN
-F 3 "http://www.digikey.com/product-detail/en/c-k-components/K8WH41GLFS/CKN10530TR-ND/4176636" H 3400 4050 60  0001 C CNN
+F 3 "http://www.ckswitches.com/media/1481/k8.pdf" H 3400 4050 60  0001 C CNN
+F 4 "CKN10530TR-ND" H 3400 4050 60  0001 C CNN "Part Number"
 	1    3400 4050
 	1    0    0    -1

Commit message: updatE
Parts:
- added U12: soft-button-4x, footprints:soft-button-4, symbol soft-button-4x
Connections:
- wire segments 31 -> 35
Changed lines of the file:
@@
 EN
 $Comp
-L GND #PWR019
+L GND #PWR22
 U 1 1 59092D1C
 P 6200 5100
-F 0 "#PWR019" H 6200 4850 50  0001 C CNN
+F 0 "#PWR22" H 6200 4850 50  0001 C CNN
 F 1 "GND" H 6200 4950 50  0000 C CNN
 F 2 "" H 6200 5100 50  0000 C CNN
@@
 $EndComp
 $Comp
-L GND #PWR020
+L GND #PWR21
 U 1 1 59092D1D
 P 5500 5100
-F 0 "#PWR020" H 5500 4850 50  0001 C CNN
+F 0 "#PWR21" H 5500 4850 50  0001 C CNN
 F 1 "GND" H 5500 4950 50  0000 C CNN
 F 2 "" H 5500 5100 50  0000 C CNN
@@
 $EndComp
 $Comp
-L GND #PWR021
+L GND #PWR20
 U 1 1 59092D28
 P 2850 4750
-F 0 "#PWR021" H 2850 4500 50  0001 C CNN
+F 0 "#PWR20" H 2850 4500 50  0001 C CNN
 F 1 "GND" H 2850 4600 50  0000 C CNN
 F 2 "" H 2850 4750 50  0000 C CNN
@@
 Text GLabel 3900 3650 1    60   Input ~ 0
 3V3
+$Comp
+L soft-button-4x U12
+U 1 1 597D230D
+P 9200 1900
+F 0 "U12" H 9550 2150 60  0000 C CNN
+F 1 "soft-button-4x" H 9650 1450 60  0000 C CNN
+F 2 "footprints:soft-button-4" H 9200 1900 60  0001 C CNN
+F 3 "" H 9200 1900 60  0001 C CNN
+	1    9200 1900
+	1    0    0    -1
+$EndComp
+Text GLabel 8750 2000 0    60   Input ~ 0
+IO32
+Text GLabel 9850 2000 2    60   Input ~ 0
+IO33
+Text GLabel 9300 1450 1    60   Input ~ 0
+IO27
+Text GLabel 9300 2550 3    60   Input ~ 0
+IO14
+Wire Wire Line
+	9300 1450 9300 1500
+Wire Wire Line
+	8750 2000 8800 2000
+Wire Wire Line
+	9300 2500 9300 2550
+Wire Wire Line
+	9850 2000 9800 2000
 $EndSCHEMATC

Commit message: update
Parts:
- removed U10, U7, U8, U9: touchpad, footprints:touch-pad, symbol touchpad
Connections:
- net labels removed: IO14
- wire segments 35 -> 31
Other:
- moved on the sheet: C5, D2, PROG1, Q2, Q3, R12, R13, R14, R15, R16, U12

Commit message: updatge
Parts:
- removed SW1: LED-switch, footprints:SMT-led-switch, symbol LED-switch
- added R8: 36, Resistors_SMD:R_0603_HandSoldering, symbol R
- added U7: RGB-LED, open-automation:RGB-LED-J-Lead-SMD-6, symbol RGB-LED
- R12: value 1K -> 36; Part Number RC0603JR-071KL -> RC0603JR-0736RL
- U12: footprint footprints:soft-button-4 -> open-automation:soft-button-4
Connections:
- net labels added: IO18, IO19
- net labels removed: IO21
- wire segments 31 -> 28
Other:
- moved on the sheet: C5, D2, PROG1, Q2, Q3, R14, R15, R16, U12

Commit message: update
Connections:
- net IO0: no longer U12.4 (DOWN)
- new net IO14: U12.4 (DOWN)
Changed lines of the file:
@@
 LIBS:open-automation
 LIBS:liger-cache
-EELAYER 26 0
+EELAYER 25 0
 EELAYER END
 $Descr A4 11693 8268
@@
 IO27
 Text GLabel 7200 3750 3    60   Input ~ 0
-IO0
+IO14
 $Comp
 L RGB-LED U7

Commit message: update
Parts:
- removed R14, R15, R16: 1K, Resistors_SMD:R_0603_HandSoldering, symbol R
- added R14, R15, R16: R_1k, Resistors_SMD:R_0603, symbol R_1k
Connections:
- net EN: now also R15.1
- net IO0: now also R16.1
- net at D2.1 (K), Q3.2 (S): now also R15.2
- net at Q3.3 (D): now also R14.1
- net at C5.2, Q2.1 (G): now also R14.2
- net at Q2.3 (D): now also R16.2
- net 5V renamed V_USB
- net IO14 renamed T_DOWN
- net IO18 renamed LED_R
- net IO19 renamed LED_G
- net IO27 renamed T_UP
- net IO32 renamed T_LEFT
- net IO33 renamed T_RIGHT
- net IO5 renamed LED_B
Changed lines of the file:
@@
 $Descr A4 11693 8268
 encoding utf-8
-Sheet 6 8
+Sheet 6 10
 Title ""
 Date ""
@@
 $EndDescr
 Text GLabel 6550 4700 0    60   Input ~ 0
-IO18
+LED_R
 $Comp
 L SW_PUSH PROG1
@@
 EN
 $Comp
-L GND #PWR019
+L GND #PWR017
 U 1 1 59092D1C
 P 3900 5000
-F 0 "#PWR019" H 3900 4750 50  0001 C CNN
+F 0 "#PWR017" H 3900 4750 50  0001 C CNN
 F 1 "GND" H 3900 4850 50  0000 C CNN
 F 2 "" H 3900 5000 50  0000 C CNN
@@
 $EndComp
 $Comp
-L GND #PWR020
+L GND #PWR018
 U 1 1 59092D1D
 P 3200 5000
-F 0 "#PWR020" H 3200 4750 50  0001 C CNN
+F 0 "#PWR018" H 3200 4750 50  0001 C CNN
 F 1 "GND" H 3200 4850 50  0000 C CNN
 F 2 "" H 3200 5000 50  0000 C CNN
@@
 $EndComp
 $Comp
-L R R14
-U 1 1 59092D20
-P 3450 4300
-F 0 "R14" V 3530 4300 50  0000 C CNN
-F 1 "1K" V 3450 4300 50  0000 C CNN
-F 2 "Resistors_SMD:R_0603_HandSoldering" V 3380 4300 50  0001 C CNN
-F 3 "http://www.digikey.com/en/resources/datasheets/yageo/rc-series-l-suffix-datasheet" H 3450 4300 50  0001 C CNN
-F 4 "RC0603JR-071KL" V 3450 4300 60  0001 C CNN "Part Number"
-	1    3450 4300
-	1    0    0    -1
-$EndComp
-$Comp
-L R R15
-U 1 1 59092D21
-P 3900 3550
-F 0 "R15" V 3980 3550 50  0000 C CNN
-F 1 "1K" V 3900 3550 50  0000 C CNN
-F 2 "Resistors_SMD:R_0603_HandSoldering" V 3830 3550 50  0001 C CNN
-F 3 "http://www.digikey.com/en/resources/datasheets/yageo/rc-series-l-suffix-datasheet" H 3900 3550 50  0001 C CNN
-F 4 "RC0603JR-071KL" V 3900 3550 60  0001 C CNN "Part Number"
-	1    3900 3550
-	1    0    0    -1
-$EndComp
-$Comp
-L R R16
-U 1 1 59092D22
-P 4200 4850
-F 0 "R16" V 4280 4850 50  0000 C CNN
-F 1 "1K" V 4200 4850 50  0000 C CNN
-F 2 "Resistors_SMD:R_0603_HandSoldering" V 4130 4850 50  0001 C CNN
-F 3 "http://www.digikey.com/en/resources/datasheets/yageo/rc-series-l-suffix-datasheet" H 4200 4850 50  0001 C CNN
-F 4 "RC0603JR-071KL" V 4200 4850 60  0001 C CNN "Part Number"
-	1    4200 4850
-	0    1    1    0
-$EndComp
-$Comp
 L C C5
 U 1 1 59092D23
@@
 Switches_N_Stuff
 Text GLabel 3900 2800 1    60   Input ~ 0
-5V
+V_USB
 $Comp
 L soft-button-4x U12
@@
 $EndComp
 Text GLabel 6650 3200 0    60   Input ~ 0
-IO32
+T_LEFT
 Text GLabel 7750 3200 2    60   Input ~ 0
-IO33
+T_RIGHT
 Text GLabel 7200 2650 1    60   Input ~ 0
-IO27
+T_UP
 Text GLabel 7200 3750 3    60   Input ~ 0
-IO14
+T_DOWN
 $Comp
 L RGB-LED U7
@@
 	7750 3200 7700 3200
 Text GLabel 6550 4850 0    60   Input ~ 0
-IO19
+LED_G
 Text GLabel 6550 4550 0    60   Input ~ 0
-IO5
+LED_B
 Wire Wire Line
 	6550 4550 6650 4550
@@
 	8150 4850 8050 4850
 Connection ~ 8150 4700
+$Comp
+L R_1k R14
+U 1 1 59BA2D07
+P 3450 4300
+F 0 "R14" V 3450 4300 50  0000 C CNN
+F 1 "R_1k" V 3375 4300 50  0000 C CNN
+F 2 "Resistors_SMD:R_0603" V 3380 4300 50  0001 C CNN
+F 3 "https://www.digikey.com/product-detail/en/yageo/RC0603JR-071KL/311-1.0KGRCT-ND/729624" V 3530 4300 50  0001 C CNN
+F 4 "RC0603JR-071KL" V 3630 4400 60  0001 C CNN "Part Number"
+	1    3450 4300
+	1    0    0    -1
+$EndComp
+$Comp
+L R_1k R16
+U 1 1 59BA2D49
+P 4200 4850
+F 0 "R16" V 4200 4850 50  0000 C CNN
+F 1 "R_1k" V 4125 4850 50  0000 C CNN
+F 2 "Resistors_SMD:R_0603" V 4130 4850 50  0001 C CNN
+F 3 "https://www.digikey.com/product-detail/en/yageo/RC0603JR-071KL/311-1.0KGRCT-ND/729624" V 4280 4850 50  0001 C CNN
+F 4 "RC0603JR-071KL" V 4380 4950 60  0001 C CNN "Part Number"
+	1    4200 4850
+	0    1    1    0
+$EndComp
+$Comp
+L R_1k R15
+U 1 1 59BA2DC7
+P 3900 3550
+F 0 "R15" V 3900 3550 50  0000 C CNN
+F 1 "R_1k" V 3825 3550 50  0000 C CNN
+F 2 "Resistors_SMD:R_0603" V 3830 3550 50  0001 C CNN
+F 3 "https://www.digikey.com/product-detail/en/yageo/RC0603JR-071KL/311-1.0KGRCT-ND/729624" V 3980 3550 50  0001 C CNN
+F 4 "RC0603JR-071KL" V 4080 3650 60  0001 C CNN "Part Number"
+	1    3900 3550
+	-1   0    0    1
+$EndComp
 $EndSCHEMATC
