File: hardware/switches.sch (KiCad schematic (older format))
At the start: 13 parts, among them Q2 Q_NMOS_GSD, Q3 Q_PMOS_GSD, U12 soft-button-4x, U7 RGB-LED

Commit message: update
Parts:
- C5: footprint Capacitors_SMD:C_0603_HandSoldering -> Capacitors_SMD:C_0603
- R12, R13, R8: footprint Resistors_SMD:R_0603_HandSoldering -> Resistors_SMD:R_0603
Changed lines of the file:
@@
 F 0 "C5" H 3225 4750 50  0000 L CNN
 F 1 "4.7uF" H 3200 4550 50  0000 L CNN
-F 2 "Capacitors_SMD:C_0603_HandSoldering" H 3238 4500 50  0001 C CNN
+F 2 "Capacitors_SMD:C_0603" H 3238 4500 50  0001 C CNN
 F 3 "http://media.digikey.com/pdf/Data%20Sheets/Samsung%20PDFs/CL_Series_MLCC_ds.pdf" H 3200 4650 50  0001 C CNN
 F 4 "CL10B475KQ8NQNC" H 3200 4650 60  0001 C CNN "Part Number"
@@
 F 0 "R8" V 7980 4550 50  0000 C CNN
 F 1 "36" V 7900 4550 50  0000 C CNN
-F 2 "Resistors_SMD:R_0603_HandSoldering" V 7830 4550 50  0001 C CNN
+F 2 "Resistors_SMD:R_0603" V 7830 4550 50  0001 C CNN
 F 3 "http://www.yageo.com.tw/exep/pages/download/literatures/PYu-R_INT-thick_7.pdf" H 7900 4550 50  0001 C CNN
 F 4 "RC0603JR-0736RL" V 7900 4550 60  0001 C CNN "Part Number"
@@
 F 0 "R12" V 7980 4700 50  0000 C CNN
 F 1 "36" V 7900 4700 50  0000 C CNN
-F 2 "Resistors_SMD:R_0603_HandSoldering" V 7830 4700 50  0001 C CNN
+F 2 "Resistors_SMD:R_0603" V 7830 4700 50  0001 C CNN
 F 3 "http://www.yageo.com.tw/exep/pages/download/literatures/PYu-R_INT-thick_7.pdf" H 7900 4700 50  0001 C CNN
 F 4 "RC0603JR-0736RL" V 7900 4700 60  0001 C CNN "Part Number"
@@
 F 0 "R13" V 7980 4850 50  0000 C CNN
 F 1 "36" V 7900 4850 50  0000 C CNN
-F 2 "Resistors_SMD:R_0603_HandSoldering" V 7830 4850 50  0001 C CNN
+F 2 "Resistors_SMD:R_0603" V 7830 4850 50  0001 C CNN
 F 3 "http://www.yageo.com.tw/exep/pages/download/literatures/PYu-R_INT-thick_7.pdf" H 7900 4850 50  0001 C CNN
 F 4 "RC0603JR-0736RL" V 7900 4850 60  0001 C CNN "Part Number"

Commit message: update
Parts:
- removed C5: 4.7uF, Capacitors_SMD:C_0603, symbol C
- removed Q2: Q_NMOS_GSD, TO_SOT_Packages_SMD:SOT-23, symbol Q_NMOS_GSD
- removed Q3: Q_PMOS_GSD, TO_SOT_Packages_SMD:SOT-23, symbol Q_PMOS_GSD
- added D4, D5: LED, LEDs:LED_0603, symbol LED
- added FACTORY1, PROG1: SW_PUSH, Buttons_Switches_SMD:SW_SPST_KMR2, symbol SW_PUSH
- renumbered PROG1 to REBOOT1
Connections:
- net labels added: FACTORY, PROG
- net labels removed: IO0, V_USB
- wire segments 28 -> 29
Changed lines of the file:
@@
 LED_R
 $Comp
-L SW_PUSH PROG1
+L SW_PUSH REBOOT1
 U 1 1 59092D1B
 P 3900 4200
-F 0 "PROG1" H 4050 4310 50  0000 C CNN
+F 0 "REBOOT1" V 4125 4375 50  0000 C CNN
 F 1 "SW_PUSH" H 3900 4120 50  0000 C CNN
 F 2 "Buttons_Switches_SMD:SW_SPST_KMR2" H 3900 4200 50  0001 C CNN
@@
 	0    1    1    0
 $EndComp
-Text GLabel 4500 4850 2    60   Input ~ 0
-IO0
+Text GLabel 3250 3800 2    60   Input ~ 0
+PROG
 Text GLabel 4150 3800 2    60   Input ~ 0
 EN
 $Comp
-L GND #PWR014
+L GND #PWR018
 U 1 1 59092D1C
-P 3900 5000
-F 0 "#PWR014" H 3900 4750 50  0001 C CNN
-F 1 "GND" H 3900 4850 50  0000 C CNN
-F 2 "" H 3900 5000 50  0000 C CNN
-F 3 "" H 3900 5000 50  0000 C CNN
-	1    3900 5000
-	1    0    0    -1
-$EndComp
-$Comp
-L GND #PWR015
-U 1 1 59092D1D
-P 3200 5000
-F 0 "#PWR015" H 3200 4750 50  0001 C CNN
-F 1 "GND" H 3200 4850 50  0000 C CNN
-F 2 "" H 3200 5000 50  0000 C CNN
-F 3 "" H 3200 5000 50  0000 C CNN
-	1    3200 5000
-	1    0    0    -1
-$EndComp
-$Comp
-L Q_PMOS_GSD Q3
-U 1 1 59092D1E
-P 3550 3800
-F 0 "Q3" H 3850 3850 50  0000 R CNN
-F 1 "Q_PMOS_GSD" H 3850 3600 50  0000 R CNN
-F 2 "TO_SOT_Packages_SMD:SOT-23" H 3750 3900 50  0001 C CNN
-F 3 "https://www.fairchildsemi.com/datasheets/BS/BSS84.pdf" H 3550 3800 50  0001 C CNN
-F 4 "BSS84" H 3550 3800 60  0001 C CNN "Part Number"
-	1    3550 3800
-	-1   0    0    1
-$EndComp
-$Comp
-L Q_NMOS_GSD Q2
-U 1 1 59092D1F
-P 3450 4750
-F 0 "Q2" V 3350 4900 50  0000 R CNN
-F 1 "Q_NMOS_GSD" V 3650 5000 50  0000 R CNN
-F 2 "TO_SOT_Packages_SMD:SOT-23" H 3650 4850 50  0001 C CNN
-F 3 "http://www.mouser.com/ds/2/308/2N7002L-D-105484.pdf" H 3450 4750 50  0001 C CNN
-F 4 "2N7002L" V 3450 4750 60  0001 C CNN "Part Number"
-	1    3450 4750
-	0    1    1    0
-$EndComp
-$Comp
-L C C5
-U 1 1 59092D23
-P 3200 4650
-F 0 "C5" H 3225 4750 50  0000 L CNN
-F 1 "4.7uF" H 3200 4550 50  0000 L CNN
-F 2 "Capacitors_SMD:C_0603" H 3238 4500 50  0001 C CNN
-F 3 "http://media.digikey.com/pdf/Data%20Sheets/Samsung%20PDFs/CL_Series_MLCC_ds.pdf" H 3200 4650 50  0001 C CNN
-F 4 "CL10B475KQ8NQNC" H 3200 4650 60  0001 C CNN "Part Number"
-	1    3200 4650
-	-1   0    0    1
+P 3900 4575
+F 0 "#PWR018" H 3900 4325 50  0001 C CNN
+F 1 "GND" H 3900 4425 50  0000 C CNN
+F 2 "" H 3900 4575 50  0000 C CNN
+F 3 "" H 3900 4575 50  0000 C CNN
+	1    3900 4575
+	1    0    0    -1
 $EndComp
 $Comp
@@
 P 3900 3100
 F 0 "D2" H 3900 3200 50  0000 C CNN
-F 1 "LED" H 4050 3050 50  0000 C CNN
+F 1 "LED" V 4025 3025 50  0000 C CNN
 F 2 "LEDs:LED_0603" H 3900 3100 50  0001 C CNN
 F 3 "http://www.osram-os.com/Graphics/XPic9/00128792_0.pdf" H 3900 3100 50  0001 C CNN
@@
 Switches_N_Stuff
 Text GLabel 3900 2800 1    60   Input ~ 0
-V_USB
+3V3
 $Comp
 L soft-button-4x U12
@@
 Wire Wire Line
 	3900 2800 3900 2950
-Wire Wire Line
-	4350 4850 4500 4850
-Wire Wire Line
-	3900 4500 3900 5000
-Wire Wire Line
-	3650 4850 4050 4850
-Wire Wire Line
-	3200 4500 3450 4500
-Connection ~ 3200 4850
-Wire Wire Line
-	3200 4800 3200 5000
-Wire Wire Line
-	3250 4850 3200 4850
-Connection ~ 3450 4500
-Wire Wire Line
-	3450 4450 3450 4550
 Connection ~ 3900 3800
 Wire Wire Line
 	3900 3700 3900 3900
-Wire Wire Line
-	3750 3800 4150 3800
-Wire Wire Line
-	3450 4150 3450 4000
-Connection ~ 3900 3350
-Wire Wire Line
-	3450 3350 3450 3600
-Wire Wire Line
-	3900 3350 3450 3350
 Wire Wire Line
 	3900 3250 3900 3400
@@
 	8150 4850 8050 4850
 Connection ~ 8150 4700
-$Comp
-L R_1k R14
-U 1 1 59BA2D07
-P 3450 4300
-F 0 "R14" V 3450 4300 50  0000 C CNN
-F 1 "R_1k" V 3375 4300 50  0000 C CNN
-F 2 "Resistors_SMD:R_0603" V 3380 4300 50  0001 C CNN
-F 3 "https://www.digikey.com/product-detail/en/yageo/RC0603JR-071KL/311-1.0KGRCT-ND/729624" V 3530 4300 50  0001 C CNN
-F 4 "RC0603JR-071KL" V 3630 4400 60  0001 C CNN "Part Number"
-	1    3450 4300
-	1    0    0    -1
-$EndComp
-$Comp
-L R_1k R16
-U 1 1 59BA2D49
-P 4200 4850
-F 0 "R16" V 4200 4850 50  0000 C CNN
-F 1 "R_1k" V 4125 4850 50  0000 C CNN
-F 2 "Resistors_SMD:R_0603" V 4130 4850 50  0001 C CNN
-F 3 "https://www.digikey.com/product-detail/en/yageo/RC0603JR-071KL/311-1.0KGRCT-ND/729624" V 4280 4850 50  0001 C CNN
-F 4 "RC0603JR-071KL" V 4380 4950 60  0001 C CNN "Part Number"
-	1    4200 4850
-	0    1    1    0
-$EndComp
 $Comp
 L R_1k R15
@@
 	-1   0    0    1
 $EndComp
+Wire Wire Line
+	4150 3800 3900 3800
+$Comp
+L SW_PUSH PROG1
+U 1 1 59CA58CF
+P 3000 4200
+F 0 "PROG1" V 3225 4400 50  0000 C CNN
+F 1 "SW_PUSH" H 3000 4120 50  0000 C CNN
+F 2 "Buttons_Switches_SMD:SW_SPST_KMR2" H 3000 4200 50  0001 C CNN
+F 3 "http://www.mouser.com/ds/2/60/KMR2_9aug12-25127.pdf" H 3000 4200 50  0001 C CNN
+F 4 "KMR211NG LFS" H 3000 4200 60  0001 C CNN "Part Number"
+	1    3000 4200
+	0    1    1    0
+$EndComp
+$Comp
+L GND #PWR019
+U 1 1 59CA58D6
+P 3000 4575
+F 0 "#PWR019" H 3000 4325 50  0001 C CNN
+F 1 "GND" H 3000 4425 50  0000 C CNN
+F 2 "" H 3000 4575 50  0000 C CNN
+F 3 "" H 3000 4575 50  0000 C CNN
+	1    3000 4575
+	1    0    0    -1
+$EndComp
+$Comp
+L LED D5
+U 1 1 59CA58DD
+P 3000 3100
+F 0 "D5" H 3000 3200 50  0000 C CNN
+F 1 "LED" V 3125 3025 50  0000 C CNN
+F 2 "LEDs:LED_0603" H 3000 3100 50  0001 C CNN
+F 3 "http://www.osram-os.com/Graphics/XPic9/00128792_0.pdf" H 3000 3100 50  0001 C CNN
+F 4 "475-2512-2-ND" H 3000 3100 60  0001 C CNN "Part Number"
+	1    3000 3100
+	0    -1   -1   0
+$EndComp
+Text GLabel 3000 2800 1    60   Input ~ 0
+3V3
+Wire Wire Line
+	3000 2800 3000 2950
+Connection ~ 3000 3800
+Wire Wire Line
+	3000 3700 3000 3900
+Wire Wire Line
+	3000 3250 3000 3400
+$Comp
+L R_1k R16
+U 1 1 59CA58E9
+P 3000 3550
+F 0 "R16" V 3000 3550 50  0000 C CNN
+F 1 "R_1k" V 2925 3550 50  0000 C CNN
+F 2 "Resistors_SMD:R_0603" V 2930 3550 50  0001 C CNN
+F 3 "https://www.digikey.com/product-detail/en/yageo/RC0603JR-071KL/311-1.0KGRCT-ND/729624" V 3080 3550 50  0001 C CNN
+F 4 "RC0603JR-071KL" V 3180 3650 60  0001 C CNN "Part Number"
+	1    3000 3550
+	-1   0    0    1
+$EndComp
+Wire Wire Line
+	3250 3800 3000 3800
+Wire Wire Line
+	3000 4500 3000 4575
+Wire Wire Line
+	3900 4500 3900 4575
+Text GLabel 2375 3800 2    60   Input ~ 0
+FACTORY
+$Comp
+L SW_PUSH FACTORY1
+U 1 1 59CA6153
+P 2125 4200
+F 0 "FACTORY1" V 2350 4400 50  0000 C CNN
+F 1 "SW_PUSH" H 2125 4120 50  0000 C CNN
+F 2 "Buttons_Switches_SMD:SW_SPST_KMR2" H 2125 4200 50  0001 C CNN
+F 3 "http://www.mouser.com/ds/2/60/KMR2_9aug12-25127.pdf" H 2125 4200 50  0001 C CNN
+F 4 "KMR211NG LFS" H 2125 4200 60  0001 C CNN "Part Number"
+	1    2125 4200
+	0    1    1    0
+$EndComp
+$Comp
+L GND #PWR020
+U 1 1 59CA6159
+P 2125 4575
+F 0 "#PWR020" H 2125 4325 50  0001 C CNN
+F 1 "GND" H 2125 4425 50  0000 C CNN
+F 2 "" H 2125 4575 50  0000 C CNN
+F 3 "" H 2125 4575 50  0000 C CNN
+	1    2125 4575
+	1    0    0    -1
+$EndComp
+$Comp
+L LED D4
+U 1 1 59CA6160
+P 2125 3100
+F 0 "D4" H 2125 3200 50  0000 C CNN
+F 1 "LED" V 2250 3025 50  0000 C CNN
+F 2 "LEDs:LED_0603" H 2125 3100 50  0001 C CNN
+F 3 "http://www.osram-os.com/Graphics/XPic9/00128792_0.pdf" H 2125 3100 50  0001 C CNN
+F 4 "475-2512-2-ND" H 2125 3100 60  0001 C CNN "Part Number"
+	1    2125 3100
+	0    -1   -1   0
+$EndComp
+Text GLabel 2125 2800 1    60   Input ~ 0
+3V3
+Wire Wire Line
+	2125 2800 2125 2950
+Connection ~ 2125 3800
+Wire Wire Line
+	2125 3700 2125 3900
+Wire Wire Line
+	2125 3250 2125 3400
+$Comp
+L R_1k R14
+U 1 1 59CA616C
+P 2125 3550
+F 0 "R14" V 2125 3550 50  0000 C CNN
+F 1 "R_1k" V 2050 3550 50  0000 C CNN
+F 2 "Resistors_SMD:R_0603" V 2055 3550 50  0001 C CNN
+F 3 "https://www.digikey.com/product-detail/en/yageo/RC0603JR-071KL/311-1.0KGRCT-ND/729624" V 2205 3550 50  0001 C CNN
+F 4 "RC0603JR-071KL" V 2305 3650 60  0001 C CNN "Part Number"
+	1    2125 3550
+	-1   0    0    1
+$EndComp
+Wire Wire Line
+	2375 3800 2125 3800
+Wire Wire Line
+	2125 4500 2125 4575
 $EndSCHEMATC

Commit message: update
Parts:
- D2, D4, D5: footprint LEDs:LED_0603 -> LEDs:LED_0603_HandSoldering
- R12, R13, R14, R15, R16, R8: footprint Resistors_SMD:R_0603 -> Resistors_SMD:R_0603_HandSoldering
Changed lines of the file:
@@
 F 0 "D2" H 3900 3200 50  0000 C CNN
 F 1 "LED" V 4025 3025 50  0000 C CNN
-F 2 "LEDs:LED_0603" H 3900 3100 50  0001 C CNN
+F 2 "LEDs:LED_0603_HandSoldering" H 3900 3100 50  0001 C CNN
 F 3 "http://www.osram-os.com/Graphics/XPic9/00128792_0.pdf" H 3900 3100 50  0001 C CNN
 F 4 "475-2512-2-ND" H 3900 3100 60  0001 C CNN "Part Number"
@@
 F 0 "R8" V 7980 4550 50  0000 C CNN
 F 1 "36" V 7900 4550 50  0000 C CNN
-F 2 "Resistors_SMD:R_0603" V 7830 4550 50  0001 C CNN
+F 2 "Resistors_SMD:R_0603_HandSoldering" V 7830 4550 50  0001 C CNN
 F 3 "http://www.yageo.com.tw/exep/pages/download/literatures/PYu-R_INT-thick_7.pdf" H 7900 4550 50  0001 C CNN
 F 4 "RC0603JR-0736RL" V 7900 4550 60  0001 C CNN "Part Number"
@@
 F 0 "R12" V 7980 4700 50  0000 C CNN
 F 1 "36" V 7900 4700 50  0000 C CNN
-F 2 "Resistors_SMD:R_0603" V 7830 4700 50  0001 C CNN
+F 2 "Resistors_SMD:R_0603_HandSoldering" V 7830 4700 50  0001 C CNN
 F 3 "http://www.yageo.com.tw/exep/pages/download/literatures/PYu-R_INT-thick_7.pdf" H 7900 4700 50  0001 C CNN
 F 4 "RC0603JR-0736RL" V 7900 4700 60  0001 C CNN "Part Number"
@@
 F 0 "R13" V 7980 4850 50  0000 C CNN
 F 1 "36" V 7900 4850 50  0000 C CNN
-F 2 "Resistors_SMD:R_0603" V 7830 4850 50  0001 C CNN
+F 2 "Resistors_SMD:R_0603_HandSoldering" V 7830 4850 50  0001 C CNN
 F 3 "http://www.yageo.com.tw/exep/pages/download/literatures/PYu-R_INT-thick_7.pdf" H 7900 4850 50  0001 C CNN
 F 4 "RC0603JR-0736RL" V 7900 4850 60  0001 C CNN "Part Number"
@@
 F 0 "R15" V 3900 3550 50  0000 C CNN
 F 1 "R_1k" V 3825 3550 50  0000 C CNN
-F 2 "Resistors_SMD:R_0603" V 3830 3550 50  0001 C CNN
+F 2 "Resistors_SMD:R_0603_HandSoldering" V 3830 3550 50  0001 C CNN
 F 3 "https://www.digikey.com/product-detail/en/yageo/RC0603JR-071KL/311-1.0KGRCT-ND/729624" V 3980 3550 50  0001 C CNN
 F 4 "RC0603JR-071KL" V 4080 3650 60  0001 C CNN "Part Number"
@@
 F 0 "D5" H 3000 3200 50  0000 C CNN
 F 1 "LED" V 3125 3025 50  0000 C CNN
-F 2 "LEDs:LED_0603" H 3000 3100 50  0001 C CNN
+F 2 "LEDs:LED_0603_HandSoldering" H 3000 3100 50  0001 C CNN
 F 3 "http://www.osram-os.com/Graphics/XPic9/00128792_0.pdf" H 3000 3100 50  0001 C CNN
 F 4 "475-2512-2-ND" H 3000 3100 60  0001 C CNN "Part Number"
@@
 F 0 "R16" V 3000 3550 50  0000 C CNN
 F 1 "R_1k" V 2925 3550 50  0000 C CNN
-F 2 "Resistors_SMD:R_0603" V 2930 3550 50  0001 C CNN
+F 2 "Resistors_SMD:R_0603_HandSoldering" V 2930 3550 50  0001 C CNN
 F 3 "https://www.digikey.com/product-detail/en/yageo/RC0603JR-071KL/311-1.0KGRCT-ND/729624" V 3080 3550 50  0001 C CNN
 F 4 "RC0603JR-071KL" V 3180 3650 60  0001 C CNN "Part Number"
@@
 F 0 "D4" H 2125 3200 50  0000 C CNN
 F 1 "LED" V 2250 3025 50  0000 C CNN
-F 2 "LEDs:LED_0603" H 2125 3100 50  0001 C CNN
+F 2 "LEDs:LED_0603_HandSoldering" H 2125 3100 50  0001 C CNN
 F 3 "http://www.osram-os.com/Graphics/XPic9/00128792_0.pdf" H 2125 3100 50  0001 C CNN
 F 4 "475-2512-2-ND" H 2125 3100 60  0001 C CNN "Part Number"
@@
 F 0 "R14" V 2125 3550 50  0000 C CNN
 F 1 "R_1k" V 2050 3550 50  0000 C CNN
-F 2 "Resistors_SMD:R_0603" V 2055 3550 50  0001 C CNN
+F 2 "Resistors_SMD:R_0603_HandSoldering" V 2055 3550 50  0001 C CNN
 F 3 "https://www.digikey.com/product-detail/en/yageo/RC0603JR-071KL/311-1.0KGRCT-ND/729624" V 2205 3550 50  0001 C CNN
 F 4 "RC0603JR-071KL" V 2305 3650 60  0001 C CNN "Part Number"

Commit message: update
Parts:
- added J1: Conn_02x08_Odd_Even, Pin_Headers:Pin_Header_Straight_2x08_Pitch2.54mm, symbol Conn_02x08_Odd_Even
Connections:
- net 3V3: now also J1.5 (Pin_5)
- net FACTORY: now also J1.7 (Pin_7)
- net GND: now also J1.1 (Pin_1), J1.2 (Pin_2)
- net PROG: now also J1.15 (Pin_15)
- new net I2S_BCLK: J1.13 (Pin_13)
- new net I2S_DATA_IN: J1.12 (Pin_12)
- new net I2S_DATA_OUT: J1.14 (Pin_14)
- new net I2S_WS: J1.11 (Pin_11)
- new net RELAY: J1.16 (Pin_16)
- new net RXD: J1.8 (Pin_8)
- new net SCL: J1.9 (Pin_9)
- new net SDA: J1.10 (Pin_10)
- new net TXD: J1.6 (Pin_6)
- new net V_BAT: J1.3 (Pin_3)
- new net V_USB: J1.4 (Pin_4)
Other:
- moved on the sheet: D2, D4, D5, FACTORY1, PROG1, R12, R13, R14, R15, R16, R8, REBOOT1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

Commit message: update
Parts:
- D2, D4, D5: symbol LED -> liger-rescue:LED
- FACTORY1, PROG1, REBOOT1: symbol SW_PUSH -> liger-rescue:SW_PUSH
- J1: symbol Conn_02x08_Odd_Even -> liger-rescue:Conn_02x08_Odd_Even
- R12, R13, R8: symbol R -> liger-rescue:R
- R14, R15, R16: symbol R_1k -> liger-rescue:R_1k
- U12: symbol soft-button-4x -> liger-rescue:soft-button-4x
- U7: symbol RGB-LED -> liger-rescue:RGB-LED
Changed lines of the file:
@@
-EESchema Schematic File Version 2
-LIBS:power
-LIBS:device
-LIBS:transistors
-LIBS:conn
-LIBS:linear
-LIBS:regul
-LIBS:74xx
-LIBS:cmos4000
-LIBS:adc-dac
-LIBS:memory
-LIBS:xilinx
-LIBS:microcontrollers
-LIBS:dsp
-LIBS:microchip
-LIBS:analog_switches
-LIBS:motorola
-LIBS:texas
-LIBS:intel
-LIBS:audio
-LIBS:interface
-LIBS:digital-audio
-LIBS:philips
-LIBS:display
-LIBS:cypress
-LIBS:siliconi
-LIBS:opto
-LIBS:atmel
-LIBS:contrib
-LIBS:valves
-LIBS:open-automation
+EESchema Schematic File Version 4
 LIBS:liger-cache
-EELAYER 25 0
+EELAYER 26 0
 EELAYER END
 $Descr A4 11693 8268
@@
 LED_R
 $Comp
-L SW_PUSH REBOOT1
+L liger-rescue:SW_PUSH REBOOT1
 U 1 1 59092D1B
 P 5350 3900
@@
 EN
 $Comp
-L GND #PWR019
+L power:GND #PWR019
 U 1 1 59092D1C
 P 5350 4275
@@
 $EndComp
 $Comp
-L LED D2
+L liger-rescue:LED D2
 U 1 1 59092D24
 P 5350 2800
@@
 3V3
 $Comp
-L soft-button-4x U12
+L liger-rescue:soft-button-4x U12
 U 1 1 597D230D
 P 7825 3325
@@
 T_DOWN
 $Comp
-L RGB-LED U7
+L liger-rescue:RGB-LED U7
 U 1 1 5980E7D1
 P 7875 4925
@@
 	7275 5075 7375 5075
 $Comp
-L R R8
+L liger-rescue:R R8
 U 1 1 5980F245
 P 8625 4775
@@
 3V3
 $Comp
-L R R12
+L liger-rescue:R R12
 U 1 1 5980F487
 P 8625 4925
@@
 $EndComp
 $Comp
-L R R13
+L liger-rescue:R R13
 U 1 1 5980F4D4
 P 8625 5075
@@
 Connection ~ 8875 4925
 $Comp
-L R_1k R15
+L liger-rescue:R_1k R15
 U 1 1 59BA2DC7
 P 5350 3250
@@
 	5600 3500 5350 3500
 $Comp
-L SW_PUSH PROG1
+L liger-rescue:SW_PUSH PROG1
 U 1 1 59CA58CF
 P 4450 3900
@@
 $EndComp
 $Comp
-L GND #PWR020
+L power:GND #PWR020
 U 1 1 59CA58D6
 P 4450 4275
@@
 $EndComp
 $Comp
-L LED D5
+L liger-rescue:LED D5
 U 1 1 59CA58DD
 P 4450 2800
@@
 	4450 2950 4450 3100
 $Comp
-L R_1k R16
+L liger-rescue:R_1k R16
 U 1 1 59CA58E9
 P 4450 3250
@@
 FACTORY
 $Comp
-L SW_PUSH FACTORY1
+L liger-rescue:SW_PUSH FACTORY1
 U 1 1 59CA6153
 P 3575 3900
@@
 $EndComp
 $Comp
-L GND #PWR021
+L power:GND #PWR021
 U 1 1 59CA6159
 P 3575 4275
@@
 $EndComp
 $Comp
-L LED D4
+L liger-rescue:LED D4
 U 1 1 59CA6160
 P 3575 2800
@@
 	3575 2950 3575 3100
 $Comp
-L R_1k R14
+L liger-rescue:R_1k R14
 U 1 1 59CA616C
 P 3575 3250
@@
 	3575 4200 3575 4275
 $Comp
-L GND #PWR022
+L power:GND #PWR022
 U 1 1 5A16D01B
 P 4050 5200
@@
 V_USB
 $Comp
-L GND #PWR023
+L power:GND #PWR023
 U 1 1 5A16D01C
 P 4650 5200
@@
 I2S_DATA_OUT
 $Comp
-L Conn_02x08_Odd_Even J1
+L liger-rescue:Conn_02x08_Odd_Even J1
 U 1 1 5A16D01F
 P 4300 5550
