File: hardware/enviroment.sch (KiCad schematic (older format))
At the start: 5 parts, among them U5 OPT3001, U6 SI7020-A20

Commit message: update
Parts:
- added C11: C_100uF, Capacitors_SMD:C_1206, symbol C_100uF
- added C12: C_1uF, Capacitors_SMD:C_0603, symbol C_1uF
- added R17: R_10, Resistors_SMD:R_0603, symbol R_10
Connections:
- wire segments 20 -> 28
Other:
- note added: "I2C ByPass CAPs"
- moved on the sheet: C23, C24, R25, U6

Commit message: update
Parts:
- removed C11: C_100uF, Capacitors_SMD:C_1206, symbol C_100uF
- removed C12: C_1uF, Capacitors_SMD:C_0603, symbol C_1uF
- removed R17: R_10, Resistors_SMD:R_0603, symbol R_10
- U5: Part Number OPT3001 -> OPT3001DNPR
Connections:
- wire segments 28 -> 20
Other:
- note removed: "I2C ByPass CAPs"
Changed lines of the file:
@@
 VCC_I2C
 $Comp
-L GND #PWR018
+L GND #PWR023
 U 1 1 5962DDD8
 P 3500 3350
-F 0 "#PWR018" H 3500 3100 50  0001 C CNN
+F 0 "#PWR023" H 3500 3100 50  0001 C CNN
 F 1 "GND" H 3500 3200 50  0000 C CNN
 F 2 "" H 3500 3350 50  0000 C CNN
@@
 $EndComp
 $Comp
-L GND #PWR019
+L GND #PWR024
 U 1 1 59B8FA16
 P 3200 3600
-F 0 "#PWR019" H 3200 3350 50  0001 C CNN
+F 0 "#PWR024" H 3200 3350 50  0001 C CNN
 F 1 "GND" H 3200 3450 50  0000 C CNN
 F 2 "" H 3200 3600 50  0000 C CNN
@@
 Text Label 7150 2700 0    60   ~ 0
 Light-Level
-$Comp
-L OPT3001 U5
-U 1 1 59B90C13
-P 7500 3200
-F 0 "U5" H 7650 2950 60  0000 C CNN
-F 1 "OPT3001" H 7500 3350 60  0000 C CNN
-F 2 "Housings_DFN_QFN:DFN-6-1EP_2x2mm_Pitch0.65mm" H 7550 2850 60  0001 C CNN
-F 3 "https://www.digikey.com/product-detail/en/texas-instruments/OPT3001DNPR/296-40474-1-ND/5178351" H 7650 2950 60  0001 C CNN
-F 4 "OPT3001" H 7750 3050 60  0001 C CNN "Part Number"
-	1    7500 3200
-	1    0    0    -1
-$EndComp
 Text GLabel 7900 3100 1    60   Input ~ 0
 SDA
@@
 SCL
 $Comp
-L GND #PWR020
+L GND #PWR025
 U 1 1 59B90C14
 P 7150 3400
-F 0 "#PWR020" H 7150 3150 50  0001 C CNN
+F 0 "#PWR025" H 7150 3150 50  0001 C CNN
 F 1 "GND" H 7150 3250 50  0000 C CNN
 F 2 "" H 7150 3400 50  0000 C CNN
@@
 $EndComp
 $Comp
-L GND #PWR021
+L GND #PWR026
 U 1 1 59B90DEC
 P 6850 3550
-F 0 "#PWR021" H 6850 3300 50  0001 C CNN
+F 0 "#PWR026" H 6850 3300 50  0001 C CNN
 F 1 "GND" H 6850 3400 50  0000 C CNN
 F 2 "" H 6850 3550 50  0000 C CNN
@@
 Connection ~ 8350 3250
 $Comp
-L R_10 R17
-U 1 1 59B8099B
-P 5100 4900
-F 0 "R17" V 5180 4900 50  0000 C CNN
-F 1 "R_10" V 5100 4900 50  0000 C CNN
-F 2 "Resistors_SMD:R_0603" V 5030 4900 50  0001 C CNN
-F 3 "https://www.digikey.com/product-detail/en/te-connectivity-passive-product/CPF0603B10RE/A119908CT-ND/4966506" V 5180 4900 50  0001 C CNN
-F 4 "CPF0603B10RE" V 5280 5000 60  0001 C CNN "Part Number"
-	1    5100 4900
-	0    1    1    0
-$EndComp
-$Comp
-L C_1uF C12
-U 1 1 59B8099C
-P 5800 5100
-F 0 "C12" H 5800 5200 50  0000 L CNN
-F 1 "C_1uF" H 5550 5000 50  0000 L CNN
-F 2 "Capacitors_SMD:C_0603" H 5900 5400 50  0001 C CNN
-F 3 "https://www.digikey.com/product-detail/en/yageo/CC0603ZRY5V7BB105/311-1372-1-ND/2103156" H 5800 4850 50  0001 C CNN
-F 4 "CC0603ZRY5V7BB105" H 5925 5300 60  0001 C CNN "Part Number"
-	1    5800 5100
+L OPT3001 U5
+U 1 1 59CC26B6
+P 7500 3200
+F 0 "U5" H 7650 2950 60  0000 C CNN
+F 1 "OPT3001" H 7500 3350 60  0000 C CNN
+F 2 "Housings_DFN_QFN:DFN-6-1EP_2x2mm_Pitch0.65mm" H 7550 2850 60  0001 C CNN
+F 3 "https://www.digikey.com/product-detail/en/texas-instruments/OPT3001DNPR/296-40474-1-ND/5178351" H 7650 2950 60  0001 C CNN
+F 4 "OPT3001DNPR" H 7750 3050 60  0001 C CNN "Part Number"
+	1    7500 3200
 	1    0    0    -1
 $EndComp
-$Comp
-L C_100uF C11
-U 1 1 59B8099D
-P 5400 5100
-F 0 "C11" H 5425 5200 50  0000 L CNN
-F 1 "C_100uF" H 5050 5000 50  0000 L CNN
-F 2 "Capacitors_SMD:C_1206" H 5500 5400 50  0001 C CNN
-F 3 "https://www.digikey.com/product-detail/en/kemet/C0603C104K5RACTU/399-5089-1-ND/1465623" H 5400 4850 50  0001 C CNN
-F 4 "C3216X5R1A107M160AC" H 5525 5300 60  0001 C CNN "Part Number"
-	1    5400 5100
-	1    0    0    -1
-$EndComp
-$Comp
-L GND #PWR022
-U 1 1 59B8099E
-P 5600 5350
-F 0 "#PWR022" H 5600 5100 50  0001 C CNN
-F 1 "GND" H 5600 5200 50  0000 C CNN
-F 2 "" H 5600 5350 50  0000 C CNN
-F 3 "" H 5600 5350 50  0000 C CNN
-	1    5600 5350
-	1    0    0    -1
-$EndComp
-Text GLabel 4850 4900 0    60   Input ~ 0
-3V3
-Text GLabel 5950 4900 2    60   Input ~ 0
-VCC_I2C
-Wire Wire Line
-	4850 4900 4950 4900
-Wire Wire Line
-	5250 4900 5950 4900
-Wire Wire Line
-	5400 4900 5400 4950
-Wire Wire Line
-	5800 4900 5800 4950
-Connection ~ 5400 4900
-Connection ~ 5800 4900
-Wire Wire Line
-	5400 5250 5400 5300
-Wire Wire Line
-	5400 5300 5800 5300
-Wire Wire Line
-	5800 5300 5800 5250
-Wire Wire Line
-	5600 5350 5600 5300
-Connection ~ 5600 5300
-Text Notes 5150 5750 0    60   ~ 0
-I2C ByPass CAPs
-Wire Notes Line
-	6400 4800 6400 5650
-Wire Notes Line
-	6400 5650 4550 5650
-Wire Notes Line
-	4550 4800 6400 4800
-Wire Notes Line
-	4550 5650 4550 4800
 $EndSCHEMATC

Commit message: update
Parts:
- removed C23, C24: C_0.1uF, Capacitors_SMD:C_0603, symbol C_0.1uF
- removed R25: R_10k, Resistors_SMD:R_0603, symbol R_10k
- removed U5: OPT3001, Housings_DFN_QFN:DFN-6-1EP_2x2mm_Pitch0.65mm, symbol OPT3001
- added C7, C9: C_0.1uF, Capacitors_SMD:C_0603_HandSoldering, symbol C_0.1uF
- added U8: TSL45315CL, open-automation:LIGHT-SENSOR-TSL45315CL, symbol TSL45315CL
Connections:
- net labels removed: LIGHT_INT, VCC_I2C
- wire segments 20 -> 16
Changed lines of the file:
@@
 Comment4 ""
 $EndDescr
-Text Label 4800 1300 0    197  ~ 0
+Text Label 5125 1950 0    197  ~ 0
 Environment
-Text GLabel 3050 3200 0    60   Input ~ 0
-VCC_I2C
+Text GLabel 3400 3425 0    60   Input ~ 0
+3V3
 $Comp
-L GND #PWR023
-U 1 1 5962DDD8
-P 3500 3350
-F 0 "#PWR023" H 3500 3100 50  0001 C CNN
-F 1 "GND" H 3500 3200 50  0000 C CNN
-F 2 "" H 3500 3350 50  0000 C CNN
-F 3 "" H 3500 3350 50  0000 C CNN
-	1    3500 3350
+L GND #PWR024
+U 1 1 59EBC48D
+P 3850 3575
+F 0 "#PWR024" H 3850 3325 50  0001 C CNN
+F 1 "GND" H 3850 3425 50  0000 C CNN
+F 2 "" H 3850 3575 50  0000 C CNN
+F 3 "" H 3850 3575 50  0000 C CNN
+	1    3850 3575
 	1    0    0    -1
 $EndComp
-Text GLabel 4500 3200 2    60   Input ~ 0
+Text GLabel 4850 3425 2    60   Input ~ 0
 SCL
-Text GLabel 4500 3300 2    60   Input ~ 0
+Text GLabel 4850 3525 2    60   Input ~ 0
 SDA
 $Comp
 L SI7020-A20 U6
-U 1 1 59AB3352
-P 4000 3300
-F 0 "U6" H 4200 3200 60  0000 C CNN
-F 1 "SI7020-A20" H 4000 3500 60  0000 C CNN
-F 2 "open-automation:SI7020-A20" H 4000 3000 60  0001 C CNN
-F 3 "https://www.digikey.com/product-detail/en/silicon-labs/SI7020-A20-GM1R/336-3596-1-ND/5823452" H 4000 3100 60  0001 C CNN
-F 4 "SI7020-A20-GM1R" H 4100 3100 60  0001 C CNN "Part Number"
-	1    4000 3300
+U 1 1 59EBC48E
+P 4350 3525
+F 0 "U6" H 4550 3425 60  0000 C CNN
+F 1 "SI7020-A20" H 4350 3725 60  0000 C CNN
+F 2 "open-automation:SI7020-A20" H 4350 3225 60  0001 C CNN
+F 3 "https://www.digikey.com/product-detail/en/silicon-labs/SI7020-A20-GM1R/336-3596-1-ND/5823452" H 4350 3325 60  0001 C CNN
+F 4 "SI7020-A20-GM1R" H 4450 3325 60  0001 C CNN "Part Number"
+	1    4350 3525
 	1    0    0    -1
 $EndComp
 $Comp
-L C_0.1uF C23
-U 1 1 59B8F8FE
-P 3200 3400
-F 0 "C23" H 3225 3500 50  0000 L CNN
-F 1 "C_0.1uF" H 2900 3300 50  0000 L CNN
-F 2 "Capacitors_SMD:C_0603" H 3300 3700 50  0001 C CNN
-F 3 "https://www.digikey.com/product-detail/en/kemet/C0603C104K5RACTU/399-5089-1-ND/1465623" H 3200 3150 50  0001 C CNN
-F 4 "C0603C104K5RACTU" H 3325 3600 60  0001 C CNN "Part Number"
-	1    3200 3400
+L C_0.1uF C7
+U 1 1 59EBC48F
+P 3550 3625
+F 0 "C7" H 3575 3725 50  0000 L CNN
+F 1 "C_0.1uF" H 3250 3525 50  0000 L CNN
+F 2 "Capacitors_SMD:C_0603_HandSoldering" H 3650 3925 50  0001 C CNN
+F 3 "https://www.digikey.com/product-detail/en/kemet/C0603C104K5RACTU/399-5089-1-ND/1465623" H 3550 3375 50  0001 C CNN
+F 4 "C0603C104K5RACTU" H 3675 3825 60  0001 C CNN "Part Number"
+	1    3550 3625
 	1    0    0    -1
 $EndComp
 $Comp
-L GND #PWR024
-U 1 1 59B8FA16
-P 3200 3600
-F 0 "#PWR024" H 3200 3350 50  0001 C CNN
-F 1 "GND" H 3200 3450 50  0000 C CNN
-F 2 "" H 3200 3600 50  0000 C CNN
-F 3 "" H 3200 3600 50  0000 C CNN
-	1    3200 3600
+L GND #PWR025
+U 1 1 59EBC490
+P 3550 3825
+F 0 "#PWR025" H 3550 3575 50  0001 C CNN
+F 1 "GND" H 3550 3675 50  0000 C CNN
+F 2 "" H 3550 3825 50  0000 C CNN
+F 3 "" H 3550 3825 50  0000 C CNN
+	1    3550 3825
 	1    0    0    -1
 $EndComp
-Text Label 7150 2700 0    60   ~ 0
+Text Label 7675 3250 0    60   ~ 0
 Light-Level
-Text GLabel 7900 3100 1    60   Input ~ 0
+Text GLabel 8425 3625 2    60   Input ~ 0
 SDA
-Text GLabel 7900 3400 3    60   Input ~ 0
+Text GLabel 8425 3500 2    60   Input ~ 0
 SCL
 $Comp
-L GND #PWR025
-U 1 1 59B90C14
-P 7150 3400
-F 0 "#PWR025" H 7150 3150 50  0001 C CNN
-F 1 "GND" H 7150 3250 50  0000 C CNN
-F 2 "" H 7150 3400 50  0000 C CNN
-F 3 "" H 7150 3400 50  0000 C CNN
-	1    7150 3400
+L GND #PWR026
+U 1 1 59EBC491
+P 7425 3675
+F 0 "#PWR026" H 7425 3425 50  0001 C CNN
+F 1 "GND" H 7425 3525 50  0000 C CNN
+F 2 "" H 7425 3675 50  0000 C CNN
+F 3 "" H 7425 3675 50  0000 C CNN
+	1    7425 3675
 	1    0    0    -1
 $EndComp
+Text GLabel 7100 3525 0    60   Input ~ 0
+3V3
 $Comp
-L R_10k R25
-U 1 1 59B90C15
-P 8350 3000
-F 0 "R25" V 8350 3000 50  0000 C CNN
-F 1 "R_10k" V 8250 3000 50  0000 C CNN
-F 2 "Resistors_SMD:R_0603" V 8280 3000 50  0001 C CNN
-F 3 "https://www.digikey.com/product-detail/en/yageo/RC0603JR-0710KL/311-10KGRCT-ND/729647" V 8430 3000 50  0001 C CNN
-F 4 "RC0603JR-0710KL" V 8530 3100 60  0001 C CNN "Part Number"
-	1    8350 3000
-	-1   0    0    1
-$EndComp
-Text GLabel 6700 3150 0    60   Input ~ 0
-VCC_I2C
-$Comp
-L C_0.1uF C24
-U 1 1 59B90DE4
-P 6850 3350
-F 0 "C24" H 6875 3450 50  0000 L CNN
-F 1 "C_0.1uF" H 6550 3250 50  0000 L CNN
-F 2 "Capacitors_SMD:C_0603" H 6950 3650 50  0001 C CNN
-F 3 "https://www.digikey.com/product-detail/en/kemet/C0603C104K5RACTU/399-5089-1-ND/1465623" H 6850 3100 50  0001 C CNN
-F 4 "C0603C104K5RACTU" H 6975 3550 60  0001 C CNN "Part Number"
-	1    6850 3350
+L C_0.1uF C9
+U 1 1 59EBC492
+P 7200 3700
+F 0 "C9" H 7225 3800 50  0000 L CNN
+F 1 "C_0.1uF" H 6900 3600 50  0000 L CNN
+F 2 "Capacitors_SMD:C_0603_HandSoldering" H 7300 4000 50  0001 C CNN
+F 3 "https://www.digikey.com/product-detail/en/kemet/C0603C104K5RACTU/399-5089-1-ND/1465623" H 7200 3450 50  0001 C CNN
+F 4 "C0603C104K5RACTU" H 7325 3900 60  0001 C CNN "Part Number"
+	1    7200 3700
 	1    0    0    -1
 $EndComp
+Text Label 4050 3200 0    60   ~ 0
+Temp-Humidty
+Wire Wire Line
+	3400 3425 3900 3425
+Wire Wire Line
+	3900 3525 3850 3525
+Wire Wire Line
+	4850 3525 4750 3525
+Wire Wire Line
+	4750 3425 4850 3425
+Wire Wire Line
+	3550 3475 3550 3425
+Connection ~ 3550 3425
+Wire Wire Line
+	3550 3825 3550 3775
+Wire Wire Line
+	3850 3525 3850 3575
+Wire Wire Line
+	7425 3675 7425 3625
+Wire Wire Line
+	7425 3625 7475 3625
+Wire Wire Line
+	7100 3525 7475 3525
+Wire Wire Line
+	7200 3525 7200 3550
 $Comp
-L GND #PWR026
-U 1 1 59B90DEC
-P 6850 3550
-F 0 "#PWR026" H 6850 3300 50  0001 C CNN
-F 1 "GND" H 6850 3400 50  0000 C CNN
-F 2 "" H 6850 3550 50  0000 C CNN
-F 3 "" H 6850 3550 50  0000 C CNN
-	1    6850 3550
+L GND #PWR027
+U 1 1 59EBC493
+P 7200 3900
+F 0 "#PWR027" H 7200 3650 50  0001 C CNN
+F 1 "GND" H 7200 3750 50  0000 C CNN
+F 2 "" H 7200 3900 50  0000 C CNN
+F 3 "" H 7200 3900 50  0000 C CNN
+	1    7200 3900
 	1    0    0    -1
 $EndComp
-Text GLabel 8350 2800 1    60   Input ~ 0
-3V3
-Text Label 3500 2900 0    60   ~ 0
-Temp-Humidty
 Wire Wire Line
-	3050 3200 3550 3200
+	7200 3900 7200 3850
+Connection ~ 7200 3525
 Wire Wire Line
-	3550 3300 3500 3300
+	8425 3625 8325 3625
 Wire Wire Line
-	4500 3300 4400 3300
+	8325 3525 8375 3525
 Wire Wire Line
-	4400 3200 4500 3200
+	8375 3525 8375 3500
 Wire Wire Line
-	3200 3250 3200 3200
-Connection ~ 3200 3200
-Wire Wire Line
-	3200 3600 3200 3550
-Wire Wire Line
-	3500 3300 3500 3350
-Wire Wire Line
-	7900 3100 7900 3150
-Wire Wire Line
-	7900 3150 7850 3150
-Wire Wire Line
-	7900 3400 7900 3350
-Wire Wire Line
-	7900 3350 7850 3350
-Wire Wire Line
-	7150 3250 7150 3400
-Wire Wire Line
-	7150 3350 7200 3350
-Wire Wire Line
-	7200 3250 7150 3250
-Connection ~ 7150 3350
-Wire Wire Line
-	7850 3250 8500 3250
-Wire Wire Line
-	6700 3150 7200 3150
-Wire Wire Line
-	6850 3200 6850 3150
-Connection ~ 6850 3150
-Wire Wire Line
-	6850 3550 6850 3500
-Wire Wire Line
-	8350 2850 8350 2800
-Text GLabel 8500 3250 2    60   Input ~ 0
-LIGHT_INT
-Wire Wire Line
-	8350 3150 8350 3250
-Connection ~ 8350 3250
+	8375 3500 8425 3500
 $Comp
-L OPT3001 U5
-U 1 1 59CC26B6
-P 7500 3200
-F 0 "U5" H 7650 2950 60  0000 C CNN
-F 1 "OPT3001" H 7500 3350 60  0000 C CNN
-F 2 "Housings_DFN_QFN:DFN-6-1EP_2x2mm_Pitch0.65mm" H 7550 2850 60  0001 C CNN
-F 3 "https://www.digikey.com/product-detail/en/texas-instruments/OPT3001DNPR/296-40474-1-ND/5178351" H 7650 2950 60  0001 C CNN
-F 4 "OPT3001DNPR" H 7750 3050 60  0001 C CNN "Part Number"
-	1    7500 3200
+L TSL45315CL U8
+U 1 1 59EBC494
+P 7925 3625
+F 0 "U8" H 8125 3525 60  0000 C CNN
+F 1 "TSL45315CL" H 7925 3825 60  0000 C CNN
+F 2 "open-automation:LIGHT-SENSOR-TSL45315CL" H 7925 3325 60  0001 C CNN
+F 3 "https://www.digikey.com/product-detail/en/ams/TSL45315CL/TSL45315-CLCT-ND/3095326" H 7925 3425 60  0001 C CNN
+F 4 "TSL45315CL" H 7925 3225 60  0001 C CNN "Part Number"
+	1    7925 3625
 	1    0    0    -1
 $EndComp

Commit message: update
Parts:
- C7, C9: symbol C_0.1uF -> liger-rescue:C_0.1uF
- U6: symbol SI7020-A20 -> liger-rescue:SI7020-A20
- U8: symbol TSL45315CL -> liger-rescue:TSL45315CL
Changed lines of the file:
@@
-EESchema Schematic File Version 2
-LIBS:power
-LIBS:device
-LIBS:transistors
-LIBS:conn
-LIBS:linear
-LIBS:regul
-LIBS:74xx
-LIBS:cmos4000
-LIBS:adc-dac
-LIBS:memory
-LIBS:xilinx
-LIBS:microcontrollers
-LIBS:dsp
-LIBS:microchip
-LIBS:analog_switches
-LIBS:motorola
-LIBS:texas
-LIBS:intel
-LIBS:audio
-LIBS:interface
-LIBS:digital-audio
-LIBS:philips
-LIBS:display
-LIBS:cypress
-LIBS:siliconi
-LIBS:opto
-LIBS:atmel
-LIBS:contrib
-LIBS:valves
-LIBS:open-automation
+EESchema Schematic File Version 4
 LIBS:liger-cache
-EELAYER 25 0
+EELAYER 26 0
 EELAYER END
 $Descr A4 11693 8268
@@
 3V3
 $Comp
-L GND #PWR024
+L power:GND #PWR024
 U 1 1 59EBC48D
 P 3850 3575
@@
 SDA
 $Comp
-L SI7020-A20 U6
+L liger-rescue:SI7020-A20 U6
 U 1 1 59EBC48E
 P 4350 3525
@@
 $EndComp
 $Comp
-L C_0.1uF C7
+L liger-rescue:C_0.1uF C7
 U 1 1 59EBC48F
 P 3550 3625
@@
 $EndComp
 $Comp
-L GND #PWR025
+L power:GND #PWR025
 U 1 1 59EBC490
 P 3550 3825
@@
 SCL
 $Comp
-L GND #PWR026
+L power:GND #PWR026
 U 1 1 59EBC491
 P 7425 3675
@@
 3V3
 $Comp
-L C_0.1uF C9
+L liger-rescue:C_0.1uF C9
 U 1 1 59EBC492
 P 7200 3700
@@
 	7200 3525 7200 3550
 $Comp
-L GND #PWR027
+L power:GND #PWR027
 U 1 1 59EBC493
 P 7200 3900
@@
 	8375 3500 8425 3500
 $Comp
-L TSL45315CL U8
+L liger-rescue:TSL45315CL U8
 U 1 1 59EBC494
 P 7925 3625

Commit message: updated schematic
Parts:
- removed C7, C9: C_0.1uF, Capacitors_SMD:C_0603_HandSoldering, symbol liger-rescue:C_0.1uF
- added C10, C11: C_0.1uF, Capacitor_SMD:C_0603_1608Metric_Pad0.99x1.00mm_HandSolder, symbol open-automation:C_0.1uF
Connections:
- net 3V3: now also C10.1, C11.1
- net GND: now also C10.2, C11.2
Changed lines of the file:
@@
 Text Label 5125 1950 0    197  ~ 0
 Environment
-Text GLabel 3400 3425 0    60   Input ~ 0
-3V3
 $Comp
 L power:GND #PWR024
@@
 	1    0    0    -1
 $EndComp
-Text GLabel 4850 3425 2    60   Input ~ 0
-SCL
-Text GLabel 4850 3525 2    60   Input ~ 0
-SDA
 $Comp
 L liger-rescue:SI7020-A20 U6
@@
 F 4 "SI7020-A20-GM1R" H 4450 3325 60  0001 C CNN "Part Number"
 	1    4350 3525
-	1    0    0    -1
-$EndComp
-$Comp
-L liger-rescue:C_0.1uF C7
-U 1 1 59EBC48F
-P 3550 3625
-F 0 "C7" H 3575 3725 50  0000 L CNN
-F 1 "C_0.1uF" H 3250 3525 50  0000 L CNN
-F 2 "Capacitors_SMD:C_0603_HandSoldering" H 3650 3925 50  0001 C CNN
-F 3 "https://www.digikey.com/product-detail/en/kemet/C0603C104K5RACTU/399-5089-1-ND/1465623" H 3550 3375 50  0001 C CNN
-F 4 "C0603C104K5RACTU" H 3675 3825 60  0001 C CNN "Part Number"
-	1    3550 3625
 	1    0    0    -1
 $EndComp
@@
 Text Label 7675 3250 0    60   ~ 0
 Light-Level
-Text GLabel 8425 3625 2    60   Input ~ 0
-SDA
-Text GLabel 8425 3500 2    60   Input ~ 0
-SCL
 $Comp
 L power:GND #PWR026
@@
 	1    0    0    -1
 $EndComp
-Text GLabel 7100 3525 0    60   Input ~ 0
-3V3
-$Comp
-L liger-rescue:C_0.1uF C9
-U 1 1 59EBC492
-P 7200 3700
-F 0 "C9" H 7225 3800 50  0000 L CNN
-F 1 "C_0.1uF" H 6900 3600 50  0000 L CNN
-F 2 "Capacitors_SMD:C_0603_HandSoldering" H 7300 4000 50  0001 C CNN
-F 3 "https://www.digikey.com/product-detail/en/kemet/C0603C104K5RACTU/399-5089-1-ND/1465623" H 7200 3450 50  0001 C CNN
-F 4 "C0603C104K5RACTU" H 7325 3900 60  0001 C CNN "Part Number"
-	1    7200 3700
-	1    0    0    -1
-$EndComp
 Text Label 4050 3200 0    60   ~ 0
 Temp-Humidty
 Wire Wire Line
-	3400 3425 3900 3425
+	3400 3425 3550 3425
 Wire Wire Line
 	3900 3525 3850 3525
@@
 	7425 3625 7475 3625
 Wire Wire Line
-	7100 3525 7475 3525
+	7100 3525 7200 3525
 Wire Wire Line
 	7200 3525 7200 3550
@@
 	1    0    0    -1
 $EndComp
+Wire Wire Line
+	3550 3425 3900 3425
+Wire Wire Line
+	7200 3525 7475 3525
+$Comp
+L open-automation:C_0.1uF C11
+U 1 1 5B1F3B9C
+P 7200 3700
+F 0 "C11" H 7315 3746 50  0000 L CNN
+F 1 "C_0.1uF" H 6800 3650 50  0000 L CNN
+F 2 "Capacitor_SMD:C_0603_1608Metric_Pad0.99x1.00mm_HandSolder" H 7300 4000 50  0001 C CNN
+F 3 "https://www.digikey.com/product-detail/en/tdk-corporation/C1608X8R1H104K080AB/445-8818-1-ND/3248223" H 7200 3450 50  0001 C CNN
+F 4 "C1608X8R1H104K080AB" H 7325 3900 60  0001 C CNN "Part Number"
+	1    7200 3700
+	1    0    0    -1
+$EndComp
+$Comp
+L open-automation:C_0.1uF C10
+U 1 1 5B1F3C43
+P 3550 3625
+F 0 "C10" H 3665 3671 50  0000 L CNN
+F 1 "C_0.1uF" H 3125 3600 50  0000 L CNN
+F 2 "Capacitor_SMD:C_0603_1608Metric_Pad0.99x1.00mm_HandSolder" H 3650 3925 50  0001 C CNN
+F 3 "https://www.digikey.com/product-detail/en/tdk-corporation/C1608X8R1H104K080AB/445-8818-1-ND/3248223" H 3550 3375 50  0001 C CNN
+F 4 "C1608X8R1H104K080AB" H 3675 3825 60  0001 C CNN "Part Number"
+	1    3550 3625
+	1    0    0    -1
+$EndComp
+Text HLabel 4850 3425 2    60   Input ~ 0
+SCL
+Text HLabel 4850 3525 2    60   Input ~ 0
+SDA
+Text HLabel 3400 3425 0    60   Input ~ 0
+3V3
+Text HLabel 7100 3525 0    60   Input ~ 0
+3V3
+Text HLabel 8425 3500 2    60   Input ~ 0
+SCL
+Text HLabel 8425 3625 2    60   Input ~ 0
+SDA
 $EndSCHEMATC

Commit message: update
Parts:
- C10, C11: footprint Capacitor_SMD:C_0603_1608Metric_Pad0.99x1.00mm_HandSolder -> Capacitor_SMD:C_0603_1608Metric_Pad1.05x0.95mm_HandSolder
Changed lines of the file:
@@
 $Descr A4 11693 8268
 encoding utf-8
-Sheet 7 9
+Sheet 6 9
 Title ""
 Date ""
@@
 F 0 "C11" H 7315 3746 50  0000 L CNN
 F 1 "C_0.1uF" H 6800 3650 50  0000 L CNN
-F 2 "Capacitor_SMD:C_0603_1608Metric_Pad0.99x1.00mm_HandSolder" H 7300 4000 50  0001 C CNN
+F 2 "Capacitor_SMD:C_0603_1608Metric_Pad1.05x0.95mm_HandSolder" H 7300 4000 50  0001 C CNN
 F 3 "https://www.digikey.com/product-detail/en/tdk-corporation/C1608X8R1H104K080AB/445-8818-1-ND/3248223" H 7200 3450 50  0001 C CNN
 F 4 "C1608X8R1H104K080AB" H 7325 3900 60  0001 C CNN "Part Number"
@@
 F 0 "C10" H 3665 3671 50  0000 L CNN
 F 1 "C_0.1uF" H 3125 3600 50  0000 L CNN
-F 2 "Capacitor_SMD:C_0603_1608Metric_Pad0.99x1.00mm_HandSolder" H 3650 3925 50  0001 C CNN
+F 2 "Capacitor_SMD:C_0603_1608Metric_Pad1.05x0.95mm_HandSolder" H 3650 3925 50  0001 C CNN
 F 3 "https://www.digikey.com/product-detail/en/tdk-corporation/C1608X8R1H104K080AB/445-8818-1-ND/3248223" H 3550 3375 50  0001 C CNN
 F 4 "C1608X8R1H104K080AB" H 3675 3825 60  0001 C CNN "Part Number"
