File: hardware/enviroment.sch (KiCad schematic (older format))
At the start: 4 parts, among them U6 SI7020-A20, U8 TSL45315CL

Commit message: order complete
Parts:
- C10, C11: Part Number C1608X8R1H104K080AB -> CL10F104ZO8NNNC
Changed lines of the file:
@@
 F 2 "Capacitor_SMD:C_0603_1608Metric_Pad1.05x0.95mm_HandSolder" H 7300 4000 50  0001 C CNN
 F 3 "https://www.digikey.com/product-detail/en/tdk-corporation/C1608X8R1H104K080AB/445-8818-1-ND/3248223" H 7200 3450 50  0001 C CNN
-F 4 "C1608X8R1H104K080AB" H 7325 3900 60  0001 C CNN "Part Number"
+F 4 "CL10F104ZO8NNNC" H 7325 3900 60  0001 C CNN "Part Number"
 	1    7200 3700
 	1    0    0    -1
@@
 F 2 "Capacitor_SMD:C_0603_1608Metric_Pad1.05x0.95mm_HandSolder" H 3650 3925 50  0001 C CNN
 F 3 "https://www.digikey.com/product-detail/en/tdk-corporation/C1608X8R1H104K080AB/445-8818-1-ND/3248223" H 3550 3375 50  0001 C CNN
-F 4 "C1608X8R1H104K080AB" H 3675 3825 60  0001 C CNN "Part Number"
+F 4 "CL10F104ZO8NNNC" H 3675 3825 60  0001 C CNN "Part Number"
 	1    3550 3625
 	1    0    0    -1
