File: hardware/relay.sch (KiCad schematic (older format))
At the start: 1 part

Commit message: order complete
Parts:
- R26: Part Number RC0603JR-0710KL -> MCT06030C1002FP500
Changed lines of the file:
@@
 F 2 "Resistor_SMD:R_0603_1608Metric_Pad1.05x0.95mm_HandSolder" V 5205 2275 50  0001 C CNN
 F 3 "https://www.digikey.com/product-detail/en/yageo/RC0603JR-0710KL/311-10KGRCT-ND/729647" V 5355 2275 50  0001 C CNN
-F 4 "RC0603JR-0710KL" V 5455 2375 60  0001 C CNN "Part Number"
+F 4 "MCT06030C1002FP500" V 5455 2375 60  0001 C CNN "Part Number"
 	1    5275 2275
 	0    -1   -1   0
