File: hardware/Interface.sch (KiCad schematic (older format))
At the start: 19 parts, among them J1 Conn_02x08_Odd_Even, J4 Conn_01x06, U12 soft-button-4x

Commit message: update
Parts:
- removed J4: Conn_01x06, Connector_PinHeader_1.00mm:PinHeader_1x06_P1.00mm_Vertical, symbol Connector_Generic:Conn_01x06
- removed R12, R13, R21, R8: R_10k, Resistor_SMD:R_0603_1608Metric_Pad0.99x1.00mm_HandSolder, symbol open-automation:R_10k
- C12: footprint Capacitor_SMD:C_0603_1608Metric_Pad0.99x1.00mm_HandSolder -> Capacitor_SMD:C_0603_1608Metric_Pad1.05x0.95mm_HandSolder
- D2, D4, D5: footprint LED_SMD:LED_0603_1608Metric_Pad0.82x1.00mm_HandSolder -> LED_SMD:LED_0603_1608Metric_Pad1.05x0.95mm_HandSolder
- FACTORY1, PROG1, REBOOT1: footprint Buttons_Switches_SMD:SW_SPST_KMR2 -> Button_Switch_SMD:SW_SPST_KMR2
- J1: footprint Pin_Headers:Pin_Header_Straight_2x08_Pitch2.54mm -> Connector_PinHeader_2.54mm:PinHeader_2x08_P2.54mm_Vertical
- R14, R15, R16, R23: footprint Resistor_SMD:R_0603_1608Metric_Pad0.99x1.00mm_HandSolder -> Resistor_SMD:R_0603_1608Metric_Pad1.05x0.95mm_HandSolder
Connections:
- net labels added: ZERO_DETECT
- net labels removed: RELAY_1, RELAY_2, RELAY_3, RELAY_4
- wire segments 69 -> 50
Other:
- moved on the sheet: D4, D5, PROG1, R15, R16, REBOOT1

Commit message: ws2812b
Parts:
- removed D7: WS2812, LED_SMD:LED_WS2812_PLCC6_5.0x5.0mm_P1.6mm, symbol LED:WS2812
- removed R23: R_150, Resistor_SMD:R_0603_1608Metric_Pad1.05x0.95mm_HandSolder, symbol open-automation:R_150
- added D7: WS2812B, LED_SMD:LED_WS2812B_PLCC4_5.0x5.0mm_P3.2mm, symbol LED:WS2812B
Connections:
- net BUTTON_LED: now also D7.4 (DIN)
- net GND: now also D7.3 (VSS)
- net V_USB: now also C12.2, D7.1 (VDD)
Changed lines of the file:
@@
 Text HLabel 5775 3500 2    60   Input ~ 0
 EN
-$Comp
-L LED:WS2812 D7
-U 1 1 5B2B9FC9
-P 7275 5475
-F 0 "D7" H 7300 5150 50  0000 L CNN
-F 1 "WS2812" H 7300 5225 50  0000 L CNN
-F 2 "LED_SMD:LED_WS2812_PLCC6_5.0x5.0mm_P1.6mm" H 7325 5175 50  0001 L TNN
-F 3 "https://www.digikey.com/product-detail/en/sparkfun-electronics/COM-11821/1568-1800-ND/6163706" H 7375 5100 50  0001 L TNN
-F 4 "COM-11821" H 7275 5475 50  0001 C CNN "Part Number"
-	1    7275 5475
-	1    0    0    -1
-$EndComp
 Wire Wire Line
 	6775 5475 6975 5475
@@
 	1    0    0    -1
 $EndComp
-Text HLabel 7275 4675 1    60   Input ~ 0
+Text HLabel 7275 4975 1    60   Input ~ 0
 V_USB
 $Comp
@@
 	1    7450 5100
 	0    1    1    0
-$EndComp
-$Comp
-L open-automation:R_150 R23
-U 1 1 5B2DE82B
-P 7275 4900
-F 0 "R23" V 7275 4825 50  0000 L CNN
-F 1 "R_150" V 7375 4800 50  0000 L CNN
-F 2 "Resistor_SMD:R_0603_1608Metric_Pad1.05x0.95mm_HandSolder" V 7205 4900 50  0001 C CNN
-F 3 "https://www.digikey.com/product-detail/en/stackpole-electronics-inc/RNCP0603FTD150R/RNCP0603FTD150RCT-ND/2240427" V 7355 4900 50  0001 C CNN
-F 4 "RNCP0603FTD150R" V 7455 5000 60  0001 C CNN "Part Number"
-	1    7275 4900
-	1    0    0    -1
 $EndComp
 $Comp
@@
 $EndComp
 Wire Wire Line
-	7275 4725 7275 4750
-Wire Wire Line
-	7275 4675 7275 4725
-Connection ~ 7275 4725
-Wire Wire Line
-	7275 4725 7175 4725
-Wire Wire Line
-	7175 4725 7175 5175
-Wire Wire Line
 	7275 5100 7275 5175
-Wire Wire Line
-	7275 5050 7275 5100
 Connection ~ 7275 5100
 Wire Wire Line
@@
 Wire Wire Line
 	7600 5100 7700 5100
+$Comp
+L LED:WS2812B D7
+U 1 1 5B7E61EB
+P 7275 5475
+F 0 "D7" H 7616 5521 50  0000 L CNN
+F 1 "WS2812B" H 7616 5430 50  0000 L CNN
+F 2 "LED_SMD:LED_WS2812B_PLCC4_5.0x5.0mm_P3.2mm" H 7325 5175 50  0001 L TNN
+F 3 "https://cdn-shop.adafruit.com/datasheets/WS2812B.pdf" H 7375 5100 50  0001 L TNN
+	1    7275 5475
+	1    0    0    -1
+$EndComp
+Wire Wire Line
+	7275 4975 7275 5100
 $EndSCHEMATC

Commit message: order complete
Parts:
- C12: Part Number CGA3E1X7R1C105M080AC -> CL10B105KP8NNNC
- R14, R15, R16: Part Number ERJ-3GEYJ102V -> ESR03EZPJ102
Changed lines of the file:
@@
 F 2 "Capacitor_SMD:C_0603_1608Metric_Pad1.05x0.95mm_HandSolder" H 7550 5400 50  0001 C CNN
 F 3 "https://www.digikey.com/product-detail/en/tdk-corporation/CGA3E1X7R1C105M080AC/445-12540-1-ND/3954206" H 7450 4850 50  0001 C CNN
-F 4 "CGA3E1X7R1C105M080AC" H 7575 5300 60  0001 C CNN "Part Number"
+F 4 "CL10B105KP8NNNC" H 7575 5300 60  0001 C CNN "Part Number"
 	1    7450 5100
 	0    1    1    0
@@
 F 2 "Resistor_SMD:R_0603_1608Metric_Pad1.05x0.95mm_HandSolder" V 4555 3250 50  0001 C CNN
 F 3 "https://www.digikey.com/product-detail/en/panasonic-electronic-components/ERJ-3GEYJ102V/P1.0KGDKR-ND/577615" V 4705 3250 50  0001 C CNN
-F 4 "ERJ-3GEYJ102V" V 4805 3350 60  0001 C CNN "Part Number"
+F 4 "ESR03EZPJ102" V 4805 3350 60  0001 C CNN "Part Number"
 	1    4625 3250
 	1    0    0    -1
@@
 F 2 "Resistor_SMD:R_0603_1608Metric_Pad1.05x0.95mm_HandSolder" V 5455 3250 50  0001 C CNN
 F 3 "https://www.digikey.com/product-detail/en/panasonic-electronic-components/ERJ-3GEYJ102V/P1.0KGDKR-ND/577615" V 5605 3250 50  0001 C CNN
-F 4 "ERJ-3GEYJ102V" V 5705 3350 60  0001 C CNN "Part Number"
+F 4 "ESR03EZPJ102" V 5705 3350 60  0001 C CNN "Part Number"
 	1    5525 3250
 	1    0    0    -1
@@
 F 2 "Resistor_SMD:R_0603_1608Metric_Pad1.05x0.95mm_HandSolder" V 3505 3250 50  0001 C CNN
 F 3 "https://www.digikey.com/product-detail/en/panasonic-electronic-components/ERJ-3GEYJ102V/P1.0KGDKR-ND/577615" V 3655 3250 50  0001 C CNN
-F 4 "ERJ-3GEYJ102V" V 3755 3350 60  0001 C CNN "Part Number"
+F 4 "ESR03EZPJ102" V 3755 3350 60  0001 C CNN "Part Number"
 	1    3575 3250
 	1    0    0    -1

Commit message: 0.7.1
Parts:
- added U7: housing-mounts, open-automation:generic-housing-mounts-md, symbol open-automation:housing-mounts
Connections:
- net GND: now also U7.1 (GND)
Changed lines of the file:
@@
 Wire Wire Line
 	7275 4975 7275 5100
+$Comp
+L open-automation:housing-mounts U7
+U 1 1 5BBF1815
+P 9275 2450
+F 0 "U7" H 9553 2503 60  0000 L CNN
+F 1 "housing-mounts" H 9553 2397 60  0000 L CNN
+F 2 "open-automation:generic-housing-mounts-md" H 9475 2250 60  0001 C CNN
+F 3 "" H 9275 2500 60  0001 C CNN
+	1    9275 2450
+	1    0    0    -1
+$EndComp
+$Comp
+L open-automation:GND #PWR0104
+U 1 1 5BBF1873
+P 8900 2475
+F 0 "#PWR0104" H 8900 2225 50  0001 C CNN
+F 1 "GND" H 8905 2302 50  0000 C CNN
+F 2 "" H 8900 2475 50  0000 C CNN
+F 3 "" H 8900 2475 50  0000 C CNN
+	1    8900 2475
+	1    0    0    -1
+$EndComp
+Wire Wire Line
+	8900 2475 8900 2450
+Wire Wire Line
+	8900 2450 8925 2450
 $EndSCHEMATC

Commit message: send board to board house, v0.7.2
Connections:
- net SCL is gone; now on net ZERO_DETECT: J1.9 (Pin_9)
- net 3V3: now also J1.7 (Pin_7); no longer J1.5 (Pin_5)
- net GND: now also J1.3 (Pin_3)
- net V_BAT: now also J1.5 (Pin_5); no longer J1.3 (Pin_3)
- net V_USB: no longer C12.2, D7.1 (VDD)
- net ZERO_DETECT: no longer J1.7 (Pin_7)
- net I2S_DATA_IN renamed RELAY_3
- net I2S_DATA_OUT renamed RELAY_2
- net RELAY renamed RELAY_1
- net SDA renamed RELAY_4
- new net V_IN: C12.2, D7.1 (VDD)
Changed lines of the file:
@@
 EESchema Schematic File Version 4
 LIBS:liger-cache
-EELAYER 26 0
+EELAYER 29 0
 EELAYER END
 $Descr A4 11693 8268
 encoding utf-8
-Sheet 9 9
+Sheet 9 8
 Title ""
 Date ""
@@
 $EndComp
 Wire Wire Line
-	4600 5950 4700 5950
-Wire Wire Line
-	4000 5950 4100 5950
-Wire Wire Line
-	4600 5850 4700 5850
-Wire Wire Line
-	4000 5750 4100 5750
-Wire Wire Line
-	4600 5750 4700 5750
-Wire Wire Line
-	4000 5850 4100 5850
-Wire Wire Line
-	4600 5650 4700 5650
-Wire Wire Line
-	4000 5650 4100 5650
-Wire Wire Line
-	4000 5450 4100 5450
-Wire Wire Line
-	4000 5550 4100 5550
-Wire Wire Line
-	4000 5350 4100 5350
-Wire Wire Line
-	4600 5450 4700 5450
-Wire Wire Line
-	4700 5550 4600 5550
-Wire Wire Line
-	4600 5350 4700 5350
-Wire Wire Line
 	4050 5200 4050 5250
 Wire Wire Line
@@
 Wire Wire Line
 	3575 3500 3575 3600
-Text HLabel 4000 5350 0    60   Input ~ 0
+Text HLabel 4050 5450 0    60   Input ~ 0
 V_BAT
-Text HLabel 4000 5450 0    60   Input ~ 0
+Text HLabel 4050 5550 0    60   Input ~ 0
 3V3
-Text HLabel 4000 5550 0    60   Input ~ 0
+Text HLabel 4050 5650 0    60   Input ~ 0
 ZERO_DETECT
-Text HLabel 4000 5650 0    60   Input ~ 0
-SCL
-Text HLabel 4000 5750 0    60   Input ~ 0
-I2S_WS
-Text HLabel 4000 5850 0    60   Input ~ 0
-I2S_BCLK
-Text HLabel 4000 5950 0    60   Input ~ 0
+Text HLabel 4650 5850 2    60   Output ~ 0
+RELAY_2
+Text HLabel 4050 5950 0    60   Input ~ 0
 PROG
-Text HLabel 4700 5350 2    60   Input ~ 0
+Text HLabel 4650 5350 2    60   Input ~ 0
 V_USB
-Text HLabel 4700 5450 2    60   Input ~ 0
+Text HLabel 4650 5450 2    60   Output ~ 0
 TXD
-Text HLabel 4700 5550 2    60   Input ~ 0
+Text HLabel 4650 5550 2    60   Input ~ 0
 RXD
-Text HLabel 4700 5650 2    60   Input ~ 0
-SDA
-Text HLabel 4700 5750 2    60   Input ~ 0
-I2S_DATA_IN
-Text HLabel 4700 5850 2    60   Input ~ 0
-I2S_DATA_OUT
-Text HLabel 4700 5950 2    60   Input ~ 0
-RELAY
+Text HLabel 4650 5750 2    60   Output ~ 0
+RELAY_3
+Text HLabel 4650 5950 2    60   Output ~ 0
+RELAY_1
 Text HLabel 6775 5475 0    60   Input ~ 0
 BUTTON_LED
@@
 $EndComp
 Text HLabel 7275 4975 1    60   Input ~ 0
-V_USB
+V_IN
 $Comp
 L open-automation:GND #PWR0102
@@
 Wire Wire Line
 	8900 2450 8925 2450
+Text HLabel 4650 5650 2    60   Output ~ 0
+RELAY_4
+Wire Wire Line
+	4650 5650 4600 5650
+Wire Wire Line
+	4650 5550 4600 5550
+Wire Wire Line
+	4600 5450 4650 5450
+Wire Wire Line
+	4650 5350 4600 5350
+Wire Wire Line
+	4600 5750 4650 5750
+Wire Wire Line
+	4650 5850 4600 5850
+Wire Wire Line
+	4600 5950 4650 5950
+Wire Wire Line
+	4100 5350 4050 5350
+Wire Wire Line
+	4050 5350 4050 5250
+Connection ~ 4050 5250
+Wire Wire Line
+	4050 5450 4100 5450
+Wire Wire Line
+	4100 5550 4050 5550
+Wire Wire Line
+	4050 5650 4100 5650
+Wire Wire Line
+	4100 5750 4050 5750
+Wire Wire Line
+	4050 5850 4100 5850
+Wire Wire Line
+	4100 5950 4050 5950
+Text HLabel 4050 5850 0    60   Input ~ 0
+I2S_BCLK
+Text HLabel 4050 5750 0    60   Input ~ 0
+I2S_WS
 $EndSCHEMATC
