File: hardware/audio.sch (KiCad schematic (older format))
At the start: 8 parts, among them U3 SPH0645LM4H-B, U5 MAX98357AETE+T

Commit message: update
Parts:
- C10: symbol C_1uF -> liger-rescue:C_1uF
- C8: symbol C_0.1uF -> liger-rescue:C_0.1uF
- LS1: symbol speaker-CVS-1508 -> liger-rescue:speaker-CVS-1508
- R11: symbol R_47.5 -> liger-rescue:R_47.5
- R17, R9: symbol R_100k -> liger-rescue:R_100k
- U3: symbol SPH0645LM4H-B -> liger-rescue:SPH0645LM4H-B
- U5: symbol MAX98357AETE+T -> liger-rescue:MAX98357AETE+T
Changed lines of the file:
@@
-EESchema Schematic File Version 2
-LIBS:power
-LIBS:device
-LIBS:transistors
-LIBS:conn
-LIBS:linear
-LIBS:regul
-LIBS:74xx
-LIBS:cmos4000
-LIBS:adc-dac
-LIBS:memory
-LIBS:xilinx
-LIBS:microcontrollers
-LIBS:dsp
-LIBS:microchip
-LIBS:analog_switches
-LIBS:motorola
-LIBS:texas
-LIBS:intel
-LIBS:audio
-LIBS:interface
-LIBS:digital-audio
-LIBS:philips
-LIBS:display
-LIBS:cypress
-LIBS:siliconi
-LIBS:opto
-LIBS:atmel
-LIBS:contrib
-LIBS:valves
-LIBS:open-automation
+EESchema Schematic File Version 4
 LIBS:liger-cache
-EELAYER 25 0
+EELAYER 26 0
 EELAYER END
 $Descr A4 11693 8268
@@
 AUDIO
 $Comp
-L SPH0645LM4H-B U3
+L liger-rescue:SPH0645LM4H-B U3
 U 1 1 5A1620A8
 P 4100 4300
@@
 $EndComp
 $Comp
-L GND #PWR06
+L power:GND #PWR06
 U 1 1 5A1620A9
 P 3650 4550
@@
 I2S_WS
 $Comp
-L C_0.1uF C8
+L liger-rescue:C_0.1uF C8
 U 1 1 5A1620AA
 P 3400 4550
@@
 $EndComp
 $Comp
-L GND #PWR07
+L power:GND #PWR07
 U 1 1 5A1620AB
 P 3400 4750
@@
 $EndComp
 $Comp
-L R_47.5 R11
+L liger-rescue:R_47.5 R11
 U 1 1 5A1620AC
 P 4750 4150
@@
 $EndComp
 $Comp
-L R_100k R9
+L liger-rescue:R_100k R9
 U 1 1 5A1620AD
 P 4750 3950
@@
 $EndComp
 $Comp
-L GND #PWR08
+L power:GND #PWR08
 U 1 1 5A1620AE
 P 4950 3950
@@
 Microphone
 $Comp
-L R_100k R17
+L liger-rescue:R_100k R17
 U 1 1 5A1620AF
 P 7000 4325
@@
 $EndComp
 $Comp
-L GND #PWR09
+L power:GND #PWR09
 U 1 1 5A1620B0
 P 7225 4550
@@
 	8450 4350 8350 4350
 $Comp
-L MAX98357AETE+T U5
+L liger-rescue:MAX98357AETE+T U5
 U 1 1 5A1620B1
 P 7600 4275
@@
 Connection ~ 7200 4450
 $Comp
-L GND #PWR010
+L power:GND #PWR010
 U 1 1 5A1620B2
 P 6750 4325
@@
 	7175 4250 7250 4250
 $Comp
-L C_1uF C10
+L liger-rescue:C_1uF C10
 U 1 1 5A1620B3
 P 7000 4625
@@
 Connection ~ 7000 4450
 $Comp
-L GND #PWR011
+L power:GND #PWR011
 U 1 1 5A1620B4
 P 7000 4825
@@
 	7000 4825 7000 4775
 $Comp
-L speaker-CVS-1508 LS1
+L liger-rescue:speaker-CVS-1508 LS1
 U 1 1 5A1620B5
 P 8825 3950

Commit message: updated schematic
Parts:
- removed C10: C_1uF, Capacitors_SMD:C_0603_HandSoldering, symbol liger-rescue:C_1uF
- removed C8: C_0.1uF, Capacitors_SMD:C_0603_HandSoldering, symbol liger-rescue:C_0.1uF
- added C5, C6: C_0.1uF, Capacitor_SMD:C_0603_1608Metric_Pad0.99x1.00mm_HandSolder, symbol open-automation:C_0.1uF
- added J2, J3: Conn_01x02, Connector_PinHeader_1.00mm:PinHeader_1x02_P1.00mm_Vertical, symbol Connector_Generic:Conn_01x02
Connections:
- wire segments 34 -> 41
Other:
- moved on the sheet: LS1
Changed lines of the file:
@@
-	1    0    0    -1
-$EndComp
-Text GLabel 4600 4450 2    60   Input ~ 0
-I2S_BCLK
-Text GLabel 5050 4150 2    60   Input ~ 0
-I2S_DATA_IN
-Text GLabel 4600 4350 2    60   Input ~ 0
-I2S_WS
-$Comp
-L liger-rescue:C_0.1uF C8
-U 1 1 5A1620AA
-P 3400 4550
-F 0 "C8" H 3425 4650 50  0000 L CNN
-F 1 "C_0.1uF" H 3075 4450 50  0000 L CNN
-F 2 "Capacitors_SMD:C_0603_HandSoldering" H 3500 4850 50  0001 C CNN
-F 3 "https://www.digikey.com/product-detail/en/kemet/C0603C104K5RACTU/399-5089-1-ND/1465623" H 3400 4300 50  0001 C CNN
-F 4 "C0603C104K5RACTU" H 3525 4750 60  0001 C CNN "Part Number"
-	1    3400 4550
 	1    0    0    -1
 $EndComp
@@
 	0    -1   -1   0
 $EndComp
-Text GLabel 3250 4250 0    60   Input ~ 0
-3V3
 Connection ~ 4550 4150
 Wire Wire Line
@@
 	4550 4150 4600 4150
 Wire Wire Line
-	4550 3950 4550 4250
+	4550 3950 4550 4150
 Wire Wire Line
 	4550 4250 4500 4250
@@
 	3400 4400 3400 4250
 Wire Wire Line
-	3250 4250 3700 4250
+	3250 4250 3400 4250
 Connection ~ 3650 4500
 Wire Wire Line
 	3700 4350 3650 4350
 Wire Wire Line
-	3650 4350 3650 4550
+	3650 4350 3650 4500
 Wire Wire Line
 	3700 4500 3650 4500
@@
 	1    0    0    -1
 $EndComp
-Text GLabel 7175 4150 0    60   Input ~ 0
-I2S_DATA_OUT
-Text GLabel 6900 4450 0    60   Input ~ 0
-V_IN
 Wire Wire Line
 	7225 4550 7225 4525
@@
 	7225 4525 7250 4525
 Wire Wire Line
-	6900 4450 7250 4450
+	6900 4450 7000 4450
 Wire Wire Line
 	7175 4150 7250 4150
@@
 Wire Wire Line
 	8350 4250 8575 4250
-Text GLabel 8450 4350 2    60   Input ~ 0
-I2S_WS
-Text GLabel 8450 4450 2    60   Input ~ 0
-I2S_BCLK
 Wire Wire Line
 	8450 4450 8350 4450
@@
 Wire Wire Line
 	7175 4250 7250 4250
-$Comp
-L liger-rescue:C_1uF C10
-U 1 1 5A1620B3
-P 7000 4625
-F 0 "C10" H 7025 4725 50  0000 L CNN
-F 1 "C_1uF" H 6775 4525 50  0000 L CNN
-F 2 "Capacitors_SMD:C_0603_HandSoldering" H 7100 4925 50  0001 C CNN
-F 3 "https://www.digikey.com/product-detail/en/yageo/CC0603ZRY5V7BB105/311-1372-1-ND/2103156" H 7000 4375 50  0001 C CNN
-F 4 "CC0603ZRY5V7BB105" H 7125 4825 60  0001 C CNN "Part Number"
-	1    7000 4625
-	1    0    0    -1
-$EndComp
 Wire Wire Line
 	7000 4475 7000 4450
@@
 L liger-rescue:speaker-CVS-1508 LS1
 U 1 1 5A1620B5
-P 8825 3950
-F 0 "LS1" H 8825 4075 50  0000 R CNN
-F 1 "speaker-CVS-1508" H 8875 4100 50  0001 R CNN
-F 2 "open-automation:speaker-1508" H 8825 3750 50  0001 C CNN
-F 3 "http://www.cui.com/product/resource/cvs-1508.pdf" H 8815 3900 50  0001 C CNN
-F 4 "CVS-1508" H 8975 4275 60  0001 C CNN "Part Number"
-	1    8825 3950
+P 9525 3950
+F 0 "LS1" H 9525 4075 50  0000 R CNN
+F 1 "speaker-CVS-1508" H 9575 4100 50  0001 R CNN
+F 2 "open-automation:speaker-1508" H 9525 3750 50  0001 C CNN
+F 3 "http://www.cui.com/product/resource/cvs-1508.pdf" H 9515 3900 50  0001 C CNN
+F 4 "CVS-1508" H 9675 4275 60  0001 C CNN "Part Number"
+	1    9525 3950
 	1    0    0    -1
 $EndComp
@@
 Text Label 7225 3525 0    197  ~ 0
 Speaker
+Wire Wire Line
+	4550 4150 4550 4250
+Wire Wire Line
+	3400 4250 3700 4250
+Wire Wire Line
+	3650 4500 3650 4550
+Wire Wire Line
+	7200 4450 7250 4450
+Wire Wire Line
+	7000 4450 7200 4450
+$Comp
+L open-automation:C_0.1uF C5
+U 1 1 5B1F056C
+P 3400 4550
+F 0 "C5" H 3515 4596 50  0000 L CNN
+F 1 "C_0.1uF" H 3515 4505 50  0000 L CNN
+F 2 "Capacitor_SMD:C_0603_1608Metric_Pad0.99x1.00mm_HandSolder" H 3500 4850 50  0001 C CNN
+F 3 "https://www.digikey.com/product-detail/en/tdk-corporation/C1608X8R1H104K080AB/445-8818-1-ND/3248223" H 3400 4300 50  0001 C CNN
+F 4 "C1608X8R1H104K080AB" H 3525 4750 60  0001 C CNN "Part Number"
+	1    3400 4550
+	1    0    0    -1
+$EndComp
+$Comp
+L open-automation:C_0.1uF C6
+U 1 1 5B1F08F4
+P 7000 4625
+F 0 "C6" H 7115 4671 50  0000 L CNN
+F 1 "C_0.1uF" H 7115 4580 50  0000 L CNN
+F 2 "Capacitor_SMD:C_0603_1608Metric_Pad0.99x1.00mm_HandSolder" H 7100 4925 50  0001 C CNN
+F 3 "https://www.digikey.com/product-detail/en/tdk-corporation/C1608X8R1H104K080AB/445-8818-1-ND/3248223" H 7000 4375 50  0001 C CNN
+F 4 "C1608X8R1H104K080AB" H 7125 4825 60  0001 C CNN "Part Number"
+	1    7000 4625
+	1    0    0    -1
+$EndComp
+Text HLabel 5050 4150 2    60   Input ~ 0
+I2S_DATA_IN
+Text HLabel 6900 4450 0    60   Input ~ 0
+V_IN
+Text HLabel 4600 4350 2    60   Input ~ 0
+I2S_WS
+Text HLabel 4600 4450 2    60   Input ~ 0
+I2S_BCLK
+Text HLabel 7175 4150 0    60   Input ~ 0
+I2S_DATA_OUT
+Text HLabel 8450 4350 2    60   Input ~ 0
+I2S_WS
+Text HLabel 8450 4450 2    60   Input ~ 0
+I2S_BCLK
+Text HLabel 3250 4250 0    60   Input ~ 0
+3V3
+Wire Wire Line
+	9325 3950 9250 3950
+$Comp
+L Connector_Generic:Conn_01x02 J2
+U 1 1 5B2BE39C
+P 8825 3950
+F 0 "J2" H 8775 4050 50  0000 L CNN
+F 1 "Conn_01x02" H 8700 3725 50  0000 L CNN
+F 2 "Connector_PinHeader_1.00mm:PinHeader_1x02_P1.00mm_Vertical" H 8825 3950 50  0001 C CNN
+F 3 "~" H 8825 3950 50  0001 C CNN
+	1    8825 3950
+	1    0    0    -1
+$EndComp
+$Comp
+L Connector_Generic:Conn_01x02 J3
+U 1 1 5B2BE409
+P 9050 4050
+F 0 "J3" H 8970 3725 50  0000 C CNN
+F 1 "Conn_01x02" H 8970 3816 50  0000 C CNN
+F 2 "Connector_PinHeader_1.00mm:PinHeader_1x02_P1.00mm_Vertical" H 9050 4050 50  0001 C CNN
+F 3 "~" H 9050 4050 50  0001 C CNN
+	1    9050 4050
+	-1   0    0    1
+$EndComp
+Wire Wire Line
+	9250 4050 9325 4050
 $EndSCHEMATC

Commit message: update
Parts:
- removed J2, J3: Conn_01x02, Connector_PinHeader_1.00mm:PinHeader_1x02_P1.00mm_Vertical, symbol Connector_Generic:Conn_01x02
- C5, C6: footprint Capacitor_SMD:C_0603_1608Metric_Pad0.99x1.00mm_HandSolder -> Capacitor_SMD:C_0603_1608Metric_Pad1.05x0.95mm_HandSolder
- R11, R17, R9: footprint Resistors_SMD:R_0603_HandSoldering -> Resistor_SMD:R_0603_1608Metric_Pad1.05x0.95mm_HandSolder
Connections:
- wire segments 41 -> 39
Other:
- moved on the sheet: LS1
Changed lines of the file:
@@
 F 0 "R11" V 4750 4150 50  0000 C CNN
 F 1 "R_47.5" V 4675 4150 50  0000 C CNN
-F 2 "Resistors_SMD:R_0603_HandSoldering" V 4680 4150 50  0001 C CNN
+F 2 "Resistor_SMD:R_0603_1608Metric_Pad1.05x0.95mm_HandSolder" V 4680 4150 50  0001 C CNN
 F 3 "https://www.digikey.com/product-detail/en/yageo/RC0603FR-0747R5L/311-47.5HRCT-ND/730201" V 4830 4150 50  0001 C CNN
 F 4 "RC0603FR-0747R5L" V 4930 4250 60  0001 C CNN "Part Number"
@@
 F 0 "R9" V 4750 3950 50  0000 C CNN
 F 1 "R_100k" V 4650 3950 50  0000 C CNN
-F 2 "Resistors_SMD:R_0603_HandSoldering" V 4680 3950 50  0001 C CNN
+F 2 "Resistor_SMD:R_0603_1608Metric_Pad1.05x0.95mm_HandSolder" V 4680 3950 50  0001 C CNN
 F 3 "https://www.digikey.com/product-detail/en/yageo/RC0603JR-07100KL/311-100KGRCT-ND/729645" V 4830 3950 50  0001 C CNN
 F 4 "RC0603JR-07100KL" V 4930 4050 60  0001 C CNN "Part Number"
@@
 F 0 "R17" V 7000 4325 50  0000 C CNN
 F 1 "R_100k" V 6925 4325 50  0000 C CNN
-F 2 "Resistors_SMD:R_0603_HandSoldering" V 6930 4325 50  0001 C CNN
+F 2 "Resistor_SMD:R_0603_1608Metric_Pad1.05x0.95mm_HandSolder" V 6930 4325 50  0001 C CNN
 F 3 "https://www.digikey.com/product-detail/en/yageo/RC0603JR-07100KL/311-100KGRCT-ND/729645" V 7080 4325 50  0001 C CNN
 F 4 "RC0603JR-07100KL" V 7180 4425 60  0001 C CNN "Part Number"
@@
 L liger-rescue:speaker-CVS-1508 LS1
 U 1 1 5A1620B5
-P 9525 3950
-F 0 "LS1" H 9525 4075 50  0000 R CNN
-F 1 "speaker-CVS-1508" H 9575 4100 50  0001 R CNN
-F 2 "open-automation:speaker-1508" H 9525 3750 50  0001 C CNN
-F 3 "http://www.cui.com/product/resource/cvs-1508.pdf" H 9515 3900 50  0001 C CNN
-F 4 "CVS-1508" H 9675 4275 60  0001 C CNN "Part Number"
-	1    9525 3950
+P 8900 3950
+F 0 "LS1" H 8900 4075 50  0000 R CNN
+F 1 "speaker-CVS-1508" H 8950 4100 50  0001 R CNN
+F 2 "open-automation:speaker-1508" H 8900 3750 50  0001 C CNN
+F 3 "http://www.cui.com/product/resource/cvs-1508.pdf" H 8890 3900 50  0001 C CNN
+F 4 "CVS-1508" H 9050 4275 60  0001 C CNN "Part Number"
+	1    8900 3950
 	1    0    0    -1
 $EndComp
@@
 	8500 4150 8500 3950
 Wire Wire Line
-	8500 3950 8625 3950
-Wire Wire Line
 	8575 4250 8575 4050
-Wire Wire Line
-	8575 4050 8625 4050
 Text Label 7225 3525 0    197  ~ 0
 Speaker
@@
 F 0 "C5" H 3515 4596 50  0000 L CNN
 F 1 "C_0.1uF" H 3515 4505 50  0000 L CNN
-F 2 "Capacitor_SMD:C_0603_1608Metric_Pad0.99x1.00mm_HandSolder" H 3500 4850 50  0001 C CNN
+F 2 "Capacitor_SMD:C_0603_1608Metric_Pad1.05x0.95mm_HandSolder" H 3500 4850 50  0001 C CNN
 F 3 "https://www.digikey.com/product-detail/en/tdk-corporation/C1608X8R1H104K080AB/445-8818-1-ND/3248223" H 3400 4300 50  0001 C CNN
 F 4 "C1608X8R1H104K080AB" H 3525 4750 60  0001 C CNN "Part Number"
@@
 F 0 "C6" H 7115 4671 50  0000 L CNN
 F 1 "C_0.1uF" H 7115 4580 50  0000 L CNN
-F 2 "Capacitor_SMD:C_0603_1608Metric_Pad0.99x1.00mm_HandSolder" H 7100 4925 50  0001 C CNN
+F 2 "Capacitor_SMD:C_0603_1608Metric_Pad1.05x0.95mm_HandSolder" H 7100 4925 50  0001 C CNN
 F 3 "https://www.digikey.com/product-detail/en/tdk-corporation/C1608X8R1H104K080AB/445-8818-1-ND/3248223" H 7000 4375 50  0001 C CNN
 F 4 "C1608X8R1H104K080AB" H 7125 4825 60  0001 C CNN "Part Number"
@@
 3V3
 Wire Wire Line
-	9325 3950 9250 3950
-$Comp
-L Connector_Generic:Conn_01x02 J2
-U 1 1 5B2BE39C
-P 8825 3950
-F 0 "J2" H 8775 4050 50  0000 L CNN
-F 1 "Conn_01x02" H 8700 3725 50  0000 L CNN
-F 2 "Connector_PinHeader_1.00mm:PinHeader_1x02_P1.00mm_Vertical" H 8825 3950 50  0001 C CNN
-F 3 "~" H 8825 3950 50  0001 C CNN
-	1    8825 3950
-	1    0    0    -1
-$EndComp
-$Comp
-L Connector_Generic:Conn_01x02 J3
-U 1 1 5B2BE409
-P 9050 4050
-F 0 "J3" H 8970 3725 50  0000 C CNN
-F 1 "Conn_01x02" H 8970 3816 50  0000 C CNN
-F 2 "Connector_PinHeader_1.00mm:PinHeader_1x02_P1.00mm_Vertical" H 9050 4050 50  0001 C CNN
-F 3 "~" H 9050 4050 50  0001 C CNN
-	1    9050 4050
-	-1   0    0    1
-$EndComp
-Wire Wire Line
-	9250 4050 9325 4050
+	8500 3950 8700 3950
+Wire Wire Line
+	8575 4050 8700 4050
 $EndSCHEMATC

Commit message: update
Connections:
- net at U5.10 (OUTN): now also LS1.1; no longer LS1.2
- net at U5.9 (OUTP): now also LS1.2; no longer LS1.1
Changed lines of the file:
@@
 	1    0    0    -1
 $EndComp
-Wire Wire Line
-	8500 4150 8500 3950
-Wire Wire Line
-	8575 4250 8575 4050
 Text Label 7225 3525 0    197  ~ 0
 Speaker
@@
 3V3
 Wire Wire Line
-	8500 3950 8700 3950
+	8700 4050 8500 4050
 Wire Wire Line
-	8575 4050 8700 4050
+	8500 4050 8500 4150
+Wire Wire Line
+	8700 3950 8575 3950
+Wire Wire Line
+	8575 3950 8575 4250
 $EndSCHEMATC

Commit message: order complete
Parts:
- C5, C6: Part Number C1608X8R1H104K080AB -> CL10F104ZO8NNNC
- R11: Part Number RC0603FR-0747R5L -> ERJ-3EKF47R5V
- R17, R9: Part Number RC0603JR-07100KL -> ERA-3AEB104V
Changed lines of the file:
@@
 F 2 "Resistor_SMD:R_0603_1608Metric_Pad1.05x0.95mm_HandSolder" V 4680 4150 50  0001 C CNN
 F 3 "https://www.digikey.com/product-detail/en/yageo/RC0603FR-0747R5L/311-47.5HRCT-ND/730201" V 4830 4150 50  0001 C CNN
-F 4 "RC0603FR-0747R5L" V 4930 4250 60  0001 C CNN "Part Number"
+F 4 "ERJ-3EKF47R5V" V 4930 4250 60  0001 C CNN "Part Number"
 	1    4750 4150
 	0    1    1    0
@@
 F 2 "Resistor_SMD:R_0603_1608Metric_Pad1.05x0.95mm_HandSolder" V 4680 3950 50  0001 C CNN
 F 3 "https://www.digikey.com/product-detail/en/yageo/RC0603JR-07100KL/311-100KGRCT-ND/729645" V 4830 3950 50  0001 C CNN
-F 4 "RC0603JR-07100KL" V 4930 4050 60  0001 C CNN "Part Number"
+F 4 "ERA-3AEB104V" V 4930 4050 60  0001 C CNN "Part Number"
 	1    4750 3950
 	0    1    1    0
@@
 F 2 "Resistor_SMD:R_0603_1608Metric_Pad1.05x0.95mm_HandSolder" V 6930 4325 50  0001 C CNN
 F 3 "https://www.digikey.com/product-detail/en/yageo/RC0603JR-07100KL/311-100KGRCT-ND/729645" V 7080 4325 50  0001 C CNN
-F 4 "RC0603JR-07100KL" V 7180 4425 60  0001 C CNN "Part Number"
+F 4 "ERA-3AEB104V" V 7180 4425 60  0001 C CNN "Part Number"
 	1    7000 4325
 	0    1    1    0
@@
 F 2 "Capacitor_SMD:C_0603_1608Metric_Pad1.05x0.95mm_HandSolder" H 3500 4850 50  0001 C CNN
 F 3 "https://www.digikey.com/product-detail/en/tdk-corporation/C1608X8R1H104K080AB/445-8818-1-ND/3248223" H 3400 4300 50  0001 C CNN
-F 4 "C1608X8R1H104K080AB" H 3525 4750 60  0001 C CNN "Part Number"
+F 4 "CL10F104ZO8NNNC" H 3525 4750 60  0001 C CNN "Part Number"
 	1    3400 4550
 	1    0    0    -1
@@
 F 2 "Capacitor_SMD:C_0603_1608Metric_Pad1.05x0.95mm_HandSolder" H 7100 4925 50  0001 C CNN
 F 3 "https://www.digikey.com/product-detail/en/tdk-corporation/C1608X8R1H104K080AB/445-8818-1-ND/3248223" H 7000 4375 50  0001 C CNN
-F 4 "C1608X8R1H104K080AB" H 7125 4825 60  0001 C CNN "Part Number"
+F 4 "CL10F104ZO8NNNC" H 7125 4825 60  0001 C CNN "Part Number"
 	1    7000 4625
 	1    0    0    -1
